File: hw/eagle/IRAMX-drv-v2.brd (EAGLE design)
At the start: 100 x 75.6 mm, 66 parts, among them IC1 IRAMTOP, IC3 LM393N, IC4 4049N, IC5 4013N, Q1 IRF740

Commit message: +values
Parts:
- C1, C2, C3: value (none) -> 4.7µ
- C10, C11, C13, C14, C16, C19, C20, C21, C7, C8, C9: value (none) -> 100n
- C12, C5: value (none) -> 0.33µ
- C15, C17: value (none) -> 1000µ
- C18, C6: value (none) -> 0.1µ
- IC6: value (none) -> 7805
- IC7: value (none) -> 7815
- LED1: value (none) -> GELB
- LED2: value (none) -> ROT
- LED3: value (none) -> GRÜN
- R1, R22: value (none) -> 10K
- R10: value (none) -> 100K
- R11, R23: value (none) -> 1K
- R12, R13, R21: value (none) -> 470
- R14, R15, R16, R17: value (none) -> 180
- R18: value (none) -> 3.9K
- R19: value (none) -> 100
- R2: value (none) -> 5K
- R20: value (none) -> 22
- R4, R8: value (none) -> 18K
- R6: value (none) -> 33K

Commit message: +values
Parts:
- C22: value (none) -> 100p
- C4: value (none) -> 1000p
- R3, R5, R7, R9: value (none) -> 10K
Changed lines of the file:
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@@
 <element name="C2" library="capacitor-wima" package="C5B5" value="4.7µ" x="84.455" y="62.23" rot="R90"/>
 <element name="C3" library="capacitor-wima" package="C5B5" value="4.7µ" x="84.455" y="69.85" rot="R270"/>
-<element name="C4" library="capacitor-wima" package="C5B5" value="" x="84.455" y="46.355" rot="R270"/>
+<element name="C4" library="capacitor-wima" package="C5B5" value="1000p" x="84.455" y="46.355" rot="R270"/>
 <element name="OK1" library="optocoupler" package="DIL08" value="6N137" x="26.67" y="29.845" rot="R270">
 <attribute name="OC_NEWARK" value="52M1895" x="26.67" y="29.845" size="1.778" layer="27" rot="R270" display="off"/>
@@
 </element>
 <element name="R1" library="rcl" package="0204/7" value="10K" x="48.895" y="14.605" rot="R180"/>
-<element name="R3" library="rcl" package="0204/7" value="" x="55.245" y="26.67" rot="R270"/>
-<element name="R5" library="rcl" package="0204/7" value="" x="52.705" y="23.495" rot="R270"/>
-<element name="R7" library="rcl" package="0204/7" value="" x="50.165" y="22.225" rot="R270"/>
+<element name="R3" library="rcl" package="0204/7" value="10K" x="55.245" y="26.67" rot="R270"/>
+<element name="R5" library="rcl" package="0204/7" value="10K" x="52.705" y="23.495" rot="R270"/>
+<element name="R7" library="rcl" package="0204/7" value="10K" x="50.165" y="22.225" rot="R270"/>
 <element name="X2" library="con-appsys" package="RJ45" value="" x="5.715" y="19.685" rot="R270"/>
 <element name="IC3" library="linear" package="DIL08" value="LM393N" x="79.375" y="10.16" rot="R180"/>
-<element name="R9" library="rcl" package="0204/7" value="" x="47.625" y="20.32" rot="R270"/>
+<element name="R9" library="rcl" package="0204/7" value="10K" x="47.625" y="20.32" rot="R270"/>
 <element name="C5" library="rcl" package="E2,5-5" value="0.33µ" x="10.16" y="45.72"/>
 <element name="C6" library="rcl" package="E2,5-5" value="0.1µ" x="5.08" y="45.72"/>
@@
 <element name="C20" library="rcl" package="C050-025X075" value="100n" x="34.29" y="18.415" rot="R270"/>
 <element name="C21" library="rcl" package="C050-025X075" value="100n" x="34.29" y="28.575" rot="R270"/>
-<element name="C22" library="rcl" package="C150-054X183" value="" x="79.375" y="50.165" rot="R270"/>
+<element name="C22" library="rcl" package="C150-054X183" value="100p" x="79.375" y="50.165" rot="R270"/>
 <element name="R23" library="rcl" package="0204/7" value="1K" x="88.9" y="17.145" rot="R90"/>
 <element name="R24" library="rcl" package="0204V" value="" x="8.89" y="59.055"/>

Commit message: pullup auf 1k und schaltplan aufgeräumt
Parts:
- R3, R5, R7, R9: value 10K -> 1K
Changed lines of the file:
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@@
 </element>
 <element name="R1" library="rcl" package="0204/7" value="10K" x="48.895" y="14.605" rot="R180"/>
-<element name="R3" library="rcl" package="0204/7" value="10K" x="55.245" y="26.67" rot="R270"/>
-<element name="R5" library="rcl" package="0204/7" value="10K" x="52.705" y="23.495" rot="R270"/>
-<element name="R7" library="rcl" package="0204/7" value="10K" x="50.165" y="22.225" rot="R270"/>
+<element name="R3" library="rcl" package="0204/7" value="1K" x="55.245" y="26.67" rot="R270"/>
+<element name="R5" library="rcl" package="0204/7" value="1K" x="52.705" y="23.495" rot="R270"/>
+<element name="R7" library="rcl" package="0204/7" value="1K" x="50.165" y="22.225" rot="R270"/>
 <element name="X2" library="con-appsys" package="RJ45" value="" x="5.715" y="19.685" rot="R270"/>
 <element name="IC3" library="linear" package="DIL08" value="LM393N" x="79.375" y="10.16" rot="R180"/>
-<element name="R9" library="rcl" package="0204/7" value="10K" x="47.625" y="20.32" rot="R270"/>
+<element name="R9" library="rcl" package="0204/7" value="1K" x="47.625" y="20.32" rot="R270"/>
 <element name="C5" library="rcl" package="E2,5-5" value="0.33µ" x="10.16" y="45.72"/>
 <element name="C6" library="rcl" package="E2,5-5" value="0.1µ" x="5.08" y="45.72"/>

Commit message: schaltplan aufgeraeumt'
Connections:
- net N$10 renamed EN
- net N$26 renamed ITRIP
Changed lines of the file:
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@@
 <?xml version="1.0" encoding="utf-8"?>
 <!DOCTYPE eagle SYSTEM "eagle.dtd">
-<eagle version="6.5.0">
+<eagle version="6.6.0">
 <drawing>
 <settings>
@@
 <contactref element="R25" pad="1"/>
 </signal>
-<signal name="N$10">
-<contactref element="IC1" pad="21"/>
-<wire x1="93.345" y1="26.165" x2="92.205" y2="26.165" width="0.254" layer="16"/>
+<signal name="EN">
 <wire x1="92.205" y1="26.165" x2="90.805" y2="24.765" width="0.254" layer="16"/>
 <wire x1="90.805" y1="24.765" x2="90.805" y2="23.495" width="0.254" layer="16"/>
 <contactref element="R23" pad="2"/>
 <wire x1="88.9" y1="20.955" x2="90.805" y2="23.495" width="0.254" layer="16"/>
+<contactref element="IC1" pad="21"/>
+<wire x1="92.205" y1="26.165" x2="93.345" y2="26.165" width="0.254" layer="16"/>
 </signal>
 <signal name="N$12">
@@
 <wire x1="80.645" y1="26.67" x2="79.375" y2="26.67" width="0.254" layer="16"/>
 </signal>
-<signal name="N$26">
+<signal name="ITRIP">
 <contactref element="R11" pad="2"/>
 <contactref element="IC1" pad="22"/>
-<wire x1="86.36" y1="24.13" x2="88.31" y2="24.13" width="0.254" layer="16"/>
-<wire x1="88.31" y1="24.13" x2="88.345" y2="24.165" width="0.254" layer="16"/>
+<wire x1="86.36" y1="24.13" x2="88.345" y2="24.13" width="0.254" layer="16"/>
+<wire x1="88.345" y1="24.13" x2="88.345" y2="24.165" width="0.254" layer="16"/>
 </signal>
 <signal name="N$29">

Commit message: iramx v2
Parts:
- removed R24, R25: (no value), rcl:0204V
- C1, C2, C3: device capacitor-wima:C5B5 -> capacitor-wima:C5B7.2
- R4, R8: device rcl:0617V -> reroolib:CER
- moved R8 38.6 mm to (49.5, 36.2)
- moved R4 2.54 mm to (45.7, 71.1)
- moved C15 1.91 mm to (62.2, 53.3)
- moved C17 1.91 mm to (36.8, 53.3)
- moved C22 1.91 mm to (77.5, 50.2)
- moved X3 1.91 mm to (72.4, 70.5)
- moved X4 1.91 mm to (58.4, 70.5)
- moved C1 0.64 mm to (83.8, 54.6)
- moved C2 0.64 mm to (83.8, 62.2)
- moved C3 0.64 mm to (83.8, 69.8)
Connections:
- removed net N$44: IC7.GND, R24.1, R25.2
- net +15V: no longer R24.2
- net GND: now also IC7.GND, R8.P$1; no longer R25.1, R8.1
- net N$11: now also R4.P$1, R8.P$2; no longer R4.1, R8.2
- net N$37: now also R4.P$2; no longer R4.2
Routing:
- net N$44: track 5.71 -> 0.00 mm
- net N$40: track 58.4 -> 63.0 mm
- net N$9: track 53.0 -> 57.0 mm
- net +15V: track 110.5 -> 114.5 mm
- net N$37: track 63.5 -> 66.8 mm
- net N$2: track 28.0 -> 30.7 mm
- net N$6: track 12.4 -> 13.8 mm
- net N$4: track 21.2 -> 22.5 mm
- net N$5: track 11.5 -> 12.1 mm

Commit message: r net
Parts:
- removed R1: 10K, rcl:0204/7
- removed R3, R5, R7, R9: 1K, rcl:0204/7
- added RN1: 1K, resistor-net:RN-6
- moved C4 0.64 mm to (83.8, 46.4)
- moved C22 0.63 mm to (77.5, 49.5)
Connections:
- net +5V: now also RN1.1; no longer R1.2, R3.2, R5.2, R7.2, R9.2
- net N$24: now also RN1.6; no longer R3.1
- net N$29: now also RN1.3; no longer R9.1
- net N$35: now also RN1.5; no longer R5.1
- net N$38: now also RN1.4; no longer R7.1
- net N$42: now also RN1.2; no longer R1.1
Routing:
- net +5V: track 216.1 -> 202.8 mm
- net N$42: track 37.7 -> 42.3 mm
- net N$24: track 92.4 -> 95.0 mm
- net N$35: track 68.5 -> 70.6 mm
- net N$40: track 63.0 -> 64.6 mm
- net N$9: track 57.0 -> 58.2 mm
- net N$29: track 51.3 -> 50.5 mm
- net +15V: track 114.5 -> 115.0 mm
- net N$11: track 68.2 -> 68.7 mm

Commit message: hw
Parts:
- moved R13 11.4 mm to (9.53, 41.9), turned to 180 degrees
- moved OK2 9.53 mm to (11.4, 27.9)
- moved R17 8.89 mm to (11.4, 21.0)
- moved X2 8.89 mm to (5.71, 10.8)
- moved C9 8.08 mm to (12.7, 35.6), turned to 0 degrees
- moved R15 3.42 mm to (19.7, 7.62), turned to 270 degrees
- moved R14 3.24 mm to (19.1, 27.9), turned to 90 degrees
- moved R16 3.24 mm to (19.1, 17.8), turned to 270 degrees
- moved R20 2.29 mm to (61.0, 31.8)
- moved C8 1.91 mm to (34.3, 6.35)
- moved LED1 1.91 mm to (15.9, 47.0)
- moved OK4 1.91 mm to (26.7, 7.62)
- moved C20 1.90 mm to (34.3, 16.5)
- moved C21 1.90 mm to (34.3, 26.7)
- moved OK1 1.90 mm to (26.7, 27.9)
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Routing:
- net +5V: track 202.8 -> 221.5 mm
- net N$20: track 10.6 -> 17.6 mm
- net N$31: track 9.09 -> 14.3 mm
- net N$9: track 58.2 -> 63.4 mm
- net +15V: track 115.0 -> 119.5 mm
- net N$16: track 8.52 -> 12.2 mm
- net N$17: track 5.34 -> 8.56 mm
- net N$40: track 64.6 -> 67.5 mm
- net N$43: track 4.86 -> 7.40 mm
- net N$23: track 8.56 -> 10.3 mm
- net N$35: track 70.6 -> 72.1 mm
- net +24V: track 29.8 -> 28.5 mm
- net N$19: track 19.1 -> 18.0 mm
- net N$18: track 15.2 -> 16.2 mm
- net N$29: track 50.5 -> 51.3 mm
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
Commit message: iramx v2
Parts:
- removed R22: 10K, rcl:0204/7
- RN1: device resistor-net:RN-6 -> resistor-net:RN-7
- moved R4 35.8 mm to (49.5, 35.6), turned to 270 degrees
- moved C19 21.0 mm to (42.5, 6.67)
- moved R21 19.6 mm to (45.7, 23.5)
- moved R20 19.3 mm to (43.5, 23.5)
- moved C7 17.3 mm to (84.1, 26.7)
- moved RN1 14.1 mm to (40.0, 13.0)
- moved R8 12.7 mm to (62.2, 35.6)
- moved R13 8.33 mm to (17.5, 39.4), turned to 270 degrees
- moved OK2 6.36 mm to (11.1, 34.3)
- moved C9 6.04 mm to (12.4, 41.6)
- moved R17 5.41 mm to (11.1, 26.4)
- moved X2 5.41 mm to (5.40, 16.2)
- moved C11 1.90 mm to (63.5, 14.0)
- moved R19 1.90 mm to (58.4, 17.8)
- moved R18 0.63 mm to (69.8, 13.3)
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Connections:
- removed net N$30: IC3.1, IC4.5, R22.1
- new net N$10: IC3.1, IC4.5, RN1.5
- net +5V: now also IC4.3; no longer R22.2
- net GND: no longer IC4.3
- net N$24: now also RN1.7; no longer RN1.6
- net N$35: now also RN1.6; no longer RN1.5
Routing:
- net N$10: track 0.00 -> 59.3 mm, vias 0 -> 2
- net N$37: track 66.9 -> 125.9 mm
- net N$30: track 33.0 -> 0.00 mm, vias 2 -> 0
- net N$11: track 68.7 -> 46.2 mm
- net N$9: track 63.4 -> 41.0 mm
- net +5V: track 221.5 -> 243.7 mm
- net N$40: track 67.5 -> 46.5 mm
- net N$39: track 13.1 -> 31.9 mm
- net N$42: track 41.7 -> 51.2 mm
- net N$35: track 72.1 -> 77.3 mm
- net N$20: track 17.6 -> 13.1 mm
- net N$24: track 95.4 -> 99.6 mm
- net N$29: track 51.3 -> 47.3 mm
- net N$43: track 7.40 -> 3.94 mm
- net N$31: track 14.3 -> 11.3 mm
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