File: hw/eagle/IRAMX-drv-v2.sch (EAGLE design)
At the start: 66 parts, among them IC1 IRAMTOP, IC3 LM393N, IC4 4049N, IC5 4013N, Q1 IRF740

Commit message: +values
Parts:
- C1, C2, C3: value (none) -> 4.7µ
- C10, C11, C13, C14, C16, C19, C20, C21, C7, C8, C9: value (none) -> 100n
- C12, C5: value (none) -> 0.33µ
- C15, C17: value (none) -> 1000µ
- C18, C6: value (none) -> 0.1µ
- IC6: value (none) -> 7805
- IC7: value (none) -> 7815
- LED1: value (none) -> GELB
- LED2: value (none) -> ROT
- LED3: value (none) -> GRÜN
- R1, R22: value (none) -> 10K
- R10: value (none) -> 100K
- R11, R23: value (none) -> 1K
- R12, R13, R21: value (none) -> 470
- R14, R15, R16, R17: value (none) -> 180
- R18: value (none) -> 3.9K
- R19: value (none) -> 100
- R2: value (none) -> 5K
- R20: value (none) -> 22
- R4, R8: value (none) -> 18K
- R6: value (none) -> 33K
Changed lines of the file:
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@@
 </classes>
 <parts>
-<part name="C1" library="capacitor-wima" deviceset="C" device="5/5"/>
-<part name="C2" library="capacitor-wima" deviceset="C" device="5/5"/>
-<part name="C3" library="capacitor-wima" deviceset="C" device="5/5"/>
+<part name="C1" library="capacitor-wima" deviceset="C" device="5/5" value="4.7µ"/>
+<part name="C2" library="capacitor-wima" deviceset="C" device="5/5" value="4.7µ"/>
+<part name="C3" library="capacitor-wima" deviceset="C" device="5/5" value="4.7µ"/>
 <part name="C4" library="capacitor-wima" deviceset="C" device="5/5"/>
 <part name="OK1" library="optocoupler" deviceset="6N137" device=""/>
@@
 <part name="OK4" library="optocoupler" deviceset="6N137" device=""/>
 <part name="GND1" library="supply1" deviceset="GND" device=""/>
-<part name="R1" library="rcl" deviceset="R-EU_" device="0204/7"/>
+<part name="R1" library="rcl" deviceset="R-EU_" device="0204/7" value="10K"/>
 <part name="GND3" library="supply1" deviceset="GND" device=""/>
 <part name="GND4" library="supply1" deviceset="GND" device=""/>
@@
 <part name="P+13" library="supply1" deviceset="+5V" device=""/>
 <part name="R9" library="rcl" deviceset="R-EU_" device="0204/7"/>
-<part name="C5" library="rcl" deviceset="CPOL-EU" device="E2.5-5"/>
-<part name="C6" library="rcl" deviceset="CPOL-EU" device="E2.5-5"/>
-<part name="C7" library="rcl" deviceset="C-EU" device="050-025X075"/>
-<part name="C8" library="rcl" deviceset="C-EU" device="050-025X075"/>
-<part name="C9" library="rcl" deviceset="C-EU" device="050-025X075"/>
+<part name="C5" library="rcl" deviceset="CPOL-EU" device="E2.5-5" value="0.33µ"/>
+<part name="C6" library="rcl" deviceset="CPOL-EU" device="E2.5-5" value="0.1µ"/>
+<part name="C7" library="rcl" deviceset="C-EU" device="050-025X075" value="100n"/>
+<part name="C8" library="rcl" deviceset="C-EU" device="050-025X075" value="100n"/>
+<part name="C9" library="rcl" deviceset="C-EU" device="050-025X075" value="100n"/>
 <part name="GND14" library="supply1" deviceset="GND" device=""/>
 <part name="GND15" library="supply1" deviceset="GND" device=""/>
@@
 <part name="GND18" library="supply1" deviceset="GND" device=""/>
 <part name="P+17" library="supply1" deviceset="+5V" device=""/>
-<part name="C10" library="rcl" deviceset="C-EU" device="050-025X075"/>
+<part name="C10" library="rcl" deviceset="C-EU" device="050-025X075" value="100n"/>
 <part name="GND19" library="supply1" deviceset="GND" device=""/>
-<part name="R11" library="rcl" deviceset="R-EU_" device="0204/7"/>
-<part name="C14" library="rcl" deviceset="C-EU" device="050-025X075"/>
+<part name="R11" library="rcl" deviceset="R-EU_" device="0204/7" value="1K"/>
+<part name="C14" library="rcl" deviceset="C-EU" device="050-025X075" value="100n"/>
 <part name="GND20" library="supply1" deviceset="GND" device=""/>
-<part name="LED1" library="led" deviceset="LED" device="5MM"/>
-<part name="LED2" library="led" deviceset="LED" device="5MM"/>
-<part name="R12" library="rcl" deviceset="R-EU_" device="0204/7"/>
+<part name="LED1" library="led" deviceset="LED" device="5MM" value="GELB"/>
+<part name="LED2" library="led" deviceset="LED" device="5MM" value="ROT"/>
+<part name="R12" library="rcl" deviceset="R-EU_" device="0204/7" value="470"/>
 <part name="P+18" library="supply1" deviceset="+5V" device=""/>
-<part name="R13" library="rcl" deviceset="R-EU_" device="0204/7"/>
+<part name="R13" library="rcl" deviceset="R-EU_" device="0204/7" value="470"/>
 <part name="GND21" library="supply1" deviceset="GND" device=""/>
-<part name="C13" library="rcl" deviceset="C-EU" device="050-025X075"/>
+<part name="C13" library="rcl" deviceset="C-EU" device="050-025X075" value="100n"/>
 <part name="GND12" library="supply1" deviceset="GND" device=""/>
-<part name="R14" library="rcl" deviceset="R-EU_" device="0204/2V"/>
-<part name="R15" library="rcl" deviceset="R-EU_" device="0204/2V"/>
-<part name="R16" library="rcl" deviceset="R-EU_" device="0204/2V"/>
-<part name="R17" library="rcl" deviceset="R-EU_" device="0204/2V"/>
+<part name="R14" library="rcl" deviceset="R-EU_" device="0204/2V" value="180"/>
+<part name="R15" library="rcl" deviceset="R-EU_" device="0204/2V" value="180"/>
+<part name="R16" library="rcl" deviceset="R-EU_" device="0204/2V" value="180"/>
+<part name="R17" library="rcl" deviceset="R-EU_" device="0204/2V" value="180"/>
 <part name="IC1" library="iram-b" deviceset="IRAM" device="TOP"/>
 <part name="IC4" library="40xx" deviceset="4049" device="N"/>
-<part name="C11" library="rcl" deviceset="C-EU" device="050-025X075"/>
-<part name="R6" library="rcl" deviceset="R-EU_" device="0204/7"/>
-<part name="R18" library="rcl" deviceset="R-EU_" device="0204/7"/>
-<part name="C16" library="rcl" deviceset="C-EU" device="050-025X075"/>
-<part name="R19" library="rcl" deviceset="R-EU_" device="0204/7"/>
+<part name="C11" library="rcl" deviceset="C-EU" device="050-025X075" value="100n"/>
+<part name="R6" library="rcl" deviceset="R-EU_" device="0204/7" value="33K"/>
+<part name="R18" library="rcl" deviceset="R-EU_" device="0204/7" value="3.9K"/>
+<part name="C16" library="rcl" deviceset="C-EU" device="050-025X075" value="100n"/>
+<part name="R19" library="rcl" deviceset="R-EU_" device="0204/7" value="100"/>
 <part name="GND7" library="supply1" deviceset="GND" device=""/>
 <part name="GND8" library="supply1" deviceset="GND" device=""/>
-<part name="R2" library="pot" deviceset="TRIM_EU-" device="CA6V"/>
+<part name="R2" library="pot" deviceset="TRIM_EU-" device="CA6V" value="5K"/>
 <part name="IC5" library="40xx" deviceset="4013" device="N"/>
 <part name="X3" library="con-wago-508" deviceset="W237-03P" device=""/>
 <part name="X4" library="con-wago-508" deviceset="W237-02P" device=""/>
-<part name="C15" library="rcl" deviceset="CPOL-EU" device="E10-25"/>
-<part name="R4" library="rcl" deviceset="R-EU_" device="0617/5V"/>
-<part name="R8" library="rcl" deviceset="R-EU_" device="0617/5V"/>
-<part name="C17" library="rcl" deviceset="CPOL-EU" device="E10-25"/>
-<part name="R10" library="rcl" deviceset="R-EU_" device="0204/7"/>
+<part name="C15" library="rcl" deviceset="CPOL-EU" device="E10-25" value="1000µ"/>
+<part name="R4" library="rcl" deviceset="R-EU_" device="0617/5V" value="18K"/>
+<part name="R8" library="rcl" deviceset="R-EU_" device="0617/5V" value="18K"/>
+<part name="C17" library="rcl" deviceset="CPOL-EU" device="E10-25" value="1000µ"/>
+<part name="R10" library="rcl" deviceset="R-EU_" device="0204/7" value="100K"/>
 <part name="P+7" library="supply1" deviceset="+5V" device=""/>
-<part name="R20" library="rcl" deviceset="R-EU_" device="0204/7"/>
+<part name="R20" library="rcl" deviceset="R-EU_" device="0204/7" value="22"/>
 <part name="Q1" library="transistor-power" deviceset="IRF740" device=""/>
 <part name="GND9" library="supply1" deviceset="GND" device=""/>
@@
 <part name="X1" library="con-wago-508" deviceset="W237-02P" device=""/>
 <part name="GND11" library="supply1" deviceset="GND" device=""/>
-<part name="IC6" library="v-reg" deviceset="78XXS" device=""/>
-<part name="IC7" library="v-reg" deviceset="78XXS" device=""/>
-<part name="C12" library="rcl" deviceset="CPOL-EU" device="E2.5-5"/>
-<part name="C18" library="rcl" deviceset="CPOL-EU" device="E2.5-5"/>
+<part name="IC6" library="v-reg" deviceset="78XXS" device="" value="7805"/>
+<part name="IC7" library="v-reg" deviceset="78XXS" device="" value="7815"/>
+<part name="C12" library="rcl" deviceset="CPOL-EU" device="E2.5-5" value="0.33µ"/>
+<part name="C18" library="rcl" deviceset="CPOL-EU" device="E2.5-5" value="0.1µ"/>
 <part name="GND13" library="supply1" deviceset="GND" device=""/>
 <part name="GND22" library="supply1" deviceset="GND" device=""/>
 <part name="GND23" library="supply1" deviceset="GND" device=""/>
-<part name="LED3" library="led" deviceset="LED" device="5MM"/>
-<part name="R21" library="rcl" deviceset="R-EU_" device="0204/7"/>
-<part name="R22" library="rcl" deviceset="R-EU_" device="0204/7"/>
+<part name="LED3" library="led" deviceset="LED" device="5MM" value="GRÜN"/>
+<part name="R21" library="rcl" deviceset="R-EU_" device="0204/7" value="470"/>
+<part name="R22" library="rcl" deviceset="R-EU_" device="0204/7" value="10K"/>
 <part name="P+22" library="supply1" deviceset="+5V" device=""/>
 <part name="P+23" library="supply1" deviceset="+5V" device=""/>
@@
 <part name="GND26" library="supply1" deviceset="GND" device=""/>
 <part name="GND27" library="supply1" deviceset="GND" device=""/>
-<part name="C19" library="rcl" deviceset="C-EU" device="050-025X075"/>
+<part name="C19" library="rcl" deviceset="C-EU" device="050-025X075" value="100n"/>
 <part name="GND28" library="supply1" deviceset="GND" device=""/>
-<part name="C20" library="rcl" deviceset="C-EU" device="050-025X075"/>
-<part name="C21" library="rcl" deviceset="C-EU" device="050-025X075"/>
+<part name="C20" library="rcl" deviceset="C-EU" device="050-025X075" value="100n"/>
+<part name="C21" library="rcl" deviceset="C-EU" device="050-025X075" value="100n"/>
 <part name="GND29" library="supply1" deviceset="GND" device=""/>
 <part name="GND30" library="supply1" deviceset="GND" device=""/>
 <part name="C22" library="rcl" deviceset="C-EU" device="150-054X183"/>
 <part name="GND31" library="supply1" deviceset="GND" device=""/>
-<part name="R23" library="rcl" deviceset="R-EU_" device="0204/7"/>
+<part name="R23" library="rcl" deviceset="R-EU_" device="0204/7" value="1K"/>
 <part name="R24" library="rcl" deviceset="R-EU_" device="0204/2V"/>
 <part name="R25" library="rcl" deviceset="R-EU_" device="0204/2V"/>

Commit message: +values
Parts:
- C22: value (none) -> 100p
- C4: value (none) -> 1000p
- R3, R5, R7, R9: value (none) -> 10K
Changed lines of the file:
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@@
 <part name="C2" library="capacitor-wima" deviceset="C" device="5/5" value="4.7µ"/>
 <part name="C3" library="capacitor-wima" deviceset="C" device="5/5" value="4.7µ"/>
-<part name="C4" library="capacitor-wima" deviceset="C" device="5/5"/>
+<part name="C4" library="capacitor-wima" deviceset="C" device="5/5" value="1000p"/>
 <part name="OK1" library="optocoupler" deviceset="6N137" device=""/>
 <part name="OK2" library="optocoupler" deviceset="6N137" device=""/>
@@
 <part name="P+3" library="supply1" deviceset="+5V" device=""/>
 <part name="P+4" library="supply1" deviceset="+5V" device=""/>
-<part name="R3" library="rcl" deviceset="R-EU_" device="0204/7"/>
+<part name="R3" library="rcl" deviceset="R-EU_" device="0204/7" value="10K"/>
 <part name="P+6" library="supply1" deviceset="+5V" device=""/>
-<part name="R5" library="rcl" deviceset="R-EU_" device="0204/7"/>
-<part name="R7" library="rcl" deviceset="R-EU_" device="0204/7"/>
+<part name="R5" library="rcl" deviceset="R-EU_" device="0204/7" value="10K"/>
+<part name="R7" library="rcl" deviceset="R-EU_" device="0204/7" value="10K"/>
 <part name="P+8" library="supply1" deviceset="+5V" device=""/>
 <part name="P+10" library="supply1" deviceset="+5V" device=""/>
@@
 <part name="GND10" library="supply1" deviceset="GND" device=""/>
 <part name="P+13" library="supply1" deviceset="+5V" device=""/>
-<part name="R9" library="rcl" deviceset="R-EU_" device="0204/7"/>
+<part name="R9" library="rcl" deviceset="R-EU_" device="0204/7" value="10K"/>
 <part name="C5" library="rcl" deviceset="CPOL-EU" device="E2.5-5" value="0.33µ"/>
 <part name="C6" library="rcl" deviceset="CPOL-EU" device="E2.5-5" value="0.1µ"/>
@@
 <part name="GND29" library="supply1" deviceset="GND" device=""/>
 <part name="GND30" library="supply1" deviceset="GND" device=""/>
-<part name="C22" library="rcl" deviceset="C-EU" device="150-054X183"/>
+<part name="C22" library="rcl" deviceset="C-EU" device="150-054X183" value="100p"/>
 <part name="GND31" library="supply1" deviceset="GND" device=""/>
 <part name="R23" library="rcl" deviceset="R-EU_" device="0204/7" value="1K"/>

Commit message: pullup auf 1k und schaltplan aufgeräumt
Parts:
- R3, R5, R7, R9: value 10K -> 1K
Other:
- moved on the sheet: C1, C10, C15, C17, C2, C22, C3, C4, IC4D, IC5B, R14, R16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

Commit message: schaltplan aufgeraeumt'
Connections:
- net N$10 renamed EN
- net N$26 renamed ITRIP
Other:
- moved on the sheet: C1, C10, C11, C12, C13, C14, C15, C16, C17, C18, C19, C2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

Commit message: iramx v2
Parts:
- removed R24, R25: (no value), rcl:R-EU_0204/2V
- C1, C2, C3: device capacitor-wima:C5/5 -> capacitor-wima:C5/7.2
- R4, R8: device rcl:R-EU_0617/5V -> reroolib:R-EU_
Connections:
- removed net N$44: IC7.GND, R24.1, R25.2
- net +15V: no longer R24.2
- net GND: now also IC7.GND; no longer R25.1
Changed lines of the file:
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@@
 <?xml version="1.0" encoding="utf-8"?>
 <!DOCTYPE eagle SYSTEM "eagle.dtd">
-<eagle version="6.6.0">
+<eagle version="6.5.0">
 <drawing>
 <settings>
@@
 </classes>
 <parts>
-<part name="C1" library="capacitor-wima" deviceset="C" device="5/5" value="4.7µ"/>
-<part name="C2" library="capacitor-wima" deviceset="C" device="5/5" value="4.7µ"/>
-<part name="C3" library="capacitor-wima" deviceset="C" device="5/5" value="4.7µ"/>
+<part name="C1" library="capacitor-wima" deviceset="C" device="5/7.2" value="4.7µ"/>
+<part name="C2" library="capacitor-wima" deviceset="C" device="5/7.2" value="4.7µ"/>
+<part name="C3" library="capacitor-wima" deviceset="C" device="5/7.2" value="4.7µ"/>
 <part name="C4" library="capacitor-wima" deviceset="C" device="5/5" value="1000p"/>
 <part name="OK1" library="optocoupler" deviceset="6N137" device=""/>
@@
 <part name="X4" library="con-wago-508" deviceset="W237-02P" device=""/>
 <part name="C15" library="rcl" deviceset="CPOL-EU" device="E10-25" value="1000µ"/>
-<part name="R4" library="rcl" deviceset="R-EU_" device="0617/5V" value="18K"/>
-<part name="R8" library="rcl" deviceset="R-EU_" device="0617/5V" value="18K"/>
+<part name="R4" library="reroolib" deviceset="R-EU_" device="" value="18K"/>
+<part name="R8" library="reroolib" deviceset="R-EU_" device="" value="18K"/>
 <part name="C17" library="rcl" deviceset="CPOL-EU" device="E10-25" value="1000µ"/>
 <part name="R10" library="rcl" deviceset="R-EU_" device="0204/7" value="100K"/>
@@
 <part name="GND31" library="supply1" deviceset="GND" device=""/>
 <part name="R23" library="rcl" deviceset="R-EU_" device="0204/7" value="1K"/>
-<part name="R24" library="rcl" deviceset="R-EU_" device="0204/2V"/>
-<part name="R25" library="rcl" deviceset="R-EU_" device="0204/2V"/>
 <part name="GND32" library="supply1" deviceset="GND" device=""/>
 <part name="P+11" library="supply1" deviceset="+15V" device=""/>
@@
 <instance part="C18" gate="G$1" x="-25.4" y="119.38"/>
 <instance part="GND13" gate="1" x="-48.26" y="104.14"/>
-<instance part="GND22" gate="1" x="-25.4" y="109.22"/>
-<instance part="GND23" gate="1" x="-15.24" y="88.9"/>
+<instance part="GND22" gate="1" x="-25.4" y="104.14"/>
+<instance part="GND23" gate="1" x="-35.56" y="104.14"/>
 <instance part="LED3" gate="G$1" x="175.26" y="-7.62"/>
 <instance part="R21" gate="G$1" x="175.26" y="0" rot="R90"/>
@@
 <instance part="GND31" gate="1" x="-93.98" y="88.9"/>
 <instance part="R23" gate="G$1" x="200.66" y="-45.72"/>
-<instance part="R24" gate="G$1" x="-15.24" y="119.38" rot="R90"/>
-<instance part="R25" gate="G$1" x="-15.24" y="99.06" rot="R90"/>
 <instance part="GND32" gate="1" x="22.86" y="63.5"/>
 <instance part="P+11" gate="1" x="22.86" y="73.66"/>
@@
 <pinref part="C18" gate="G$1" pin="-"/>
 <pinref part="GND22" gate="1" pin="GND"/>
-<wire x1="-25.4" y1="114.3" x2="-25.4" y2="111.76" width="0.1524" layer="91"/>
-</segment>
-<segment>
-<pinref part="R25" gate="G$1" pin="1"/>
+<wire x1="-25.4" y1="114.3" x2="-25.4" y2="106.68" width="0.1524" layer="91"/>
+</segment>
+<segment>
+<pinref part="IC7" gate="1" pin="GND"/>
+<wire x1="-35.56" y1="116.84" x2="-35.56" y2="106.68" width="0.1524" layer="91"/>
 <pinref part="GND23" gate="1" pin="GND"/>
-<wire x1="-15.24" y1="93.98" x2="-15.24" y2="91.44" width="0.1524" layer="91"/>
 </segment>
 </net>
@@
 <wire x1="-27.94" y1="124.46" x2="-25.4" y2="124.46" width="0.1524" layer="91"/>
 <pinref part="C18" gate="G$1" pin="+"/>
-<wire x1="-25.4" y1="124.46" x2="-15.24" y2="124.46" width="0.1524" layer="91"/>
-<wire x1="-15.24" y1="124.46" x2="-7.62" y2="124.46" width="0.1524" layer="91"/>
+<wire x1="-25.4" y1="124.46" x2="-7.62" y2="124.46" width="0.1524" layer="91"/>
 <wire x1="-25.4" y1="121.92" x2="-25.4" y2="124.46" width="0.1524" layer="91"/>
 <pinref part="IC6" gate="1" pin="IN"/>
 <junction x="-7.62" y="124.46"/>
 <junction x="-25.4" y="124.46"/>
-<pinref part="R24" gate="G$1" pin="2"/>
-<junction x="-15.24" y="124.46"/>
 </segment>
 </net>
@@
 </segment>
 </net>
-<net name="N$44" class="0">
-<segment>
-<pinref part="R24" gate="G$1" pin="1"/>
-<pinref part="R25" gate="G$1" pin="2"/>
-<wire x1="-15.24" y1="114.3" x2="-15.24" y2="106.68" width="0.1524" layer="91"/>
-<pinref part="IC7" gate="1" pin="GND"/>
-<wire x1="-15.24" y1="106.68" x2="-15.24" y2="104.14" width="0.1524" layer="91"/>
-<wire x1="-35.56" y1="116.84" x2="-35.56" y2="106.68" width="0.1524" layer="91"/>
-<wire x1="-35.56" y1="106.68" x2="-15.24" y2="106.68" width="0.1524" layer="91"/>
-<junction x="-15.24" y="106.68"/>
-</segment>
-</net>

Commit message: r net
Parts:
- removed R1: 10K, rcl:R-EU_0204/7
- removed R3, R5, R7, R9: 1K, rcl:R-EU_0204/7
- added RN1: 1K, resistor-net:RN05
Connections:
- net +5V: now also RN1.1; no longer R1.2, R3.2, R5.2, R7.2, R9.2
- net N$24: now also RN1.6; no longer R3.1
- net N$29: now also RN1.3; no longer R9.1
- net N$35: now also RN1.5; no longer R5.1
- net N$38: now also RN1.4; no longer R7.1
- net N$42: now also RN1.2; no longer R1.1
Other:
- moved on the sheet: IC4C, IC4D, IC4E
