File: hw/eagle/IRAMX-drv-v2.sch (EAGLE design)
At the start: 60 parts, among them IC1 IRAMTOP, IC3 LM393N, IC4 4049N, IC5 4013N, IC6 7805, IC7 7815, Q1 IRF740

Commit message: iramx v2
Parts:
- removed R22: 10K, rcl:R-EU_0204/7
- RN1: device resistor-net:RN05 -> resistor-net:RN06
Connections:
- removed net N$30: IC3A.OUT, IC4B.I, R22.1
- new net N$10: IC3A.OUT, IC4B.I, RN1.5
- net +5V: now also IC4A.I; no longer R22.2
- net GND: no longer IC4A.I
- net N$24: now also RN1.7; no longer RN1.6
- net N$35: now also RN1.6; no longer RN1.5
Changed lines of the file:
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@@
 <part name="LED3" library="led" deviceset="LED" device="5MM" value="GRÜN"/>
 <part name="R21" library="rcl" deviceset="R-EU_" device="0204/7" value="470"/>
-<part name="R22" library="rcl" deviceset="R-EU_" device="0204/7" value="10K"/>
-<part name="P+22" library="supply1" deviceset="+5V" device=""/>
 <part name="GND2" library="supply1" deviceset="GND" device=""/>
-<part name="GND24" library="supply1" deviceset="GND" device=""/>
 <part name="GND25" library="supply1" deviceset="GND" device=""/>
 <part name="P+24" library="supply1" deviceset="+5V" device=""/>
@@
 <part name="GND32" library="supply1" deviceset="GND" device=""/>
 <part name="P+11" library="supply1" deviceset="+15V" device=""/>
-<part name="RN1" library="resistor-net" deviceset="RN05" device="" value="1K"/>
+<part name="RN1" library="resistor-net" deviceset="RN06" device="" value="1K"/>
 <part name="P+5" library="supply1" deviceset="+5V" device=""/>
+<part name="P+6" library="supply1" deviceset="+5V" device=""/>
 </parts>
 <sheets>
@@
 <instance part="LED3" gate="G$1" x="175.26" y="-7.62"/>
 <instance part="R21" gate="G$1" x="175.26" y="0" rot="R90"/>
-<instance part="R22" gate="G$1" x="124.46" y="10.16" rot="R90"/>
-<instance part="P+22" gate="1" x="124.46" y="20.32"/>
 <instance part="GND2" gate="1" x="96.52" y="53.34"/>
-<instance part="GND24" gate="1" x="-93.98" y="116.84"/>
 <instance part="GND25" gate="1" x="152.4" y="-50.8"/>
 <instance part="P+24" gate="1" x="147.32" y="-40.64" rot="R90"/>
@@
 <instance part="GND32" gate="1" x="22.86" y="63.5"/>
 <instance part="P+11" gate="1" x="22.86" y="73.66"/>
-<instance part="RN1" gate="1" x="-7.62" y="86.36" rot="R270"/>
-<instance part="P+5" gate="1" x="-7.62" y="96.52"/>
+<instance part="RN1" gate="1" x="-7.62" y="91.44" rot="R270"/>
+<instance part="P+5" gate="1" x="-7.62" y="99.06"/>
+<instance part="P+6" gate="1" x="-91.44" y="124.46"/>
 </instances>
 <busses>
@@
 <pinref part="GND13" gate="1" pin="GND"/>
 <wire x1="-48.26" y1="106.68" x2="-48.26" y2="114.3" width="0.1524" layer="91"/>
-</segment>
-<segment>
-<pinref part="IC4" gate="A" pin="I"/>
-<pinref part="GND24" gate="1" pin="GND"/>
-<wire x1="-93.98" y1="119.38" x2="-91.44" y2="119.38" width="0.1524" layer="91"/>
 </segment>
 <segment>
@@
 <wire x1="-25.4" y1="10.16" x2="-25.4" y2="7.62" width="0.1524" layer="91"/>
 <pinref part="RN1" gate="1" pin="3"/>
-<wire x1="-7.62" y1="76.2" x2="-30.48" y2="76.2" width="0.1524" layer="91"/>
-<wire x1="-30.48" y1="76.2" x2="-30.48" y2="10.16" width="0.1524" layer="91"/>
+<wire x1="-7.62" y1="81.28" x2="-30.48" y2="81.28" width="0.1524" layer="91"/>
+<wire x1="-30.48" y1="81.28" x2="-30.48" y2="10.16" width="0.1524" layer="91"/>
 <junction x="-30.48" y="10.16"/>
 </segment>
@@
 <pinref part="OK1" gate="A" pin="VO"/>
 <wire x1="-20.32" y1="63.5" x2="-25.4" y2="63.5" width="0.1524" layer="91"/>
-<pinref part="RN1" gate="1" pin="5"/>
 <wire x1="-25.4" y1="63.5" x2="-35.56" y2="63.5" width="0.1524" layer="91"/>
+<junction x="-25.4" y="63.5"/>
+<pinref part="RN1" gate="1" pin="6"/>
+<wire x1="-25.4" y1="66.04" x2="-25.4" y2="63.5" width="0.1524" layer="91"/>
 <wire x1="-7.62" y1="66.04" x2="-25.4" y2="66.04" width="0.1524" layer="91"/>
-<wire x1="-25.4" y1="66.04" x2="-25.4" y2="63.5" width="0.1524" layer="91"/>
-<junction x="-25.4" y="63.5"/>
 </segment>
 </net>
@@
 <pinref part="RN1" gate="1" pin="4"/>
 <wire x1="-27.94" y1="27.94" x2="-22.86" y2="27.94" width="0.1524" layer="91"/>
-<wire x1="-7.62" y1="71.12" x2="-27.94" y2="71.12" width="0.1524" layer="91"/>
-<wire x1="-27.94" y1="71.12" x2="-27.94" y2="27.94" width="0.1524" layer="91"/>
+<wire x1="-7.62" y1="76.2" x2="-27.94" y2="76.2" width="0.1524" layer="91"/>
+<wire x1="-27.94" y1="76.2" x2="-27.94" y2="27.94" width="0.1524" layer="91"/>
 <junction x="-27.94" y="27.94"/>
 </segment>
@@
 <wire x1="27.94" y1="45.72" x2="-15.24" y2="45.72" width="0.1524" layer="91"/>
 <pinref part="IC4" gate="F" pin="I"/>
-<pinref part="RN1" gate="1" pin="6"/>
-<wire x1="-7.62" y1="60.96" x2="-17.78" y2="60.96" width="0.1524" layer="91"/>
 <wire x1="-17.78" y1="60.96" x2="-17.78" y2="45.72" width="0.1524" layer="91"/>
 <junction x="-17.78" y="45.72"/>
+<pinref part="RN1" gate="1" pin="7"/>
+<wire x1="-17.78" y1="60.96" x2="-7.62" y2="60.96" width="0.1524" layer="91"/>
 </segment>
 </net>
@@
 </segment>
 </net>
-<net name="N$30" class="0">
-<segment>
-<pinref part="IC3" gate="A" pin="OUT"/>
-<wire x1="121.92" y1="5.08" x2="124.46" y2="5.08" width="0.1524" layer="91"/>
-<pinref part="R22" gate="G$1" pin="1"/>
-<pinref part="IC4" gate="B" pin="I"/>
-<wire x1="124.46" y1="5.08" x2="154.94" y2="5.08" width="0.1524" layer="91"/>
-<junction x="124.46" y="5.08"/>
-</segment>
-</net>
 <net name="N$39" class="0">
 <segment>
@@
 </net>
 <net name="+5V" class="0">
-<segment>
-<pinref part="R22" gate="G$1" pin="2"/>
-<pinref part="P+22" gate="1" pin="+5V"/>
-<wire x1="124.46" y1="17.78" x2="124.46" y2="15.24" width="0.1524" layer="91"/>
-</segment>
 <segment>
 <pinref part="IC5" gate="A" pin="D"/>
@@
 <pinref part="RN1" gate="1" pin="1"/>
 <pinref part="P+5" gate="1" pin="+5V"/>
-<wire x1="-7.62" y1="93.98" x2="-7.62" y2="91.44" width="0.1524" layer="91"/>
+</segment>
+<segment>
+<pinref part="IC4" gate="A" pin="I"/>
+<pinref part="P+6" gate="1" pin="+5V"/>
+<wire x1="-91.44" y1="121.92" x2="-91.44" y2="119.38" width="0.1524" layer="91"/>
 </segment>
 </net>
@@
 <pinref part="IC5" gate="A" pin="R"/>
 <pinref part="RN1" gate="1" pin="2"/>
-<wire x1="-7.62" y1="81.28" x2="63.5" y2="81.28" width="0.1524" layer="91"/>
-<wire x1="63.5" y1="81.28" x2="63.5" y2="88.9" width="0.1524" layer="91"/>
+<wire x1="-7.62" y1="86.36" x2="63.5" y2="86.36" width="0.1524" layer="91"/>
+<wire x1="63.5" y1="86.36" x2="63.5" y2="88.9" width="0.1524" layer="91"/>
 <wire x1="63.5" y1="88.9" x2="152.4" y2="88.9" width="0.1524" layer="91"/>
 <wire x1="152.4" y1="88.9" x2="152.4" y2="25.4" width="0.1524" layer="91"/>
@@
 </segment>
 </net>
+<net name="N$10" class="0">
+<segment>
+<wire x1="5.08" y1="71.12" x2="5.08" y2="83.82" width="0.1524" layer="91"/>
+<wire x1="5.08" y1="83.82" x2="66.04" y2="83.82" width="0.1524" layer="91"/>
+<wire x1="66.04" y1="83.82" x2="66.04" y2="86.36" width="0.1524" layer="91"/>
+<wire x1="66.04" y1="86.36" x2="124.46" y2="86.36" width="0.1524" layer="91"/>
+<pinref part="IC3" gate="A" pin="OUT"/>
+<wire x1="121.92" y1="5.08" x2="124.46" y2="5.08" width="0.1524" layer="91"/>
+<pinref part="IC4" gate="B" pin="I"/>
+<wire x1="124.46" y1="5.08" x2="154.94" y2="5.08" width="0.1524" layer="91"/>
+<junction x="124.46" y="5.08"/>
+<wire x1="124.46" y1="86.36" x2="124.46" y2="5.08" width="0.1524" layer="91"/>
+<pinref part="RN1" gate="1" pin="5"/>
+<wire x1="-7.62" y1="71.12" x2="5.08" y2="71.12" width="0.1524" layer="91"/>
+</segment>
+</net>
 </nets>
 </sheet>
 </sheets>
+<errors>
+</errors>
 </schematic>
 </drawing>
