File: hw/eagle/res-standalone.sch (EAGLE design)
At the start: 66 parts, among them IC2 7805T, IC3 L272M, IC4 L272M, IC5 STM32F415RGT, X5 22-23-2021

Commit message: slider gain offset
Parts:
- removed ADM485: (no value), ic-package:DIL8
- removed C7: (no value), rcl:C-EU050-025X075
- removed R21, R22: 1k, resistor:R-EU_0204/7
- removed R23: 100, resistor:R-EU_0204/7
- removed R24: (no value), resistor:R-EU_0204/7
- removed U$1: STM32F4-DISCOVERY, STM32F4-DISCOVERY:STM32F4-DISCOVERY
- removed X4, X6: (no value), con-appsys:RJ45
Connections:
- removed net N$37: ADM485.4, U$1.PD8
- removed net N$41: ADM485.1, U$1.PD9
- removed net N$42: ADM485.2, ADM485.3, U$1.PD11
- removed net N$43: ADM485.6, R21.1, R24.2, X4-.5, X6-.5
- removed net N$44: ADM485.7, R22.2, R24.1, X4-.4, X6-.4
- removed net N$45: R23.2, X4-.8, X6-.8
- removed net N$47: R26.2, U$1.PC9
- removed net N$48: R27.1, U$1.PC6
- removed net N$49: R28.1, U$1.PC8
- removed net N$51: R25.2, U$1.PA8
- net +5V: no longer ADM485.8, C7.1, R21.2
- net CRS: no longer U$1.PA7
- net GND: no longer ADM485.5, C7.2, R22.1, R23.1, U$1.GND, U$1.GND1, U$1.GND2, U$1.GND3, U$1.GND4, U$1.GND5, U$1.GND6, U$1.GND7, U$1.GND8, U$1.GND9
- net MDC: no longer U$1.PC1
- net MDIO: no longer U$1.PA2
- net N$14: no longer U$1.PD15
- net N$16: no longer U$1.PD12
- net N$18: no longer U$1.PD14
- net N$19: no longer U$1.PD13
- net N$20: no longer U$1.PA3
- net N$22: no longer U$1.PB4
- net N$23: no longer U$1.PB5
- net N$4: no longer U$1.PC2
- net N$40: no longer U$1.PB1
- net OSCIN: no longer U$1.PA1
- net RX1: no longer U$1.PC5
- net RXO: no longer U$1.PC4
- net TX1: no longer U$1.PB13
- net TXO: no longer U$1.PB12
- net TX_EN: no longer U$1.PB11
- net VCC: no longer U$1.5V, U$1.5V2
- net VDD: no longer U$1.VDD2, U$1.VDD3
Other:
- moved on the sheet: IC5
