File: hw/eagle/IRAMX-drv-v3.brd (EAGLE design)
At the start: 100 x 75.3 mm, 54 parts, among them IC1 IRAMTOP, IC2 STM32F103R6T, IC4 78L05SMD

Commit message: iramx v3
Parts:
- added D2: (no value), diode:SOD80C
- moved C6 6.02 mm to (52.8, 35.2), turned to 180 degrees
- moved R7 2.50 mm to (85.8, 22.8)
- moved R6 1.50 mm to (87.8, 21.8)
- moved C27 1.27 mm to (78.5, 24.0)
- moved IC4 1.25 mm to (52.2, 30.0)
- moved C8 1.12 mm to (69.7, 9.50), turned to 0 degrees
- moved C5 1.00 mm to (52.8, 24.8)
- moved C18 0.71 mm to (79.2, 10.5), turned to 90 degrees
- moved C23 0.56 mm to (81.2, 14.0)
- moved C25 0.56 mm to (65.5, 22.2), turned to 0 degrees
- moved C28 0.56 mm to (83.8, 13.2)
- moved C13 0.25 mm to (65.8, 13.5)
- moved C14 0.25 mm to (63.5, 15.5)
- moved LED1 0.25 mm to (63.7, 3.25)
- moved LED3 0.25 mm to (59.2, 3.25)
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Connections:
- net GND: now also D2.A
- net VLT: now also D2.C
Routing:
- net +3V3: track 113.8 -> 159.1 mm, vias 0 -> 8
- net TX: track 37.6 -> 59.7 mm, vias 0 -> 2
- net GND: track 0.00 -> 17.0 mm, vias 0 -> 2
- net RX: track 37.5 -> 53.1 mm, vias 0 -> 2
- net +15V: track 45.1 -> 55.5 mm, vias 0 -> 2
- net N$37: track 51.8 -> 58.8 mm
- net E: track 11.7 -> 14.6 mm
- net AMP: track 68.8 -> 67.8 mm
- net VTH: track 55.3 -> 56.2 mm
- net VLT: track 60.4 -> 61.2 mm

Commit message: iramxv3 rj45
Parts:
- added IC3: 78L05SMD, linear:SO08
Connections:
- new net ISO_GND: IC3.2, IC3.3, IC3.6, IC3.7, U$1.4, U$2.VIN-, X2.8
- new net N$11: IC3.1, U$1.1
- new net N$13: U$1.2, X2.4
- new net N$14: U$1.3, X2.5
- new net N$17: IC3.8, U$2.VIN+, X2.7
Routing:
- net N$17: track 0.00 -> 24.8 mm
- net N$14: track 0.00 -> 14.9 mm
- net N$11: track 0.00 -> 12.2 mm
- net N$13: track 0.00 -> 11.0 mm
- added copper zone on layer 16, net ISO_GND
Changed lines of the file:
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@@
 <?xml version="1.0" encoding="utf-8"?>
 <!DOCTYPE eagle SYSTEM "eagle.dtd">
-<eagle version="6.5.0">
+<eagle version="7.1.0">
 <drawing>
 <settings>
@@
 <pass name="Default">
 <param name="RoutingGrid" value="50mil"/>
+<param name="AutoGrid" value="1"/>
+<param name="Efforts" value="0"/>
+<param name="TopRouterVariant" value="1"/>
 <param name="tpViaShape" value="round"/>
 <param name="PrefDir.1" value="|"/>
@@
 <element name="R7" library="rcl" package="R0805" value="1K" x="85.75" y="22.75" rot="MR90"/>
 <element name="D2" library="diode" package="SOD80C" value="" x="64.25" y="32.5" rot="MR90"/>
+<element name="IC3" library="linear" package="SO08" value="78L05SMD" x="51.25" y="58.75" rot="MR270"/>
 </elements>
 <signals>
@@
 <signal name="N$7">
 </signal>
+<signal name="N$11">
+<contactref element="IC3" pad="1"/>
+<contactref element="U$1" pad="1"/>
+<wire x1="53.85" y1="60.655" x2="52.405" y2="60.655" width="0.4064" layer="16"/>
+<wire x1="52.405" y1="60.655" x2="51.5" y2="59.75" width="0.4064" layer="16"/>
+<wire x1="51.5" y1="59.75" x2="51.5" y2="56.25" width="0.4064" layer="16"/>
+<wire x1="51.5" y1="56.25" x2="52.5" y2="55.25" width="0.4064" layer="16"/>
+<wire x1="52.5" y1="55.25" x2="54.25" y2="55.25" width="0.4064" layer="16"/>
+<wire x1="54.25" y1="55.25" x2="55" y2="54.5" width="0.4064" layer="16"/>
+<wire x1="55" y1="54.5" x2="55" y2="52.9184" width="0.4064" layer="16"/>
+<wire x1="55" y1="52.9184" x2="55.095" y2="52.8234" width="0.4064" layer="16"/>
+</signal>
+<signal name="ISO_GND">
+<contactref element="U$1" pad="4"/>
+<contactref element="IC3" pad="7"/>
+<contactref element="IC3" pad="6"/>
+<contactref element="IC3" pad="3"/>
+<contactref element="IC3" pad="2"/>
+<contactref element="U$2" pad="VIN-"/>
+<polygon width="0.4064" layer="16">
+<vertex x="46" y="72.75"/>
+<vertex x="63.75" y="72.75"/>
+<vertex x="63.75" y="50.5"/>
+<vertex x="46" y="50.5"/>
+</polygon>
+<contactref element="X2" pad="8"/>
+</signal>
+<signal name="N$17">
+<contactref element="U$2" pad="VIN+"/>
+<contactref element="IC3" pad="8"/>
+<wire x1="48.65" y1="60.655" x2="47" y2="60.655" width="0.4064" layer="16"/>
+<wire x1="47" y1="60.655" x2="47" y2="54" width="0.4064" layer="16"/>
+<wire x1="47" y1="54" x2="49.75" y2="51.25" width="0.4064" layer="16"/>
+<wire x1="49.75" y1="51.25" x2="52.27" y2="51.25" width="0.4064" layer="16"/>
+<wire x1="52.27" y1="51.25" x2="52.5" y2="51.02" width="0.4064" layer="16"/>
+<contactref element="X2" pad="7"/>
+<wire x1="52.0375" y1="66.185" x2="48.435" y2="66.185" width="0.4064" layer="16"/>
+<wire x1="48.435" y1="66.185" x2="47" y2="64.75" width="0.4064" layer="16"/>
+<wire x1="47" y1="64.75" x2="47" y2="60.655" width="0.4064" layer="16"/>
+</signal>
+<signal name="N$13">
+<contactref element="X2" pad="4"/>
+<contactref element="U$1" pad="2"/>
+<wire x1="56.365" y1="52.8234" x2="56.365" y2="63.1275" width="0.4064" layer="16"/>
+<wire x1="56.365" y1="63.1275" x2="55.8475" y2="63.645" width="0.4064" layer="16"/>
+</signal>
+<signal name="N$14">
+<contactref element="U$1" pad="3"/>
+<contactref element="X2" pad="5"/>
+<wire x1="57.635" y1="52.8234" x2="57.635" y2="61.865" width="0.4064" layer="16"/>
+<wire x1="57.635" y1="61.865" x2="57.25" y2="62.25" width="0.4064" layer="16"/>
+<wire x1="57.25" y1="62.25" x2="57.25" y2="64" width="0.4064" layer="16"/>
+<wire x1="57.25" y1="64" x2="56" y2="65.25" width="0.4064" layer="16"/>
+<wire x1="56" y1="65.25" x2="55.5125" y2="65.25" width="0.4064" layer="16"/>
+<wire x1="55.5125" y1="65.25" x2="54.5775" y2="66.185" width="0.4064" layer="16"/>
+</signal>
 </signals>

Commit message: iramx v3
Parts:
- removed H4: MOUNT-PAD-ROUND3.2, holes:3,2-PAD
- added C20, C21: (no value), rcl:A/3216-18R
- moved H3 45.0 mm to (50.0, 5.00)
- moved IC3 1.46 mm to (52.5, 58.0)
Connections:
- net ISO_GND: now also C20.-, C21.-
- net N$11: now also C21.+
- net N$17: now also C20.+
Routing:
- net N$14: track 14.9 -> 19.4 mm
- net N$13: track 11.0 -> 15.4 mm
- net N$17: track 24.8 -> 22.4 mm
- removed copper zone on layer 16, net FOO
Other:
- board size 100 x 75.3 mm -> 55 x 75 mm
Changed lines of the file:
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@@
 <?xml version="1.0" encoding="utf-8"?>
 <!DOCTYPE eagle SYSTEM "eagle.dtd">
-<eagle version="7.1.0">
+<eagle version="6.5.0">
 <drawing>
 <settings>
@@
 <board>
 <plain>
-<wire x1="0" y1="0" x2="100" y2="0" width="0" layer="20"/>
-<wire x1="100" y1="0" x2="100" y2="75.3175" width="0" layer="20"/>
-<wire x1="100" y1="75.3175" x2="0" y2="75.3175" width="0" layer="20"/>
-<wire x1="0" y1="75.3175" x2="0" y2="0" width="0" layer="20"/>
+<wire x1="45" y1="0" x2="100" y2="0" width="0" layer="20"/>
+<wire x1="100" y1="0" x2="100" y2="74.9975" width="0" layer="20"/>
+<wire x1="100" y1="74.9975" x2="45" y2="74.9975" width="0" layer="20"/>
+<wire x1="45" y1="74.9975" x2="45" y2="0" width="0" layer="20"/>
+<dimension x1="50" y1="5" x2="95" y2="5" x3="72.5" y3="-4.75" textsize="1.778" layer="16"/>
+<dimension x1="95" y1="70" x2="95" y2="5" x3="106.5" y3="37.5" textsize="1.778" layer="16"/>
+<dimension x1="45" y1="74.9975" x2="100" y2="75.0075" x3="72.49819375" y3="84.935" textsize="1.778" layer="16"/>
+<dimension x1="45" y1="74.9975" x2="45" y2="0" x3="37.75" y3="37.49875" textsize="1.778" layer="16"/>
 </plain>
 <attributes>
@@
 <pass name="Default">
 <param name="RoutingGrid" value="50mil"/>
-<param name="AutoGrid" value="1"/>
-<param name="Efforts" value="0"/>
-<param name="TopRouterVariant" value="1"/>
 <param name="tpViaShape" value="round"/>
 <param name="PrefDir.1" value="|"/>
@@
 <element name="H1" library="holes" package="3,2-PAD" value="MOUNT-PAD-ROUND3.2" x="95" y="70"/>
 <element name="H2" library="holes" package="3,2-PAD" value="MOUNT-PAD-ROUND3.2" x="95" y="5"/>
-<element name="H3" library="holes" package="3,2-PAD" value="MOUNT-PAD-ROUND3.2" x="5" y="5"/>
-<element name="H4" library="holes" package="3,2-PAD" value="MOUNT-PAD-ROUND3.2" x="5" y="70"/>
+<element name="H3" library="holes" package="3,2-PAD" value="MOUNT-PAD-ROUND3.2" x="50" y="5"/>
 <element name="IC2" library="micro-stm_v2" package="LQFP64" value="STM32F103R6T" x="73.49246875" y="17.25305625" rot="MR0"/>
 <element name="C4" library="rcl" package="C1206K" value="" x="89.255" y="44.4975" rot="MR270"/>
@@
 <element name="R7" library="rcl" package="R0805" value="1K" x="85.75" y="22.75" rot="MR90"/>
 <element name="D2" library="diode" package="SOD80C" value="" x="64.25" y="32.5" rot="MR90"/>
-<element name="IC3" library="linear" package="SO08" value="78L05SMD" x="51.25" y="58.75" rot="MR270"/>
+<element name="IC3" library="linear" package="SO08" value="78L05SMD" x="52.5" y="58" rot="MR270"/>
+<element name="C20" library="rcl" package="A/3216-18R" value="" x="47.75" y="58.75" rot="MR90"/>
+<element name="C21" library="rcl" package="A/3216-18R" value="" x="57.25" y="58.75" rot="MR90"/>
 </elements>
 <signals>
@@
 <contactref element="C10" pad="2"/>
 <polygon width="0.2" layer="16" orphans="yes">
-<vertex x="46.7" y="48.57"/>
+<vertex x="44.95" y="48.57"/>
 <vertex x="65" y="48.57"/>
 <vertex x="65" y="42"/>
@@
 <vertex x="100.08" y="41.68"/>
 <vertex x="100.2625" y="-0.5"/>
-<vertex x="46.97" y="-0.5025"/>
+<vertex x="45.22" y="-0.5025"/>
 </polygon>
 <contactref element="LED1" pad="K"/>
@@
 <wire x1="63.7975" y1="6.2525" x2="63.7975" y2="4.315" width="0.3" layer="16"/>
 <wire x1="63.7975" y1="4.315" x2="63.7475" y2="4.515" width="0.3" layer="16"/>
-</signal>
-<signal name="FOO">
-<polygon width="0.1" layer="16" orphans="yes" rank="6">
-<vertex x="0.3175" y="33.02"/>
-<vertex x="25.7175" y="33.02"/>
-<vertex x="25.7175" y="0.3175"/>
-<vertex x="0.3175" y="0.3175"/>
-</polygon>
 </signal>
 <signal name="TIM1_1">
@@
 <contactref element="IC3" pad="1"/>
 <contactref element="U$1" pad="1"/>
-<wire x1="53.85" y1="60.655" x2="52.405" y2="60.655" width="0.4064" layer="16"/>
-<wire x1="52.405" y1="60.655" x2="51.5" y2="59.75" width="0.4064" layer="16"/>
-<wire x1="51.5" y1="59.75" x2="51.5" y2="56.25" width="0.4064" layer="16"/>
-<wire x1="51.5" y1="56.25" x2="52.5" y2="55.25" width="0.4064" layer="16"/>
-<wire x1="52.5" y1="55.25" x2="54.25" y2="55.25" width="0.4064" layer="16"/>
-<wire x1="54.25" y1="55.25" x2="55" y2="54.5" width="0.4064" layer="16"/>
-<wire x1="55" y1="54.5" x2="55" y2="52.9184" width="0.4064" layer="16"/>
-<wire x1="55" y1="52.9184" x2="55.095" y2="52.8234" width="0.4064" layer="16"/>
+<contactref element="C21" pad="+"/>
+<wire x1="55.1" y1="59.905" x2="57.25" y2="59.905" width="0.3" layer="16"/>
+<wire x1="57.25" y1="59.905" x2="57.25" y2="60.125" width="0.3" layer="16"/>
+<wire x1="55.1" y1="59.905" x2="53.655" y2="59.905" width="0.3" layer="16"/>
+<wire x1="53.655" y1="59.905" x2="53" y2="59.25" width="0.3" layer="16"/>
+<wire x1="53" y1="59.25" x2="53" y2="56" width="0.3" layer="16"/>
+<wire x1="53" y1="56" x2="55" y2="54" width="0.3" layer="16"/>
+<wire x1="55" y1="54" x2="55" y2="52.9184" width="0.3" layer="16"/>
+<wire x1="55" y1="52.9184" x2="55.095" y2="52.8234" width="0.3" layer="16"/>
 </signal>
 <signal name="ISO_GND">
@@
 <contactref element="U$2" pad="VIN-"/>
 <polygon width="0.4064" layer="16">
-<vertex x="46" y="72.75"/>
-<vertex x="63.75" y="72.75"/>
+<vertex x="45" y="75"/>
+<vertex x="63.75" y="75"/>
 <vertex x="63.75" y="50.5"/>
-<vertex x="46" y="50.5"/>
+<vertex x="45" y="50.5"/>
 </polygon>
 <contactref element="X2" pad="8"/>
+<contactref element="C20" pad="-"/>
+<contactref element="C21" pad="-"/>
 </signal>
 <signal name="N$17">
 <contactref element="U$2" pad="VIN+"/>
 <contactref element="IC3" pad="8"/>
-<wire x1="48.65" y1="60.655" x2="47" y2="60.655" width="0.4064" layer="16"/>
-<wire x1="47" y1="60.655" x2="47" y2="54" width="0.4064" layer="16"/>
-<wire x1="47" y1="54" x2="49.75" y2="51.25" width="0.4064" layer="16"/>
-<wire x1="49.75" y1="51.25" x2="52.27" y2="51.25" width="0.4064" layer="16"/>
-<wire x1="52.27" y1="51.25" x2="52.5" y2="51.02" width="0.4064" layer="16"/>
 <contactref element="X2" pad="7"/>
-<wire x1="52.0375" y1="66.185" x2="48.435" y2="66.185" width="0.4064" layer="16"/>
-<wire x1="48.435" y1="66.185" x2="47" y2="64.75" width="0.4064" layer="16"/>
-<wire x1="47" y1="64.75" x2="47" y2="60.655" width="0.4064" layer="16"/>
+<contactref element="C20" pad="+"/>
+<wire x1="49.9" y1="59.905" x2="47.75" y2="59.905" width="0.3" layer="16"/>
+<wire x1="47.75" y1="59.905" x2="47.75" y2="60.125" width="0.3" layer="16"/>
+<wire x1="52.0375" y1="66.185" x2="52.0375" y2="60.655" width="0.3" layer="16"/>
+<wire x1="52.0375" y1="60.655" x2="52.0375" y2="56.0375" width="0.3" layer="16"/>
+<wire x1="52.0375" y1="56.0375" x2="50.25" y2="54.25" width="0.3" layer="16"/>
+<wire x1="50.25" y1="54.25" x2="50.25" y2="51.75" width="0.3" layer="16"/>
+<wire x1="50.25" y1="51.75" x2="51" y2="51" width="0.3" layer="16"/>
+<wire x1="51" y1="51" x2="52.48" y2="51" width="0.3" layer="16"/>
+<wire x1="52.48" y1="51" x2="52.5" y2="51.02" width="0.3" layer="16"/>
+<wire x1="49.9" y1="59.905" x2="52.0375" y2="60.655" width="0.3" layer="16"/>
 </signal>
 <signal name="N$13">
 <contactref element="X2" pad="4"/>
 <contactref element="U$1" pad="2"/>
-<wire x1="56.365" y1="52.8234" x2="56.365" y2="63.1275" width="0.4064" layer="16"/>
-<wire x1="56.365" y1="63.1275" x2="55.8475" y2="63.645" width="0.4064" layer="16"/>
+<wire x1="55.8475" y1="63.645" x2="55.8475" y2="62.9025" width="0.3" layer="16"/>
+<wire x1="55.8475" y1="62.9025" x2="56.25" y2="62.5" width="0.3" layer="16"/>
+<wire x1="56.25" y1="62.5" x2="58.5" y2="62.5" width="0.3" layer="16"/>
+<wire x1="58.5" y1="62.5" x2="59.75" y2="61.25" width="0.3" layer="16"/>
+<wire x1="59.75" y1="61.25" x2="59.75" y2="57" width="0.3" layer="16"/>
+<wire x1="59.75" y1="57" x2="56.5" y2="54" width="0.3" layer="16"/>
+<wire x1="56.5" y1="54" x2="56.5" y2="53" width="0.3" layer="16"/>
+<wire x1="56.5" y1="53" x2="56.4384" y2="52.9384" width="0.3" layer="16"/>
+<wire x1="56.4384" y1="52.9384" x2="56.25" y2="52.9384" width="0.3" layer="16"/>
+<wire x1="56.25" y1="52.9384" x2="56.365" y2="52.8234" width="0.3" layer="16"/>
 </signal>
 <signal name="N$14">
 <contactref element="U$1" pad="3"/>
 <contactref element="X2" pad="5"/>
-<wire x1="57.635" y1="52.8234" x2="57.635" y2="61.865" width="0.4064" layer="16"/>
-<wire x1="57.635" y1="61.865" x2="57.25" y2="62.25" width="0.4064" layer="16"/>
-<wire x1="57.25" y1="62.25" x2="57.25" y2="64" width="0.4064" layer="16"/>
-<wire x1="57.25" y1="64" x2="56" y2="65.25" width="0.4064" layer="16"/>
-<wire x1="56" y1="65.25" x2="55.5125" y2="65.25" width="0.4064" layer="16"/>
-<wire x1="55.5125" y1="65.25" x2="54.5775" y2="66.185" width="0.4064" layer="16"/>
+<wire x1="54.5775" y1="66.185" x2="54.5775" y2="66.1725" width="0.3" layer="16"/>
+<wire x1="54.5775" y1="66.1725" x2="55.75" y2="65" width="0.3" layer="16"/>
+<wire x1="55.75" y1="65" x2="59" y2="65" width="0.3" layer="16"/>
+<wire x1="59" y1="65" x2="60.75" y2="63" width="0.3" layer="16"/>
+<wire x1="60.75" y1="63" x2="60.75" y2="56.75" width="0.3" layer="16"/>
+<wire x1="60.75" y1="56.75" x2="57.75" y2="54" width="0.3" layer="16"/>
+<wire x1="57.75" y1="54" x2="57.75" y2="53" width="0.3" layer="16"/>
+<wire x1="57.75" y1="53" x2="57.7084" y2="52.9584" width="0.3" layer="16"/>
+<wire x1="57.7084" y1="52.9584" x2="57.5" y2="52.9584" width="0.3" layer="16"/>
+<wire x1="57.5" y1="52.9584" x2="57.635" y2="52.8234" width="0.3" layer="16"/>
 </signal>
 </signals>

Commit message: iramx v3
Parts:
- added H4: MOUNT-PAD-ROUND3.2, holes:3,2-PAD
- added R8: (no value), rcl:R0805
- moved R2 27.0 mm to (66.5, 33.5), turned to 90 degrees
- moved C26 3.20 mm to (56.0, 41.2), turned to 270 degrees
- moved R13 1.25 mm to (65.5, 5.25), turned to 90 degrees
- moved D2 1.03 mm to (64.5, 33.5)
- moved C10 1.00 mm to (89.2, 39.2)
- moved C24 1.00 mm to (87.3, 39.2)
- moved C11 0.79 mm to (87.5, 45.0)
- moved R4 0.71 mm to (64.5, 25.5)
- moved C4 0.35 mm to (89.5, 44.7)
- moved C15 0.25 mm to (93.8, 44.7)
- moved C16 0.25 mm to (91.5, 45.0)
- moved R1 0.25 mm to (96.5, 44.0)
- moved R23 0.25 mm to (87.2, 16.5)
- moved R6 0.25 mm to (87.5, 21.8)
- moved R7 0.25 mm to (85.5, 22.8)
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Connections:
- net N$2 renamed U
- net N$37 renamed V+
- net N$4 renamed V
- net N$6 renamed W
- new net V-: C11.2, C15.2, C16.2, C17.-, C4.2, IC1.12, R8.2, X4.2
- net GND: now also R8.1; no longer C11.2, C15.2, C16.2, C17.-, C4.2, IC1.12, X4.2
Routing:
- net V+: track 58.8 -> 2.08 mm
- net U: track 27.6 -> 2.23 mm
- net V: track 19.7 -> 2.36 mm
- net W: track 11.6 -> 2.35 mm
- net VLT: track 61.2 -> 63.2 mm
- net +3V3: track 159.1 -> 160.9 mm
- net +15V: track 55.5 -> 54.8 mm
- added copper zone on layer 16, net U
- added copper zone on layer 16, net V
- added copper zone on layer 16, net V+
- added copper zone on layer 16, net V-
- added copper zone on layer 16, net W

Commit message: iramx v3
Parts:
- moved R2 4.61 mm to (63.0, 30.5), turned to 0 degrees
- moved D2 1.25 mm to (65.8, 33.5)
Routing:
- net VLT: track 63.2 -> 61.5 mm

Commit message: iramx v3
Parts:
- moved R8 0.25 mm to (83.2, 41.0)
Changed lines of the file:
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@@
 <element name="C21" library="rcl" package="A/3216-18R" value="" x="57.25" y="58.75" rot="MR90"/>
 <element name="H4" library="holes" package="3,2-PAD" value="MOUNT-PAD-ROUND3.2" x="50" y="40"/>
-<element name="R8" library="rcl" package="R0805" value="" x="83.25" y="41.25" rot="MR90"/>
+<element name="R8" library="rcl" package="R0805" value="" x="83.25" y="41" rot="MR90"/>
 </elements>
 <signals>

Commit message: iramx v3
Parts:
- removed X2: (no value), con-appsys:RJ45
- added X1: (no value), reroolib:RJ45
- moved H2 90.0 mm to (5.00, 5.00), turned to 270 degrees
- moved JP1 78.4 mm to (4.00, 19.0), turned to 270 degrees
- moved C12 73.8 mm to (5.50, 22.8), turned to 90 degrees
- moved R11 73.0 mm to (19.3, 8.50), turned to 180 degrees
- moved Q1 72.0 mm to (6.50, 23.5), turned to 0 degrees
- moved C7 71.4 mm to (7.50, 22.8), turned to 90 degrees
- moved LED4 71.0 mm to (3.25, 31.8), turned to 180 degrees
- moved R23 70.8 mm to (16.5, 12.8), turned to 270 degrees
- moved R5 70.7 mm to (4.50, 29.2), turned to 270 degrees
- moved C28 70.6 mm to (13.2, 16.2), turned to 0 degrees
- moved H1 69.6 mm to (70.0, 5.00), turned to 270 degrees
- moved C18 69.5 mm to (10.5, 20.8), turned to 180 degrees
- moved LED1 68.9 mm to (3.25, 36.3), turned to 180 degrees
- moved C23 67.4 mm to (14.0, 18.8), turned to 180 degrees
- moved LED3 67.4 mm to (3.25, 40.8), turned to 180 degrees
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Connections:
- net ISO_GND: now also X1.8; no longer X2.8
- net N$13: now also X1.4; no longer X2.4
- net N$14: now also X1.5; no longer X2.5
- net N$17: now also X1.7; no longer X2.7
Routing:
- net N$17: track 22.6 -> 24.6 mm
- net N$14: track 19.6 -> 19.0 mm
Other:
- board size 55 x 75 mm -> 75 x 55 mm
