File: hw/eagle/IRAMX-drv-v3.brd (EAGLE design)
At the start: 75 x 55 mm, 59 parts, among them IC1 IRAMTOP, IC2 STM32F103R6T, IC3 78L05SMD, IC4 78L05SMD

Commit message: iramxv3
Parts:
- moved X3 0.50 mm to (70.0, 16.5)
- moved X4 0.50 mm to (70.0, 30.5)
Routing:
- net AMP: track 67.8 -> 67.1 mm
Changed lines of the file:
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@@
 <element name="R13" library="rcl" package="R0805" value="470" x="5.2475" y="34.5025" rot="MR180"/>
 <element name="IC1" library="iram-b" package="SIP23_TOP" value="IRAMTOP" x="62.9975" y="8.505"/>
-<element name="X3" library="con-wago-508" package="W237-133" value="" x="69.9975" y="16.995" rot="R90">
-<attribute name="OC_NEWARK" value="unknown" x="69.9975" y="16.995" size="1.778" layer="27" rot="R90" display="off"/>
-<attribute name="MPN" value="" x="69.9975" y="16.995" size="1.778" layer="27" rot="R90" display="off"/>
-<attribute name="MF" value="" x="69.9975" y="16.995" size="1.778" layer="27" rot="R90" display="off"/>
-<attribute name="OC_FARNELL" value="unknown" x="69.9975" y="16.995" size="1.778" layer="27" rot="R90" display="off"/>
+<element name="X3" library="con-wago-508" package="W237-133" value="" x="69.9975" y="16.495" rot="R90">
+<attribute name="OC_NEWARK" value="unknown" x="69.9975" y="16.495" size="1.778" layer="27" rot="R90" display="off"/>
+<attribute name="MPN" value="" x="69.9975" y="16.495" size="1.778" layer="27" rot="R90" display="off"/>
+<attribute name="MF" value="" x="69.9975" y="16.495" size="1.778" layer="27" rot="R90" display="off"/>
+<attribute name="OC_FARNELL" value="unknown" x="69.9975" y="16.495" size="1.778" layer="27" rot="R90" display="off"/>
 </element>
-<element name="X4" library="con-wago-508" package="W237-132" value="" x="69.9975" y="30" rot="R90">
-<attribute name="OC_NEWARK" value="unknown" x="69.9975" y="30" size="1.778" layer="27" rot="R90" display="off"/>
-<attribute name="MPN" value="" x="69.9975" y="30" size="1.778" layer="27" rot="R90" display="off"/>
-<attribute name="MF" value="" x="69.9975" y="30" size="1.778" layer="27" rot="R90" display="off"/>
-<attribute name="OC_FARNELL" value="unknown" x="69.9975" y="30" size="1.778" layer="27" rot="R90" display="off"/>
+<element name="X4" library="con-wago-508" package="W237-132" value="" x="69.9975" y="30.5" rot="R90">
+<attribute name="OC_NEWARK" value="unknown" x="69.9975" y="30.5" size="1.778" layer="27" rot="R90" display="off"/>
+<attribute name="MPN" value="" x="69.9975" y="30.5" size="1.778" layer="27" rot="R90" display="off"/>
+<attribute name="MF" value="" x="69.9975" y="30.5" size="1.778" layer="27" rot="R90" display="off"/>
+<attribute name="OC_FARNELL" value="unknown" x="69.9975" y="30.5" size="1.778" layer="27" rot="R90" display="off"/>
 </element>
 <element name="C17" library="rcl" package="EB35D" value="1000µ" x="47.749071875" y="27.003028125" rot="R135"/>
@@
 <wire x1="16.4975" y1="36.5" x2="16.4975" y2="34.0025" width="0.3" layer="16"/>
 <wire x1="16.4975" y1="34.0025" x2="17.00305625" y2="33.49694375" width="0.3" layer="16"/>
-<wire x1="18.3025" y1="8.5" x2="10" y2="8.5" width="0.3" layer="16"/>
-<wire x1="10" y1="8.5" x2="1.75" y2="16.75" width="0.3" layer="16"/>
-<wire x1="1.75" y1="16.75" x2="1.75" y2="30" width="0.3" layer="16"/>
+<wire x1="18.3025" y1="8.5" x2="11.25" y2="8.5" width="0.3" layer="16"/>
+<wire x1="11.25" y1="8.5" x2="1.75" y2="18" width="0.3" layer="16"/>
+<wire x1="1.75" y1="18" x2="1.75" y2="30" width="0.3" layer="16"/>
 <wire x1="1.75" y1="30" x2="3.25" y2="31.25" width="0.3" layer="16"/>
 <wire x1="3.25" y1="31.25" x2="3.25" y2="41.75" width="0.3" layer="16"/>
@@
 <wire x1="35.25" y1="45.875" x2="35.47" y2="45.875" width="0.3" layer="16"/>
 <wire x1="35.47" y1="45.875" x2="35.5" y2="45.845" width="0.3" layer="16"/>
-<via x="33.5" y="43" extent="1-16" drill="0.8" diameter="1.4224"/>
-<wire x1="33.5" y1="43" x2="33.5" y2="37.5" width="0.3" layer="1"/>
-<via x="33.5" y="37.5" extent="1-16" drill="0.8" diameter="1.4224"/>
-<wire x1="33.5" y1="37.5" x2="33.5" y2="31.75" width="0.3" layer="16"/>
-<wire x1="33.5" y1="43" x2="33.5" y2="45.745" width="0.3" layer="16"/>
-<wire x1="33.5" y1="45.745" x2="32.6" y2="45.845" width="0.3" layer="16"/>
+<via x="33.25" y="43" extent="1-16" drill="0.8" diameter="1.4224"/>
+<wire x1="33.25" y1="43" x2="33.25" y2="37.5" width="0.3" layer="1"/>
+<via x="33.25" y="37.5" extent="1-16" drill="0.8" diameter="1.4224"/>
+<wire x1="33.25" y1="37.5" x2="33.25" y2="32" width="0.3" layer="16"/>
+<wire x1="33.25" y1="43" x2="33.25" y2="45.745" width="0.3" layer="16"/>
+<wire x1="33.25" y1="45.745" x2="32.6" y2="45.845" width="0.3" layer="16"/>
 <wire x1="39.0275" y1="8.425" x2="38.25" y2="9.2025" width="0.3" layer="16"/>
 <wire x1="38.25" y1="9.2025" x2="38.25" y2="10.75" width="0.3" layer="16"/>
 <wire x1="38.25" y1="10.75" x2="38.2475" y2="10.7525" width="0.3" layer="16"/>
 <wire x1="38.2475" y1="10.7525" x2="38.2475" y2="12.7475" width="0.3" layer="16"/>
-<wire x1="38.2475" y1="27.0025" x2="33.5" y2="31.75" width="0.3" layer="16"/>
+<wire x1="38.2475" y1="27.0025" x2="33.25" y2="32" width="0.3" layer="16"/>
 <wire x1="38.2475" y1="27.0025" x2="38.2475" y2="12.7475" width="0.3" layer="16"/>
 </signal>
@@
 <wire x1="59.905" y1="42.75" x2="60.125" y2="42.75" width="0.3" layer="16"/>
 <wire x1="59.905" y1="44.9" x2="59.905" y2="46.345" width="0.3" layer="16"/>
-<wire x1="59.905" y1="46.345" x2="59.25" y2="47" width="0.3" layer="16"/>
-<wire x1="59.25" y1="47" x2="56" y2="47" width="0.3" layer="16"/>
-<wire x1="56" y1="47" x2="54" y2="45" width="0.3" layer="16"/>
+<wire x1="59.905" y1="46.345" x2="59.5" y2="46.75" width="0.3" layer="16"/>
+<wire x1="59.5" y1="46.75" x2="55.75" y2="46.75" width="0.3" layer="16"/>
+<wire x1="55.75" y1="46.75" x2="54" y2="45" width="0.3" layer="16"/>
 <wire x1="54" y1="45" x2="52.9184" y2="45" width="0.3" layer="16"/>
 <wire x1="52.9184" y1="45" x2="52.5734" y2="44.905" width="0.3" layer="16"/>
@@
 <wire x1="59.905" y1="50.1" x2="59.905" y2="52.25" width="0.3" layer="16"/>
 <wire x1="59.905" y1="52.25" x2="60.125" y2="52.25" width="0.3" layer="16"/>
-<wire x1="59.905" y1="47.9625" x2="56.0375" y2="47.9625" width="0.3" layer="16"/>
-<wire x1="56.0375" y1="47.9625" x2="54" y2="50" width="0.3" layer="16"/>
+<wire x1="59.905" y1="48.2125" x2="55.7875" y2="48.2125" width="0.3" layer="16"/>
+<wire x1="55.7875" y1="48.2125" x2="54" y2="50" width="0.3" layer="16"/>
 <wire x1="54" y1="50" x2="52" y2="50" width="0.3" layer="16"/>
 <wire x1="52" y1="50" x2="51" y2="49" width="0.3" layer="16"/>
@@
 <wire x1="51" y1="47.52" x2="51.02" y2="47.5" width="0.3" layer="16"/>
 <wire x1="59.905" y1="50.1" x2="59.905" y2="48.5" width="0.3" layer="16"/>
-<wire x1="59.905" y1="48.5" x2="59.905" y2="47.9625" width="0.3" layer="16"/>
+<wire x1="59.905" y1="48.5" x2="59.905" y2="48.2125" width="0.3" layer="16"/>
 <wire x1="59.905" y1="50.1" x2="59.905" y2="52" width="0.3" layer="16"/>
 <contactref element="X1" pad="7"/>
