File: hw/eagle/IRAMX-drv-v3.sch (EAGLE design)
At the start: 54 parts, among them IC1 IRAMTOP, IC2 STM32F103R6T, IC4 78L05SMD

Commit message: iramx v3
Parts:
- added D2: (no value), diode:ZENER-DIODESOD80C
Connections:
- net GND: now also D2.A
- net VLT: now also D2.C
Changed lines of the file:
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@@
 <grid distance="0.1" unitdist="inch" unit="inch" style="lines" multiple="1" display="no" altdistance="0.01" altunitdist="inch" altunit="inch"/>
 <layers>
-<layer number="1" name="Top" color="4" fill="1" visible="no" active="no"/>
-<layer number="16" name="Bottom" color="1" fill="1" visible="no" active="no"/>
-<layer number="17" name="Pads" color="2" fill="1" visible="no" active="no"/>
-<layer number="18" name="Vias" color="2" fill="1" visible="no" active="no"/>
-<layer number="19" name="Unrouted" color="6" fill="1" visible="no" active="no"/>
-<layer number="20" name="Dimension" color="15" fill="1" visible="no" active="no"/>
-<layer number="21" name="tPlace" color="7" fill="1" visible="no" active="no"/>
-<layer number="22" name="bPlace" color="7" fill="1" visible="no" active="no"/>
-<layer number="23" name="tOrigins" color="15" fill="1" visible="no" active="no"/>
-<layer number="24" name="bOrigins" color="15" fill="1" visible="no" active="no"/>
-<layer number="25" name="tNames" color="7" fill="1" visible="no" active="no"/>
-<layer number="26" name="bNames" color="7" fill="1" visible="no" active="no"/>
-<layer number="27" name="tValues" color="7" fill="1" visible="no" active="no"/>
-<layer number="28" name="bValues" color="7" fill="1" visible="no" active="no"/>
+<layer number="1" name="Top" color="4" fill="1" visible="yes" active="no"/>
+<layer number="16" name="Bottom" color="1" fill="1" visible="yes" active="no"/>
+<layer number="17" name="Pads" color="2" fill="1" visible="yes" active="no"/>
+<layer number="18" name="Vias" color="2" fill="1" visible="yes" active="no"/>
+<layer number="19" name="Unrouted" color="6" fill="1" visible="yes" active="no"/>
+<layer number="20" name="Dimension" color="15" fill="1" visible="yes" active="no"/>
+<layer number="21" name="tPlace" color="7" fill="1" visible="yes" active="no"/>
+<layer number="22" name="bPlace" color="7" fill="1" visible="yes" active="no"/>
+<layer number="23" name="tOrigins" color="15" fill="1" visible="yes" active="no"/>
+<layer number="24" name="bOrigins" color="15" fill="1" visible="yes" active="no"/>
+<layer number="25" name="tNames" color="7" fill="1" visible="yes" active="no"/>
+<layer number="26" name="bNames" color="7" fill="1" visible="yes" active="no"/>
+<layer number="27" name="tValues" color="7" fill="1" visible="yes" active="no"/>
+<layer number="28" name="bValues" color="7" fill="1" visible="yes" active="no"/>
 <layer number="29" name="tStop" color="7" fill="3" visible="no" active="no"/>
 <layer number="30" name="bStop" color="7" fill="6" visible="no" active="no"/>
@@
 <layer number="35" name="tGlue" color="7" fill="4" visible="no" active="no"/>
 <layer number="36" name="bGlue" color="7" fill="5" visible="no" active="no"/>
-<layer number="37" name="tTest" color="7" fill="1" visible="no" active="no"/>
-<layer number="38" name="bTest" color="7" fill="1" visible="no" active="no"/>
+<layer number="37" name="tTest" color="7" fill="1" visible="yes" active="no"/>
+<layer number="38" name="bTest" color="7" fill="1" visible="yes" active="no"/>
 <layer number="39" name="tKeepout" color="4" fill="11" visible="no" active="no"/>
 <layer number="40" name="bKeepout" color="1" fill="11" visible="no" active="no"/>
@@
 <layer number="44" name="Drills" color="7" fill="1" visible="no" active="no"/>
 <layer number="45" name="Holes" color="7" fill="1" visible="no" active="no"/>
-<layer number="46" name="Milling" color="3" fill="1" visible="no" active="no"/>
-<layer number="47" name="Measures" color="7" fill="1" visible="no" active="no"/>
-<layer number="48" name="Document" color="7" fill="1" visible="no" active="no"/>
-<layer number="49" name="Reference" color="7" fill="1" visible="no" active="no"/>
-<layer number="50" name="dxf" color="7" fill="1" visible="no" active="no"/>
-<layer number="51" name="tDocu" color="7" fill="1" visible="no" active="no"/>
-<layer number="52" name="bDocu" color="7" fill="1" visible="no" active="no"/>
-<layer number="53" name="tGND_GNDA" color="7" fill="9" visible="no" active="no"/>
-<layer number="54" name="bGND_GNDA" color="1" fill="9" visible="no" active="no"/>
-<layer number="56" name="wert" color="7" fill="1" visible="no" active="no"/>
+<layer number="46" name="Milling" color="3" fill="1" visible="yes" active="no"/>
+<layer number="47" name="Measures" color="7" fill="1" visible="yes" active="no"/>
+<layer number="48" name="Document" color="7" fill="1" visible="yes" active="no"/>
+<layer number="49" name="Reference" color="7" fill="1" visible="yes" active="no"/>
+<layer number="50" name="dxf" color="7" fill="1" visible="yes" active="no"/>
+<layer number="51" name="tDocu" color="7" fill="1" visible="yes" active="no"/>
+<layer number="52" name="bDocu" color="7" fill="1" visible="yes" active="no"/>
+<layer number="53" name="tGND_GNDA" color="7" fill="9" visible="yes" active="no"/>
+<layer number="54" name="bGND_GNDA" color="1" fill="9" visible="yes" active="no"/>
+<layer number="56" name="wert" color="7" fill="1" visible="yes" active="no"/>
 <layer number="91" name="Nets" color="2" fill="1" visible="yes" active="yes"/>
 <layer number="92" name="Busses" color="1" fill="1" visible="yes" active="yes"/>
@@
 <part name="GND11" library="supply1" deviceset="GND" device=""/>
 <part name="+3V5" library="supply1" deviceset="+3V3" device=""/>
+<part name="D2" library="diode" deviceset="ZENER-DIODE" device="SOD80C"/>
+<part name="GND13" library="supply1" deviceset="GND" device=""/>
 </parts>
 <sheets>
@@
 <instance part="GND11" gate="1" x="195.58" y="-58.42"/>
 <instance part="+3V5" gate="G$1" x="195.58" y="-33.02"/>
+<instance part="D2" gate="G$1" x="96.52" y="83.82" rot="R270"/>
+<instance part="GND13" gate="1" x="96.52" y="96.52" rot="R180"/>
 </instances>
 <busses>
@@
 <pinref part="GND11" gate="1" pin="GND"/>
 </segment>
+<segment>
+<pinref part="D2" gate="G$1" pin="A"/>
+<pinref part="GND13" gate="1" pin="GND"/>
+<wire x1="96.52" y1="93.98" x2="96.52" y2="86.36" width="0.1524" layer="91"/>
+</segment>
 </net>
 <net name="EN" class="0">
@@
 <pinref part="R10" gate="G$1" pin="2"/>
 <junction x="96.52" y="22.86"/>
+<label x="106.68" y="22.86" size="1.778" layer="95"/>
 <wire x1="114.3" y1="22.86" x2="96.52" y2="22.86" width="0.1524" layer="91"/>
-<label x="106.68" y="22.86" size="1.778" layer="95"/>
 </segment>
 <segment>
@@
 <wire x1="109.22" y1="81.28" x2="104.14" y2="81.28" width="0.1524" layer="91"/>
 <junction x="104.14" y="81.28"/>
-<wire x1="104.14" y1="81.28" x2="88.9" y2="81.28" width="0.1524" layer="91"/>
+<wire x1="104.14" y1="81.28" x2="96.52" y2="81.28" width="0.1524" layer="91"/>
 <label x="88.9" y="81.28" size="1.778" layer="95"/>
-</segment>
-<segment>
+<pinref part="D2" gate="G$1" pin="C"/>
+<wire x1="96.52" y1="81.28" x2="88.9" y2="81.28" width="0.1524" layer="91"/>
+<junction x="96.52" y="81.28"/>
+</segment>
+<segment>

Commit message: iramxv3 rj45
Parts:
- added IC3: 78L05SMD, linear:78L05SMD
Connections:
- new net ISO_GND: IC3G$1.GND@1, IC3G$1.GND@2, IC3G$1.GND@3, IC3G$1.GND@4, U$1.GND1, U$2.VIN-, X2-.8
- new net N$11: IC3G$1.VOUT, U$1.VDD1
- new net N$13: U$1.IN1, X2-.4
- new net N$14: U$1.OUT2, X2-.5
- new net N$17: IC3G$1.VIN, U$2.VIN+, X2-.7
Other:
- moved on the sheet: X2-
Changed lines of the file:
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@@
 <?xml version="1.0" encoding="utf-8"?>
 <!DOCTYPE eagle SYSTEM "eagle.dtd">
-<eagle version="6.5.0">
+<eagle version="7.1.0">
 <drawing>
 <settings>
@@
 <grid distance="0.1" unitdist="inch" unit="inch" style="lines" multiple="1" display="no" altdistance="0.01" altunitdist="inch" altunit="inch"/>
 <layers>
-<layer number="1" name="Top" color="4" fill="1" visible="yes" active="no"/>
-<layer number="16" name="Bottom" color="1" fill="1" visible="yes" active="no"/>
-<layer number="17" name="Pads" color="2" fill="1" visible="yes" active="no"/>
-<layer number="18" name="Vias" color="2" fill="1" visible="yes" active="no"/>
-<layer number="19" name="Unrouted" color="6" fill="1" visible="yes" active="no"/>
-<layer number="20" name="Dimension" color="15" fill="1" visible="yes" active="no"/>
-<layer number="21" name="tPlace" color="7" fill="1" visible="yes" active="no"/>
-<layer number="22" name="bPlace" color="7" fill="1" visible="yes" active="no"/>
-<layer number="23" name="tOrigins" color="15" fill="1" visible="yes" active="no"/>
-<layer number="24" name="bOrigins" color="15" fill="1" visible="yes" active="no"/>
-<layer number="25" name="tNames" color="7" fill="1" visible="yes" active="no"/>
-<layer number="26" name="bNames" color="7" fill="1" visible="yes" active="no"/>
-<layer number="27" name="tValues" color="7" fill="1" visible="yes" active="no"/>
-<layer number="28" name="bValues" color="7" fill="1" visible="yes" active="no"/>
+<layer number="1" name="Top" color="4" fill="1" visible="no" active="no"/>
+<layer number="16" name="Bottom" color="1" fill="1" visible="no" active="no"/>
+<layer number="17" name="Pads" color="2" fill="1" visible="no" active="no"/>
+<layer number="18" name="Vias" color="2" fill="1" visible="no" active="no"/>
+<layer number="19" name="Unrouted" color="6" fill="1" visible="no" active="no"/>
+<layer number="20" name="Dimension" color="15" fill="1" visible="no" active="no"/>
+<layer number="21" name="tPlace" color="7" fill="1" visible="no" active="no"/>
+<layer number="22" name="bPlace" color="7" fill="1" visible="no" active="no"/>
+<layer number="23" name="tOrigins" color="15" fill="1" visible="no" active="no"/>
+<layer number="24" name="bOrigins" color="15" fill="1" visible="no" active="no"/>
+<layer number="25" name="tNames" color="7" fill="1" visible="no" active="no"/>
+<layer number="26" name="bNames" color="7" fill="1" visible="no" active="no"/>
+<layer number="27" name="tValues" color="7" fill="1" visible="no" active="no"/>
+<layer number="28" name="bValues" color="7" fill="1" visible="no" active="no"/>
 <layer number="29" name="tStop" color="7" fill="3" visible="no" active="no"/>
 <layer number="30" name="bStop" color="7" fill="6" visible="no" active="no"/>
@@
 <layer number="35" name="tGlue" color="7" fill="4" visible="no" active="no"/>
 <layer number="36" name="bGlue" color="7" fill="5" visible="no" active="no"/>
-<layer number="37" name="tTest" color="7" fill="1" visible="yes" active="no"/>
-<layer number="38" name="bTest" color="7" fill="1" visible="yes" active="no"/>
+<layer number="37" name="tTest" color="7" fill="1" visible="no" active="no"/>
+<layer number="38" name="bTest" color="7" fill="1" visible="no" active="no"/>
 <layer number="39" name="tKeepout" color="4" fill="11" visible="no" active="no"/>
 <layer number="40" name="bKeepout" color="1" fill="11" visible="no" active="no"/>
@@
 <layer number="44" name="Drills" color="7" fill="1" visible="no" active="no"/>
 <layer number="45" name="Holes" color="7" fill="1" visible="no" active="no"/>
-<layer number="46" name="Milling" color="3" fill="1" visible="yes" active="no"/>
-<layer number="47" name="Measures" color="7" fill="1" visible="yes" active="no"/>
-<layer number="48" name="Document" color="7" fill="1" visible="yes" active="no"/>
-<layer number="49" name="Reference" color="7" fill="1" visible="yes" active="no"/>
-<layer number="50" name="dxf" color="7" fill="1" visible="yes" active="no"/>
-<layer number="51" name="tDocu" color="7" fill="1" visible="yes" active="no"/>
-<layer number="52" name="bDocu" color="7" fill="1" visible="yes" active="no"/>
-<layer number="53" name="tGND_GNDA" color="7" fill="9" visible="yes" active="no"/>
-<layer number="54" name="bGND_GNDA" color="1" fill="9" visible="yes" active="no"/>
-<layer number="56" name="wert" color="7" fill="1" visible="yes" active="no"/>
+<layer number="46" name="Milling" color="3" fill="1" visible="no" active="no"/>
+<layer number="47" name="Measures" color="7" fill="1" visible="no" active="no"/>
+<layer number="48" name="Document" color="7" fill="1" visible="no" active="no"/>
+<layer number="49" name="Reference" color="7" fill="1" visible="no" active="no"/>
+<layer number="50" name="dxf" color="7" fill="1" visible="no" active="no"/>
+<layer number="51" name="tDocu" color="7" fill="1" visible="no" active="no"/>
+<layer number="52" name="bDocu" color="7" fill="1" visible="no" active="no"/>
+<layer number="53" name="tGND_GNDA" color="7" fill="9" visible="no" active="no"/>
+<layer number="54" name="bGND_GNDA" color="1" fill="9" visible="no" active="no"/>
+<layer number="56" name="wert" color="7" fill="1" visible="no" active="no"/>
 <layer number="91" name="Nets" color="2" fill="1" visible="yes" active="yes"/>
 <layer number="92" name="Busses" color="1" fill="1" visible="yes" active="yes"/>
@@
 <part name="D2" library="diode" deviceset="ZENER-DIODE" device="SOD80C"/>
 <part name="GND13" library="supply1" deviceset="GND" device=""/>
+<part name="IC3" library="linear" deviceset="78L*SMD" device="" technology="05"/>
 </parts>
 <sheets>
@@
 <instance part="C2" gate="G$1" x="63.5" y="45.72" rot="R90"/>
 <instance part="C3" gate="G$1" x="63.5" y="35.56" rot="R90"/>
-<instance part="X2" gate="-" x="-129.54" y="53.34" rot="MR0"/>
+<instance part="X2" gate="-" x="-137.16" y="35.56" rot="MR0"/>
 <instance part="X2" gate="SHIELD@1" x="-136.906" y="64.77" rot="R180"/>
 <instance part="X2" gate="SHIELD@2" x="-140.462" y="64.77" rot="R180"/>
@@
 <instance part="D2" gate="G$1" x="96.52" y="83.82" rot="R270"/>
 <instance part="GND13" gate="1" x="96.52" y="96.52" rot="R180"/>
+<instance part="IC3" gate="G$1" x="-104.14" y="45.72"/>
 </instances>
 <busses>
@@
 </segment>
 </net>
+<net name="N$11" class="0">
+<segment>
+<pinref part="IC3" gate="G$1" pin="VOUT"/>
+<pinref part="U$1" gate="G$1" pin="VDD1"/>
+<wire x1="-91.44" y1="45.72" x2="-83.82" y2="45.72" width="0.1524" layer="91"/>
+</segment>
+</net>
+<net name="ISO_GND" class="0">
+<segment>
+<pinref part="U$1" gate="G$1" pin="GND1"/>
+<wire x1="-83.82" y1="38.1" x2="-86.36" y2="38.1" width="0.1524" layer="91"/>
+<wire x1="-86.36" y1="38.1" x2="-86.36" y2="27.94" width="0.1524" layer="91"/>
+<pinref part="IC3" gate="G$1" pin="GND@4"/>
+<wire x1="-86.36" y1="27.94" x2="-99.06" y2="27.94" width="0.1524" layer="91"/>
+<wire x1="-99.06" y1="27.94" x2="-99.06" y2="33.02" width="0.1524" layer="91"/>
+<pinref part="IC3" gate="G$1" pin="GND@3"/>
+<wire x1="-101.6" y1="33.02" x2="-101.6" y2="27.94" width="0.1524" layer="91"/>
+<wire x1="-101.6" y1="27.94" x2="-99.06" y2="27.94" width="0.1524" layer="91"/>
+<pinref part="IC3" gate="G$1" pin="GND@2"/>
+<wire x1="-104.14" y1="33.02" x2="-104.14" y2="27.94" width="0.1524" layer="91"/>
+<wire x1="-104.14" y1="27.94" x2="-101.6" y2="27.94" width="0.1524" layer="91"/>
+<pinref part="IC3" gate="G$1" pin="GND@1"/>
+<wire x1="-106.68" y1="33.02" x2="-106.68" y2="27.94" width="0.1524" layer="91"/>
+<wire x1="-106.68" y1="27.94" x2="-104.14" y2="27.94" width="0.1524" layer="91"/>
+<wire x1="-86.36" y1="27.94" x2="-38.1" y2="27.94" width="0.1524" layer="91"/>
+<wire x1="-38.1" y1="27.94" x2="-38.1" y2="111.76" width="0.1524" layer="91"/>
+<pinref part="U$2" gate="G$1" pin="VIN-"/>
+<wire x1="-38.1" y1="111.76" x2="-60.96" y2="111.76" width="0.1524" layer="91"/>
+<wire x1="-60.96" y1="111.76" x2="-60.96" y2="119.38" width="0.1524" layer="91"/>
+<junction x="-86.36" y="27.94"/>
+<junction x="-99.06" y="27.94"/>
+<junction x="-101.6" y="27.94"/>
+<junction x="-104.14" y="27.94"/>
+<pinref part="X2" gate="-" pin="8"/>
+<wire x1="-134.62" y1="27.94" x2="-106.68" y2="27.94" width="0.1524" layer="91"/>
+<junction x="-106.68" y="27.94"/>
+</segment>
+</net>
+<net name="N$17" class="0">
+<segment>
+<pinref part="U$2" gate="G$1" pin="VIN+"/>
+<wire x1="-60.96" y1="124.46" x2="-121.92" y2="124.46" width="0.1524" layer="91"/>
+<wire x1="-121.92" y1="124.46" x2="-121.92" y2="45.72" width="0.1524" layer="91"/>
+<pinref part="IC3" gate="G$1" pin="VIN"/>
+<wire x1="-121.92" y1="45.72" x2="-114.3" y2="45.72" width="0.1524" layer="91"/>
+<pinref part="X2" gate="-" pin="7"/>
+<wire x1="-134.62" y1="30.48" x2="-121.92" y2="30.48" width="0.1524" layer="91"/>
+<wire x1="-121.92" y1="30.48" x2="-121.92" y2="45.72" width="0.1524" layer="91"/>
+<junction x="-121.92" y="45.72"/>
+</segment>
+</net>
+<net name="N$13" class="0">
+<segment>
+<pinref part="X2" gate="-" pin="4"/>
+<wire x1="-134.62" y1="38.1" x2="-129.54" y2="38.1" width="0.1524" layer="91"/>
+<wire x1="-129.54" y1="38.1" x2="-129.54" y2="55.88" width="0.1524" layer="91"/>
+<wire x1="-129.54" y1="55.88" x2="-86.36" y2="55.88" width="0.1524" layer="91"/>
+<wire x1="-86.36" y1="55.88" x2="-86.36" y2="43.18" width="0.1524" layer="91"/>
+<pinref part="U$1" gate="G$1" pin="IN1"/>
+<wire x1="-86.36" y1="43.18" x2="-83.82" y2="43.18" width="0.1524" layer="91"/>
+</segment>
+</net>
+<net name="N$14" class="0">
+<segment>
+<pinref part="U$1" gate="G$1" pin="OUT2"/>
+<wire x1="-83.82" y1="40.64" x2="-88.9" y2="40.64" width="0.1524" layer="91"/>
+<wire x1="-88.9" y1="40.64" x2="-88.9" y2="58.42" width="0.1524" layer="91"/>
+<wire x1="-88.9" y1="58.42" x2="-132.08" y2="58.42" width="0.1524" layer="91"/>
+<wire x1="-132.08" y1="58.42" x2="-132.08" y2="35.56" width="0.1524" layer="91"/>
+<pinref part="X2" gate="-" pin="5"/>
+<wire x1="-132.08" y1="35.56" x2="-134.62" y2="35.56" width="0.1524" layer="91"/>
+</segment>
+</net>

Commit message: iramx v3
Parts:
- removed H4: MOUNT-PAD-ROUND3.2, holes:MOUNT-PAD-ROUND3.2
- added C20, C21: (no value), rcl:CPOL-EUA/3216-18R
Connections:
- net ISO_GND: now also C20.-, C21.-
- net N$11: now also C21.+
- net N$17: now also C20.+
Changed lines of the file:
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@@
 <?xml version="1.0" encoding="utf-8"?>
 <!DOCTYPE eagle SYSTEM "eagle.dtd">
-<eagle version="7.1.0">
+<eagle version="6.5.0">
 <drawing>
 <settings>
@@
 <part name="H2" library="holes" deviceset="MOUNT-PAD-ROUND" device="3.2"/>
 <part name="H3" library="holes" deviceset="MOUNT-PAD-ROUND" device="3.2"/>
-<part name="H4" library="holes" deviceset="MOUNT-PAD-ROUND" device="3.2"/>
 <part name="IC2" library="micro-stm_v2" deviceset="STM32F103R*T" device="" technology="6"/>
 <part name="C4" library="rcl" deviceset="C-EU" device="C1206K"/>
@@
 <part name="GND13" library="supply1" deviceset="GND" device=""/>
 <part name="IC3" library="linear" deviceset="78L*SMD" device="" technology="05"/>
+<part name="C20" library="rcl" deviceset="CPOL-EU" device="A/3216-18R"/>
+<part name="C21" library="rcl" deviceset="CPOL-EU" device="A/3216-18R"/>
 </parts>
 <sheets>
@@
 <instance part="H2" gate="G$1" x="175.26" y="109.22"/>
 <instance part="H3" gate="G$1" x="175.26" y="101.6"/>
-<instance part="H4" gate="G$1" x="175.26" y="93.98"/>
 <instance part="IC2" gate="MCU" x="45.72" y="-27.94"/>
 <instance part="C4" gate="G$1" x="66.04" y="68.58"/>
@@
 <instance part="GND13" gate="1" x="96.52" y="96.52" rot="R180"/>
 <instance part="IC3" gate="G$1" x="-104.14" y="45.72"/>
+<instance part="C20" gate="G$1" x="-116.84" y="43.18"/>
+<instance part="C21" gate="G$1" x="-91.44" y="43.18"/>
 </instances>
 <busses>
@@
 <pinref part="U$1" gate="G$1" pin="VDD1"/>
 <wire x1="-91.44" y1="45.72" x2="-83.82" y2="45.72" width="0.1524" layer="91"/>
+<pinref part="C21" gate="G$1" pin="+"/>
+<junction x="-91.44" y="45.72"/>
 </segment>
 </net>
@@
 <wire x1="-86.36" y1="38.1" x2="-86.36" y2="27.94" width="0.1524" layer="91"/>
 <pinref part="IC3" gate="G$1" pin="GND@4"/>
-<wire x1="-86.36" y1="27.94" x2="-99.06" y2="27.94" width="0.1524" layer="91"/>
+<wire x1="-86.36" y1="27.94" x2="-91.44" y2="27.94" width="0.1524" layer="91"/>
+<wire x1="-91.44" y1="27.94" x2="-99.06" y2="27.94" width="0.1524" layer="91"/>
 <wire x1="-99.06" y1="27.94" x2="-99.06" y2="33.02" width="0.1524" layer="91"/>
 <pinref part="IC3" gate="G$1" pin="GND@3"/>
@@
 <junction x="-104.14" y="27.94"/>
 <pinref part="X2" gate="-" pin="8"/>
-<wire x1="-134.62" y1="27.94" x2="-106.68" y2="27.94" width="0.1524" layer="91"/>
+<wire x1="-134.62" y1="27.94" x2="-116.84" y2="27.94" width="0.1524" layer="91"/>
 <junction x="-106.68" y="27.94"/>
+<pinref part="C20" gate="G$1" pin="-"/>
+<wire x1="-116.84" y1="27.94" x2="-106.68" y2="27.94" width="0.1524" layer="91"/>
+<wire x1="-116.84" y1="38.1" x2="-116.84" y2="27.94" width="0.1524" layer="91"/>
+<pinref part="C21" gate="G$1" pin="-"/>
+<wire x1="-91.44" y1="38.1" x2="-91.44" y2="27.94" width="0.1524" layer="91"/>
+<junction x="-116.84" y="27.94"/>
+<junction x="-91.44" y="27.94"/>
 </segment>
 </net>
@@
 <wire x1="-121.92" y1="124.46" x2="-121.92" y2="45.72" width="0.1524" layer="91"/>
 <pinref part="IC3" gate="G$1" pin="VIN"/>
-<wire x1="-121.92" y1="45.72" x2="-114.3" y2="45.72" width="0.1524" layer="91"/>
+<wire x1="-121.92" y1="45.72" x2="-116.84" y2="45.72" width="0.1524" layer="91"/>
 <pinref part="X2" gate="-" pin="7"/>
+<wire x1="-116.84" y1="45.72" x2="-114.3" y2="45.72" width="0.1524" layer="91"/>
 <wire x1="-134.62" y1="30.48" x2="-121.92" y2="30.48" width="0.1524" layer="91"/>
 <wire x1="-121.92" y1="30.48" x2="-121.92" y2="45.72" width="0.1524" layer="91"/>
 <junction x="-121.92" y="45.72"/>
-</segment>
-</net>
+<pinref part="C20" gate="G$1" pin="+"/>
+<junction x="-116.84" y="45.72"/>
+</segment>
+</net>
