File: hw/eagle/IRAMX-drv-v3.sch (EAGLE design)
At the start: 57 parts, among them IC1 IRAMTOP, IC2 STM32F103R6T, IC3 78L05SMD, IC4 78L05SMD

Commit message: iramx v3
Parts:
- added H4: MOUNT-PAD-ROUND3.2, holes:MOUNT-PAD-ROUND3.2
- added R8: (no value), rcl:R-EU_R0805
Connections:
- net N$2 renamed U
- net N$37 renamed V+
- net N$4 renamed V
- net N$6 renamed W
- new net V-: C11.2, C15.2, C16.2, C17.-, C4.2, IC1.V-, R8.2, X4-2.KL
- net GND: now also R8.1; no longer C11.2, C15.2, C16.2, C17.-, C4.2, IC1.V-, X4-2.KL
Changed lines of the file:
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@@
 <part name="C20" library="rcl" deviceset="CPOL-EU" device="A/3216-18R"/>
 <part name="C21" library="rcl" deviceset="CPOL-EU" device="A/3216-18R"/>
+<part name="H4" library="holes" deviceset="MOUNT-PAD-ROUND" device="3.2"/>
+<part name="R8" library="rcl" deviceset="R-EU_" device="R0805"/>
 </parts>
 <sheets>
@@
 <instance part="P+9" gate="1" x="-7.62" y="127"/>
 <instance part="GND22" gate="1" x="-25.4" y="104.14"/>
-<instance part="GND2" gate="1" x="96.52" y="53.34"/>
+<instance part="GND2" gate="1" x="96.52" y="48.26"/>
 <instance part="R23" gate="G$1" x="200.66" y="-45.72"/>
 <instance part="GND32" gate="1" x="10.16" y="63.5"/>
@@
 <instance part="C20" gate="G$1" x="-116.84" y="43.18"/>
 <instance part="C21" gate="G$1" x="-91.44" y="43.18"/>
+<instance part="H4" gate="G$1" x="175.26" y="93.98"/>
+<instance part="R8" gate="G$1" x="96.52" y="58.42" rot="R90"/>
 </instances>
 <busses>
@@
 </segment>
 </net>
-<net name="N$2" class="1">
+<net name="U" class="1">
 <segment>
 <wire x1="58.42" y1="50.8" x2="68.58" y2="50.8" width="0.1524" layer="91"/>
@@
 </segment>
 </net>
-<net name="N$4" class="1">
+<net name="V" class="1">
 <segment>
 <wire x1="58.42" y1="40.64" x2="68.58" y2="40.64" width="0.1524" layer="91"/>
@@
 </segment>
 </net>
-<net name="N$6" class="1">
+<net name="W" class="1">
 <segment>
 <wire x1="58.42" y1="30.48" x2="68.58" y2="30.48" width="0.1524" layer="91"/>
@@
 <wire x1="27.94" y1="66.04" x2="10.16" y2="66.04" width="0.1524" layer="91"/>
 <pinref part="GND32" gate="1" pin="GND"/>
-</segment>
-<segment>
-<wire x1="58.42" y1="63.5" x2="66.04" y2="63.5" width="0.1524" layer="91"/>
-<pinref part="IC1" gate="G$1" pin="V-"/>
-<wire x1="66.04" y1="63.5" x2="71.12" y2="63.5" width="0.1524" layer="91"/>
-<wire x1="71.12" y1="63.5" x2="76.2" y2="63.5" width="0.1524" layer="91"/>
-<wire x1="76.2" y1="63.5" x2="81.28" y2="63.5" width="0.1524" layer="91"/>
-<wire x1="81.28" y1="63.5" x2="96.52" y2="63.5" width="0.1524" layer="91"/>
-<wire x1="96.52" y1="55.88" x2="96.52" y2="63.5" width="0.1524" layer="91"/>
-<pinref part="C17" gate="G$1" pin="-"/>
-<junction x="96.52" y="63.5"/>
-<pinref part="GND2" gate="1" pin="GND"/>
-<pinref part="X4" gate="-2" pin="KL"/>
-<wire x1="109.22" y1="63.5" x2="96.52" y2="63.5" width="0.1524" layer="91"/>
-<junction x="96.52" y="63.5"/>
-<pinref part="C4" gate="G$1" pin="2"/>
-<junction x="66.04" y="63.5"/>
-<pinref part="C11" gate="G$1" pin="2"/>
-<junction x="81.28" y="63.5"/>
-<pinref part="C15" gate="G$1" pin="2"/>
-<junction x="76.2" y="63.5"/>
-<pinref part="C16" gate="G$1" pin="2"/>
-<junction x="71.12" y="63.5"/>
 </segment>
 <segment>
@@
 <wire x1="96.52" y1="93.98" x2="96.52" y2="86.36" width="0.1524" layer="91"/>
 </segment>
+<segment>
+<pinref part="R8" gate="G$1" pin="1"/>
+<pinref part="GND2" gate="1" pin="GND"/>
+<wire x1="96.52" y1="50.8" x2="96.52" y2="53.34" width="0.1524" layer="91"/>
+</segment>
 </net>
 <net name="EN" class="0">
@@
 </segment>
 </net>
-<net name="N$37" class="1">
+<net name="V+" class="1">
 <segment>
 <pinref part="X4" gate="-1" pin="KL"/>
@@
 </segment>
 </net>
+<net name="V-" class="0">
+<segment>
+<wire x1="58.42" y1="63.5" x2="66.04" y2="63.5" width="0.1524" layer="91"/>
+<pinref part="IC1" gate="G$1" pin="V-"/>
+<wire x1="66.04" y1="63.5" x2="71.12" y2="63.5" width="0.1524" layer="91"/>
+<wire x1="71.12" y1="63.5" x2="76.2" y2="63.5" width="0.1524" layer="91"/>
+<wire x1="76.2" y1="63.5" x2="81.28" y2="63.5" width="0.1524" layer="91"/>
+<wire x1="81.28" y1="63.5" x2="96.52" y2="63.5" width="0.1524" layer="91"/>
+<pinref part="C17" gate="G$1" pin="-"/>
+<junction x="96.52" y="63.5"/>
+<pinref part="X4" gate="-2" pin="KL"/>
+<wire x1="109.22" y1="63.5" x2="96.52" y2="63.5" width="0.1524" layer="91"/>
+<junction x="96.52" y="63.5"/>
+<pinref part="C4" gate="G$1" pin="2"/>
+<junction x="66.04" y="63.5"/>
+<pinref part="C11" gate="G$1" pin="2"/>
+<junction x="81.28" y="63.5"/>
+<pinref part="C15" gate="G$1" pin="2"/>
+<junction x="76.2" y="63.5"/>
+<pinref part="C16" gate="G$1" pin="2"/>
+<junction x="71.12" y="63.5"/>
+<pinref part="R8" gate="G$1" pin="2"/>
+</segment>
+</net>

Commit message: iramx v3
Parts:
- removed X2: (no value), con-appsys:RJ45
- added X1: (no value), reroolib:RJ45
Connections:
- net ISO_GND: now also X1.8; no longer X2-.8
- net N$13: now also X1.4; no longer X2-.4
- net N$14: now also X1.5; no longer X2-.5
- net N$17: now also X1.7; no longer X2-.7
Other:
- moved on the sheet: C20, C21, IC3

Commit message: aufgebaut
Parts:
- C15, C4: value (none) -> 100p
- C17: value 1000µ -> 820µ
- R13, R3, R5: value 470 -> 180
- R4: value 100K -> 10K
Changed lines of the file:
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@@
 <part name="C14" library="rcl" deviceset="C-EU" device="C0805K" value="100n"/>
 <part name="LED1" library="led" deviceset="LED" device="3MM" value="GELB"/>
-<part name="R13" library="rcl" deviceset="R-EU_" device="R0805" value="470"/>
+<part name="R13" library="rcl" deviceset="R-EU_" device="R0805" value="180"/>
 <part name="GND21" library="supply1" deviceset="GND" device=""/>
 <part name="IC1" library="iram-b" deviceset="IRAM" device="TOP"/>
 <part name="X3" library="con-wago-508" deviceset="W237-03P" device=""/>
 <part name="X4" library="con-wago-508" deviceset="W237-02P" device=""/>
-<part name="C17" library="rcl" deviceset="CPOL-EU" device="E10-35" value="1000µ"/>
+<part name="C17" library="rcl" deviceset="CPOL-EU" device="E10-35" value="820µ"/>
 <part name="R10" library="rcl" deviceset="R-EU_" device="R0805" value="100K"/>
 <part name="P+9" library="supply1" deviceset="+15V" device=""/>
@@
 <part name="H3" library="holes" deviceset="MOUNT-PAD-ROUND" device="3.2"/>
 <part name="IC2" library="micro-stm_v2" deviceset="STM32F103R*T" device="" technology="6"/>
-<part name="C4" library="rcl" deviceset="C-EU" device="C1206K"/>
+<part name="C4" library="rcl" deviceset="C-EU" device="C1206K" value="100p"/>
 <part name="C11" library="rcl" deviceset="C-EU" device="C0805K" value="4.7µ"/>
-<part name="C15" library="rcl" deviceset="C-EU" device="C1206K"/>
+<part name="C15" library="rcl" deviceset="C-EU" device="C1206K" value="100p"/>
 <part name="C16" library="rcl" deviceset="C-EU" device="C0805K" value="4.7µ"/>
 <part name="GND3" library="supply1" deviceset="GND" device=""/>
@@
 <part name="C19" library="rcl" deviceset="C-EU" device="C0805K" value="100n"/>
 <part name="GND18" library="supply1" deviceset="GND" device=""/>
-<part name="R4" library="rcl" deviceset="R-EU_" device="R0805" value="100K"/>
+<part name="R4" library="rcl" deviceset="R-EU_" device="R0805" value="10K"/>
 <part name="U$1" library="reroolib" deviceset="SI8621" device=""/>
 <part name="+3V3" library="supply1" deviceset="+3V3" device=""/>
@@
 <part name="U$2" library="reroolib" deviceset="RO-XXXX" device=""/>
 <part name="IC4" library="linear" deviceset="78L*SMD" device="" technology="05"/>
-<part name="R3" library="rcl" deviceset="R-EU_" device="R0805" value="470"/>
+<part name="R3" library="rcl" deviceset="R-EU_" device="R0805" value="180"/>
 <part name="LED3" library="led" deviceset="LED" device="3MM" value="GRÜN"/>
 <part name="GND1" library="supply1" deviceset="GND" device=""/>
-<part name="R5" library="rcl" deviceset="R-EU_" device="R0805" value="470"/>
+<part name="R5" library="rcl" deviceset="R-EU_" device="R0805" value="180"/>
 <part name="LED4" library="led" deviceset="LED" device="3MM" value="ROT"/>
 <part name="GND5" library="supply1" deviceset="GND" device=""/>

Commit message: iramx v3
Parts:
- R1: value (none) -> 100K
- R10: value 100K -> 10K
- R2: value (none) -> 800
Changed lines of the file:
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@@
 <part name="X4" library="con-wago-508" deviceset="W237-02P" device=""/>
 <part name="C17" library="rcl" deviceset="CPOL-EU" device="E10-35" value="820µ"/>
-<part name="R10" library="rcl" deviceset="R-EU_" device="R0805" value="100K"/>
+<part name="R10" library="rcl" deviceset="R-EU_" device="R0805" value="10K"/>
 <part name="P+9" library="supply1" deviceset="+15V" device=""/>
 <part name="GND22" library="supply1" deviceset="GND" device=""/>
@@
 <part name="+3V1" library="supply1" deviceset="+3V3" device=""/>
 <part name="+3V2" library="supply1" deviceset="+3V3" device=""/>
-<part name="R1" library="rcl" deviceset="R-EU_" device="R0805"/>
-<part name="R2" library="rcl" deviceset="R-EU_" device="R0805"/>
+<part name="R1" library="rcl" deviceset="R-EU_" device="R0805" value="100K"/>
+<part name="R2" library="rcl" deviceset="R-EU_" device="R0805" value="800"/>
 <part name="C9" library="rcl" deviceset="C-EU" device="C0805K" value="100n"/>
 <part name="GND8" library="supply1" deviceset="GND" device=""/>
