File: hw/eagle/IRAMX-drv-v3.1.brd (EAGLE design)
At the start: 100 x 75 mm, 146 parts, among them IC1 IRAMTOP, IC2 STM32F103R6T, IC3 78L05SMD, IC4 78L05SMD, IC5 STM32F405RGT, IC6 7805TV, IC7 7812TV, Q1 8Mhz, Q2 8Mhz

Commit message: iramx 3.1 todo
Parts:
- added C65, C66: (no value), rcl:E2,5-6
- added C68: 18p, rcl:C0805
- added D1: 3v3, diode:SOD80C
- added JP10: (no value), pinhead:1X01
- moved C34 0.75 mm to (47.0, 36.2)
- moved C31 0.25 mm to (44.2, 36.8)
- moved C35 0.25 mm to (40.2, 32.2)
- moved R39 0.25 mm to (7.75, 16.2)
- moved R40 0.25 mm to (5.75, 16.2)
Connections:
- net +12V_RES: now also C65.+
- net +5V_RES: now also C66.+
- net AMP: now also D1.C
- net GND_DRV: now also C68.1, D1.A
- net GND_RES: now also C65.-, C66.-
- net NRST_RES: now also JP10.1
- net RST: now also C68.2
Routing:
- net RST: track 16.3 -> 19.4 mm
- net NRST_RES: track 0.00 -> 2.45 mm
- net N$6: track 8.76 -> 7.34 mm
- net AMP: track 67.1 -> 68.3 mm
- net N$26: track 11.2 -> 10.3 mm
- net N$32: track 12.0 -> 11.2 mm
- net N$28: track 11.5 -> 10.7 mm
- net N$18: track 9.60 -> 8.88 mm
- net N$40: track 50.5 -> 49.8 mm

Commit message: drc
Parts:
- moved C65 16.2 mm to (20.0, 10.5), turned to 270 degrees
- moved C60 0.25 mm to (33.2, 17.0)
- moved C66 0.25 mm to (19.0, 58.0)
- moved R39 0.25 mm to (7.50, 16.2)
Routing:
- net +24V_RES: track 97.7 -> 96.3 mm

Commit message: iramxv3.1
Parts:
- added C67: (no value), rcl:E2,5-6
- added LOGO1, LOGO2: OSHW-LOGOL, wz:OSHW-LOGO-L
- moved C66 1.00 mm to (19.0, 57.0)
- moved C52 0.71 mm to (48.0, 25.2)
- moved C35 0.56 mm to (40.0, 31.8)
- moved R35 0.50 mm to (24.2, 58.0)
- moved R36 0.50 mm to (26.2, 58.0)
- moved R37 0.50 mm to (22.2, 58.0)
- moved C64 0.25 mm to (54.5, 25.8)
Connections:
- net +24V_RES: now also C67.+
- net GND_RES: now also C67.-
Routing:
- net VLT: track 54.0 -> 52.2 mm
- net +24V_RES: track 96.3 -> 97.5 mm
- net Y_RES: track 18.4 -> 17.3 mm
- net N$20: track 10.1 -> 10.9 mm
- net R_RES: track 19.9 -> 19.4 mm

Commit message: iramx 3.1 final
Parts:
- removed C68: 18p, rcl:C0805
- added C69: 100n, rcl:C0805K
- C11, C16: value 4.7µ -> 10n
- C22, C48, C49, C50, C51, C52, C6: value (none) -> 0.33µ
- C28, C33, C34, C47, C5: value (none) -> 10µ
- C31, C35: value 2.2u -> 100n
- C57, C58: value 2.2u -> 2.2µ
- C65, C66, C67: value (none) -> 4.7µ
- R10, R4: value 10K -> 10k
- R11, R23, R6, R7: value 1K -> 1k
- R17, R22, R25, R28: value 3.6k -> 3.9k
- R2, R9: value 280 -> 560
Connections:
- net GND_DRV: now also C69.2; no longer C68.1
- net RST: now also C69.1; no longer C68.2

Commit message: iramx3.1 werte
Parts:
- R29: value 500 -> 470
Changed lines of the file:
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@@
 <grid distance="0.25" unitdist="mm" unit="mm" style="lines" multiple="4" display="yes" altdistance="0.01" altunitdist="mm" altunit="mm"/>
 <layers>
-<layer number="1" name="Top" color="4" fill="1" visible="no" active="yes"/>
+<layer number="1" name="Top" color="4" fill="1" visible="yes" active="yes"/>
 <layer number="16" name="Bottom" color="1" fill="1" visible="yes" active="yes"/>
 <layer number="17" name="Pads" color="2" fill="1" visible="yes" active="yes"/>
@@
 </element>
 <element name="IC5" library="micro-stm_v2" package="LQFP64" value="STM32F405RGT" x="36.25" y="40.5" rot="MR270"/>
-<element name="R29" library="rcl" package="R0805" value="500" x="45.25" y="7.25" rot="MR270"/>
+<element name="R29" library="rcl" package="R0805" value="470" x="45.25" y="7.25" rot="MR270"/>
 <element name="C41" library="rcl" package="C0805K" value="100n" x="48" y="5.5" rot="MR180"/>
 <element name="C42" library="rcl" package="C0805K" value="100n" x="45.25" y="3.75" rot="MR90"/>

Commit message: IC1 value
Parts:
- IC1: value IRAMTOP -> IRAMX16UP60B
Changed lines of the file:
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@@
 <element name="LED1" library="led" package="LED3MM" value="GELB" x="63.7475" y="3.255" rot="R270"/>
 <element name="R13" library="rcl" package="R0805" value="180" x="65.4975" y="5.2475" rot="MR90"/>
-<element name="IC1" library="iram-b" package="SIP23_TOP" value="IRAMTOP" x="91.495" y="62.9975" rot="R90"/>
+<element name="IC1" library="iram-b" package="SIP23_TOP" value="IRAMX16UP60B" x="91.495" y="62.9975" rot="R90"/>
 <element name="X3" library="con-wago-508" package="W237-133" value="" x="83.505" y="69.9975" rot="R180">
 <attribute name="OC_NEWARK" value="unknown" x="83.505" y="69.9975" size="1.778" layer="27" rot="R180" display="off"/>
