File: hw/eagle/IRAMX-drv-v3.1.sch (EAGLE design)
At the start: 146 parts, among them IC1 IRAMTOP, IC2 STM32F103R6T, IC3 78L05SMD, IC4 78L05SMD, IC5 STM32F405RGT, IC6 7805TV, IC7 7812TV

Commit message: iramx v3.1
Connections:
- removed net N$48: IC5MCU.PC0
- removed net N$49: IC5MCU.PC2
- removed net N$57: IC5MCU.PC1
Changed lines of the file:
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@@
-</segment>
-</net>
-<net name="N$48" class="0">
-<segment>
-<pinref part="IC5" gate="MCU" pin="PC0"/>
-<wire x1="-360.68" y1="144.78" x2="-370.84" y2="144.78" width="0.1524" layer="91"/>
-<label x="-370.84" y="144.78" size="1.778" layer="95"/>
-</segment>
-</net>
-<net name="N$49" class="0">
-<segment>
-<pinref part="IC5" gate="MCU" pin="PC2"/>
-<wire x1="-360.68" y1="149.86" x2="-370.84" y2="149.86" width="0.1524" layer="91"/>
-<label x="-370.84" y="149.86" size="1.778" layer="95"/>
 </segment>
 </net>
@@
 <wire x1="-256.54" y1="160.02" x2="-238.76" y2="160.02" width="0.1524" layer="91"/>
 <label x="-251.46" y="160.02" size="1.778" layer="95"/>
-</segment>
-</net>
-<net name="N$57" class="0">
-<segment>
-<pinref part="IC5" gate="MCU" pin="PC1"/>
-<wire x1="-360.68" y1="147.32" x2="-370.84" y2="147.32" width="0.1524" layer="91"/>
-<label x="-370.84" y="147.32" size="1.778" layer="95"/>
 </segment>
 </net>
@@
 <wire x1="-447.04" y1="35.56" x2="-454.66" y2="35.56" width="0.1524" layer="91"/>
 <wire x1="-454.66" y1="35.56" x2="-454.66" y2="43.18" width="0.1524" layer="91"/>
+<junction x="-447.04" y="35.56"/>
 </segment>
 <segment>
@@
 <wire x1="-485.14" y1="170.18" x2="-482.6" y2="170.18" width="0.1524" layer="91"/>
 <pinref part="GND50" gate="1" pin="GND"/>
-<junction x="-482.6" y="170.18"/>
 </segment>
 <segment>
@@
 <pinref part="U$2" gate="G$1" pin="VIN+"/>
 <pinref part="P+4" gate="1" pin="+24V"/>
+<junction x="-99.06" y="124.46"/>
+<junction x="-109.22" y="124.46"/>
 </segment>
 </net>
@@
 <wire x1="-454.66" y1="55.88" x2="-447.04" y2="55.88" width="0.1524" layer="91"/>
 <pinref part="U$3" gate="G$1" pin="VCC"/>
+<junction x="-447.04" y="55.88"/>
 </segment>
 <segment>
@@
 <pinref part="JP8" gate="A" pin="1"/>
 <wire x1="-396.24" y1="160.02" x2="-396.24" y2="172.72" width="0.1524" layer="91"/>
-</segment>
-<segment>
+<label x="-396.24" y="172.72" size="1.778" layer="95"/>
+</segment>
+<segment>

Commit message: iramx v3.1
Parts:
- C12, C43, C44, C7: value (none) -> 18p
- D2: value (none) -> 3v3
- Q1, Q2: value (none) -> 8Mhz
Other:
- moved on the sheet: C10, C20, C21, C22, C24, C29, C30, C31, C32, C33, C34, C35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

Commit message: iramx 3.1 todo
Parts:
- added C65, C66: (no value), rcl:CPOL-EUE2.5-6
- added C68: 18p, rcl:C-EUC0805
- added D1: 3v3, diode:ZENER-DIODESOD80C
- added JP10: (no value), pinhead:PINHD-1X1
Connections:
- net +12V_RES: now also C65.+
- net +5V_RES: now also C66.+
- net AMP: now also D1.C
- net GND_DRV: now also C68.1, D1.A
- net GND_RES: now also C65.-, C66.-
- net NRST_RES: now also JP10.1
- net RST: now also C68.2
Changed lines of the file:
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@@
 <part name="GND55" library="supply1" deviceset="GND" device=""/>
 <part name="GND56" library="supply1" deviceset="GND" device=""/>
+<part name="D1" library="diode" deviceset="ZENER-DIODE" device="SOD80C" value="3v3"/>
+<part name="GND57" library="supply1" deviceset="GND" device=""/>
+<part name="C65" library="rcl" deviceset="CPOL-EU" device="E2.5-6"/>
+<part name="C66" library="rcl" deviceset="CPOL-EU" device="E2.5-6"/>
+<part name="JP10" library="pinhead" deviceset="PINHD-1X1" device=""/>
+<part name="C68" library="rcl" deviceset="C-EU" device="C0805" value="18p"/>
 </parts>
 <sheets>
@@
 <instance part="GND55" gate="1" x="-203.2" y="96.52" rot="R270"/>
 <instance part="GND56" gate="1" x="-203.2" y="91.44" rot="R270"/>
+<instance part="D1" gate="G$1" x="109.22" y="17.78" rot="R90"/>
+<instance part="GND57" gate="1" x="109.22" y="10.16"/>
+<instance part="C65" gate="G$1" x="-185.42" y="165.1"/>
+<instance part="C66" gate="G$1" x="-187.96" y="127"/>
+<instance part="JP10" gate="G$1" x="-218.44" y="-68.58" rot="R180"/>
+<instance part="C68" gate="G$1" x="-15.24" y="-73.66" rot="R180"/>
 </instances>
 <busses>
@@
 <junction x="96.52" y="22.86"/>
 <label x="106.68" y="22.86" size="1.778" layer="95"/>
-<wire x1="114.3" y1="22.86" x2="96.52" y2="22.86" width="0.1524" layer="91"/>
+<wire x1="114.3" y1="22.86" x2="109.22" y2="22.86" width="0.1524" layer="91"/>
+<pinref part="D1" gate="G$1" pin="C"/>
+<wire x1="109.22" y1="22.86" x2="96.52" y2="22.86" width="0.1524" layer="91"/>
+<wire x1="109.22" y1="22.86" x2="109.22" y2="20.32" width="0.1524" layer="91"/>
+<junction x="109.22" y="22.86"/>
 </segment>
 <segment>
@@
 <segment>
 <pinref part="JP1" gate="G$1" pin="1"/>
-<wire x1="-2.54" y1="-66.04" x2="-12.7" y2="-66.04" width="0.1524" layer="91"/>
+<wire x1="-2.54" y1="-66.04" x2="-15.24" y2="-66.04" width="0.1524" layer="91"/>
 <label x="-12.7" y="-66.04" size="1.778" layer="95"/>
+<pinref part="C68" gate="G$1" pin="2"/>
+<wire x1="-15.24" y1="-66.04" x2="-15.24" y2="-68.58" width="0.1524" layer="91"/>
 </segment>
 </net>
@@
 <wire x1="0" y1="-30.48" x2="5.08" y2="-30.48" width="0.1524" layer="91"/>
 <junction x="-5.08" y="-30.48"/>
+<pinref part="C68" gate="G$1" pin="1"/>
+<wire x1="-15.24" y1="-76.2" x2="-15.24" y2="-78.74" width="0.1524" layer="91"/>
+<wire x1="-15.24" y1="-78.74" x2="-30.48" y2="-78.74" width="0.1524" layer="91"/>
+<wire x1="-30.48" y1="-78.74" x2="-30.48" y2="-58.42" width="0.1524" layer="91"/>
+<junction x="-30.48" y="-58.42"/>
 </segment>
 <segment>
@@
 <label x="101.6" y="-53.34" size="1.778" layer="95"/>
 <pinref part="JP2" gate="A" pin="2"/>
+</segment>
+<segment>
+<pinref part="D1" gate="G$1" pin="A"/>
+<pinref part="GND57" gate="1" pin="GND"/>
+<wire x1="109.22" y1="15.24" x2="109.22" y2="12.7" width="0.1524" layer="91"/>
 </segment>
 </net>
@@
 <pinref part="GND29" gate="1" pin="GND"/>
 <wire x1="-195.58" y1="160.02" x2="-195.58" y2="152.4" width="0.1524" layer="91"/>
+<pinref part="C65" gate="G$1" pin="-"/>
+<wire x1="-185.42" y1="160.02" x2="-195.58" y2="160.02" width="0.1524" layer="91"/>
+<junction x="-195.58" y="160.02"/>
 </segment>
 <segment>
@@
 <pinref part="GND31" gate="1" pin="GND"/>
 <wire x1="-200.66" y1="121.92" x2="-200.66" y2="111.76" width="0.1524" layer="91"/>
+<pinref part="C66" gate="G$1" pin="-"/>
+<wire x1="-187.96" y1="121.92" x2="-200.66" y2="121.92" width="0.1524" layer="91"/>
+<junction x="-200.66" y="121.92"/>
 </segment>
 <segment>
@@
 <wire x1="-210.82" y1="129.54" x2="-208.28" y2="129.54" width="0.1524" layer="91"/>
 <wire x1="-208.28" y1="129.54" x2="-200.66" y2="129.54" width="0.1524" layer="91"/>
-<wire x1="-200.66" y1="129.54" x2="-175.26" y2="129.54" width="0.1524" layer="91"/>
+<wire x1="-200.66" y1="129.54" x2="-187.96" y2="129.54" width="0.1524" layer="91"/>
 <junction x="-175.26" y="129.54"/>
 <pinref part="IC3" gate="G$1" pin="VIN"/>
@@
 <junction x="-200.66" y="129.54"/>
 <pinref part="P+5" gate="1" pin="+5V"/>
+<pinref part="C66" gate="G$1" pin="+"/>
+<wire x1="-187.96" y1="129.54" x2="-175.26" y2="129.54" width="0.1524" layer="91"/>
+<junction x="-187.96" y="129.54"/>
 </segment>
 <segment>
@@
 <junction x="-195.58" y="167.64"/>
 <junction x="-203.2" y="167.64"/>
+<pinref part="C65" gate="G$1" pin="+"/>
+<wire x1="-185.42" y1="167.64" x2="-195.58" y2="167.64" width="0.1524" layer="91"/>
 </segment>
 <segment>
@@
 <label x="-198.12" y="-38.1" size="1.778" layer="95"/>
 </segment>
-</net>
+<segment>
+<pinref part="JP10" gate="G$1" pin="1"/>
+<wire x1="-215.9" y1="-68.58" x2="-187.96" y2="-68.58" width="0.1524" layer="91"/>
+</segment>
+</net>

Commit message: iramxv3.1
Parts:
- added C67: (no value), rcl:CPOL-EUE2.5-6
- added LOGO1, LOGO2: OSHW-LOGOL, wz:OSHW-LOGOL
Connections:
- net +24V_RES: now also C67.+
- net GND_RES: now also C67.-
Changed lines of the file:
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@@
 <layer number="54" name="bGND_GNDA" color="1" fill="9" visible="no" active="no"/>
 <layer number="56" name="wert" color="7" fill="1" visible="no" active="no"/>
+<layer number="57" name="tCAD" color="7" fill="1" visible="no" active="no"/>
+<layer number="90" name="Modules" color="5" fill="1" visible="yes" active="yes"/>
 <layer number="91" name="Nets" color="2" fill="1" visible="yes" active="yes"/>
 <layer number="92" name="Busses" color="1" fill="1" visible="yes" active="yes"/>
@@
 <layer number="109" name="fp9" color="7" fill="1" visible="yes" active="yes"/>
 <layer number="110" name="fp0" color="7" fill="1" visible="yes" active="yes"/>
+<layer number="111" name="LPC17xx" color="7" fill="1" visible="yes" active="yes"/>
+<layer number="112" name="tSilk" color="7" fill="1" visible="yes" active="yes"/>
 <layer number="116" name="Patch_BOT" color="9" fill="4" visible="yes" active="yes"/>
 <layer number="121" name="_tsilk" color="7" fill="1" visible="yes" active="yes"/>
@@
 <layer number="124" name="bTestmark" color="7" fill="1" visible="yes" active="yes"/>
 <layer number="125" name="_tNames" color="7" fill="1" visible="yes" active="yes"/>
+<layer number="126" name="_bNames" color="7" fill="1" visible="yes" active="yes"/>
+<layer number="127" name="_tValues" color="7" fill="1" visible="yes" active="yes"/>
+<layer number="128" name="_bValues" color="7" fill="1" visible="yes" active="yes"/>
 <layer number="131" name="tAdjust" color="7" fill="1" visible="yes" active="yes"/>
 <layer number="132" name="bAdjust" color="7" fill="1" visible="yes" active="yes"/>
 <layer number="144" name="Drill_legend" color="7" fill="1" visible="yes" active="yes"/>
+<layer number="150" name="Notes" color="7" fill="1" visible="yes" active="yes"/>
 <layer number="151" name="HeatSink" color="7" fill="1" visible="yes" active="yes"/>
+<layer number="152" name="_bDocu" color="7" fill="1" visible="yes" active="yes"/>
+<layer number="153" name="FabDoc1" color="7" fill="1" visible="yes" active="yes"/>
+<layer number="154" name="FabDoc2" color="7" fill="1" visible="yes" active="yes"/>
+<layer number="155" name="FabDoc3" color="7" fill="1" visible="yes" active="yes"/>
 <layer number="199" name="Contour" color="7" fill="1" visible="yes" active="yes"/>
 <layer number="200" name="200bmp" color="1" fill="10" visible="yes" active="yes"/>
@@
 <layer number="223" name="223bmp" color="7" fill="1" visible="yes" active="yes"/>
 <layer number="224" name="224bmp" color="7" fill="1" visible="yes" active="yes"/>
+<layer number="248" name="Housing" color="7" fill="1" visible="yes" active="yes"/>
+<layer number="249" name="Edge" color="7" fill="1" visible="yes" active="yes"/>
 <layer number="250" name="Descript" color="3" fill="1" visible="no" active="no"/>
 <layer number="251" name="SMDround" color="12" fill="11" visible="no" active="no"/>
@@
 <part name="JP10" library="pinhead" deviceset="PINHD-1X1" device=""/>
 <part name="C68" library="rcl" deviceset="C-EU" device="C0805" value="18p"/>
+<part name="C67" library="rcl" deviceset="CPOL-EU" device="E2.5-6"/>
+<part name="LOGO1" library="wz" deviceset="OSHW-LOGO" device="L"/>
+<part name="LOGO2" library="wz" deviceset="OSHW-LOGO" device="L"/>
 </parts>
 <sheets>
@@
 <instance part="JP10" gate="G$1" x="-218.44" y="-68.58" rot="R180"/>
 <instance part="C68" gate="G$1" x="-15.24" y="-73.66" rot="R180"/>
+<instance part="C67" gate="G$1" x="-254" y="127"/>
+<instance part="LOGO1" gate="G$1" x="-160.02" y="157.48"/>
+<instance part="LOGO2" gate="G$1" x="20.32" y="-96.52"/>
 </instances>
 <busses>
@@
 <wire x1="-243.84" y1="121.92" x2="-236.22" y2="121.92" width="0.1524" layer="91"/>
 <junction x="-236.22" y="121.92"/>
+<pinref part="C67" gate="G$1" pin="-"/>
+<wire x1="-254" y1="121.92" x2="-243.84" y2="121.92" width="0.1524" layer="91"/>
+<junction x="-243.84" y="121.92"/>
 </segment>
 <segment>
@@
 <pinref part="C63" gate="G$1" pin="1"/>
 <wire x1="-236.22" y1="129.54" x2="-243.84" y2="129.54" width="0.1524" layer="91"/>
-</segment>
-<segment>
+<pinref part="C67" gate="G$1" pin="+"/>
+<wire x1="-254" y1="129.54" x2="-243.84" y2="129.54" width="0.1524" layer="91"/>
+<junction x="-243.84" y="129.54"/>
+</segment>
+<segment>

Commit message: iramx 3.1 final
Parts:
- removed C68: 18p, rcl:C-EUC0805
- added C69: 100n, rcl:C-EUC0805K
- C11, C16: value 4.7µ -> 10n
- C22, C48, C49, C50, C51, C52, C6: value (none) -> 0.33µ
- C28, C33, C34, C47, C5: value (none) -> 10µ
- C31, C35: value 2.2u -> 100n
- C57, C58: value 2.2u -> 2.2µ
- C65, C66, C67: value (none) -> 4.7µ
- R10, R4: value 10K -> 10k
- R11, R23, R6, R7: value 1K -> 1k
- R17, R22, R25, R28: value 3.6k -> 3.9k
- R2, R9: value 280 -> 560
Connections:
- net GND_DRV: now also C69.2; no longer C68.1
- net RST: now also C69.1; no longer C68.2
Other:
- moved on the sheet: C11, C13, C15, C16, C18, C28, C31, C33, C5, C62, C9, D2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

Commit message: iramx3.1 werte
Parts:
- R29: value 500 -> 470
Changed lines of the file:
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@@
 <part name="X6" library="con-wago-508" deviceset="W237-02P" device=""/>
 <part name="IC5" library="micro-stm_v2" deviceset="STM32F405R*T" device="" technology="G"/>
-<part name="R29" library="rcl" deviceset="R-EU_" device="R0805" value="500"/>
+<part name="R29" library="rcl" deviceset="R-EU_" device="R0805" value="470"/>
 <part name="C41" library="rcl" deviceset="C-EU" device="C0805K" value="100n"/>
 <part name="C42" library="rcl" deviceset="C-EU" device="C0805K" value="100n"/>

Commit message: IC1 value
Parts:
- IC1: value IRAMTOP -> IRAMX16UP60B
Changed lines of the file:
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@@
 <part name="R13" library="rcl" deviceset="R-EU_" device="R0805" value="180"/>
 <part name="GND21" library="supply1" deviceset="GND" device=""/>
-<part name="IC1" library="iram-b" deviceset="IRAM" device="TOP"/>
+<part name="IC1" library="iram-b" deviceset="IRAM" device="TOP" value="IRAMX16UP60B"/>
 <part name="X3" library="con-wago-508" deviceset="W237-03P" device=""/>
 <part name="X4" library="con-wago-508" deviceset="W237-02P" device=""/>
