File: hw/eagle/IRAMX-drv-v3.2.sch (EAGLE design)
At the start: 159 parts, among them IC1 IRAMX16UP60B, IC2 STM32F103R6T, IC5 STM32F405RGT, IC6 7805TV, IC7 7812TV, Q1 8Mhz, Q2 8Mhz, T1 zldo1117, T2 zldo1117

Commit message: drv 3.2
Connections:
- new net N$55: IC5MCU.PB11
- new net N$56: IC5MCU.PB10
Changed lines of the file:
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@@
+</segment>
+</net>
+<net name="N$55" class="0">
+<segment>
+<pinref part="IC5" gate="MCU" pin="PB11"/>
+<wire x1="-134.62" y1="22.86" x2="-124.46" y2="22.86" width="0.1524" layer="91"/>
+</segment>
+</net>
+<net name="N$56" class="0">
+<segment>
+<pinref part="IC5" gate="MCU" pin="PB10"/>
+<wire x1="-134.62" y1="20.32" x2="-124.46" y2="20.32" width="0.1524" layer="91"/>
 </segment>
 </net>

Commit message: iramx32
Parts:
- removed JP10: (no value), pinhead:PINHD-1X1
- removed JP4: (no value), pinhead:PINHD-1X3
- added JP7: (no value), pinhead:PINHD-1X4
- C30, C68: device rcl:C-EUC0805K -> rcl:C-EUC0603
Connections:
- new net +5V: U$6.VCC, U$7.VCC
- new net N$57: U$6.A, X2-.5
- new net N$58: U$6.B, X2-.4
- new net N$59: U$6.DE, U$6.RE
- new net N$60: U$7.DE, U$7.RE
- net GND: now also U$6.GND, U$7.GND
- net GND_RES: now also JP7.2; no longer JP4.2
- net N$27: now also U$7.B
- net N$34: now also U$7.A
- net NRST_RES: now also JP7.4; no longer JP10.1
- net SWCLK_RES: now also JP7.1; no longer JP4.1
- net SWDIO_RES: now also JP7.3; no longer JP4.3
Other:
- moved on the sheet: JP11, JP3, JP5

Commit message: fiducials
Parts:
- added U$8, U$9: FIDUCIAL, adafruit:FIDUCIAL
Changed lines of the file:
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@@
 <?xml version="1.0" encoding="utf-8"?>
 <!DOCTYPE eagle SYSTEM "eagle.dtd">
-<eagle version="7.2.0">
+<eagle version="7.1.0">
 <drawing>
 <settings>
@@
 <grid distance="0.1" unitdist="inch" unit="inch" style="lines" multiple="1" display="no" altdistance="0.01" altunitdist="inch" altunit="inch"/>
 <layers>
-<layer number="1" name="Top" color="4" fill="1" visible="yes" active="no"/>
-<layer number="16" name="Bottom" color="1" fill="1" visible="yes" active="no"/>
-<layer number="17" name="Pads" color="2" fill="1" visible="yes" active="no"/>
-<layer number="18" name="Vias" color="2" fill="1" visible="yes" active="no"/>
-<layer number="19" name="Unrouted" color="6" fill="1" visible="yes" active="no"/>
-<layer number="20" name="Dimension" color="15" fill="1" visible="yes" active="no"/>
-<layer number="21" name="tPlace" color="7" fill="1" visible="yes" active="no"/>
-<layer number="22" name="bPlace" color="7" fill="1" visible="yes" active="no"/>
-<layer number="23" name="tOrigins" color="15" fill="1" visible="yes" active="no"/>
-<layer number="24" name="bOrigins" color="15" fill="1" visible="yes" active="no"/>
-<layer number="25" name="tNames" color="7" fill="1" visible="yes" active="no"/>
-<layer number="26" name="bNames" color="7" fill="1" visible="yes" active="no"/>
-<layer number="27" name="tValues" color="7" fill="1" visible="yes" active="no"/>
-<layer number="28" name="bValues" color="7" fill="1" visible="yes" active="no"/>
+<layer number="1" name="Top" color="4" fill="1" visible="no" active="no"/>
+<layer number="16" name="Bottom" color="1" fill="1" visible="no" active="no"/>
+<layer number="17" name="Pads" color="2" fill="1" visible="no" active="no"/>
+<layer number="18" name="Vias" color="2" fill="1" visible="no" active="no"/>
+<layer number="19" name="Unrouted" color="6" fill="1" visible="no" active="no"/>
+<layer number="20" name="Dimension" color="15" fill="1" visible="no" active="no"/>
+<layer number="21" name="tPlace" color="7" fill="1" visible="no" active="no"/>
+<layer number="22" name="bPlace" color="7" fill="1" visible="no" active="no"/>
+<layer number="23" name="tOrigins" color="15" fill="1" visible="no" active="no"/>
+<layer number="24" name="bOrigins" color="15" fill="1" visible="no" active="no"/>
+<layer number="25" name="tNames" color="7" fill="1" visible="no" active="no"/>
+<layer number="26" name="bNames" color="7" fill="1" visible="no" active="no"/>
+<layer number="27" name="tValues" color="7" fill="1" visible="no" active="no"/>
+<layer number="28" name="bValues" color="7" fill="1" visible="no" active="no"/>
 <layer number="29" name="tStop" color="7" fill="3" visible="no" active="no"/>
 <layer number="30" name="bStop" color="7" fill="6" visible="no" active="no"/>
@@
 <layer number="35" name="tGlue" color="7" fill="4" visible="no" active="no"/>
 <layer number="36" name="bGlue" color="7" fill="5" visible="no" active="no"/>
-<layer number="37" name="tTest" color="7" fill="1" visible="yes" active="no"/>
-<layer number="38" name="bTest" color="7" fill="1" visible="yes" active="no"/>
+<layer number="37" name="tTest" color="7" fill="1" visible="no" active="no"/>
+<layer number="38" name="bTest" color="7" fill="1" visible="no" active="no"/>
 <layer number="39" name="tKeepout" color="4" fill="11" visible="no" active="no"/>
 <layer number="40" name="bKeepout" color="1" fill="11" visible="no" active="no"/>
@@
 <layer number="44" name="Drills" color="7" fill="1" visible="no" active="no"/>
 <layer number="45" name="Holes" color="7" fill="1" visible="no" active="no"/>
-<layer number="46" name="Milling" color="3" fill="1" visible="yes" active="no"/>
-<layer number="47" name="Measures" color="7" fill="1" visible="yes" active="no"/>
-<layer number="48" name="Document" color="7" fill="1" visible="yes" active="no"/>
-<layer number="49" name="Reference" color="7" fill="1" visible="yes" active="no"/>
-<layer number="50" name="dxf" color="7" fill="1" visible="yes" active="no"/>
-<layer number="51" name="tDocu" color="7" fill="1" visible="yes" active="no"/>
-<layer number="52" name="bDocu" color="7" fill="1" visible="yes" active="no"/>
-<layer number="53" name="tGND_GNDA" color="7" fill="9" visible="yes" active="no"/>
-<layer number="54" name="bGND_GNDA" color="1" fill="9" visible="yes" active="no"/>
-<layer number="56" name="wert" color="7" fill="1" visible="yes" active="no"/>
-<layer number="57" name="tCAD" color="7" fill="1" visible="yes" active="no"/>
+<layer number="46" name="Milling" color="3" fill="1" visible="no" active="no"/>
+<layer number="47" name="Measures" color="7" fill="1" visible="no" active="no"/>
+<layer number="48" name="Document" color="7" fill="1" visible="no" active="no"/>
+<layer number="49" name="Reference" color="7" fill="1" visible="no" active="no"/>
+<layer number="50" name="dxf" color="7" fill="1" visible="no" active="no"/>
+<layer number="51" name="tDocu" color="7" fill="1" visible="no" active="no"/>
+<layer number="52" name="bDocu" color="7" fill="1" visible="no" active="no"/>
+<layer number="53" name="tGND_GNDA" color="7" fill="9" visible="no" active="no"/>
+<layer number="54" name="bGND_GNDA" color="1" fill="9" visible="no" active="no"/>
+<layer number="56" name="wert" color="7" fill="1" visible="no" active="no"/>
+<layer number="57" name="tCAD" color="7" fill="1" visible="no" active="no"/>
 <layer number="90" name="Modules" color="5" fill="1" visible="yes" active="yes"/>
 <layer number="91" name="Nets" color="2" fill="1" visible="yes" active="yes"/>
@@
 <layer number="111" name="LPC17xx" color="7" fill="1" visible="yes" active="yes"/>
 <layer number="112" name="tSilk" color="7" fill="1" visible="yes" active="yes"/>
+<layer number="113" name="ReferenceLS" color="7" fill="1" visible="no" active="no"/>
 <layer number="116" name="Patch_BOT" color="9" fill="4" visible="yes" active="yes"/>
+<layer number="118" name="Rect_Pads" color="7" fill="1" visible="no" active="no"/>
 <layer number="121" name="_tsilk" color="7" fill="1" visible="yes" active="yes"/>
 <layer number="122" name="_bsilk" color="7" fill="1" visible="yes" active="yes"/>
@@
 <layer number="223" name="223bmp" color="7" fill="1" visible="yes" active="yes"/>
 <layer number="224" name="224bmp" color="7" fill="1" visible="yes" active="yes"/>
+<layer number="231" name="Eagle3D_PG1" color="7" fill="1" visible="no" active="no"/>
+<layer number="232" name="Eagle3D_PG2" color="7" fill="1" visible="no" active="no"/>
+<layer number="233" name="Eagle3D_PG3" color="7" fill="1" visible="no" active="no"/>
 <layer number="248" name="Housing" color="7" fill="1" visible="yes" active="yes"/>
 <layer number="249" name="Edge" color="7" fill="1" visible="yes" active="yes"/>
@@
 <part name="P+15" library="supply1" deviceset="+5V" device=""/>
 <part name="GND59" library="supply1" deviceset="GND" device=""/>
+<part name="U$8" library="adafruit" deviceset="FIDUCIAL" device=""/>
+<part name="U$9" library="adafruit" deviceset="FIDUCIAL" device=""/>
 </parts>
 <sheets>
@@
 <instance part="P+15" gate="1" x="-317.5" y="38.1"/>
 <instance part="GND59" gate="1" x="-317.5" y="20.32"/>
+<instance part="U$8" gate="G$1" x="157.48" y="93.98"/>
+<instance part="U$9" gate="G$1" x="167.64" y="93.98"/>
 </instances>
 <busses>

Commit message: routing iramx32
Parts:
- removed JP8: (no value), pinhead:PINHD-1X4
Connections:
- removed net +5V: U$6.VCC, U$7.VCC
- net +5V_RES: now also U$6.VCC, U$7.VCC
- net COS: no longer JP8.3
- net GND: no longer U$6.GND, U$7.GND
- net GND_RES: now also U$6.GND, U$7.GND; no longer JP8.4
- net RES: no longer JP8.1
- net SIN: no longer JP8.2
Changed lines of the file:
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@@
 <?xml version="1.0" encoding="utf-8"?>
 <!DOCTYPE eagle SYSTEM "eagle.dtd">
-<eagle version="7.1.0">
+<eagle version="7.2.0">
 <drawing>
 <settings>
@@
 <part name="C63" library="rcl" deviceset="C-EU" device="C0603" value="100n"/>
 <part name="GND52" library="supply1" deviceset="GND" device=""/>
-<part name="JP8" library="pinhead" deviceset="PINHD-1X4" device=""/>
 <part name="C64" library="rcl" deviceset="C-EU" device="C0805K" value="4.7µ"/>
 <part name="GND53" library="supply1" deviceset="GND" device=""/>
@@
 <instance part="C63" gate="G$1" x="-243.84" y="127"/>
 <instance part="GND52" gate="1" x="-215.9" y="-7.62"/>
-<instance part="JP8" gate="A" x="-213.36" y="5.08"/>
 <instance part="C64" gate="G$1" x="10.16" y="106.68"/>
 <instance part="X1" gate="G$1" x="-307.34" y="48.26"/>
@@
 <wire x1="-215.9" y1="5.08" x2="-220.98" y2="5.08" width="0.1524" layer="91"/>
 <wire x1="-220.98" y1="5.08" x2="-220.98" y2="-17.78" width="0.1524" layer="91"/>
-<pinref part="JP8" gate="A" pin="3"/>
 </segment>
 <segment>
@@
 <wire x1="-215.9" y1="7.62" x2="-220.98" y2="7.62" width="0.1524" layer="91"/>
 <wire x1="-220.98" y1="7.62" x2="-220.98" y2="22.86" width="0.1524" layer="91"/>
-<pinref part="JP8" gate="A" pin="2"/>
 </segment>
 <segment>
@@
 <wire x1="-215.9" y1="2.54" x2="-215.9" y2="-5.08" width="0.1524" layer="91"/>
 <pinref part="GND52" gate="1" pin="GND"/>
-<pinref part="JP8" gate="A" pin="4"/>
 </segment>
 <segment>
@@
 <pinref part="GND56" gate="1" pin="GND"/>
 <wire x1="-200.66" y1="91.44" x2="-198.12" y2="91.44" width="0.1524" layer="91"/>
+</segment>
+<segment>
+<pinref part="U$7" gate="G$1" pin="GND"/>
+<pinref part="GND59" gate="1" pin="GND"/>
+<wire x1="-320.04" y1="25.4" x2="-317.5" y2="25.4" width="0.1524" layer="91"/>
+<wire x1="-317.5" y1="25.4" x2="-317.5" y2="22.86" width="0.1524" layer="91"/>
+</segment>
+<segment>
+<pinref part="GND26" gate="1" pin="GND"/>
+<wire x1="-187.96" y1="68.58" x2="-187.96" y2="71.12" width="0.1524" layer="91"/>
+<pinref part="U$6" gate="G$1" pin="GND"/>
+<wire x1="-187.96" y1="71.12" x2="-185.42" y2="71.12" width="0.1524" layer="91"/>
 </segment>
 </net>
@@
 <pinref part="P+13" gate="1" pin="+5V"/>
 <wire x1="-266.7" y1="73.66" x2="-264.16" y2="73.66" width="0.1524" layer="91"/>
+</segment>
+<segment>
+<pinref part="U$7" gate="G$1" pin="VCC"/>
+<pinref part="P+15" gate="1" pin="+5V"/>
+<wire x1="-320.04" y1="33.02" x2="-317.5" y2="33.02" width="0.1524" layer="91"/>
+<wire x1="-317.5" y1="33.02" x2="-317.5" y2="35.56" width="0.1524" layer="91"/>
+</segment>
+<segment>
+<pinref part="P+14" gate="1" pin="+5V"/>
+<wire x1="-187.96" y1="81.28" x2="-187.96" y2="78.74" width="0.1524" layer="91"/>
+<pinref part="U$6" gate="G$1" pin="VCC"/>
+<wire x1="-187.96" y1="78.74" x2="-185.42" y2="78.74" width="0.1524" layer="91"/>
 </segment>
 </net>
@@
 </segment>
 <segment>
-<pinref part="JP8" gate="A" pin="1"/>
 <wire x1="-215.9" y1="10.16" x2="-215.9" y2="22.86" width="0.1524" layer="91"/>
 <label x="-215.9" y="22.86" size="1.778" layer="95"/>
@@
 <pinref part="GND58" gate="1" pin="GND"/>
 </segment>
-<segment>
-<pinref part="GND26" gate="1" pin="GND"/>
-<wire x1="-187.96" y1="68.58" x2="-187.96" y2="71.12" width="0.1524" layer="91"/>
-<pinref part="U$6" gate="G$1" pin="GND"/>
-<wire x1="-187.96" y1="71.12" x2="-185.42" y2="71.12" width="0.1524" layer="91"/>
-</segment>
-<segment>
-<pinref part="U$7" gate="G$1" pin="GND"/>
-<pinref part="GND59" gate="1" pin="GND"/>
-<wire x1="-320.04" y1="25.4" x2="-317.5" y2="25.4" width="0.1524" layer="91"/>
-<wire x1="-317.5" y1="25.4" x2="-317.5" y2="22.86" width="0.1524" layer="91"/>
-</segment>
 </net>
 <net name="N$22" class="0">
@@
 </segment>
 </net>
-<net name="+5V" class="0">
-<segment>
-<pinref part="P+14" gate="1" pin="+5V"/>
-<wire x1="-187.96" y1="81.28" x2="-187.96" y2="78.74" width="0.1524" layer="91"/>
-<pinref part="U$6" gate="G$1" pin="VCC"/>
-<wire x1="-187.96" y1="78.74" x2="-185.42" y2="78.74" width="0.1524" layer="91"/>
-</segment>
-<segment>
-<pinref part="U$7" gate="G$1" pin="VCC"/>
-<pinref part="P+15" gate="1" pin="+5V"/>
-<wire x1="-320.04" y1="33.02" x2="-317.5" y2="33.02" width="0.1524" layer="91"/>
-<wire x1="-317.5" y1="33.02" x2="-317.5" y2="35.56" width="0.1524" layer="91"/>
-</segment>
-</net>

Commit message: iramx32
Parts:
- removed C33, C34: 10µ, rcl:CPOL-EUA/3216-18R
- removed C50, C51, C52: 0.33µ, rcl:CPOL-EUA/3216-18R
- removed C66, C67: 4.7µ, rcl:CPOL-EUE2.5-6
- removed Q2: 8Mhz, special:XTAL/S
- added C22, C47: 100n, rcl:C-EUC0603
- added D3: (no value), adafruit:DIODESOD-123
- added Q3: IRLML5203, transistor-power:IRLML5203
- added Q4: (no value), crystal:CRYSTALCTS406
- added R47: 1k, rcl:R-EU_R0603
- added R48: 33, rcl:R-EU_R0603
- added R49, R50: 180, rcl:R-EU_R0603
- added X5: (no value), con-wago-508:W237-02P
- C31: device rcl:C-EUC0805K -> rcl:C-EUC0603
- IC6: value 7805TV -> 78; device linear:7805TV -> reroolib:78
- JP6: device pinhead:PINHD-1X3 -> jumper:SJ2W
Connections:
- removed net GND: C68.2
- new net N$61: D3.C, Q3.S, X5-2.KL
- new net N$62: Q3.G, R47.1, R48.1
- new net N$63: R48.2
- net +12V_RES: no longer C51.+
- net +24V: now also C70.+, X5-1.KL
- net +24V_RES: no longer C50.+, C52.+, C67.+
- net +3V3_RES: no longer C33.+
- net +5V_RES: now also C22.2, C47.2; no longer C66.+
- net GND_RES: now also C22.1, C47.1, C68.2, C70.-, D3.A, Q3.D, R47.2; no longer C33.-, C34.-, C50.-, C51.-, C52.-, C66.-, C67.-
- net N$15: now also Q4.1; no longer Q2.1
- net N$27: now also R50.1
- net N$34: now also R50.2
- net N$39: now also Q4.2; no longer Q2.2
- net N$46: no longer C34.+
- net N$57: now also R49.2
- net N$58: now also R49.1
Other:
- moved on the sheet: C70

Commit message: iramx32
Parts:
- removed JP2: (no value), pinhead:PINHD-1X3
- removed Q1: 8Mhz, special:XTAL/S
- added Q2: (no value), crystal:CRYSTALCTS406
- JP1: device pinhead:PINHD-1X1 -> pinhead:PINHD-1X4
Connections:
- removed net +24V: C62.1, C70.+, IC7.VI, X5-1.KL, X6-1.KL
- net +24V_RES: now also C62.1, C70.+, IC7.VI, X5-1.KL, X6-1.KL
- net GND_DRV: now also JP1.2; no longer JP2.2
- net N$10: now also Q2.2; no longer Q1.2
- net N$12: now also Q2.1; no longer Q1.1
- net RST: now also JP1.4; no longer JP1.1
- net SWCLK: now also JP1.1; no longer JP2.1
- net SWDIO: now also JP1.3; no longer JP2.3
