File: hw/eagle/IRAMX-drv-v3.2.sch (EAGLE design)
At the start: 160 parts, among them IC1 IRAMX16UP60B, IC2 STM32F103R6T, IC5 STM32F405RGT, IC6 78, IC7 7812TV, Q3 IRLML5203, T1 zldo1117, T2 zldo1117

Commit message: iramx 32
Parts:
- removed R30, R38, R41, R42: 180, rcl:R-EU_R0603
- added U$10, U$11, U$12: ACS712, SparkFun-AnalogIC:ACS712
Connections:
- removed net N$35: R30.1, U$5.2Y
- removed net N$42: R42.2, U$5.3Y
- removed net N$44: R41.2, U$5.4Y
- removed net N$45: R38.1, U$5.1Y
- net +24V_RES: now also D3.C
- net GND_RES: now also C61.2; no longer D3.A
- net N$61: now also D3.A; no longer D3.C
- net TIM1_A: now also U$5.4Y; no longer R41.1
- net TIM1_B: now also U$5.3Y; no longer R42.1
- net TIM3_A: now also U$5.1Y; no longer R38.2
- net TIM3_B: now also U$5.2Y; no longer R30.2
Other:
- moved on the sheet: D3, Q3, R47, R48
Changed lines of the file:
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@@
 <layer number="251" name="SMDround" color="12" fill="11" visible="no" active="no"/>
 <layer number="254" name="cooling" color="7" fill="1" visible="yes" active="yes"/>
+<layer number="255" name="routoute" color="7" fill="1" visible="yes" active="yes"/>
 </layers>
 <schematic xreflabel="%F%N/%S.%C%R" xrefpart="/%S.%C%R">
@@
 </variantdefs>
 <classes>
-<class number="0" name="default" width="0.2" drill="0">
+<class number="0" name="default" width="0.2" drill="0.1">
 <clearance class="0" value="0.19"/>
 </class>
@@
 <part name="C60" library="rcl" deviceset="C-EU" device="C0603" value="100n"/>
 <part name="P+13" library="supply1" deviceset="+5V" device=""/>
-<part name="R30" library="rcl" deviceset="R-EU_" device="R0603" value="180"/>
-<part name="R38" library="rcl" deviceset="R-EU_" device="R0603" value="180"/>
-<part name="R41" library="rcl" deviceset="R-EU_" device="R0603" value="180"/>
-<part name="R42" library="rcl" deviceset="R-EU_" device="R0603" value="180"/>
 <part name="L1" library="resistor" deviceset="L-EU" device="L2825P"/>
 <part name="L2" library="resistor" deviceset="L-EU" device="L2825P"/>
@@
 <part name="Q2" library="crystal" deviceset="CRYSTAL" device="CTS406"/>
 <part name="JP1" library="pinhead" deviceset="PINHD-1X4" device=""/>
+<part name="U$10" library="SparkFun-AnalogIC" deviceset="ACS712" device=""/>
+<part name="U$11" library="SparkFun-AnalogIC" deviceset="ACS712" device=""/>
+<part name="U$12" library="SparkFun-AnalogIC" deviceset="ACS712" device=""/>
 </parts>
 <sheets>
@@
 <instance part="C60" gate="G$1" x="-274.32" y="-101.6"/>
 <instance part="P+13" gate="1" x="-269.24" y="73.66" rot="R90"/>
-<instance part="R30" gate="G$1" x="-269.24" y="68.58" rot="R180"/>
-<instance part="R38" gate="G$1" x="-269.24" y="78.74" rot="R180"/>
-<instance part="R41" gate="G$1" x="-228.6" y="73.66" rot="R180"/>
-<instance part="R42" gate="G$1" x="-228.6" y="63.5" rot="R180"/>
 <instance part="L1" gate="G$1" x="-215.9" y="-30.48" rot="R90"/>
 <instance part="L2" gate="G$1" x="96.52" y="58.42" rot="R180"/>
@@
 <instance part="X5" gate="-1" x="-297.18" y="157.48"/>
 <instance part="X5" gate="-2" x="-297.18" y="147.32"/>
-<instance part="Q3" gate="G$1" x="-284.48" y="139.7" rot="MR0"/>
-<instance part="D3" gate="G$1" x="-292.1" y="139.7" rot="R90"/>
-<instance part="GND60" gate="1" x="-292.1" y="129.54"/>
+<instance part="Q3" gate="G$1" x="-289.56" y="137.16" rot="MR0"/>
+<instance part="D3" gate="G$1" x="-292.1" y="152.4" rot="R90"/>
+<instance part="GND60" gate="1" x="-292.1" y="121.92"/>
 <instance part="P+16" gate="1" x="-289.56" y="162.56"/>
-<instance part="R47" gate="G$1" x="-276.86" y="137.16" rot="R270"/>
-<instance part="R48" gate="G$1" x="-266.7" y="142.24"/>
+<instance part="R47" gate="G$1" x="-276.86" y="134.62" rot="R270"/>
+<instance part="R48" gate="G$1" x="-266.7" y="139.7"/>
 <instance part="R49" gate="G$1" x="-205.74" y="76.2" rot="R180"/>
 <instance part="R50" gate="G$1" x="-294.64" y="27.94" rot="R180"/>
@@
 <instance part="Q2" gate="G$1" x="12.7" y="-45.72" rot="R90"/>
 <instance part="JP1" gate="A" x="119.38" y="-55.88"/>
+<instance part="U$10" gate="G$1" x="195.58" y="127"/>
+<instance part="U$11" gate="G$1" x="195.58" y="106.68"/>
+<instance part="U$12" gate="G$1" x="195.58" y="86.36"/>
 </instances>
 <busses>
@@
 <segment>
 <label x="-223.52" y="73.66" size="1.778" layer="95"/>
-<pinref part="R41" gate="G$1" pin="1"/>
-<wire x1="-223.52" y1="73.66" x2="-218.44" y2="73.66" width="0.1524" layer="91"/>
+<wire x1="-233.68" y1="73.66" x2="-218.44" y2="73.66" width="0.1524" layer="91"/>
+<pinref part="U$5" gate="G$1" pin="4Y"/>
 </segment>
 </net>
@@
 <segment>
 <label x="-223.52" y="63.5" size="1.778" layer="95"/>
-<pinref part="R42" gate="G$1" pin="1"/>
-<wire x1="-223.52" y1="63.5" x2="-218.44" y2="63.5" width="0.1524" layer="91"/>
+<wire x1="-233.68" y1="63.5" x2="-218.44" y2="63.5" width="0.1524" layer="91"/>
+<pinref part="U$5" gate="G$1" pin="3Y"/>
 </segment>
 </net>
@@
 <segment>
 <label x="-281.94" y="78.74" size="1.778" layer="95"/>
-<pinref part="R38" gate="G$1" pin="2"/>
-<wire x1="-274.32" y1="78.74" x2="-281.94" y2="78.74" width="0.1524" layer="91"/>
+<wire x1="-264.16" y1="78.74" x2="-281.94" y2="78.74" width="0.1524" layer="91"/>
+<pinref part="U$5" gate="G$1" pin="1Y"/>
 </segment>
 </net>
@@
 <segment>
 <label x="-281.94" y="68.58" size="1.778" layer="95"/>
-<pinref part="R30" gate="G$1" pin="2"/>
-<wire x1="-274.32" y1="68.58" x2="-281.94" y2="68.58" width="0.1524" layer="91"/>
+<wire x1="-264.16" y1="68.58" x2="-281.94" y2="68.58" width="0.1524" layer="91"/>
+<pinref part="U$5" gate="G$1" pin="2Y"/>
 </segment>
 </net>
@@
 <pinref part="GND27" gate="1" pin="GND"/>
 <wire x1="-127" y1="111.76" x2="-127" y2="121.92" width="0.1524" layer="91"/>
+<pinref part="C61" gate="G$1" pin="2"/>
 </segment>
 <segment>
@@
 </segment>
 <segment>
-<pinref part="D3" gate="G$1" pin="A"/>
-<wire x1="-292.1" y1="137.16" x2="-292.1" y2="132.08" width="0.1524" layer="91"/>
 <pinref part="GND60" gate="1" pin="GND"/>
 <pinref part="R47" gate="G$1" pin="2"/>
-<wire x1="-276.86" y1="132.08" x2="-287.02" y2="132.08" width="0.1524" layer="91"/>
+<wire x1="-276.86" y1="129.54" x2="-292.1" y2="129.54" width="0.1524" layer="91"/>
 <pinref part="Q3" gate="G$1" pin="D"/>
-<wire x1="-287.02" y1="132.08" x2="-292.1" y2="132.08" width="0.1524" layer="91"/>
-<wire x1="-287.02" y1="134.62" x2="-287.02" y2="132.08" width="0.1524" layer="91"/>
-<junction x="-287.02" y="132.08"/>
-<junction x="-292.1" y="132.08"/>
+<wire x1="-292.1" y1="129.54" x2="-292.1" y2="124.46" width="0.1524" layer="91"/>
+<wire x1="-292.1" y1="132.08" x2="-292.1" y2="129.54" width="0.1524" layer="91"/>
+<junction x="-292.1" y="129.54"/>
 </segment>
 <segment>
@@
 <pinref part="P+16" gate="1" pin="+24V"/>
 <wire x1="-289.56" y1="157.48" x2="-289.56" y2="160.02" width="0.1524" layer="91"/>
+<pinref part="D3" gate="G$1" pin="C"/>
+<wire x1="-292.1" y1="154.94" x2="-292.1" y2="157.48" width="0.1524" layer="91"/>
+<junction x="-292.1" y="157.48"/>
 </segment>
 <segment>
@@
 </segment>
 </net>
-<net name="N$35" class="0">
-<segment>
-<pinref part="U$5" gate="G$1" pin="2Y"/>
-<pinref part="R30" gate="G$1" pin="1"/>
-</segment>
-</net>
-<net name="N$42" class="0">
-<segment>
-<pinref part="U$5" gate="G$1" pin="3Y"/>
-<pinref part="R42" gate="G$1" pin="2"/>
-</segment>
-</net>
-<net name="N$44" class="0">
-<segment>
-<pinref part="U$5" gate="G$1" pin="4Y"/>
-<pinref part="R41" gate="G$1" pin="2"/>
-</segment>
-</net>
-<net name="N$45" class="0">
-<segment>
-<pinref part="U$5" gate="G$1" pin="1Y"/>
-<pinref part="R38" gate="G$1" pin="1"/>
-</segment>
-</net>
 <net name="N$46" class="0">
 <segment>
@@
 <segment>
 <pinref part="X5" gate="-2" pin="KL"/>
-<pinref part="D3" gate="G$1" pin="C"/>
-<wire x1="-292.1" y1="147.32" x2="-292.1" y2="144.78" width="0.1524" layer="91"/>
 <pinref part="Q3" gate="G$1" pin="S"/>
-<wire x1="-292.1" y1="144.78" x2="-292.1" y2="142.24" width="0.1524" layer="91"/>
-<wire x1="-287.02" y1="144.78" x2="-292.1" y2="144.78" width="0.1524" layer="91"/>
-<junction x="-292.1" y="144.78"/>
+<wire x1="-292.1" y1="142.24" x2="-292.1" y2="147.32" width="0.1524" layer="91"/>
+<pinref part="D3" gate="G$1" pin="A"/>
+<wire x1="-292.1" y1="149.86" x2="-292.1" y2="147.32" width="0.1524" layer="91"/>
+<junction x="-292.1" y="147.32"/>
 </segment>
 </net>
@@
 <segment>
 <pinref part="Q3" gate="G$1" pin="G"/>
-<wire x1="-281.94" y1="142.24" x2="-276.86" y2="142.24" width="0.1524" layer="91"/>
+<wire x1="-287.02" y1="139.7" x2="-276.86" y2="139.7" width="0.1524" layer="91"/>
 <pinref part="R47" gate="G$1" pin="1"/>
-<wire x1="-276.86" y1="142.24" x2="-271.78" y2="142.24" width="0.1524" layer="91"/>
-<junction x="-276.86" y="142.24"/>
+<wire x1="-276.86" y1="139.7" x2="-271.78" y2="139.7" width="0.1524" layer="91"/>
+<junction x="-276.86" y="139.7"/>
 <pinref part="R48" gate="G$1" pin="1"/>
 </segment>
@@
 <segment>
 <pinref part="R48" gate="G$1" pin="2"/>
-<wire x1="-261.62" y1="142.24" x2="-254" y2="142.24" width="0.1524" layer="91"/>
-</segment>
-</net>
+<wire x1="-261.62" y1="139.7" x2="-254" y2="139.7" width="0.1524" layer="91"/>
+</segment>
+</net>

Commit message: iramx32
Parts:
- removed U$10, U$11, U$12: ACS712, SparkFun-AnalogIC:ACS712
Changed lines of the file:
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@@
 <part name="Q2" library="crystal" deviceset="CRYSTAL" device="CTS406"/>
 <part name="JP1" library="pinhead" deviceset="PINHD-1X4" device=""/>
-<part name="U$10" library="SparkFun-AnalogIC" deviceset="ACS712" device=""/>
-<part name="U$11" library="SparkFun-AnalogIC" deviceset="ACS712" device=""/>
-<part name="U$12" library="SparkFun-AnalogIC" deviceset="ACS712" device=""/>
 </parts>
 <sheets>
@@
 <instance part="Q2" gate="G$1" x="12.7" y="-45.72" rot="R90"/>
 <instance part="JP1" gate="A" x="119.38" y="-55.88"/>
-<instance part="U$10" gate="G$1" x="195.58" y="127"/>
-<instance part="U$11" gate="G$1" x="195.58" y="106.68"/>
-<instance part="U$12" gate="G$1" x="195.58" y="86.36"/>
 </instances>
 <busses>
