File: hw/eagle/IRAMX-drv-v3.2.brd (EAGLE design)
At the start: 100 x 75 mm, 189 parts, among them IC1 IRAMX16UP60B, IC2 STM32F103R6T, IC5 STM32F405RGT, IC6 78, IC7 7812TV, J1 22-27-2031-03, Q1 IRLML5203, Q3 IRLML5203, T1 zldo1117, T2 zldo1117

Commit message: iramx32
Parts:
- moved C36 0.25 mm to (20.0, 6.75)
- moved C38 0.25 mm to (20.0, 16.5)
- moved C40 0.25 mm to (20.0, 13.5)
- moved C55 0.25 mm to (20.0, 19.5)
- moved C56 0.25 mm to (20.0, 10.5)
Routing:
- net +5V_RES: track 213.6 -> 214.1 mm

Commit message: values
Parts:
- C34, C48, C50, C51, C70: value (none) -> 2.2u
- R43, R8: value 1k -> 22
Changed lines of the file:
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@@
 <element name="C69" library="rcl" package="C0603" value="100n" x="72.75" y="6.25" rot="MR270"/>
 <element name="C68" library="rcl" package="C0603" value="100n" x="40.5" y="33.5" rot="MR180"/>
-<element name="R8" library="rcl" package="R0805" value="1k" x="9.25" y="48.25" rot="MR180"/>
-<element name="R43" library="rcl" package="R0805" value="1k" x="9.25" y="46.25" rot="MR180"/>
+<element name="R8" library="rcl" package="R0805" value="22" x="9.25" y="48.25" rot="MR180"/>
+<element name="R43" library="rcl" package="R0805" value="22" x="9.25" y="46.25" rot="MR180"/>
 <element name="JP11" library="daspilker" package="FCI-10103594-0001LF" value="USB-RECEPTABLE" x="0" y="51.25" rot="MR90"/>
 <element name="U$6" library="reroolib" package="SOIC08" value="ADM485SOIC8" x="19.75" y="28.75" rot="MR270"/>
 <element name="U$7" library="reroolib" package="SOIC08" value="ADM485SOIC8" x="19.75" y="23.5" rot="MR270"/>
-<element name="C70" library="rcl" package="153CLV-0405" value="" x="36.75" y="61" rot="MR180"/>
+<element name="C70" library="rcl" package="153CLV-0405" value="2.2u" x="36.75" y="61" rot="MR180"/>
 <element name="C5" library="rcl" package="C0805" value="4.7u" x="50.5" y="39.5" rot="MR0"/>
 <element name="C6" library="rcl" package="C0805" value="4.7u" x="49" y="35.5" rot="MR0"/>
@@
 <element name="JP1" library="pinhead" package="1X04" value="" x="57.75" y="25.25"/>
 <element name="C33" library="rcl" package="C0603" value="100n" x="14.25" y="10.25" rot="MR270"/>
-<element name="C34" library="rcl" package="153CLV-0405" value="" x="36.75" y="61"/>
-<element name="C48" library="rcl" package="E2,5-6E" value="" x="32.25" y="61.5" rot="R270"/>
+<element name="C34" library="rcl" package="153CLV-0405" value="2.2u" x="36.75" y="61"/>
+<element name="C48" library="rcl" package="E2,5-6E" value="2.2u" x="32.25" y="61.5" rot="R270"/>
 <element name="C49" library="rcl" package="C0603" value="100n" x="9.5" y="31.5" rot="MR180"/>
 <element name="J1" library="con-molex" package="6410-03" value="22-27-2031-03" x="13.25" y="70.5" rot="R180">
@@
 <element name="TP13" library="SparkFun-Passives" package="PAD.03X.03" value="TEST-POINT3" x="56.25" y="35"/>
 <element name="TP14" library="SparkFun-Passives" package="PAD.03X.03" value="TEST-POINT3" x="56.25" y="31"/>
-<element name="C50" library="rcl" package="153CLV-0405" value="" x="50.5" y="35"/>
+<element name="C50" library="rcl" package="153CLV-0405" value="2.2u" x="50.5" y="35"/>
 <element name="TP15" library="SparkFun-Passives" package="PAD.03X.03" value="TEST-POINT3" x="47.75" y="21.25"/>
 <element name="TP16" library="SparkFun-Passives" package="PAD.03X.03" value="TEST-POINT3" x="47.75" y="22.75"/>
-<element name="C51" library="rcl" package="E2,5-6E" value="" x="50.5" y="37.5" rot="R180"/>
+<element name="C51" library="rcl" package="E2,5-6E" value="2.2u" x="50.5" y="37.5" rot="R180"/>
 <element name="TP17" library="SparkFun-Passives" package="PAD.03X.03" value="TEST-POINT3" x="28" y="60.5"/>
 <element name="TP18" library="SparkFun-Passives" package="PAD.03X.03" value="TEST-POINT3" x="35" y="28.75"/>

Commit message: assembly things
Parts:
- C1, C2, C24, C3: value 4.7µ -> 4.7u; device rcl:C0805K -> rcl:C0805
- C57, C58: value 2.2µ -> 2.2u
- R43, R8: device rcl:R0805 -> rcl:R0603
Routing:
- net +5V_RES: track 214.1 -> 213.6 mm
Changed lines of the file:
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@@
 <grid distance="0.25" unitdist="mm" unit="mm" style="lines" multiple="4" display="yes" altdistance="0.001" altunitdist="mm" altunit="mm"/>
 <layers>
-<layer number="1" name="Top" color="4" fill="1" visible="yes" active="yes"/>
+<layer number="1" name="Top" color="4" fill="1" visible="no" active="yes"/>
 <layer number="16" name="Bottom" color="1" fill="1" visible="yes" active="yes"/>
 <layer number="17" name="Pads" color="2" fill="1" visible="yes" active="yes"/>
@@
 <layer number="27" name="tValues" color="7" fill="1" visible="no" active="yes"/>
 <layer number="28" name="bValues" color="7" fill="1" visible="no" active="yes"/>
-<layer number="29" name="tStop" color="7" fill="3" visible="yes" active="yes"/>
-<layer number="30" name="bStop" color="7" fill="6" visible="yes" active="yes"/>
+<layer number="29" name="tStop" color="7" fill="3" visible="no" active="yes"/>
+<layer number="30" name="bStop" color="7" fill="6" visible="no" active="yes"/>
 <layer number="31" name="tCream" color="7" fill="4" visible="no" active="yes"/>
 <layer number="32" name="bCream" color="7" fill="5" visible="no" active="yes"/>
@@
 </autorouter>
 <elements>
-<element name="C1" library="rcl" package="C0805K" value="4.7µ" x="95.5025" y="51.0025" rot="MR0"/>
-<element name="C2" library="rcl" package="C0805K" value="4.7µ" x="95.5025" y="57.005" rot="MR0"/>
-<element name="C3" library="rcl" package="C0805K" value="4.7µ" x="95.5025" y="62.9975" rot="MR0"/>
+<element name="C1" library="rcl" package="C0805" value="4.7u" x="95.5025" y="51.0025" rot="MR0"/>
+<element name="C2" library="rcl" package="C0805" value="4.7u" x="95.5025" y="57.005" rot="MR0"/>
+<element name="C3" library="rcl" package="C0805" value="4.7u" x="95.5025" y="62.9975" rot="MR0"/>
 <element name="C8" library="rcl" package="C0603" value="100n" x="67.7475" y="11.0025" rot="MR0"/>
 <element name="C10" library="rcl" package="C0603" value="100n" x="88.5" y="37.75" rot="MR270"/>
@@
 <element name="C15" library="rcl" package="C1206K" value="100p" x="83.255" y="44.9975" rot="MR270"/>
 <element name="C16" library="rcl" package="C1206K" value="10n" x="89.255" y="45" rot="MR270"/>
-<element name="C24" library="rcl" package="C0805K" value="4.7µ" x="86.4975" y="37.7525" rot="MR270"/>
+<element name="C24" library="rcl" package="C0805" value="4.7u" x="86.4975" y="37.7525" rot="MR270"/>
 <element name="C23" library="rcl" package="C0603" value="100n" x="81.25" y="14" rot="MR90"/>
 <element name="C25" library="rcl" package="C0603" value="100n" x="65.75" y="22" rot="MR0"/>
@@
 <element name="C55" library="rcl" package="C0603" value="100n" x="20" y="19.5" rot="MR270"/>
 <element name="C56" library="rcl" package="C0603" value="100n" x="20" y="10.5" rot="MR90"/>
-<element name="C57" library="rcl" package="C0603" value="2.2µ" x="27" y="27.25" rot="MR90"/>
-<element name="C58" library="rcl" package="C0603" value="2.2µ" x="24.25" y="41.5" rot="MR270"/>
+<element name="C57" library="rcl" package="C0603" value="2.2u" x="27" y="27.25" rot="MR90"/>
+<element name="C58" library="rcl" package="C0603" value="2.2u" x="24.25" y="41.5" rot="MR270"/>
 <element name="C31" library="rcl" package="C0603" value="100n" x="40.5" y="31.5" rot="MR0"/>
 <element name="C36" library="rcl" package="C0603" value="100n" x="20" y="6.75" rot="MR90"/>
@@
 <element name="C69" library="rcl" package="C0603" value="100n" x="72.75" y="6.25" rot="MR270"/>
 <element name="C68" library="rcl" package="C0603" value="100n" x="40.5" y="33.5" rot="MR180"/>
-<element name="R8" library="rcl" package="R0805" value="22" x="9.25" y="48.25" rot="MR180"/>
-<element name="R43" library="rcl" package="R0805" value="22" x="9.25" y="46.25" rot="MR180"/>
+<element name="R8" library="rcl" package="R0603" value="22" x="9.25" y="48.25" rot="MR180"/>
+<element name="R43" library="rcl" package="R0603" value="22" x="9.25" y="46.25" rot="MR180"/>
 <element name="JP11" library="daspilker" package="FCI-10103594-0001LF" value="USB-RECEPTABLE" x="0" y="51.25" rot="MR90"/>
 <element name="U$6" library="reroolib" package="SOIC08" value="ADM485SOIC8" x="19.75" y="28.75" rot="MR270"/>
@@
 <contactref element="IC1" pad="7"/>
 <wire x1="96.5" y1="52.9995" x2="96.5" y2="51.005" width="1" layer="16"/>
-<wire x1="96.5" y1="51.005" x2="96.5025" y2="51.0025" width="1" layer="16"/>
+<wire x1="96.5" y1="51.005" x2="96.4525" y2="51.0025" width="1" layer="16"/>
 </signal>
 <signal name="U" class="1">
@@
 <vertex x="77" y="64.25"/>
 </polygon>
-<wire x1="94.5025" y1="51.0025" x2="91.503" y2="51.0025" width="1" layer="16"/>
+<wire x1="94.5525" y1="51.0025" x2="91.503" y2="51.0025" width="1" layer="16"/>
 <wire x1="91.503" y1="51.0025" x2="91.5" y2="50.9995" width="1" layer="16"/>
 <contactref element="X3" pad="1"/>
@@
 <contactref element="IC1" pad="4"/>
 <wire x1="96.5" y1="58.9995" x2="96.5" y2="57.0075" width="1" layer="16"/>
-<wire x1="96.5" y1="57.0075" x2="96.5025" y2="57.005" width="1" layer="16"/>
+<wire x1="96.5" y1="57.0075" x2="96.4525" y2="57.005" width="1" layer="16"/>
 </signal>
 <signal name="V" class="1">
@@
 </polygon>
 <wire x1="91.5975" y1="57.005" x2="91.5" y2="56.9995" width="1" layer="16"/>
-<wire x1="94.5025" y1="57.005" x2="91.5055" y2="57.005" width="1" layer="16"/>
+<wire x1="94.5525" y1="57.005" x2="91.5055" y2="57.005" width="1" layer="16"/>
 <wire x1="91.5055" y1="57.005" x2="91.5" y2="56.9995" width="1" layer="16"/>
 <contactref element="X3" pad="2"/>
@@
 <contactref element="C3" pad="1"/>
 <contactref element="IC1" pad="1"/>
-<wire x1="96.5025" y1="64.99" x2="96.5025" y2="62.9975" width="1" layer="16"/>
+<wire x1="96.5025" y1="64.99" x2="96.4525" y2="62.9975" width="1" layer="16"/>
 <wire x1="96.5025" y1="64.99" x2="96.5025" y2="64.997" width="0.2" layer="16"/>
 <wire x1="96.5025" y1="64.997" x2="96.5" y2="64.9995" width="0.2" layer="16"/>
@@
 <vertex x="87" y="66.25"/>
 </polygon>
-<wire x1="94.5025" y1="62.9975" x2="91.502" y2="62.9975" width="1" layer="16"/>
+<wire x1="94.5525" y1="62.9975" x2="91.502" y2="62.9975" width="1" layer="16"/>
 <wire x1="91.502" y1="62.9975" x2="91.5" y2="62.9995" width="1" layer="16"/>
 <contactref element="X3" pad="3"/>
@@
 <contactref element="R8" pad="1"/>
 <contactref element="JP11" pad="3"/>
-<wire x1="8.3" y1="48.25" x2="7.75" y2="48.25" width="0.2" layer="16"/>
+<wire x1="8.4" y1="48.25" x2="7.75" y2="48.25" width="0.2" layer="16"/>
 <wire x1="7.75" y1="48.25" x2="6.75" y2="49.25" width="0.2" layer="16"/>
 <wire x1="6.75" y1="49.25" x2="6.75" y2="50.75" width="0.2" layer="16"/>
@@
 <wire x1="6.25" y1="50.25" x2="6.25" y2="47.75" width="0.2" layer="16"/>
 <wire x1="6.25" y1="47.75" x2="7.75" y2="46.25" width="0.2" layer="16"/>
-<wire x1="7.75" y1="46.25" x2="8.3" y2="46.25" width="0.2" layer="16"/>
+<wire x1="7.75" y1="46.25" x2="8.4" y2="46.25" width="0.2" layer="16"/>
 </signal>
 <signal name="TIM1_A">
@@
 <via x="20.25" y="22" extent="1-16" drill="0.3302"/>
 <wire x1="20.25" y1="22" x2="20.25" y2="7.25" width="0.2" layer="1"/>
-<wire x1="20.25" y1="29.5" x2="20.25" y2="29" width="0.2" layer="16"/>
 <wire x1="20.25" y1="29" x2="20.25" y2="25.405" width="0.2" layer="16"/>
 <wire x1="20.25" y1="25.405" x2="20.25" y2="22" width="0.2" layer="16"/>
@@
 <wire x1="86.5" y1="38.9995" x2="88.5" y2="38.9995" width="0.4" layer="16"/>
 <wire x1="88.5" y1="38.9995" x2="91.5" y2="38.9995" width="0.4" layer="16"/>
-<wire x1="86.4975" y1="38.7525" x2="86.5" y2="38.755" width="0.4" layer="16"/>
+<wire x1="86.4975" y1="38.7025" x2="86.5" y2="38.755" width="0.4" layer="16"/>
 <wire x1="86.5" y1="38.755" x2="86.5" y2="38.9995" width="0.4" layer="16"/>
 <wire x1="88.5" y1="38.6" x2="88.5" y2="38.9995" width="0.4" layer="16"/>
@@
 <wire x1="13.75" y1="44.75" x2="10.5" y2="48" width="0.2" layer="16"/>
 <wire x1="10.5" y1="48" x2="10.25" y2="48" width="0.2" layer="16"/>
-<wire x1="10.25" y1="48" x2="10.2" y2="48.25" width="0.2" layer="16"/>
+<wire x1="10.25" y1="48" x2="10.1" y2="48.25" width="0.2" layer="16"/>
 </signal>
 <signal name="N$23">
@@
 <wire x1="21.5" y1="44.25" x2="13.25" y2="44.25" width="0.2" layer="16"/>
 <wire x1="13.25" y1="44.25" x2="11.25" y2="46.25" width="0.2" layer="16"/>
-<wire x1="11.25" y1="46.25" x2="10.2" y2="46.25" width="0.2" layer="16"/>
+<wire x1="11.25" y1="46.25" x2="10.1" y2="46.25" width="0.2" layer="16"/>
 </signal>
 <signal name="N$6">

Commit message: led res
Parts:
- R13, R3, R36, R37, R5: value 180 -> 330
Changed lines of the file:
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@@
 <element name="C14" library="rcl" package="C0603" value="100n" x="63.5" y="15.4975" rot="MR270"/>
 <element name="LED1" library="led" package="LED3MM" value="GELB" x="63.7475" y="3.255" rot="R270"/>
-<element name="R13" library="rcl" package="R0603" value="180" x="65.4975" y="5.2475" rot="MR90"/>
+<element name="R13" library="rcl" package="R0603" value="330" x="65.4975" y="5.2475" rot="MR90"/>
 <element name="IC1" library="iram-b" package="SIP23_TOP" value="IRAMX16UP60B" x="91.5" y="62.9995" rot="R90"/>
 <element name="C17" library="rcl" package="EB35D" value="820µ" x="73" y="47.75" rot="R225"/>
@@
 <element name="R4" library="rcl" package="R0603" value="10k" x="68.75" y="26.75" rot="MR90"/>
 <element name="U$1" library="reroolib" package="SOIC08" value="SI8621" x="44" y="22" rot="MR90"/>
-<element name="R3" library="rcl" package="R0603" value="180" x="59.25" y="7" rot="MR90"/>
+<element name="R3" library="rcl" package="R0603" value="330" x="59.25" y="7" rot="MR90"/>
 <element name="LED3" library="led" package="LED3MM" value="GRÜN" x="59.25" y="3.25" rot="R270"/>
-<element name="R5" library="rcl" package="R0603" value="180" x="70.25" y="6" rot="MR90"/>
+<element name="R5" library="rcl" package="R0603" value="330" x="70.25" y="6" rot="MR90"/>
 <element name="LED4" library="led" package="LED3MM" value="ROT" x="68.25" y="3.25" rot="R270"/>
 <element name="C7" library="rcl" package="C0603" value="18p" x="79.75" y="7.25" rot="MR0"/>
@@
 <element name="C31" library="rcl" package="C0603" value="100n" x="40.5" y="31.5" rot="MR0"/>
 <element name="C36" library="rcl" package="C0603" value="100n" x="20" y="6.75" rot="MR90"/>
-<element name="R36" library="rcl" package="R0603" value="180" x="5.75" y="61.75" rot="MR180"/>
+<element name="R36" library="rcl" package="R0603" value="330" x="5.75" y="61.75" rot="MR180"/>
 <element name="LED5" library="led" package="LED3MM" value="GRÜN" x="3" y="63" rot="R90"/>
-<element name="R37" library="rcl" package="R0603" value="180" x="5.75" y="56.75" rot="MR180"/>
+<element name="R37" library="rcl" package="R0603" value="330" x="5.75" y="56.75" rot="MR180"/>
 <element name="LED6" library="led" package="LED3MM" value="ROT" x="3" y="58" rot="R90"/>
 <element name="JP5" library="pinhead" package="1X03" value="" x="17.5" y="5.5" rot="R90"/>

Commit message: led res
Parts:
- R13, R3, R36, R37, R5: value 330 -> 470
Changed lines of the file:
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@@
 <element name="C14" library="rcl" package="C0603" value="100n" x="63.5" y="15.4975" rot="MR270"/>
 <element name="LED1" library="led" package="LED3MM" value="GELB" x="63.7475" y="3.255" rot="R270"/>
-<element name="R13" library="rcl" package="R0603" value="330" x="65.4975" y="5.2475" rot="MR90"/>
+<element name="R13" library="rcl" package="R0603" value="470" x="65.4975" y="5.2475" rot="MR90"/>
 <element name="IC1" library="iram-b" package="SIP23_TOP" value="IRAMX16UP60B" x="91.5" y="62.9995" rot="R90"/>
 <element name="C17" library="rcl" package="EB35D" value="820µ" x="73" y="47.75" rot="R225"/>
@@
 <element name="R4" library="rcl" package="R0603" value="10k" x="68.75" y="26.75" rot="MR90"/>
 <element name="U$1" library="reroolib" package="SOIC08" value="SI8621" x="44" y="22" rot="MR90"/>
-<element name="R3" library="rcl" package="R0603" value="330" x="59.25" y="7" rot="MR90"/>
+<element name="R3" library="rcl" package="R0603" value="470" x="59.25" y="7" rot="MR90"/>
 <element name="LED3" library="led" package="LED3MM" value="GRÜN" x="59.25" y="3.25" rot="R270"/>
-<element name="R5" library="rcl" package="R0603" value="330" x="70.25" y="6" rot="MR90"/>
+<element name="R5" library="rcl" package="R0603" value="470" x="70.25" y="6" rot="MR90"/>
 <element name="LED4" library="led" package="LED3MM" value="ROT" x="68.25" y="3.25" rot="R270"/>
 <element name="C7" library="rcl" package="C0603" value="18p" x="79.75" y="7.25" rot="MR0"/>
@@
 <element name="C31" library="rcl" package="C0603" value="100n" x="40.5" y="31.5" rot="MR0"/>
 <element name="C36" library="rcl" package="C0603" value="100n" x="20" y="6.75" rot="MR90"/>
-<element name="R36" library="rcl" package="R0603" value="330" x="5.75" y="61.75" rot="MR180"/>
+<element name="R36" library="rcl" package="R0603" value="470" x="5.75" y="61.75" rot="MR180"/>
 <element name="LED5" library="led" package="LED3MM" value="GRÜN" x="3" y="63" rot="R90"/>
-<element name="R37" library="rcl" package="R0603" value="330" x="5.75" y="56.75" rot="MR180"/>
+<element name="R37" library="rcl" package="R0603" value="470" x="5.75" y="56.75" rot="MR180"/>
 <element name="LED6" library="led" package="LED3MM" value="ROT" x="3" y="58" rot="R90"/>
 <element name="JP5" library="pinhead" package="1X03" value="" x="17.5" y="5.5" rot="R90"/>

Commit message: 3.3
Parts:
- added C26: 10n, rcl:C0603
- added JP4: (no value), jumper:SJ_2
- added R52: 10k, rcl:R0603
- JP11: device daspilker:FCI-10103594-0001LF -> reroolib:FCI-10103594-0001LF
- Q1, Q3: value IRLML5203 -> IRLML6344; device transistor-power:MICRO3 -> reroolib:MICRO3
- moved JP1 0.25 mm to (57.8, 25.0)
Connections:
- new net N$52: D5.C, J1.2, JP4.2
- new net USB_SHIELD: C26.1, JP11.6, JP11.7, JP11.8, JP11.9, R52.1
- net +12V_RES: now also JP4.3; no longer D5.C, J1.2
- net +24V_RES: now also JP4.1
- net GND_RES: now also C26.2, Q1.2, Q3.2, R52.2; no longer Q1.3, Q3.3
- net N$42: now also Q1.3; no longer Q1.2
- net N$61: now also Q3.3; no longer Q3.2
Routing:
- net N$52: track 0.00 -> 16.4 mm
- net +12V_RES: track 136.2 -> 121.1 mm
- net GND_RES: track 0.00 -> 5.87 mm, vias 101 -> 124
- net +24V_RES: track 103.2 -> 108.4 mm
- net N$61: track 7.75 -> 6.12 mm
- net N$42: track 7.89 -> 7.31 mm
- added copper zone on layer 1, net USB_SHIELD
- added copper zone on layer 16, net USB_SHIELD
Other:
- outline, holes or cut-outs redrawn

Commit message: cool
Parts:
- moved C50 1.25 mm to (50.5, 36.2)
- moved TP13 0.75 mm to (57.0, 35.0)
- moved TP14 0.75 mm to (57.0, 31.0)
- moved TP19 0.75 mm to (57.0, 33.0)
Routing:
- net +3V3_DRV: track 126.6 -> 106.9 mm, vias 22 -> 24
- net +15V_DRV: track 66.0 -> 62.7 mm
- net GND_DRV: track 0.00 -> 2.55 mm, vias 83 -> 80
