File: hw/eagle/IRAMX-drv-v3.3.sch (EAGLE design)
At the start: 192 parts, among them IC1 IRAMX16UP60B, IC2 STM32F103R6T, IC5 STM32F405RGT, IC6 78, IC7 7812TV, J1 22-27-2031-03, Q1 IRLML6344, Q3 IRLML6344, T1 zldo1117, T2 zldo1117

Commit message: 3.3
Parts:
- added LOGO1: OSHW-LOGOL, SparkFun-Aesthetics:OSHW-LOGOL
Changed lines of the file:
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@@
 <layer number="56" name="wert" color="7" fill="1" visible="no" active="no"/>
 <layer number="57" name="tCAD" color="7" fill="1" visible="no" active="no"/>
+<layer number="59" name="tCarbon" color="7" fill="1" visible="no" active="no"/>
+<layer number="60" name="bCarbon" color="7" fill="1" visible="no" active="no"/>
 <layer number="90" name="Modules" color="5" fill="1" visible="yes" active="yes"/>
 <layer number="91" name="Nets" color="2" fill="1" visible="yes" active="yes"/>
@@
 <layer number="127" name="_tValues" color="7" fill="1" visible="yes" active="yes"/>
 <layer number="128" name="_bValues" color="7" fill="1" visible="yes" active="yes"/>
+<layer number="129" name="Mask" color="7" fill="1" visible="yes" active="yes"/>
 <layer number="131" name="tAdjust" color="7" fill="1" visible="yes" active="yes"/>
 <layer number="132" name="bAdjust" color="7" fill="1" visible="yes" active="yes"/>
@@
 <layer number="223" name="223bmp" color="7" fill="1" visible="yes" active="yes"/>
 <layer number="224" name="224bmp" color="7" fill="1" visible="yes" active="yes"/>
+<layer number="225" name="225bmp" color="7" fill="1" visible="yes" active="yes"/>
+<layer number="226" name="226bmp" color="7" fill="1" visible="yes" active="yes"/>
+<layer number="227" name="227bmp" color="7" fill="1" visible="yes" active="yes"/>
+<layer number="228" name="228bmp" color="7" fill="1" visible="yes" active="yes"/>
+<layer number="229" name="229bmp" color="7" fill="1" visible="yes" active="yes"/>
+<layer number="230" name="230bmp" color="7" fill="1" visible="yes" active="yes"/>
 <layer number="231" name="Eagle3D_PG1" color="7" fill="1" visible="no" active="no"/>
 <layer number="232" name="Eagle3D_PG2" color="7" fill="1" visible="no" active="no"/>
@@
 <part name="C26" library="rcl" deviceset="C-EU" device="C0603" value="10n"/>
 <part name="R52" library="rcl" deviceset="R-EU_" device="R0603" value="10k"/>
+<part name="LOGO1" library="SparkFun-Aesthetics" deviceset="OSHW-LOGO" device="L"/>
 </parts>
 <sheets>
@@
 <instance part="C26" gate="G$1" x="-99.06" y="60.96"/>
 <instance part="R52" gate="G$1" x="-106.68" y="58.42" rot="R270"/>
+<instance part="LOGO1" gate="G$1" x="-27.94" y="33.02"/>
 </instances>
 <busses>

Commit message: 3.3
Parts:
- C31: value 100n -> 2.2u
- SV2: device con-lstb:MA05-1 -> pinhead:PINHD-1X5
Changed lines of the file:
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@@
 <?xml version="1.0" encoding="utf-8"?>
 <!DOCTYPE eagle SYSTEM "eagle.dtd">
-<eagle version="7.1.0">
+<eagle version="7.2.0">
 <drawing>
 <settings>
@@
 <part name="GND41" library="supply1" deviceset="GND" device=""/>
 <part name="+3V11" library="supply1" deviceset="+3V3" device=""/>
-<part name="C31" library="rcl" deviceset="C-EU" device="C0603" value="100n"/>
+<part name="C31" library="rcl" deviceset="C-EU" device="C0603" value="2.2u"/>
 <part name="GND42" library="supply1" deviceset="GND" device=""/>
 <part name="+3V13" library="supply1" deviceset="+3V3" device=""/>
@@
 <part name="R51" library="rcl" deviceset="R-EU_" device="R0603" value="1k"/>
 <part name="+3V9" library="supply1" deviceset="+3V3" device=""/>
-<part name="SV2" library="con-lstb" deviceset="MA05-1" device=""/>
+<part name="SV2" library="pinhead" deviceset="PINHD-1X5" device=""/>
 <part name="JP2" library="pinhead" deviceset="PINHD-1X2" device=""/>
 <part name="JP4" library="jumper" deviceset="SJ2W" device=""/>
@@
 <instance part="R51" gate="G$1" x="-314.96" y="165.1" rot="R270"/>
 <instance part="+3V9" gate="G$1" x="-314.96" y="175.26"/>
-<instance part="SV2" gate="G$1" x="91.44" y="-53.34" rot="R180"/>
+<instance part="SV2" gate="A" x="91.44" y="-53.34" rot="R180"/>
 <instance part="JP2" gate="G$1" x="-5.08" y="121.92" rot="R90"/>
 <instance part="JP4" gate="G$1" x="-320.04" y="213.36" rot="R90"/>
@@
 <pinref part="GND18" gate="1" pin="GND"/>
 <wire x1="99.06" y1="-22.86" x2="99.06" y2="-20.32" width="0.1524" layer="91"/>
-<wire x1="83.82" y1="-48.26" x2="81.28" y2="-48.26" width="0.1524" layer="91"/>
+<wire x1="93.98" y1="-58.42" x2="81.28" y2="-48.26" width="0.1524" layer="91"/>
 <wire x1="81.28" y1="-48.26" x2="81.28" y2="-22.86" width="0.1524" layer="91"/>
 <wire x1="81.28" y1="-22.86" x2="99.06" y2="-22.86" width="0.1524" layer="91"/>
 <junction x="99.06" y="-22.86"/>
-<pinref part="SV2" gate="G$1" pin="1"/>
+<pinref part="SV2" gate="A" pin="1"/>
 </segment>
 <segment>
@@
 <pinref part="+3V4" gate="G$1" pin="+3V3"/>
 <wire x1="99.06" y1="0" x2="99.06" y2="-2.54" width="0.1524" layer="91"/>
-<wire x1="83.82" y1="-58.42" x2="78.74" y2="-58.42" width="0.1524" layer="91"/>
+<wire x1="93.98" y1="-48.26" x2="78.74" y2="-58.42" width="0.1524" layer="91"/>
 <wire x1="78.74" y1="-58.42" x2="78.74" y2="-2.54" width="0.1524" layer="91"/>
 <wire x1="78.74" y1="-2.54" x2="99.06" y2="-2.54" width="0.1524" layer="91"/>
 <junction x="99.06" y="-2.54"/>
-<pinref part="SV2" gate="G$1" pin="5"/>
+<pinref part="SV2" gate="A" pin="5"/>
 </segment>
 <segment>
@@
 <segment>
 <pinref part="IC2" gate="MCU" pin="PA5"/>
-<wire x1="68.58" y1="-55.88" x2="83.82" y2="-55.88" width="0.1524" layer="91"/>
-<pinref part="SV2" gate="G$1" pin="4"/>
+<wire x1="68.58" y1="-55.88" x2="93.98" y2="-50.8" width="0.1524" layer="91"/>
+<pinref part="SV2" gate="A" pin="4"/>
 </segment>
 </net>
@@
 <segment>
 <pinref part="IC2" gate="MCU" pin="PA6"/>
-<wire x1="68.58" y1="-53.34" x2="83.82" y2="-53.34" width="0.1524" layer="91"/>
-<pinref part="SV2" gate="G$1" pin="3"/>
+<wire x1="68.58" y1="-53.34" x2="93.98" y2="-53.34" width="0.1524" layer="91"/>
+<pinref part="SV2" gate="A" pin="3"/>
 </segment>
 </net>
@@
 <segment>
 <pinref part="IC2" gate="MCU" pin="PA7"/>
-<wire x1="68.58" y1="-50.8" x2="83.82" y2="-50.8" width="0.1524" layer="91"/>
-<pinref part="SV2" gate="G$1" pin="2"/>
+<wire x1="68.58" y1="-50.8" x2="93.98" y2="-55.88" width="0.1524" layer="91"/>
+<pinref part="SV2" gate="A" pin="2"/>
 </segment>
 </net>

Commit message: 3.3
Parts:
- removed LED6: ROT, led:LED3MM
- added LED2: GELB, led:LED3MM
- LED1: value GELB -> GRÜN
- LED3, LED5: value GRÜN -> ROT
- LED4: value ROT -> GRÜN
Connections:
- net GND_DRV: now also LED2.C; no longer LED4.C
- net GND_RES: now also LED4.C; no longer LED6.C
- net N$11: now also LED4.A; no longer LED5.A
- net N$20: now also LED5.A; no longer LED6.A
- net N$43: now also LED2.A; no longer LED1.A
- net N$8: now also LED1.A; no longer LED3.A
- net N$9: now also LED3.A; no longer LED4.A
Other:
- moved on the sheet: LED1, LED3, LED4, LED5
Changed lines of the file:
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@@
 <?xml version="1.0" encoding="utf-8"?>
 <!DOCTYPE eagle SYSTEM "eagle.dtd">
-<eagle version="7.2.0">
+<eagle version="7.1.0">
 <drawing>
 <settings>
@@
 <part name="R11" library="rcl" deviceset="R-EU_" device="R0603" value="180"/>
 <part name="C14" library="rcl" deviceset="C-EU" device="C0603" value="100n"/>
-<part name="LED1" library="led" deviceset="LED" device="3MM" value="GELB"/>
+<part name="LED2" library="led" deviceset="LED" device="3MM" value="GELB"/>
 <part name="R13" library="rcl" deviceset="R-EU_" device="R0603" value="470"/>
 <part name="GND21" library="supply1" deviceset="GND" device=""/>
@@
 <part name="+3V6" library="supply1" deviceset="+3V3" device=""/>
 <part name="R3" library="rcl" deviceset="R-EU_" device="R0603" value="470"/>
-<part name="LED3" library="led" deviceset="LED" device="3MM" value="GRÜN"/>
+<part name="LED1" library="led" deviceset="LED" device="3MM" value="GRÜN"/>
 <part name="GND1" library="supply1" deviceset="GND" device=""/>
 <part name="R5" library="rcl" deviceset="R-EU_" device="R0603" value="470"/>
-<part name="LED4" library="led" deviceset="LED" device="3MM" value="ROT"/>
+<part name="LED3" library="led" deviceset="LED" device="3MM" value="ROT"/>
 <part name="GND5" library="supply1" deviceset="GND" device=""/>
 <part name="GND6" library="supply1" deviceset="GND" device=""/>
@@
 <part name="GND46" library="supply1" deviceset="GND" device=""/>
 <part name="R36" library="rcl" deviceset="R-EU_" device="R0603" value="470"/>
-<part name="LED5" library="led" deviceset="LED" device="3MM" value="GRÜN"/>
+<part name="LED4" library="led" deviceset="LED" device="3MM" value="GRÜN"/>
 <part name="GND48" library="supply1" deviceset="GND" device=""/>
 <part name="R37" library="rcl" deviceset="R-EU_" device="R0603" value="470"/>
-<part name="LED6" library="led" deviceset="LED" device="3MM" value="ROT"/>
+<part name="LED5" library="led" deviceset="LED" device="3MM" value="ROT"/>
 <part name="GND49" library="supply1" deviceset="GND" device=""/>
 <part name="JP5" library="pinhead" deviceset="PINHD-1X3" device=""/>
@@
 <instance part="R11" gate="G$1" x="91.44" y="22.86" rot="R180"/>
 <instance part="C14" gate="G$1" x="96.52" y="20.32"/>
-<instance part="LED1" gate="G$1" x="132.08" y="-17.78"/>
+<instance part="LED2" gate="G$1" x="132.08" y="-17.78"/>
 <instance part="R13" gate="G$1" x="132.08" y="-10.16" rot="R90"/>
 <instance part="GND21" gate="1" x="132.08" y="-27.94"/>
@@
 <instance part="+3V6" gate="G$1" x="96.52" y="10.16" rot="R180"/>
 <instance part="R3" gate="G$1" x="147.32" y="-10.16" rot="R90"/>
-<instance part="LED3" gate="G$1" x="147.32" y="-17.78"/>
+<instance part="LED1" gate="G$1" x="147.32" y="-17.78"/>
 <instance part="GND1" gate="1" x="147.32" y="-27.94"/>
 <instance part="R5" gate="G$1" x="157.48" y="-10.16" rot="R90"/>
-<instance part="LED4" gate="G$1" x="157.48" y="-17.78"/>
+<instance part="LED3" gate="G$1" x="157.48" y="-17.78"/>
 <instance part="GND5" gate="1" x="157.48" y="-27.94"/>
 <instance part="GND6" gate="1" x="35.56" y="88.9"/>
@@
 <instance part="GND46" gate="1" x="-238.76" y="10.16"/>
 <instance part="R36" gate="G$1" x="-157.48" y="-93.98" rot="R90"/>
-<instance part="LED5" gate="G$1" x="-157.48" y="-101.6"/>
+<instance part="LED4" gate="G$1" x="-157.48" y="-101.6"/>
 <instance part="GND48" gate="1" x="-157.48" y="-111.76"/>
 <instance part="R37" gate="G$1" x="-147.32" y="-93.98" rot="R90"/>
-<instance part="LED6" gate="G$1" x="-147.32" y="-101.6"/>
+<instance part="LED5" gate="G$1" x="-147.32" y="-101.6"/>
 <instance part="GND49" gate="1" x="-147.32" y="-111.76"/>
 <instance part="JP5" gate="A" x="-314.96" y="7.62" rot="R180"/>
@@
 <net name="N$43" class="0">
 <segment>
-<pinref part="LED1" gate="G$1" pin="A"/>
+<pinref part="LED2" gate="G$1" pin="A"/>
 <pinref part="R13" gate="G$1" pin="1"/>
 </segment>
@@
 <net name="N$8" class="0">
 <segment>
+<pinref part="LED1" gate="G$1" pin="A"/>
+<pinref part="R3" gate="G$1" pin="1"/>
+</segment>
+</net>
+<net name="N$9" class="0">
+<segment>
 <pinref part="LED3" gate="G$1" pin="A"/>
-<pinref part="R3" gate="G$1" pin="1"/>
-</segment>
-</net>
-<net name="N$9" class="0">
-<segment>
-<pinref part="LED4" gate="G$1" pin="A"/>
 <pinref part="R5" gate="G$1" pin="1"/>
 </segment>
@@
 <segment>
 <pinref part="GND21" gate="1" pin="GND"/>
+<pinref part="LED2" gate="G$1" pin="C"/>
+<wire x1="132.08" y1="-25.4" x2="132.08" y2="-22.86" width="0.1524" layer="91"/>
+</segment>
+<segment>
 <pinref part="LED1" gate="G$1" pin="C"/>
-<wire x1="132.08" y1="-25.4" x2="132.08" y2="-22.86" width="0.1524" layer="91"/>
-</segment>
-<segment>
-<pinref part="LED3" gate="G$1" pin="C"/>
 <pinref part="GND1" gate="1" pin="GND"/>
 <wire x1="147.32" y1="-25.4" x2="147.32" y2="-22.86" width="0.1524" layer="91"/>
 </segment>
 <segment>
-<pinref part="LED4" gate="G$1" pin="C"/>
+<pinref part="LED3" gate="G$1" pin="C"/>
 <pinref part="GND5" gate="1" pin="GND"/>
 <wire x1="157.48" y1="-25.4" x2="157.48" y2="-22.86" width="0.1524" layer="91"/>
@@
 </segment>
 <segment>
-<pinref part="LED5" gate="G$1" pin="C"/>
+<pinref part="LED4" gate="G$1" pin="C"/>
 <pinref part="GND48" gate="1" pin="GND"/>
 <wire x1="-157.48" y1="-109.22" x2="-157.48" y2="-106.68" width="0.1524" layer="91"/>
 </segment>
 <segment>
-<pinref part="LED6" gate="G$1" pin="C"/>
+<pinref part="LED5" gate="G$1" pin="C"/>
 <pinref part="GND49" gate="1" pin="GND"/>
 <wire x1="-147.32" y1="-109.22" x2="-147.32" y2="-106.68" width="0.1524" layer="91"/>
@@
 <net name="N$11" class="0">
 <segment>
+<pinref part="LED4" gate="G$1" pin="A"/>
+<pinref part="R36" gate="G$1" pin="1"/>
+</segment>
+</net>
+<net name="N$20" class="0">
+<segment>
 <pinref part="LED5" gate="G$1" pin="A"/>
-<pinref part="R36" gate="G$1" pin="1"/>
-</segment>
-</net>
-<net name="N$20" class="0">
-<segment>
-<pinref part="LED6" gate="G$1" pin="A"/>
 <pinref part="R37" gate="G$1" pin="1"/>
 </segment>

Commit message: 3.3
Other:
- moved on the sheet: C13, C18, C23, C25, C27, C69, C8, J1-1, J1-3, Q1, R30, R35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

Commit message: 3.3
Parts:
- renumbered U$1 to IC12, U$2 to IC14, U$3 to IC10, U$4 to IC11, U$5 to IC13, U$6 to IC8, U$7 to IC9

Commit message: 3.3
Parts:
- renumbered D5 to D4, T1 to IC3, T2 to IC4
Changed lines of the file:
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@@
 <part name="C5" library="rcl" deviceset="C-EU" device="C0805" value="4.7u"/>
 <part name="C6" library="rcl" deviceset="C-EU" device="C0805" value="4.7u"/>
-<part name="T1" library="zetex" deviceset="NPNSOT223" device="" value="zldo1117"/>
-<part name="T2" library="zetex" deviceset="NPNSOT223" device="" value="zldo1117"/>
+<part name="IC3" library="zetex" deviceset="NPNSOT223" device="" value="zldo1117"/>
+<part name="IC4" library="zetex" deviceset="NPNSOT223" device="" value="zldo1117"/>
 <part name="R32" library="rcl" deviceset="R-EU_" device="R0603" value="3.9k"/>
 <part name="R44" library="rcl" deviceset="R-EU_" device="R0603" value="1k"/>
@@
 <part name="J1" library="con-molex" deviceset="22-?-03" device="27-2031"/>
 <part name="Q1" library="reroolib" deviceset="IRLML6344" device=""/>
-<part name="D5" library="adafruit" deviceset="DIODE" device="SOD-123"/>
+<part name="D4" library="adafruit" deviceset="DIODE" device="SOD-123"/>
 <part name="GND62" library="supply1" deviceset="GND" device=""/>
 <part name="R30" library="rcl" deviceset="R-EU_" device="R0603" value="1k"/>
@@
 <instance part="C5" gate="G$1" x="35.56" y="106.68"/>
 <instance part="C6" gate="G$1" x="71.12" y="106.68"/>
-<instance part="T1" gate="A" x="-154.94" y="127" rot="MR90"/>
-<instance part="T2" gate="A" x="45.72" y="106.68" rot="MR90"/>
+<instance part="IC3" gate="A" x="-154.94" y="127" rot="MR90"/>
+<instance part="IC4" gate="A" x="45.72" y="106.68" rot="MR90"/>
 <instance part="R32" gate="G$1" x="-254" y="-45.72" rot="R180"/>
 <instance part="R44" gate="G$1" x="-274.32" y="-40.64" rot="R180"/>
@@
 <instance part="J1" gate="-3" x="-330.2" y="152.4" rot="R180"/>
 <instance part="Q1" gate="1" x="-317.5" y="187.96" rot="MR0"/>
-<instance part="D5" gate="G$1" x="-320.04" y="200.66" rot="R90"/>
+<instance part="D4" gate="G$1" x="-320.04" y="200.66" rot="R90"/>
 <instance part="GND62" gate="1" x="-320.04" y="170.18"/>
 <instance part="R30" gate="G$1" x="-312.42" y="180.34" rot="R270"/>
@@
 <segment>
 <pinref part="GND15" gate="1" pin="GND"/>
-<pinref part="T2" gate="A" pin="B"/>
+<pinref part="IC4" gate="A" pin="B"/>
 <wire x1="45.72" y1="104.14" x2="45.72" y2="91.44" width="0.1524" layer="91"/>
 </segment>
@@
 <segment>
 <pinref part="GND23" gate="1" pin="GND"/>
-<pinref part="T1" gate="A" pin="B"/>
+<pinref part="IC3" gate="A" pin="B"/>
 <wire x1="-154.94" y1="124.46" x2="-157.48" y2="124.46" width="0.1524" layer="91"/>
 <wire x1="-157.48" y1="124.46" x2="-157.48" y2="111.76" width="0.1524" layer="91"/>
@@
 <pinref part="C61" gate="G$1" pin="1"/>
 <wire x1="-127" y1="129.54" x2="-134.62" y2="129.54" width="0.1524" layer="91"/>
-<pinref part="T1" gate="A" pin="C"/>
+<pinref part="IC3" gate="A" pin="C"/>
 <wire x1="-149.86" y1="129.54" x2="-147.32" y2="129.54" width="0.1524" layer="91"/>
 <pinref part="TP20" gate="G$1" pin="1"/>
@@
 <pinref part="P+5" gate="1" pin="+5V"/>
 <wire x1="-200.66" y1="129.54" x2="-175.26" y2="129.54" width="0.1524" layer="91"/>
-<pinref part="T1" gate="A" pin="E"/>
+<pinref part="IC3" gate="A" pin="E"/>
 <pinref part="TP11" gate="G$1" pin="1"/>
 </segment>
@@
 <pinref part="C6" gate="G$1" pin="1"/>
 <junction x="71.12" y="109.22"/>
-<pinref part="T2" gate="A" pin="C"/>
+<pinref part="IC4" gate="A" pin="C"/>
 <wire x1="50.8" y1="109.22" x2="71.12" y2="109.22" width="0.1524" layer="91"/>
 <pinref part="TP14" gate="G$1" pin="1"/>
@@
 <pinref part="C5" gate="G$1" pin="1"/>
 <junction x="35.56" y="109.22"/>
-<pinref part="T2" gate="A" pin="E"/>
+<pinref part="IC4" gate="A" pin="E"/>
 <wire x1="35.56" y1="109.22" x2="40.64" y2="109.22" width="0.1524" layer="91"/>
 <pinref part="TP13" gate="G$1" pin="1"/>
@@
 <net name="N$42" class="0">
 <segment>
-<pinref part="D5" gate="G$1" pin="A"/>
+<pinref part="D4" gate="G$1" pin="A"/>
 <pinref part="J1" gate="-1" pin="S"/>
 <wire x1="-320.04" y1="195.58" x2="-320.04" y2="198.12" width="0.1524" layer="91"/>
@@
 <segment>
 <pinref part="J1" gate="-2" pin="S"/>
-<pinref part="D5" gate="G$1" pin="C"/>
+<pinref part="D4" gate="G$1" pin="C"/>
 <wire x1="-320.04" y1="203.2" x2="-320.04" y2="205.74" width="0.1524" layer="91"/>
 <pinref part="JP4" gate="G$1" pin="2"/>
