File: hw/eagle/bene2stmbl-smd.sch (EAGLE design)
At the start: 15 parts, among them IC2 7414D

Commit message: bene adapter vaules
Parts:
- C1, C2: value (none) -> 100n
- R1, R2: value (none) -> 330
- R4, R5: value (none) -> 3k9
Changed lines of the file:
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@@
 <part name="X1" library="reroolib" deviceset="RJ45" device=""/>
 <part name="X2" library="reroolib" deviceset="RJ45" device=""/>
-<part name="R1" library="resistor" deviceset="R-EU_" device="R0603"/>
-<part name="R2" library="resistor" deviceset="R-EU_" device="R0603"/>
-<part name="C1" library="resistor" deviceset="C-EU" device="C0603"/>
-<part name="C2" library="resistor" deviceset="C-EU" device="C0603"/>
+<part name="R1" library="resistor" deviceset="R-EU_" device="R0603" value="330"/>
+<part name="R2" library="resistor" deviceset="R-EU_" device="R0603" value="330"/>
+<part name="C1" library="resistor" deviceset="C-EU" device="C0603" value="100n"/>
+<part name="C2" library="resistor" deviceset="C-EU" device="C0603" value="100n"/>
 <part name="R3" library="resistor" deviceset="R-EU_" device="R0603"/>
-<part name="R4" library="resistor" deviceset="R-EU_" device="R0603"/>
-<part name="R5" library="resistor" deviceset="R-EU_" device="R0603"/>
+<part name="R4" library="resistor" deviceset="R-EU_" device="R0603" value="3k9"/>
+<part name="R5" library="resistor" deviceset="R-EU_" device="R0603" value="3k9"/>
 <part name="U$1" library="reroolib" deviceset="HCPL-053L-SMD" device=""/>
 <part name="SUPPLY2" library="SparkFun-Aesthetics" deviceset="VCC" device=""/>
