File: hw/eagle/IRAMX-drv-v3.4.brd (EAGLE design)
At the start: 100 x 75 mm, 175 parts, among them IC1 IRAMX16UP60B, IC10 TCA0372DWDM2, IC12 SI8621, IC13 AM26LS32ACD, IC14 rk-2415s, IC2 STM32F103R6T, IC3 LD117AS33TR, IC4 LD117AS33TR, IC5 STM32F405RGT, IC6 78, IC7 7812TV, IC8 ADM485SOIC8, IC9 ADM485SOIC8, J1 22-27-2031-03, Q1 IRLML6344, Q2 8M, Q3 IRLML6344, Q4 8M

Commit message: fixed 3v3 regulator footprint
Parts:
- IC3, IC4: device v-reg:SOT223 -> reroolib:SOT223
Connections:
- net +3V3_DRV: now also IC4.2
- net +3V3_RES: now also IC3.2
Changed lines of the file:
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@@
 <?xml version="1.0" encoding="utf-8"?>
 <!DOCTYPE eagle SYSTEM "eagle.dtd">
-<eagle version="7.5.0">
+<eagle version="7.2.0">
 <drawing>
 <settings>
@@
 </element>
 <element name="LOGO1" library="SparkFun-Aesthetics" package="OSHW-LOGO-L" value="OSHW-LOGOL" x="26.25" y="11.25" smashed="yes"/>
-<element name="IC3" library="v-reg" package="SOT223" value="LD117AS33TR" x="37.75" y="14.75" rot="MR270"/>
-<element name="IC4" library="v-reg" package="SOT223" value="LD117AS33TR" x="50" y="30" rot="MR180"/>
+<element name="IC3" library="reroolib" package="SOT223" value="LD117AS33TR" x="37.75" y="14.75" rot="MR270"/>
+<element name="IC4" library="reroolib" package="SOT223" value="LD117AS33TR" x="50" y="30" rot="MR180"/>
 </elements>
 <signals>
@@
 <wire x1="36" y1="43" x2="35.5" y2="43" width="0.2" layer="1"/>
 <contactref element="IC3" pad="4"/>
+<contactref element="IC3" pad="2"/>
 </signal>
 <signal name="+5V_RES">
@@
 <via x="63.25" y="9.75" extent="1-16" drill="0.3302"/>
 <contactref element="IC4" pad="4"/>
+<contactref element="IC4" pad="2"/>
 </signal>
 <signal name="+24V_RES">

Commit message: name signals
Connections:
- net N$13 renamed VCAP2
- net N$14 renamed VCAP1
- net N$15 renamed OSC_OUT
- net N$22 renamed USB_DP_
- net N$23 renamed USB_DM_
- net N$39 renamed OSC_IN
- net N$4 renamed PA5
- net N$46 renamed VDDA
- net N$49 renamed PA6
- net N$51 renamed PA7
Routing:
- net N$40: track 48.7 -> 47.4 mm
Changed lines of the file:
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@@
 <?xml version="1.0" encoding="utf-8"?>
 <!DOCTYPE eagle SYSTEM "eagle.dtd">
-<eagle version="7.2.0">
+<eagle version="7.7.0">
 <drawing>
 <settings>
@@
 <wire x1="5.25" y1="35.25" x2="5.5" y2="35.4" width="0.2" layer="16"/>
 </signal>
-<signal name="N$15">
+<signal name="OSC_OUT">
 <contactref element="C44" pad="2"/>
 <contactref element="IC5" pad="6"/>
@@
 <wire x1="41.6" y1="37" x2="40.5" y2="37" width="0.2" layer="16"/>
 </signal>
-<signal name="N$39">
+<signal name="OSC_IN">
 <contactref element="C43" pad="2"/>
 <contactref element="IC5" pad="5"/>
@@
 <wire x1="52.3114" y1="33.15" x2="52.3114" y2="37.5" width="0.4" layer="16"/>
 </signal>
-<signal name="N$13">
+<signal name="VCAP2">
 <contactref element="C58" pad="2"/>
 <contactref element="IC5" pad="47"/>
@@
 <wire x1="25.25" y1="38" x2="26" y2="38" width="0.2" layer="16"/>
 </signal>
-<signal name="N$14">
+<signal name="VCAP1">
 <contactref element="IC5" pad="31"/>
 <contactref element="C57" pad="2"/>
@@
 <wire x1="8.235" y1="17.615" x2="7.35" y2="18.5" width="0.2" layer="16"/>
 </signal>
-<signal name="N$46">
+<signal name="VDDA">
 <contactref element="C31" pad="2"/>
 <contactref element="IC5" pad="13"/>
@@
 <wire x1="14.5" y1="32.75" x2="11.5" y2="29.75" width="0.2" layer="16"/>
 <wire x1="11.5" y1="29.75" x2="11.5" y2="28.5" width="0.2" layer="16"/>
-<wire x1="4.5" y1="21.5" x2="4.5" y2="16" width="0.2" layer="16"/>
-<wire x1="4.5" y1="16" x2="8.25" y2="16" width="0.2" layer="16"/>
-<wire x1="8.25" y1="16" x2="8.595" y2="16.345" width="0.2" layer="16"/>
-<wire x1="8.595" y1="16.345" x2="11.89" y2="16.345" width="0.2" layer="16"/>
+<wire x1="4.5" y1="21.5" x2="4.5" y2="17.75" width="0.2" layer="16"/>
 <wire x1="4.5" y1="21.5" x2="11.5" y2="28.5" width="0.2" layer="16"/>
 <wire x1="15" y1="12.9" x2="14.85" y2="12.9" width="0.2" layer="16"/>
@@
 <wire x1="16.65" y1="12.25" x2="16" y2="12.9" width="0.2" layer="16"/>
 <wire x1="16" y1="12.9" x2="15" y2="12.9" width="0.2" layer="16"/>
+<wire x1="4.5" y1="17.75" x2="5.905" y2="16.345" width="0.2" layer="16"/>
+<wire x1="5.905" y1="16.345" x2="11.89" y2="16.345" width="0.2" layer="16"/>
 </signal>
 <signal name="N$50">
@@
 <wire x1="12" y1="28.25" x2="7.5" y2="23.75" width="0.2" layer="16"/>
 </signal>
-<signal name="N$22">
+<signal name="USB_DP_">
 <contactref element="R8" pad="2"/>
 <contactref element="IC5" pad="45"/>
@@
 <wire x1="10.25" y1="48" x2="10.1" y2="48.25" width="0.2" layer="16"/>
 </signal>
-<signal name="N$23">
+<signal name="USB_DM_">
 <contactref element="IC5" pad="44"/>
 <contactref element="R43" pad="2"/>
@@
 <wire x1="18" y1="63.9" x2="17.85" y2="64" width="0.2" layer="16"/>
 </signal>
-<signal name="N$4">
+<signal name="PA5">
 <contactref element="IC2" pad="21"/>
 <contactref element="SV2" pad="4"/>
@@
 <wire x1="54.21" y1="9.75" x2="54" y2="9.96" width="0.2" layer="1"/>
 </signal>
-<signal name="N$49">
+<signal name="PA6">
 <contactref element="IC2" pad="22"/>
 <contactref element="SV2" pad="3"/>
@@
 <wire x1="55.75" y1="12.5" x2="54" y2="12.5" width="0.2" layer="1"/>
 </signal>
-<signal name="N$51">
+<signal name="PA7">
 <contactref element="IC2" pad="23"/>
 <contactref element="SV2" pad="2"/>
