File: hw/eagle/uhu-adapter.sch (EAGLE design)
At the start: 17 parts, among them IC1 STM32F303CBT

Commit message: uhu adapter
Parts:
- added D1: (no value), diode:DIODE-SOD123
- added R4: 10k, rcl:R-EU_R0603
- C1, C2, C3, C4, C5, C6: value (none) -> 100n
Connections:
- removed net IO0: SV4.3
- removed net IO2: SV3.1
- new net 5VUSB: D1.A, JP1.VCC
- new net N$21: IC1MCU.PC13
- new net N$22: IC1MCU.PC14
- new net N$25: IC1MCU.PC15
- new net SWCLK: IC1MCU.PA14, SV3.1
- new net SWDIO: IC1MCU.PA13, SV4.3
- net 3V3: now also R4.1
- net 5V: now also D1.C
- net GND: now also IC1MCU.BOOT0
- net IO1: now also IC1MCU.PA15
- net IO3: now also IC1MCU.PA0-WKUP
- net IO4: now also IC1MCU.PA1, R4.2
- net START: now also IC1MCU.PA10; no longer IC1MCU.PA15
Other:
- moved on the sheet: C1
Changed lines of the file:
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@@
 <layer number="113" name="IDFDebug" color="7" fill="1" visible="yes" active="yes"/>
 <layer number="116" name="Patch_BOT" color="9" fill="4" visible="yes" active="yes"/>
+<layer number="118" name="Rect_Pads" color="7" fill="1" visible="no" active="no"/>
 <layer number="121" name="_tsilk" color="7" fill="1" visible="yes" active="yes"/>
 <layer number="122" name="_bsilk" color="7" fill="1" visible="yes" active="yes"/>
@@
 <layer number="230" name="230bmp" color="7" fill="1" visible="yes" active="yes"/>
 <layer number="231" name="231bmp" color="7" fill="1" visible="yes" active="yes"/>
+<layer number="232" name="Eagle3D_PG2" color="7" fill="1" visible="no" active="no"/>
+<layer number="233" name="Eagle3D_PG3" color="7" fill="1" visible="no" active="no"/>
 <layer number="248" name="Housing" color="7" fill="1" visible="yes" active="yes"/>
 <layer number="249" name="Edge" color="7" fill="1" visible="yes" active="yes"/>
@@
 <part name="GND1" library="supply1" deviceset="GND" device=""/>
 <part name="GND2" library="supply1" deviceset="GND" device=""/>
-<part name="C1" library="rcl" deviceset="C-EU" device="C0603"/>
+<part name="C1" library="rcl" deviceset="C-EU" device="C0603" value="100n"/>
 <part name="R1" library="rcl" deviceset="R-EU_" device="R0603" value="22"/>
 <part name="R2" library="rcl" deviceset="R-EU_" device="R0603" value="22"/>
 <part name="R3" library="rcl" deviceset="R-EU_" device="R0603" value="1k5"/>
 <part name="GND3" library="supply1" deviceset="GND" device=""/>
-<part name="C2" library="rcl" deviceset="C-EU" device="C0603"/>
-<part name="C3" library="rcl" deviceset="C-EU" device="C0603"/>
-<part name="C4" library="rcl" deviceset="C-EU" device="C0603"/>
-<part name="C5" library="rcl" deviceset="C-EU" device="C0603"/>
-<part name="C6" library="rcl" deviceset="C-EU" device="C0603"/>
+<part name="C2" library="rcl" deviceset="C-EU" device="C0603" value="100n"/>
+<part name="C3" library="rcl" deviceset="C-EU" device="C0603" value="100n"/>
+<part name="C4" library="rcl" deviceset="C-EU" device="C0603" value="100n"/>
+<part name="C5" library="rcl" deviceset="C-EU" device="C0603" value="100n"/>
+<part name="C6" library="rcl" deviceset="C-EU" device="C0603" value="100n"/>
+<part name="R4" library="rcl" deviceset="R-EU_" device="R0603" value="10k"/>
+<part name="D1" library="diode" deviceset="DIODE-" device="SOD123"/>
 </parts>
 <sheets>
@@
 <instance part="GND1" gate="1" x="81.28" y="144.78"/>
 <instance part="GND2" gate="1" x="5.08" y="76.2" rot="R90"/>
-<instance part="C1" gate="G$1" x="43.18" y="33.02"/>
+<instance part="C1" gate="G$1" x="38.1" y="33.02"/>
 <instance part="R1" gate="G$1" x="27.94" y="71.12" rot="R180"/>
 <instance part="R2" gate="G$1" x="20.32" y="68.58" rot="R180"/>
 <instance part="R3" gate="G$1" x="12.7" y="76.2" rot="R270"/>
-<instance part="GND3" gate="1" x="43.18" y="22.86"/>
+<instance part="GND3" gate="1" x="38.1" y="22.86"/>
 <instance part="C2" gate="G$1" x="88.9" y="187.96"/>
 <instance part="C3" gate="G$1" x="43.18" y="187.96"/>
@@
 <instance part="C5" gate="G$1" x="129.54" y="170.18"/>
 <instance part="C6" gate="G$1" x="137.16" y="170.18"/>
+<instance part="R4" gate="G$1" x="111.76" y="43.18" rot="R270"/>
+<instance part="D1" gate="G$1" x="5.08" y="66.04"/>
 </instances>
 <busses>
@@
 <wire x1="210.82" y1="63.5" x2="203.2" y2="63.5" width="0.1524" layer="91"/>
 <label x="203.2" y="63.5" size="1.778" layer="95"/>
+</segment>
+<segment>
+<pinref part="D1" gate="G$1" pin="C"/>
+<wire x1="7.62" y1="66.04" x2="15.24" y2="66.04" width="0.1524" layer="91"/>
+<label x="12.7" y="66.04" size="1.778" layer="95"/>
 </segment>
 </net>
@@
 <pinref part="C1" gate="G$1" pin="2"/>
 <pinref part="GND3" gate="1" pin="GND"/>
-<wire x1="43.18" y1="27.94" x2="43.18" y2="25.4" width="0.1524" layer="91"/>
+<wire x1="38.1" y1="27.94" x2="38.1" y2="25.4" width="0.1524" layer="91"/>
 </segment>
 <segment>
@@
 <wire x1="185.42" y1="40.64" x2="193.04" y2="40.64" width="0.1524" layer="91"/>
 <label x="187.96" y="40.64" size="1.778" layer="95"/>
+</segment>
+<segment>
+<pinref part="IC1" gate="MCU" pin="BOOT0"/>
+<wire x1="53.34" y1="33.02" x2="45.72" y2="33.02" width="0.1524" layer="91"/>
+<label x="45.72" y="33.02" size="1.778" layer="95"/>
 </segment>
 </net>
@@
 <segment>
 <pinref part="IC1" gate="MCU" pin="PA11"/>
-<wire x1="99.06" y1="60.96" x2="111.76" y2="60.96" width="0.1524" layer="91"/>
+<wire x1="99.06" y1="60.96" x2="109.22" y2="60.96" width="0.1524" layer="91"/>
 <label x="104.14" y="60.96" size="1.778" layer="95"/>
 </segment>
@@
 <segment>
 <pinref part="IC1" gate="MCU" pin="PA12"/>
-<wire x1="99.06" y1="63.5" x2="111.76" y2="63.5" width="0.1524" layer="91"/>
+<wire x1="99.06" y1="63.5" x2="109.22" y2="63.5" width="0.1524" layer="91"/>
 <label x="104.14" y="63.5" size="1.778" layer="95"/>
 </segment>
@@
 <label x="45.72" y="45.72" size="1.778" layer="95"/>
 </segment>
+<segment>
+<pinref part="R4" gate="G$1" pin="1"/>
+<wire x1="111.76" y1="48.26" x2="111.76" y2="53.34" width="0.1524" layer="91"/>
+<label x="111.76" y="50.8" size="1.778" layer="95" rot="R90"/>
+</segment>
 </net>
 <net name="NRST" class="0">
@@
 <pinref part="IC1" gate="MCU" pin="NRST"/>
 <pinref part="C1" gate="G$1" pin="1"/>
-<wire x1="53.34" y1="35.56" x2="43.18" y2="35.56" width="0.1524" layer="91"/>
+<wire x1="53.34" y1="35.56" x2="38.1" y2="35.56" width="0.1524" layer="91"/>
 <label x="45.72" y="35.56" size="1.778" layer="95"/>
 </segment>
@@
 </segment>
 <segment>
+<pinref part="IC1" gate="MCU" pin="PA10"/>
+<wire x1="99.06" y1="58.42" x2="109.22" y2="58.42" width="0.1524" layer="91"/>
+<label x="104.14" y="58.42" size="1.778" layer="95"/>
+</segment>
+</net>
+<net name="IO3" class="0">
+<segment>
+<pinref part="SV3" gate="1" pin="8"/>
+<wire x1="210.82" y1="58.42" x2="203.2" y2="58.42" width="0.1524" layer="91"/>
+<label x="203.2" y="58.42" size="1.778" layer="95"/>
+</segment>
+<segment>
+<pinref part="IC1" gate="MCU" pin="PA0-WKUP"/>
+<wire x1="99.06" y1="33.02" x2="111.76" y2="33.02" width="0.1524" layer="91"/>
+<label x="104.14" y="33.02" size="1.778" layer="95"/>
+</segment>
+</net>
+<net name="IO4" class="0">
+<segment>
+<pinref part="SV3" gate="1" pin="9"/>
+<wire x1="210.82" y1="60.96" x2="203.2" y2="60.96" width="0.1524" layer="91"/>
+<label x="203.2" y="60.96" size="1.778" layer="95"/>
+</segment>
+<segment>
+<pinref part="IC1" gate="MCU" pin="PA1"/>
+<wire x1="99.06" y1="35.56" x2="109.22" y2="35.56" width="0.1524" layer="91"/>
+<label x="104.14" y="35.56" size="1.778" layer="95"/>
+<pinref part="R4" gate="G$1" pin="2"/>
+<wire x1="109.22" y1="35.56" x2="111.76" y2="35.56" width="0.1524" layer="91"/>
+<wire x1="111.76" y1="35.56" x2="111.76" y2="38.1" width="0.1524" layer="91"/>
+</segment>
+</net>
+<net name="IO1" class="0">
+<segment>
+<pinref part="SV4" gate="1" pin="2"/>
+<wire x1="185.42" y1="43.18" x2="193.04" y2="43.18" width="0.1524" layer="91"/>
+<label x="187.96" y="43.18" size="1.778" layer="95"/>
+</segment>
+<segment>
 <pinref part="IC1" gate="MCU" pin="PA15"/>
 <wire x1="99.06" y1="71.12" x2="109.22" y2="71.12" width="0.1524" layer="91"/>
@@
 </segment>
 </net>
-<net name="IO3" class="0">
-<segment>
-<pinref part="SV3" gate="1" pin="8"/>
-<wire x1="210.82" y1="58.42" x2="203.2" y2="58.42" width="0.1524" layer="91"/>
-<label x="203.2" y="58.42" size="1.778" layer="95"/>
-</segment>
-</net>
-<net name="IO4" class="0">
-<segment>
-<pinref part="SV3" gate="1" pin="9"/>
-<wire x1="210.82" y1="60.96" x2="203.2" y2="60.96" width="0.1524" layer="91"/>
-<label x="203.2" y="60.96" size="1.778" layer="95"/>
-</segment>
-</net>
-<net name="IO1" class="0">
-<segment>
-<pinref part="SV4" gate="1" pin="2"/>
-<wire x1="185.42" y1="43.18" x2="193.04" y2="43.18" width="0.1524" layer="91"/>
-<label x="187.96" y="43.18" size="1.778" layer="95"/>
-</segment>
-</net>
-<net name="IO0" class="0">
+<net name="SWDIO" class="0">
 <segment>
 <pinref part="SV4" gate="1" pin="3"/>
@@
 <label x="187.96" y="45.72" size="1.778" layer="95"/>
 </segment>
-</net>
-<net name="IO2" class="0">
+<segment>
+<pinref part="IC1" gate="MCU" pin="PA13"/>
+<wire x1="99.06" y1="66.04" x2="109.22" y2="66.04" width="0.1524" layer="91"/>
+<label x="104.14" y="66.04" size="1.778" layer="95"/>
+</segment>
+</net>
+<net name="SWCLK" class="0">
 <segment>
 <pinref part="SV3" gate="1" pin="1"/>
@@
 <label x="203.2" y="40.64" size="1.778" layer="95"/>
 </segment>
-</net>
+<segment>
+<pinref part="IC1" gate="MCU" pin="PA14"/>
+<wire x1="99.06" y1="68.58" x2="109.22" y2="68.58" width="0.1524" layer="91"/>
+<label x="104.14" y="68.58" size="1.778" layer="95"/>
+</segment>
+</net>
+<net name="N$21" class="0">
+<segment>
+<pinref part="IC1" gate="MCU" pin="PC13"/>
+<wire x1="53.34" y1="76.2" x2="45.72" y2="76.2" width="0.1524" layer="91"/>
+</segment>
+</net>
+<net name="N$22" class="0">
+<segment>
+<pinref part="IC1" gate="MCU" pin="PC14"/>
+<wire x1="53.34" y1="78.74" x2="45.72" y2="78.74" width="0.1524" layer="91"/>
+</segment>
+</net>
+<net name="N$25" class="0">
+<segment>
+<pinref part="IC1" gate="MCU" pin="PC15"/>
+<wire x1="53.34" y1="81.28" x2="45.72" y2="81.28" width="0.1524" layer="91"/>
+</segment>
+</net>
+<net name="5VUSB" class="0">
+<segment>
+<pinref part="JP1" gate="G$1" pin="VCC"/>
+<pinref part="D1" gate="G$1" pin="A"/>
+<wire x1="-2.54" y1="66.04" x2="2.54" y2="66.04" width="0.1524" layer="91"/>
+</segment>
+</net>
