File: hw/kicad/v3.4/fb.sch (KiCad schematic (older format))
At the start: 44 parts

Commit message: fb fix, cleanup
Parts:
- added R?: 10k, symbol R
Connections:
- net +12V: now also R?.2
- net at JP?.2, R?.1, R?.2: now also R?.1
Changed lines of the file:
@@
 $Descr A4 11693 8268
 encoding utf-8
-Sheet 10 14
+Sheet 12 14
 Title ""
 Date ""
@@
 Wire Wire Line
 	3100 4650 3300 4650
-Connection ~ 3200 4650
 Wire Wire Line
 	3200 4350 3000 4350
@@
 Connection ~ 3700 3150
 Connection ~ 3600 3550
+$Comp
+L R R?
+U 1 1 56666171
+P 3200 4800
+F 0 "R?" V 3280 4800 50  0000 C CNN
+F 1 "10k" V 3200 4800 50  0000 C CNN
+F 2 "" V 3130 4800 30  0000 C CNN
+F 3 "" H 3200 4800 30  0000 C CNN
+	1    3200 4800
+	1    0    0    -1
+$EndComp
+Connection ~ 3200 4650
+Wire Wire Line
+	3200 4950 3000 4950
+Connection ~ 3000 4950
 $EndSCHEMATC

Commit message: hw v3.4
Connections:
- net at C?.1, R?.1, R?.2: now also U?.3 (+); no longer U?.5 (+)
- net at C?.2, R?.1, R?.2: now also U?.2 (-); no longer U?.6 (-)
- net at R?.1, R?.2: now also U?.1; no longer U?.7

Commit message: hw v3.4 +testpoints
Parts:
- added T? (x8): testpoint, symbol testpoint
Connections:
- net +1V8: now also T?.1
- net A12: now also T?.1
- net A35: now also T?.1
- net C8: now also T?.1
- net D12: now also T?.1
- net D36: now also T?.1
- net D45: now also T?.1
- net GND: now also T?.1
Changed lines of the file:
@@
 EESchema Schematic File Version 2
-LIBS:conn
 LIBS:power
 LIBS:stmbl_3.4-cache
@@
 Connection ~ 8600 1250
 Wire Wire Line
-	8550 1450 8900 1450
+	8900 1450 8550 1450
 Wire Wire Line
 	8550 2550 8600 2550
@@
 Connection ~ 8600 2650
 Wire Wire Line
-	8550 2850 8900 2850
+	8900 2850 8550 2850
 Wire Wire Line
 	8550 3950 8600 3950
@@
 Connection ~ 8600 4050
 Wire Wire Line
-	8550 4250 8900 4250
+	8900 4250 8550 4250
 Wire Wire Line
 	2200 2950 6300 2950
@@
 	4450 4050 4450 4000
 Wire Wire Line
-	6100 4500 6100 4600
+	6100 4400 6100 4600
 Wire Wire Line
 	6000 4600 6200 4600
@@
 	5500 5600 5700 5600
 Wire Wire Line
-	6100 5600 6100 5700
+	6100 5500 6100 5700
 Wire Wire Line
 	6000 5700 6200 5700
@@
 	2700 6150 2700 6250
 Wire Wire Line
-	2700 6250 2500 6250
+	2500 6250 2800 6250
 Wire Wire Line
 	2600 6350 2600 6250
@@
 	3000 4900 3000 5000
 Wire Wire Line
-	8900 1450 8900 1050
+	8900 950  8900 1450
 Connection ~ 8900 1050
 Wire Wire Line
-	8900 2850 8900 2450
+	8900 2350 8900 2850
 Connection ~ 8900 2450
 Wire Wire Line
-	8900 4250 8900 3850
+	8900 3750 8900 4250
 Connection ~ 8900 3850
 Wire Wire Line
@@
 	2600 4150 2600 4100
 Wire Wire Line
-	2400 4100 2650 4100
+	2200 4100 2650 4100
 Wire Wire Line
 	2600 4500 2600 4450
@@
 	3200 4950 3000 4950
 Connection ~ 3000 4950
+$Comp
+L testpoint T?
+U 1 1 5681BCA9
+P 8900 750
+AR Path="/56590966/5659191C/5681BCA9" Ref="T?"  Part="1"
+AR Path="/56590966/565F7162/5681BCA9" Ref="T?"  Part="1"
+F 0 "T?" H 8900 850 60  0000 C CNN
+F 1 "testpoint" H 8900 650 60  0000 C CNN
+F 2 "" H 8900 750 60  0000 C CNN
+F 3 "" H 8900 750 60  0000 C CNN
+	1    8900 750
+	0    -1   -1   0
+$EndComp
+$Comp
+L testpoint T?
+U 1 1 5681BE5B
+P 8900 2150
+AR Path="/56590966/5659191C/5681BE5B" Ref="T?"  Part="1"
+AR Path="/56590966/565F7162/5681BE5B" Ref="T?"  Part="1"
+F 0 "T?" H 8900 2250 60  0000 C CNN
+F 1 "testpoint" H 8900 2050 60  0000 C CNN
+F 2 "" H 8900 2150 60  0000 C CNN
+F 3 "" H 8900 2150 60  0000 C CNN
+	1    8900 2150
+	0    -1   -1   0
+$EndComp
+$Comp
+L testpoint T?
+U 1 1 5681C17F
+P 8900 3550
+AR Path="/56590966/5659191C/5681C17F" Ref="T?"  Part="1"
+AR Path="/56590966/565F7162/5681C17F" Ref="T?"  Part="1"
+F 0 "T?" H 8900 3650 60  0000 C CNN
+F 1 "testpoint" H 8900 3450 60  0000 C CNN
+F 2 "" H 8900 3550 60  0000 C CNN
+F 3 "" H 8900 3550 60  0000 C CNN
+	1    8900 3550
+	0    -1   -1   0
+$EndComp
+$Comp
+L testpoint T?
+U 1 1 5681CB1F
+P 6100 4200
+AR Path="/56590966/5659191C/5681CB1F" Ref="T?"  Part="1"
+AR Path="/56590966/565F7162/5681CB1F" Ref="T?"  Part="1"
+F 0 "T?" H 6100 4300 60  0000 C CNN
+F 1 "testpoint" H 6100 4100 60  0000 C CNN
+F 2 "" H 6100 4200 60  0000 C CNN
+F 3 "" H 6100 4200 60  0000 C CNN
+	1    6100 4200
+	0    -1   -1   0
+$EndComp
+$Comp
+L testpoint T?
+U 1 1 5681CBE7
+P 6100 5300
+AR Path="/56590966/565F7162/5681CBE7" Ref="T?"  Part="1"
+AR Path="/56590966/5659191C/5681CBE7" Ref="T?"  Part="1"
+F 0 "T?" H 6100 5400 60  0000 C CNN
+F 1 "testpoint" H 6100 5200 60  0000 C CNN
+F 2 "" H 6100 5300 60  0000 C CNN
+F 3 "" H 6100 5300 60  0000 C CNN
+	1    6100 5300
+	0    -1   -1   0
+$EndComp
+$Comp
+L testpoint T?
+U 1 1 5681D090
+P 2000 4100
+AR Path="/56590966/5659191C/5681D090" Ref="T?"  Part="1"
+AR Path="/56590966/565F7162/5681D090" Ref="T?"  Part="1"
+F 0 "T?" H 2000 4200 60  0000 C CNN
+F 1 "testpoint" H 2000 4000 60  0000 C CNN
+F 2 "" H 2000 4100 60  0000 C CNN
+F 3 "" H 2000 4100 60  0000 C CNN
+	1    2000 4100
+	-1   0    0    1
+$EndComp
+$Comp
+L testpoint T?
+U 1 1 568217DB
+P 2300 5750
+AR Path="/56590966/565F7162/568217DB" Ref="T?"  Part="1"
+AR Path="/56590966/5659191C/568217DB" Ref="T?"  Part="1"
+F 0 "T?" H 2300 5850 60  0000 C CNN
+F 1 "testpoint" H 2300 5650 60  0000 C CNN
+F 2 "" H 2300 5750 60  0000 C CNN
+F 3 "" H 2300 5750 60  0000 C CNN
+	1    2300 5750
+	-1   0    0    1
+$EndComp
+$Comp
+L testpoint T?
+U 1 1 5682DB05
+P 3000 6250
+F 0 "T?" H 3000 6350 60  0000 C CNN
+F 1 "testpoint" H 3000 6150 60  0000 C CNN
+F 2 "" H 3000 6250 60  0000 C CNN
+F 3 "" H 3000 6250 60  0000 C CNN
+	1    3000 6250
+	1    0    0    -1
+$EndComp
+Connection ~ 2700 6250
 $EndSCHEMATC
