File: hw/kicad/v3.4/cur.sch (KiCad schematic (older format))
At the start: 31 parts

Commit message: v3.4
Parts:
- removed U? (x4): LM358, symbol LM358
- added U? (x4): LM358, symbol LM358
Connections:
- net +15V: now also U?.8 (V+), U?.8 (V+), U?.8 (V+)
- net GNDPWR: now also U?.4 (V-), U?.4 (V-), U?.4 (V-), U?.5 (+), U?.6 (-)
- net at R?.1: now also R?.2, U?.6 (-); no longer R?.1
- net at R?.1: now also R?.1, U?.5 (+); no longer R?.2
- net at R?.1, R?.2: now also U?.7
- net at R?.1: now also R?.2, U?.2 (-); no longer R?.1 (x2)
- net at R?.1: now also R?.1, U?.3 (+); no longer R?.2 (x2)
- net at R?.1, R?.2: now also U?.1 (x2)
Other:
- moved on the sheet: R?
Changed lines of the file:
@@
 $EndDescr
-$Comp
-L LM358 U?
-U 1 1 56697CF0
-P 6050 2450
-F 0 "U?" H 6000 2650 60  0000 L CNN
-F 1 "LM358" H 6000 2200 60  0000 L CNN
-F 2 "" H 6050 2450 60  0000 C CNN
-F 3 "" H 6050 2450 60  0000 C CNN
-	1    6050 2450
-	1    0    0    -1
-$EndComp
-$Comp
-L LM358 U?
-U 1 1 56697D11
-P 2900 2450
-F 0 "U?" H 2850 2650 60  0000 L CNN
-F 1 "LM358" H 2850 2200 60  0000 L CNN
-F 2 "" H 2900 2450 60  0000 C CNN
-F 3 "" H 2900 2450 60  0000 C CNN
-	1    2900 2450
-	1    0    0    -1
-$EndComp
 $Comp
 L R R?
@@
 L R R?
 U 1 1 56690D3E
-P 5700 2150
-F 0 "R?" V 5780 2150 50  0000 C CNN
-F 1 "10k" V 5700 2150 50  0000 C CNN
-F 2 "" V 5630 2150 30  0000 C CNN
-F 3 "" H 5700 2150 30  0000 C CNN
-	1    5700 2150
-	0    1    1    0
-$EndComp
-Wire Wire Line
-	5550 2150 5500 2150
-Wire Wire Line
-	5500 2150 5500 2350
+P 5700 2750
+F 0 "R?" V 5780 2750 50  0000 C CNN
+F 1 "10k" V 5700 2750 50  0000 C CNN
+F 2 "" V 5630 2750 30  0000 C CNN
+F 3 "" H 5700 2750 30  0000 C CNN
+	1    5700 2750
+	0    1    1    0
+$EndComp
 Wire Wire Line
 	5450 2350 5550 2350
@@
 Wire Wire Line
 	6550 2450 6650 2450
-Wire Wire Line
-	6600 2150 6600 2450
 Connection ~ 6600 2450
 $Comp
@@
 	7050 2350 7050 2550
 Wire Wire Line
-	7050 2850 7050 2950
-Wire Wire Line
-	7050 2950 5950 2950
+	7050 2950 7050 2850
+Wire Wire Line
+	5950 2950 7050 2950
 Wire Wire Line
 	5950 2950 5950 2850
-Wire Wire Line
-	5450 2750 5500 2750
 Wire Wire Line
 	5500 2750 5500 2550
@@
 L +1V5 #PWR?
 U 1 1 56691046
-P 5050 2750
-F 0 "#PWR?" H 5050 2600 50  0001 C CNN
-F 1 "+1V5" H 5050 2890 50  0000 C CNN
-F 2 "" H 5050 2750 50  0000 C CNN
-F 3 "" H 5050 2750 50  0000 C CNN
-	1    5050 2750
+P 5050 2150
+F 0 "#PWR?" H 5050 2000 50  0001 C CNN
+F 1 "+1V5" H 5050 2290 50  0000 C CNN
+F 2 "" H 5050 2150 50  0000 C CNN
+F 3 "" H 5050 2150 50  0000 C CNN
+	1    5050 2150
 	0    -1   -1   0
 $EndComp
@@
 $EndComp
 Wire Wire Line
-	5950 2050 5950 1950
-Wire Wire Line
-	5850 2150 6600 2150
+	5950 1950 5950 2050
 $Comp
 L R R?
 U 1 1 5669140D
-P 5300 2750
-F 0 "R?" V 5380 2750 50  0000 C CNN
-F 1 "10k" V 5300 2750 50  0000 C CNN
-F 2 "" V 5230 2750 30  0000 C CNN
-F 3 "" H 5300 2750 30  0000 C CNN
-	1    5300 2750
-	0    1    1    0
-$EndComp
-Wire Wire Line
-	5050 2750 5150 2750
+P 5300 2150
+F 0 "R?" V 5380 2150 50  0000 C CNN
+F 1 "10k" V 5300 2150 50  0000 C CNN
+F 2 "" V 5230 2150 30  0000 C CNN
+F 3 "" H 5300 2150 30  0000 C CNN
+	1    5300 2150
+	0    1    1    0
+$EndComp
 $Comp
 L C C?
@@
 L R R?
 U 1 1 56691AA6
-P 8900 2300
-F 0 "R?" V 8980 2300 50  0000 C CNN
-F 1 "10k" V 8900 2300 50  0000 C CNN
-F 2 "" V 8830 2300 30  0000 C CNN
-F 3 "" H 8900 2300 30  0000 C CNN
-	1    8900 2300
-	0    1    1    0
-$EndComp
-Wire Wire Line
-	8750 2300 8700 2300
+P 8900 2900
+F 0 "R?" V 8980 2900 50  0000 C CNN
+F 1 "10k" V 8900 2900 50  0000 C CNN
+F 2 "" V 8830 2900 30  0000 C CNN
+F 3 "" H 8900 2900 30  0000 C CNN
+	1    8900 2900
+	0    1    1    0
+$EndComp
 Wire Wire Line
 	8700 2300 8700 2500
@@
 Wire Wire Line
 	9750 2600 9850 2600
-Wire Wire Line
-	9800 2300 9800 2600
 Connection ~ 9800 2600
 $Comp
@@
 	10250 2500 10250 2700
 Wire Wire Line
-	10250 3000 10250 3100
-Wire Wire Line
-	10250 3100 9150 3100
+	10250 3100 10250 3000
+Wire Wire Line
+	9150 3100 10250 3100
 Wire Wire Line
 	9150 3100 9150 3000
-Wire Wire Line
-	8650 2900 8700 2900
 Wire Wire Line
 	8700 2900 8700 2700
@@
 L +1V5 #PWR?
 U 1 1 56691AC8
-P 8250 2900
-F 0 "#PWR?" H 8250 2750 50  0001 C CNN
-F 1 "+1V5" H 8250 3040 50  0000 C CNN
-F 2 "" H 8250 2900 50  0000 C CNN
-F 3 "" H 8250 2900 50  0000 C CNN
-	1    8250 2900
+P 8250 2300
+F 0 "#PWR?" H 8250 2150 50  0001 C CNN
+F 1 "+1V5" H 8250 2440 50  0000 C CNN
+F 2 "" H 8250 2300 50  0000 C CNN
+F 3 "" H 8250 2300 50  0000 C CNN
+	1    8250 2300
 	0    -1   -1   0
 $EndComp
@@
 $EndComp
 Wire Wire Line
-	9150 2200 9150 2100
-Wire Wire Line
-	9050 2300 9800 2300
+	9150 2100 9150 2200
 $Comp
 L R R?
 U 1 1 56691ADD
-P 8500 2900
-F 0 "R?" V 8580 2900 50  0000 C CNN
-F 1 "10k" V 8500 2900 50  0000 C CNN
-F 2 "" V 8430 2900 30  0000 C CNN
-F 3 "" H 8500 2900 30  0000 C CNN
-	1    8500 2900
-	0    1    1    0
-$EndComp
-Wire Wire Line
-	8250 2900 8350 2900
+P 8500 2300
+F 0 "R?" V 8580 2300 50  0000 C CNN
+F 1 "10k" V 8500 2300 50  0000 C CNN
+F 2 "" V 8430 2300 30  0000 C CNN
+F 3 "" H 8500 2300 30  0000 C CNN
+	1    8500 2300
+	0    1    1    0
+$EndComp
 $Comp
 L C C?
@@
 L R R?
 U 1 1 56691D2C
-P 2550 2150
-F 0 "R?" V 2630 2150 50  0000 C CNN
-F 1 "10k" V 2550 2150 50  0000 C CNN
-F 2 "" V 2480 2150 30  0000 C CNN
-F 3 "" H 2550 2150 30  0000 C CNN
-	1    2550 2150
-	0    1    1    0
-$EndComp
-Wire Wire Line
-	2400 2150 2350 2150
+P 2550 2750
+F 0 "R?" V 2630 2750 50  0000 C CNN
+F 1 "10k" V 2550 2750 50  0000 C CNN
+F 2 "" V 2480 2750 30  0000 C CNN
+F 3 "" H 2550 2750 30  0000 C CNN
+	1    2550 2750
+	0    1    1    0
+$EndComp
 Wire Wire Line
 	2350 2150 2350 2350
@@
 Wire Wire Line
 	3400 2450 3500 2450
-Wire Wire Line
-	3450 2150 3450 2450
 Connection ~ 3450 2450
 $Comp
@@
 	2800 2850 2800 3050
 Wire Wire Line
-	2300 2750 2350 2750
-Wire Wire Line
 	2350 2750 2350 2550
 Connection ~ 2350 2550
@@
 L +1V5 #PWR?
 U 1 1 56691D4E
-P 1900 2750
-F 0 "#PWR?" H 1900 2600 50  0001 C CNN
-F 1 "+1V5" H 1900 2890 50  0000 C CNN
-F 2 "" H 1900 2750 50  0000 C CNN
-F 3 "" H 1900 2750 50  0000 C CNN
-	1    1900 2750
+P 1900 2150
+F 0 "#PWR?" H 1900 2000 50  0001 C CNN
+F 1 "+1V5" H 1900 2290 50  0000 C CNN
+F 2 "" H 1900 2150 50  0000 C CNN
+F 3 "" H 1900 2150 50  0000 C CNN
+	1    1900 2150
 	0    -1   -1   0
 $EndComp
@@
 Wire Wire Line
 	2800 2050 2800 1950
-Wire Wire Line
-	2700 2150 3450 2150
 $Comp
 L R R?
 U 1 1 56691D63
-P 2150 2750
-F 0 "R?" V 2230 2750 50  0000 C CNN
-F 1 "10k" V 2150 2750 50  0000 C CNN
-F 2 "" V 2080 2750 30  0000 C CNN
-F 3 "" H 2150 2750 30  0000 C CNN
-	1    2150 2750
+P 2150 2150
+F 0 "R?" V 2230 2150 50  0000 C CNN
+F 1 "10k" V 2150 2150 50  0000 C CNN
+F 2 "" V 2080 2150 30  0000 C CNN
+F 3 "" H 2150 2150 30  0000 C CNN
+	1    2150 2150
 	0    1    1    0
 $EndComp
@@
 Wire Wire Line
 	1900 2550 2000 2550
-$Comp
-L LM358 U?
-U 1 1 5669211F
-P 9250 2600
-F 0 "U?" H 9200 2800 60  0000 L CNN
-F 1 "LM358" H 9200 2350 60  0000 L CNN
-F 2 "" H 9250 2600 60  0000 C CNN
-F 3 "" H 9250 2600 60  0000 C CNN
-	1    9250 2600
-	1    0    0    -1
-$EndComp
-$Comp
-L LM358 U?
-U 1 1 566922D2
-P 9250 1300
-F 0 "U?" H 9200 1500 60  0000 L CNN
-F 1 "LM358" H 9200 1050 60  0000 L CNN
-F 2 "" H 9250 1300 60  0000 C CNN
-F 3 "" H 9250 1300 60  0000 C CNN
-	1    9250 1300
-	1    0    0    -1
-$EndComp
 $Comp
 L GNDPWR #PWR?
@@
 	8750 1400 8650 1400
 Connection ~ 8650 1400
-Wire Wire Line
-	1900 2750 2000 2750
 $Comp
 L R R?
@@
 	4300 1900 4300 2100
 Wire Wire Line
-	4300 1600 4300 1400
+	4300 1400 4300 1600
 Wire Wire Line
 	4300 1100 4300 1000
@@
 	0    -1   -1   0
 $EndComp
+Wire Wire Line
+	2350 2750 2400 2750
+Wire Wire Line
+	2700 2750 3450 2750
+Wire Wire Line
+	3450 2750 3450 2450
+Wire Wire Line
+	2300 2150 2350 2150
+Wire Wire Line
+	1900 2150 2000 2150
+Wire Wire Line
+	5500 2750 5550 2750
+Wire Wire Line
+	6600 2750 5850 2750
+Wire Wire Line
+	6600 2750 6600 2450
+Wire Wire Line
+	5450 2150 5500 2150
+Wire Wire Line
+	5500 2150 5500 2350
+Wire Wire Line
+	5050 2150 5150 2150
+Wire Wire Line
+	8250 2300 8350 2300
+Wire Wire Line
+	8700 2900 8750 2900
+Wire Wire Line
+	9050 2900 9800 2900
+Wire Wire Line
+	9800 2900 9800 2600
+Wire Wire Line
+	8650 2300 8700 2300
+$Comp
+L LM358 U?
+U 1 1 56BF1407
+P 2900 2450
+F 0 "U?" H 3441 2503 60  0000 L CNN
+F 1 "LM358" H 3441 2397 60  0000 L CNN
+F 2 "" H 2900 2450 60  0000 C CNN
+F 3 "" H 2900 2450 60  0000 C CNN
+	1    2900 2450
+	1    0    0    -1
+$EndComp
+$Comp
+L LM358 U?
+U 2 1 56BF1487
+P 6050 2450
+F 0 "U?" H 6591 2503 60  0000 L CNN
+F 1 "LM358" H 6591 2397 60  0000 L CNN
+F 2 "" H 6050 2450 60  0000 C CNN
+F 3 "" H 6050 2450 60  0000 C CNN
+	2    6050 2450
+	1    0    0    -1
+$EndComp
+$Comp
+L LM358 U?
+U 1 1 56BF16F2
+P 9250 2600
+F 0 "U?" H 9791 2653 60  0000 L CNN
+F 1 "LM358" H 9791 2547 60  0000 L CNN
+F 2 "" H 9250 2600 60  0000 C CNN
+F 3 "" H 9250 2600 60  0000 C CNN
+	1    9250 2600
+	1    0    0    -1
+$EndComp
+$Comp
+L LM358 U?
+U 2 1 56BF176D
+P 9250 1300
+F 0 "U?" H 9791 1353 60  0000 L CNN
+F 1 "LM358" H 9791 1247 60  0000 L CNN
+F 2 "" H 9250 1300 60  0000 C CNN
+F 3 "" H 9250 1300 60  0000 C CNN
+	2    9250 1300
+	1    0    0    -1
+$EndComp
 $EndSCHEMATC
