File: hw/kicad/v3.4/hv.sch (KiCad schematic (older format))
At the start: 7 parts

Commit message: hw v3.4
Parts:
- added P?: CONN_01X02, symbol CONN_01X02
- added R?: 1k, symbol R
- added R?: 10k, symbol R
Connections:
- net +3.3VP: now also R?.1
- net GNDPWR: now also P?.1 (P1)
- net f1/A_T_MOT: now also R?.1
- new net: P?.2 (P2), R?.2, R?.2
Changed lines of the file:
@@
 EESchema Schematic File Version 2
 LIBS:conn
+LIBS:power
 LIBS:stmbl_3.4-cache
 EELAYER 25 0
@@
 Wire Wire Line
 	5150 3500 4150 3500
+$Comp
+L CONN_01X02 P?
+U 1 1 568233C2
+P 2700 3150
+F 0 "P?" H 2700 3300 50  0000 C CNN
+F 1 "CONN_01X02" V 2800 3150 50  0000 C CNN
+F 2 "" H 2700 3150 50  0000 C CNN
+F 3 "" H 2700 3150 50  0000 C CNN
+	1    2700 3150
+	-1   0    0    1
+$EndComp
+$Comp
+L R R?
+U 1 1 5682376B
+P 3000 2850
+F 0 "R?" V 3080 2850 50  0000 C CNN
+F 1 "1k" V 3000 2850 50  0000 C CNN
+F 2 "" V 2930 2850 30  0000 C CNN
+F 3 "" H 3000 2850 30  0000 C CNN
+	1    3000 2850
+	1    0    0    -1
+$EndComp
+$Comp
+L R R?
+U 1 1 568238FC
+P 3250 3100
+F 0 "R?" V 3330 3100 50  0000 C CNN
+F 1 "10k" V 3250 3100 50  0000 C CNN
+F 2 "" V 3180 3100 30  0000 C CNN
+F 3 "" H 3250 3100 30  0000 C CNN
+	1    3250 3100
+	0    1    1    0
+$EndComp
+$Comp
+L GNDPWR #PWR?
+U 1 1 56823A9D
+P 3000 3300
+F 0 "#PWR?" H 3000 3100 50  0001 C CNN
+F 1 "GNDPWR" H 3000 3170 50  0000 C CNN
+F 2 "" H 3000 3250 60  0000 C CNN
+F 3 "" H 3000 3250 60  0000 C CNN
+	1    3000 3300
+	1    0    0    -1
+$EndComp
+Wire Wire Line
+	2900 3100 3100 3100
+Wire Wire Line
+	3000 3000 3000 3100
+Connection ~ 3000 3100
+Wire Wire Line
+	2900 3200 3000 3200
+Wire Wire Line
+	3000 3200 3000 3300
+$Comp
+L +3.3VP #PWR?
+U 1 1 56824435
+P 3000 2600
+F 0 "#PWR?" H 3150 2550 50  0001 C CNN
+F 1 "+3.3VP" H 3000 2700 50  0000 C CNN
+F 2 "" H 3000 2600 60  0000 C CNN
+F 3 "" H 3000 2600 60  0000 C CNN
+	1    3000 2600
+	1    0    0    -1
+$EndComp
+Wire Wire Line
+	3000 2700 3000 2600
+Wire Wire Line
+	3400 3100 5050 3100
+Wire Wire Line
+	5050 3100 5050 2200
+Wire Wire Line
+	5050 2200 6000 2200
 $EndSCHEMATC

Commit message: hw v3.4 +testpoints
Parts:
- added T? (x4): testpoint, symbol testpoint
Connections:
- net f1/A_T_MOT: now also T?.1
- net f1/BKIN: now also T?.1
- net f1/HV_RX: now also T?.1
- net f1/HV_TX: now also T?.1
Changed lines of the file:
@@
 EESchema Schematic File Version 2
-LIBS:conn
 LIBS:power
 LIBS:stmbl_3.4-cache
@@
 F8 "HV_TX" I L 6000 2000 60
 F9 "HV_RX" I L 6000 1900 60
-F10 "A_15V" I L 6000 2300 60
-F11 "A_HV" I L 6000 2750 60
-F12 "A_U" I L 6000 3100 60
-F13 "A_V" I L 6000 3000 60
-F14 "A_W" I L 6000 2900 60
-F15 "A_T_HV" I R 7000 2900 60
-F16 "A_T_MOT" I L 6000 2200 60
-F17 "HV_EN" I R 7000 2600 60
-F18 "HV_FLT" I R 7000 2700 60
-F19 "BKIN" I L 6000 2100 60
-F20 "A_IU" I L 6000 2400 60
-F21 "A_IV" I L 6000 2500 60
-F22 "A_IW" I L 6000 2600 60
+F10 "A_HV" I L 6000 2750 60
+F11 "A_U" I L 6000 3100 60
+F12 "A_V" I L 6000 3000 60
+F13 "A_W" I L 6000 2900 60
+F14 "A_T_HV" I R 7000 2900 60
+F15 "A_T_MOT" I L 6000 2200 60
+F16 "HV_EN" I R 7000 2600 60
+F17 "HV_FLT" I R 7000 2700 60
+F18 "BKIN" I L 6000 2100 60
+F19 "A_IU" I L 6000 2400 60
+F20 "A_IV" I L 6000 2500 60
+F21 "A_IW" I L 6000 2600 60
 $EndSheet
 $Sheet
@@
 F0 "viper" 60
 F1 "viper.sch" 60
-F2 "A_15V" I R 4150 3500 60
 $EndSheet
 $Sheet
@@
 Connection ~ 5400 1800
 Wire Wire Line
-	5400 1300 5750 1300
+	5400 1300 5850 1300
 Wire Wire Line
 	5750 1200 5750 2100
@@
 	5750 2100 6000 2100
 Connection ~ 5750 1300
-Wire Wire Line
-	5150 2300 6000 2300
 $Sheet
 S 8450 3350 750  600
@@
 Wire Wire Line
 	7000 3850 7100 3850
-Wire Wire Line
-	5150 2300 5150 3500
-Wire Wire Line
-	5150 3500 4150 3500
 $Comp
 L CONN_01X02 P?
@@
 Wire Wire Line
 	5050 2200 6000 2200
+$Comp
+L testpoint T?
+U 1 1 568248AF
+P 4050 2850
+F 0 "T?" H 4050 2950 60  0000 C CNN
+F 1 "testpoint" H 4050 2750 60  0000 C CNN
+F 2 "" H 4050 2850 60  0000 C CNN
+F 3 "" H 4050 2850 60  0000 C CNN
+	1    4050 2850
+	0    -1   -1   0
+$EndComp
+Wire Wire Line
+	4050 3050 4050 3100
+Connection ~ 4050 3100
+$Comp
+L testpoint T?
+U 1 1 56828AEB
+P 6050 1300
+F 0 "T?" H 6050 1400 60  0000 C CNN
+F 1 "testpoint" H 6050 1200 60  0000 C CNN
+F 2 "" H 6050 1300 60  0000 C CNN
+F 3 "" H 6050 1300 60  0000 C CNN
+	1    6050 1300
+	1    0    0    -1
+$EndComp
+$Comp
+L testpoint T?
+U 1 1 56829511
+P 5700 1800
+F 0 "T?" H 5700 1900 60  0000 C CNN
+F 1 "testpoint" H 5700 1700 60  0000 C CNN
+F 2 "" H 5700 1800 60  0000 C CNN
+F 3 "" H 5700 1800 60  0000 C CNN
+	1    5700 1800
+	1    0    0    -1
+$EndComp
+$Comp
+L testpoint T?
+U 1 1 568296AA
+P 5700 2100
+F 0 "T?" H 5700 2200 60  0000 C CNN
+F 1 "testpoint" H 5700 2000 60  0000 C CNN
+F 2 "" H 5700 2100 60  0000 C CNN
+F 3 "" H 5700 2100 60  0000 C CNN
+	1    5700 2100
+	1    0    0    -1
+$EndComp
+Connection ~ 5500 2100
+Connection ~ 5500 1800
 $EndSCHEMATC
