File: hw/kicad/v3.4/hv_drive.sch (KiCad schematic (older format))
At the start: 12 parts

Commit message: +iram256
Parts:
- removed C?: CP, symbol CP
- removed C? (x2): 4.7µ, symbol C
- removed IC?: iramxb, symbol iramxb
- added C? (x3): 100n, symbol C
- added C? (x3): 2.2µ, symbol C
- added R? (x3): 0.002, symbol R
- added U?: IRAM256a, symbol IRAM256a
- C?: value 4.7µ -> 2.2µ
Connections:
- net labels added: CUH, CUL, CVH, CVL, CWH, CWL
- net labels removed: V-
- wire segments 28 -> 34
Other:
- moved on the sheet: C?

Commit message: +f1 3.3V, viper fix
Parts:
- removed X?: akl230-03, symbol akl230-03
- added P?: CONN_01X03, symbol CONN_01X03
- added P?: CONN_01X02, symbol CONN_01X02
Connections:
- net labels added: VPP
- net labels removed: V+
- wire segments 34 -> 64
Changed lines of the file:
@@
 Connection ~ 4550 4550
 Connection ~ 4250 4550
-Wire Wire Line
-	3800 4250 5850 4250
 Connection ~ 4250 4250
 Connection ~ 4550 4250
@@
 	5850 3050 5750 3050
 Wire Wire Line
-	5350 3150 5850 3150
-Wire Wire Line
-	5450 2850 5450 3150
+	5350 3150 5450 3150
+Wire Wire Line
+	5450 3150 5850 3150
+Wire Wire Line
+	5450 2850 5450 3050
+Wire Wire Line
+	5450 3050 5450 3150
 Text HLabel 5350 3150 0    60   Input ~ 0
 W
@@
 Text HLabel 5350 3950 0    60   Input ~ 0
 U
-Text HLabel 3800 4250 0    60   Input ~ 0
-V+
 Connection ~ 3950 4250
 Connection ~ 5450 3150
-$Comp
-L akl230-03 X?
-U 1 1 5669783C
-P 5450 2000
-F 0 "X?" H 5500 2200 60  0000 C CNN
-F 1 "akl230-03" H 5600 1800 60  0000 C CNN
-F 2 "" H 5450 1900 60  0000 C CNN
-F 3 "" H 5450 1900 60  0000 C CNN
-	1    5450 2000
-	1    0    0    -1
-$EndComp
 Text HLabel 5150 1900 0    60   Input ~ 0
 U
@@
 	5850 3450 5750 3450
 Wire Wire Line
-	5350 3550 5850 3550
-Wire Wire Line
-	5450 3250 5450 3550
+	5350 3550 5450 3550
+Wire Wire Line
+	5450 3550 5850 3550
+Wire Wire Line
+	5450 3250 5450 3450
+Wire Wire Line
+	5450 3450 5450 3550
 Connection ~ 5450 3550
 $Comp
@@
 	5850 3850 5750 3850
 Wire Wire Line
-	5350 3950 5850 3950
-Wire Wire Line
-	5450 3650 5450 3950
+	5350 3950 5450 3950
+Wire Wire Line
+	5450 3950 5850 3950
+Wire Wire Line
+	5450 3650 5450 3850
+Wire Wire Line
+	5450 3850 5450 3950
 Connection ~ 5450 3950
 $Comp
@@
 $EndComp
 Wire Wire Line
-	5550 4950 5850 4950
-Wire Wire Line
-	5550 4750 5850 4750
-Wire Wire Line
-	5550 4550 5850 4550
-Wire Wire Line
-	5000 4950 5250 4950
-Wire Wire Line
-	5150 4550 5150 4950
-Wire Wire Line
-	5000 4750 5250 4750
+	5550 4950 5700 4950
+Wire Wire Line
+	5700 4950 5850 4950
+Wire Wire Line
+	5550 4750 5700 4750
+Wire Wire Line
+	5700 4750 5850 4750
+Wire Wire Line
+	5550 4550 5700 4550
+Wire Wire Line
+	5700 4550 5850 4550
+Wire Wire Line
+	5000 4950 5150 4950
+Wire Wire Line
+	5150 4950 5250 4950
+Wire Wire Line
+	5150 4550 5150 4750
+Wire Wire Line
+	5150 4750 5150 4850
+Wire Wire Line
+	5150 4850 5150 4950
+Wire Wire Line
+	5000 4750 5150 4750
+Wire Wire Line
+	5150 4750 5250 4750
 Connection ~ 5150 4750
 Wire Wire Line
-	3850 4550 5250 4550
+	3850 4550 3950 4550
+Wire Wire Line
+	3950 4550 4250 4550
+Wire Wire Line
+	4250 4550 4550 4550
+Wire Wire Line
+	4550 4550 4850 4550
+Wire Wire Line
+	4850 4550 5150 4550
+Wire Wire Line
+	5150 4550 5250 4550
 Text HLabel 5000 4750 0    60   Input ~ 0
 CUL
@@
 Connection ~ 3950 4550
 Wire Wire Line
-	7050 5050 7800 5050
+	7050 5050 7550 5050
+Wire Wire Line
+	7550 5050 7800 5050
 Wire Wire Line
 	7050 4850 7400 4850
@@
 	7400 4850 7400 4750
 Wire Wire Line
-	7400 4750 7800 4750
+	7400 4750 7550 4750
+Wire Wire Line
+	7550 4750 7800 4750
 Wire Wire Line
 	7550 4750 7550 4650
@@
 Connection ~ 7550 5050
 Connection ~ 7550 4750
+$Comp
+L CONN_01X03 P?
+U 1 1 566CEA04
+P 5450 2000
+F 0 "P?" H 5450 2200 50  0000 C CNN
+F 1 "CONN_01X03" V 5550 2000 50  0000 C CNN
+F 2 "" H 5450 2000 60  0000 C CNN
+F 3 "" H 5450 2000 60  0000 C CNN
+	1    5450 2000
+	1    0    0    -1
+$EndComp
+$Comp
+L CONN_01X02 P?
+U 1 1 566CF01F
+P 3900 1950
+F 0 "P?" H 3900 2100 50  0000 C CNN
+F 1 "CONN_01X02" V 4000 1950 50  0000 C CNN
+F 2 "" H 3900 1950 60  0000 C CNN
+F 3 "" H 3900 1950 60  0000 C CNN
+	1    3900 1950
+	-1   0    0    1
+$EndComp
+$Comp
+L GNDPWR #PWR?
+U 1 1 566CF13E
+P 4200 2100
+F 0 "#PWR?" H 4200 1900 50  0001 C CNN
+F 1 "GNDPWR" H 4200 1970 50  0000 C CNN
+F 2 "" H 4200 2050 60  0000 C CNN
+F 3 "" H 4200 2050 60  0000 C CNN
+	1    4200 2100
+	1    0    0    -1
+$EndComp
+$Comp
+L VPP #PWR?
+U 1 1 566CF184
+P 4200 1800
+F 0 "#PWR?" H 4200 1650 50  0001 C CNN
+F 1 "VPP" H 4200 1950 50  0000 C CNN
+F 2 "" H 4200 1800 60  0000 C CNN
+F 3 "" H 4200 1800 60  0000 C CNN
+	1    4200 1800
+	1    0    0    -1
+$EndComp
+Wire Wire Line
+	4100 2000 4200 2000
+Wire Wire Line
+	4200 2000 4200 2100
+Wire Wire Line
+	4100 1900 4200 1900
+Wire Wire Line
+	4200 1900 4200 1800
+Wire Wire Line
+	3850 4250 3950 4250
+Wire Wire Line
+	3950 4250 4250 4250
+Wire Wire Line
+	4250 4250 4550 4250
+Wire Wire Line
+	4550 4250 4850 4250
+Wire Wire Line
+	4850 4250 5150 4250
+Wire Wire Line
+	5150 4250 5850 4250
+$Comp
+L VPP #PWR?
+U 1 1 566CF322
+P 3850 4150
+F 0 "#PWR?" H 3850 4000 50  0001 C CNN
+F 1 "VPP" H 3850 4300 50  0000 C CNN
+F 2 "" H 3850 4150 60  0000 C CNN
+F 3 "" H 3850 4150 60  0000 C CNN
+	1    3850 4150
+	1    0    0    -1
+$EndComp
+Wire Wire Line
+	3850 4250 3850 4150
 $EndSCHEMATC

Commit message: hw v3.4
Parts:
- removed C? (x4): 100n, symbol C
- added R?: 10k, symbol R
- C?: value C -> 470n
Connections:
- net HU: now also U?.20 (HINU)
- net HV: now also U?.22 (HINV)
- net HW: now also U?.23 (HINW)
- net LU: now also U?.24 (LINU)
- net LV: now also U?.25 (LINV)
- net LW: now also U?.26 (LINW)
- net Vth: now also U?.27 (VTH), R?.2
- net en: now also U?.18 (!FLT/EN)
- net itirp: now also U?.16 (ITrip)
- new net +3.3VP: R?.1
Changed lines of the file:
@@
 EESchema Schematic File Version 2
 LIBS:conn
+LIBS:power
 LIBS:stmbl_3.4-cache
 EELAYER 25 0
@@
 P 5150 4400
 F 0 "C?" H 5175 4500 50  0000 L CNN
-F 1 "C" H 5175 4300 50  0000 L CNN
+F 1 "470n" H 5175 4300 50  0000 L CNN
 F 2 "" H 5188 4250 30  0000 C CNN
 F 3 "" H 5150 4400 60  0000 C CNN
@@
 	5850 3050 5750 3050
 Wire Wire Line
-	5350 3150 5450 3150
-Wire Wire Line
-	5450 3150 5850 3150
-Wire Wire Line
-	5450 2850 5450 3050
-Wire Wire Line
-	5450 3050 5450 3150
+	5350 3150 5850 3150
 Text HLabel 5350 3150 0    60   Input ~ 0
 W
@@
 $EndComp
 $Comp
-L C C?
-U 1 1 56697FB6
-P 7550 4900
-F 0 "C?" H 7575 5000 50  0000 L CNN
-F 1 "100n" H 7575 4800 50  0000 L CNN
-F 2 "" H 7588 4750 30  0000 C CNN
-F 3 "" H 7550 4900 60  0000 C CNN
-	1    7550 4900
-	1    0    0    -1
-$EndComp
-$Comp
 L IRAM256a U?
 U 1 1 5668DD3B
@@
 $Comp
 L C C?
-U 1 1 5668DF00
-P 5600 2850
-F 0 "C?" H 5625 2950 50  0000 L CNN
-F 1 "100n" H 5625 2750 50  0000 L CNN
-F 2 "" H 5638 2700 30  0000 C CNN
-F 3 "" H 5600 2850 60  0000 C CNN
-	1    5600 2850
-	0    -1   -1   0
-$EndComp
-Wire Wire Line
-	5750 3050 5750 2850
-Connection ~ 5450 3050
-Connection ~ 5750 3050
-$Comp
-L C C?
 U 1 1 5668E03D
 P 5600 3450
@@
 	5850 3450 5750 3450
 Wire Wire Line
-	5350 3550 5450 3550
-Wire Wire Line
-	5450 3550 5850 3550
-Wire Wire Line
-	5450 3250 5450 3450
+	5350 3550 5850 3550
 Wire Wire Line
 	5450 3450 5450 3550
 Connection ~ 5450 3550
-$Comp
-L C C?
-U 1 1 5668E047
-P 5600 3250
-F 0 "C?" H 5625 3350 50  0000 L CNN
-F 1 "100n" H 5625 3150 50  0000 L CNN
-F 2 "" H 5638 3100 30  0000 C CNN
-F 3 "" H 5600 3250 60  0000 C CNN
-	1    5600 3250
-	0    -1   -1   0
-$EndComp
-Wire Wire Line
-	5750 3450 5750 3250
-Connection ~ 5450 3450
-Connection ~ 5750 3450
 $Comp
 L C C?
@@
 	5850 3850 5750 3850
 Wire Wire Line
-	5350 3950 5450 3950
-Wire Wire Line
-	5450 3950 5850 3950
-Wire Wire Line
-	5450 3650 5450 3850
+	5350 3950 5850 3950
 Wire Wire Line
 	5450 3850 5450 3950
 Connection ~ 5450 3950
-$Comp
-L C C?
-U 1 1 5668E1B6
-P 5600 3650
-F 0 "C?" H 5625 3750 50  0000 L CNN
-F 1 "100n" H 5625 3550 50  0000 L CNN
-F 2 "" H 5638 3500 30  0000 C CNN
-F 3 "" H 5600 3650 60  0000 C CNN
-	1    5600 3650
-	0    -1   -1   0
-$EndComp
-Wire Wire Line
-	5750 3850 5750 3650
-Connection ~ 5450 3850
-Connection ~ 5750 3850
 $Comp
 L R R?
@@
 $EndComp
 Wire Wire Line
-	5550 4950 5700 4950
-Wire Wire Line
-	5700 4950 5850 4950
-Wire Wire Line
-	5550 4750 5700 4750
-Wire Wire Line
-	5700 4750 5850 4750
-Wire Wire Line
-	5550 4550 5700 4550
-Wire Wire Line
-	5700 4550 5850 4550
-Wire Wire Line
-	5000 4950 5150 4950
-Wire Wire Line
-	5150 4950 5250 4950
-Wire Wire Line
-	5150 4550 5150 4750
-Wire Wire Line
-	5150 4750 5150 4850
-Wire Wire Line
-	5150 4850 5150 4950
-Wire Wire Line
-	5000 4750 5150 4750
-Wire Wire Line
-	5150 4750 5250 4750
+	5550 4950 5850 4950
+Wire Wire Line
+	5550 4750 5850 4750
+Wire Wire Line
+	5550 4550 5850 4550
+Wire Wire Line
+	5000 4950 5250 4950
+Wire Wire Line
+	5150 4550 5150 4950
+Wire Wire Line
+	5000 4750 5250 4750
 Connection ~ 5150 4750
 Wire Wire Line
-	3850 4550 3950 4550
-Wire Wire Line
-	3950 4550 4250 4550
-Wire Wire Line
-	4250 4550 4550 4550
-Wire Wire Line
-	4550 4550 4850 4550
-Wire Wire Line
-	4850 4550 5150 4550
-Wire Wire Line
-	5150 4550 5250 4550
+	3850 4550 5250 4550
 Text HLabel 5000 4750 0    60   Input ~ 0
 CUL
@@
 Connection ~ 3950 4550
 Wire Wire Line
-	7050 5050 7550 5050
-Wire Wire Line
-	7550 5050 7800 5050
+	7050 5050 7800 5050
 Wire Wire Line
 	7050 4850 7400 4850
@@
 	7400 4850 7400 4750
 Wire Wire Line
-	7400 4750 7550 4750
-Wire Wire Line
-	7550 4750 7800 4750
+	7400 4750 7800 4750
 Wire Wire Line
 	7550 4750 7550 4650
@@
 	4200 1900 4200 1800
 Wire Wire Line
-	3850 4250 3950 4250
-Wire Wire Line
-	3950 4250 4250 4250
-Wire Wire Line
-	4250 4250 4550 4250
-Wire Wire Line
-	4550 4250 4850 4250
-Wire Wire Line
-	4850 4250 5150 4250
-Wire Wire Line
-	5150 4250 5850 4250
+	3850 4250 5850 4250
 $Comp
 L VPP #PWR?
@@
 Wire Wire Line
 	3850 4250 3850 4150
+Wire Wire Line
+	7050 3050 7150 3050
+Wire Wire Line
+	7050 3250 7150 3250
+Wire Wire Line
+	7050 3450 7150 3450
+Wire Wire Line
+	7050 3650 7150 3650
+Wire Wire Line
+	7050 3850 7150 3850
+Wire Wire Line
+	7050 4050 7150 4050
+Wire Wire Line
+	7050 4250 7150 4250
+Wire Wire Line
+	7050 4450 7150 4450
+Wire Wire Line
+	7050 4650 7150 4650
+$Comp
+L +3.3VP #PWR?
+U 1 1 566DE47B
+P 7800 4050
+F 0 "#PWR?" H 7950 4000 50  0001 C CNN
+F 1 "+3.3VP" H 7800 4150 50  0000 C CNN
+F 2 "" H 7800 4050 60  0000 C CNN
+F 3 "" H 7800 4050 60  0000 C CNN
+	1    7800 4050
+	1    0    0    -1
+$EndComp
+$Comp
+L R R?
+U 1 1 566DE4EC
+P 7800 4300
+F 0 "R?" V 7880 4300 50  0000 C CNN
+F 1 "10k" V 7800 4300 50  0000 C CNN
+F 2 "" V 7730 4300 30  0000 C CNN
+F 3 "" H 7800 4300 30  0000 C CNN
+	1    7800 4300
+	1    0    0    -1
+$EndComp
+Text HLabel 7900 4550 2    60   Input ~ 0
+Vth
+Wire Wire Line
+	7800 4050 7800 4150
+Wire Wire Line
+	7800 4450 7800 4550
+Wire Wire Line
+	7800 4550 7900 4550
+Wire Wire Line
+	5450 3050 5450 3150
 $EndSCHEMATC
