File: hw/kicad/v3.4/lmr.sch (KiCad schematic (older format))
At the start: 16 parts

Commit message: +f1 3.3V, viper fix
Parts:
- removed X?: akl230-02, symbol akl230-02
- added P?: CONN_01X02, symbol CONN_01X02
Changed lines of the file:
@@
 $Descr A4 11693 8268
 encoding utf-8
-Sheet 8 15
+Sheet 9 15
 Title ""
 Date ""
@@
 $EndComp
 $Comp
-L akl230-02 X?
-U 1 1 566022A6
-P 2200 2350
-F 0 "X?" H 2250 2500 60  0000 C CNN
-F 1 "akl230-02" H 2300 2200 60  0000 C CNN
-F 2 "" H 2200 2200 60  0000 C CNN
-F 3 "" H 2200 2200 60  0000 C CNN
-	1    2200 2350
-	-1   0    0    1
-$EndComp
-$Comp
 L C C?
 U 1 1 56606890
@@
 	6300 4000 6300 4100
 Connection ~ 6300 4100
+$Comp
+L CONN_01X02 P?
+U 1 1 566CDEAC
+P 2200 2350
+F 0 "P?" H 2200 2500 50  0000 C CNN
+F 1 "CONN_01X02" V 2300 2350 50  0000 C CNN
+F 2 "" H 2200 2350 60  0000 C CNN
+F 3 "" H 2200 2350 60  0000 C CNN
+	1    2200 2350
+	-1   0    0    1
+$EndComp
 $EndSCHEMATC

Commit message: hw v3.4
Parts:
- C? (x2): value 2.2µ 30V -> 2.2µ; Voltage (none) -> 30V
- C?: value 47µ 6.3V -> 47µ; Voltage (none) -> 6.3V
- C? (x3): value 4.7µ 16V -> 4.7µ; Voltage (none) -> 16V
Changed lines of the file:
@@
 EESchema Schematic File Version 2
 LIBS:conn
+LIBS:power
 LIBS:stmbl_3.4-cache
 EELAYER 25 0
@@
 P 3350 3850
 F 0 "C?" H 3375 3950 50  0000 L CNN
-F 1 "2.2µ 30V" H 3375 3750 50  0000 L CNN
+F 1 "2.2µ" H 3375 3750 50  0000 L CNN
 F 2 "" H 3388 3700 30  0000 C CNN
 F 3 "" H 3350 3850 60  0000 C CNN
+F 4 "30V" H 3350 3850 60  0001 C CNN "Voltage"
 	1    3350 3850
 	1    0    0    -1
@@
 P 5800 3850
 F 0 "C?" H 5825 3950 50  0000 L CNN
-F 1 "47µ 6.3V" H 5825 3750 50  0000 L CNN
+F 1 "47µ" H 5825 3750 50  0000 L CNN
 F 2 "" H 5838 3700 30  0000 C CNN
 F 3 "" H 5800 3850 60  0000 C CNN
+F 4 "6.3V" H 5800 3850 60  0001 C CNN "Voltage"
 	1    5800 3850
 	1    0    0    -1
@@
 P 7550 3850
 F 0 "C?" H 7575 3950 50  0000 L CNN
-F 1 "4.7µ 16V" H 7575 3750 50  0000 L CNN
+F 1 "4.7µ" H 7575 3750 50  0000 L CNN
 F 2 "" H 7588 3700 30  0000 C CNN
 F 3 "" H 7550 3850 60  0000 C CNN
+F 4 "16V" H 7550 3850 60  0001 C CNN "Voltage"
 	1    7550 3850
 	1    0    0    -1
@@
 P 6550 3850
 F 0 "C?" H 6575 3950 50  0000 L CNN
-F 1 "4.7µ 16V" H 6575 3750 50  0000 L CNN
+F 1 "4.7µ" H 6575 3750 50  0000 L CNN
 F 2 "" H 6588 3700 30  0000 C CNN
 F 3 "" H 6550 3850 60  0000 C CNN
+F 4 "16V" H 6550 3850 60  0001 C CNN "Voltage"
 	1    6550 3850
 	1    0    0    -1
@@
 P 2950 3850
 F 0 "C?" H 2975 3950 50  0000 L CNN
-F 1 "2.2µ 30V" H 2975 3750 50  0000 L CNN
+F 1 "2.2µ" H 2975 3750 50  0000 L CNN
 F 2 "" H 2988 3700 30  0000 C CNN
 F 3 "" H 2950 3850 60  0000 C CNN
+F 4 "30V" H 2950 3850 60  0001 C CNN "Voltage"
 	1    2950 3850
 	1    0    0    -1
@@
 P 1950 3750
 F 0 "C?" H 1975 3850 50  0000 L CNN
-F 1 "4.7µ 16V" H 1975 3650 50  0000 L CNN
+F 1 "4.7µ" H 1975 3650 50  0000 L CNN
 F 2 "" H 1988 3600 30  0000 C CNN
 F 3 "" H 1950 3750 60  0000 C CNN
+F 4 "16V" H 1950 3750 60  0001 C CNN "Voltage"
 	1    1950 3750
 	1    0    0    -1

Commit message: hw v3.4 +testpoints
Parts:
- added T? (x5): testpoint, symbol testpoint
Connections:
- net +12V: now also T?.1
- net +24V: now also T?.1
- net +3V3: now also T?.1
- net +5V: now also T?.1
- net GND: now also T?.1
Changed lines of the file:
@@
 EESchema Schematic File Version 2
-LIBS:conn
 LIBS:power
 LIBS:stmbl_3.4-cache
@@
 	5800 3500 5800 3700
 Wire Wire Line
-	1950 4100 7550 4100
+	1950 4100 7650 4100
 Wire Wire Line
 	5800 3700 5000 3700
@@
 Connection ~ 6550 3500
 Wire Wire Line
-	7450 3500 7550 3500
+	7450 3500 7800 3500
 Wire Wire Line
 	7550 3400 7550 3700
@@
 Connection ~ 2450 4100
 Wire Wire Line
-	2050 3500 1950 3500
+	1700 3500 2050 3500
 Wire Wire Line
 	1950 3400 1950 3600
@@
 	-1   0    0    1
 $EndComp
+$Comp
+L testpoint T?
+U 1 1 5681960A
+P 2950 3300
+F 0 "T?" H 2950 3400 60  0000 C CNN
+F 1 "testpoint" H 2950 3200 60  0000 C CNN
+F 2 "" H 2950 3300 60  0000 C CNN
+F 3 "" H 2950 3300 60  0000 C CNN
+	1    2950 3300
+	0    -1   -1   0
+$EndComp
+$Comp
+L testpoint T?
+U 1 1 56819741
+P 6300 3300
+F 0 "T?" H 6300 3400 60  0000 C CNN
+F 1 "testpoint" H 6300 3200 60  0000 C CNN
+F 2 "" H 6300 3300 60  0000 C CNN
+F 3 "" H 6300 3300 60  0000 C CNN
+	1    6300 3300
+	0    -1   -1   0
+$EndComp
+$Comp
+L testpoint T?
+U 1 1 568197A1
+P 7800 3300
+F 0 "T?" H 7800 3400 60  0000 C CNN
+F 1 "testpoint" H 7800 3200 60  0000 C CNN
+F 2 "" H 7800 3300 60  0000 C CNN
+F 3 "" H 7800 3300 60  0000 C CNN
+	1    7800 3300
+	0    -1   -1   0
+$EndComp
+$Comp
+L testpoint T?
+U 1 1 568197F9
+P 1700 3300
+F 0 "T?" H 1700 3400 60  0000 C CNN
+F 1 "testpoint" H 1700 3200 60  0000 C CNN
+F 2 "" H 1700 3300 60  0000 C CNN
+F 3 "" H 1700 3300 60  0000 C CNN
+	1    1700 3300
+	0    -1   -1   0
+$EndComp
+Wire Wire Line
+	1950 3500 1950 3450
+Connection ~ 1950 3450
+$Comp
+L testpoint T?
+U 1 1 5682CF3A
+P 7850 4100
+F 0 "T?" H 7850 4200 60  0000 C CNN
+F 1 "testpoint" H 7850 4000 60  0000 C CNN
+F 2 "" H 7850 4100 60  0000 C CNN
+F 3 "" H 7850 4100 60  0000 C CNN
+	1    7850 4100
+	1    0    0    -1
+$EndComp
+Connection ~ 7550 4100
 $EndSCHEMATC

Commit message: v3.4 pdf
Changed lines of the file:
@@
 Wire Wire Line
 	1950 3400 1950 3600
-$Comp
-L +12V #PWR?
-U 1 1 5660831D
-P 1950 3400
-F 0 "#PWR?" H 1950 3250 50  0001 C CNN
-F 1 "+12V" H 1950 3540 50  0000 C CNN
-F 2 "" H 1950 3400 60  0000 C CNN
-F 3 "" H 1950 3400 60  0000 C CNN
-	1    1950 3400
-	1    0    0    -1
-$EndComp
 Connection ~ 1950 3500
 $Comp
@@
 	0    -1   -1   0
 $EndComp
-Wire Wire Line
-	1950 3500 1950 3450
-Connection ~ 1950 3450
 $Comp
 L testpoint T?
@@
 $EndComp
 Connection ~ 7550 4100
+$Comp
+L +12V #PWR?
+U 1 1 5660831D
+P 1950 3400
+F 0 "#PWR?" H 1950 3250 50  0001 C CNN
+F 1 "+12V" H 1950 3540 50  0000 C CNN
+F 2 "" H 1950 3400 60  0000 C CNN
+F 3 "" H 1950 3400 60  0000 C CNN
+	1    1950 3400
+	1    0    0    -1
+$EndComp
 $EndSCHEMATC
