File: hw/kicad/v4.0/cmd.sch (KiCad schematic (older format))
At the start: 31 parts

Commit message: v4.0
Parts:
- added R? (x4): 1k, symbol R
- U? (x4): value SP3485EN -> SN65176B
Connections:
- wire segments 142 -> 154
Changed lines of the file:
@@
 LIBS:transistors
 LIBS:stm32
-LIBS:stmbl_3.4-cache
+LIBS:texas
+LIBS:diode
+LIBS:opto
+LIBS:display
+LIBS:device
+LIBS:stmbl_4.0-cache
 EELAYER 25 0
 EELAYER END
@@
 P 5450 1400
 F 0 "U?" H 5150 1750 50  0000 L CNN
-F 1 "SP3485EN" H 5550 1750 50  0000 L CNN
+F 1 "SN65176B" H 5550 1750 50  0000 L CNN
 F 2 "SO-8" H 5450 1400 50  0000 C CIN
 F 3 "" H 5450 1400 60  0000 C CNN
@@
 P 5450 2800
 F 0 "U?" H 5150 3150 50  0000 L CNN
-F 1 "SP3485EN" H 5550 3150 50  0000 L CNN
+F 1 "SN65176B" H 5550 3150 50  0000 L CNN
 F 2 "SO-8" H 5450 2800 50  0000 C CIN
 F 3 "" H 5450 2800 60  0000 C CNN
@@
 P 5450 4200
 F 0 "U?" H 5150 4550 50  0000 L CNN
-F 1 "SP3485EN" H 5550 4550 50  0000 L CNN
+F 1 "SN65176B" H 5550 4550 50  0000 L CNN
 F 2 "SO-8" H 5450 4200 50  0000 C CIN
 F 3 "" H 5450 4200 60  0000 C CNN
@@
 P 5450 5600
 F 0 "U?" H 5150 5950 50  0000 L CNN
-F 1 "SP3485EN" H 5550 5950 50  0000 L CNN
+F 1 "SN65176B" H 5550 5950 50  0000 L CNN
 F 2 "SO-8" H 5450 5600 50  0000 C CIN
 F 3 "" H 5450 5600 60  0000 C CNN
@@
 Wire Wire Line
 	5150 2150 5150 2350
+$Comp
+L R R?
+U 1 1 57758B35
+P 6900 1600
+F 0 "R?" V 6980 1600 50  0000 C CNN
+F 1 "1k" V 6900 1600 50  0000 C CNN
+F 2 "" V 6830 1600 30  0000 C CNN
+F 3 "" H 6900 1600 30  0000 C CNN
+	1    6900 1600
+	1    0    0    -1
+$EndComp
+$Comp
+L GND #PWR?
+U 1 1 57758BC5
+P 6900 1800
+F 0 "#PWR?" H 6900 1550 50  0001 C CNN
+F 1 "GND" H 6900 1650 50  0000 C CNN
+F 2 "" H 6900 1800 60  0000 C CNN
+F 3 "" H 6900 1800 60  0000 C CNN
+	1    6900 1800
+	1    0    0    -1
+$EndComp
+Wire Wire Line
+	6950 1400 6900 1400
+Wire Wire Line
+	6900 1400 6900 1450
+Wire Wire Line
+	6900 1750 6900 1800
+$Comp
+L R R?
+U 1 1 57758F9B
+P 6900 3000
+F 0 "R?" V 6980 3000 50  0000 C CNN
+F 1 "1k" V 6900 3000 50  0000 C CNN
+F 2 "" V 6830 3000 30  0000 C CNN
+F 3 "" H 6900 3000 30  0000 C CNN
+	1    6900 3000
+	1    0    0    -1
+$EndComp
+$Comp
+L GND #PWR?
+U 1 1 57758FA1
+P 6900 3200
+F 0 "#PWR?" H 6900 2950 50  0001 C CNN
+F 1 "GND" H 6900 3050 50  0000 C CNN
+F 2 "" H 6900 3200 60  0000 C CNN
+F 3 "" H 6900 3200 60  0000 C CNN
+	1    6900 3200
+	1    0    0    -1
+$EndComp
+Wire Wire Line
+	6950 2800 6900 2800
+Wire Wire Line
+	6900 2800 6900 2850
+Wire Wire Line
+	6900 3150 6900 3200
+$Comp
+L R R?
+U 1 1 577591B1
+P 6900 4400
+F 0 "R?" V 6980 4400 50  0000 C CNN
+F 1 "1k" V 6900 4400 50  0000 C CNN
+F 2 "" V 6830 4400 30  0000 C CNN
+F 3 "" H 6900 4400 30  0000 C CNN
+	1    6900 4400
+	1    0    0    -1
+$EndComp
+$Comp
+L GND #PWR?
+U 1 1 577591B7
+P 6900 4600
+F 0 "#PWR?" H 6900 4350 50  0001 C CNN
+F 1 "GND" H 6900 4450 50  0000 C CNN
+F 2 "" H 6900 4600 60  0000 C CNN
+F 3 "" H 6900 4600 60  0000 C CNN
+	1    6900 4600
+	1    0    0    -1
+$EndComp
+Wire Wire Line
+	6950 4200 6900 4200
+Wire Wire Line
+	6900 4200 6900 4250
+Wire Wire Line
+	6900 4550 6900 4600
+$Comp
+L R R?
+U 1 1 5775928B
+P 6900 5800
+F 0 "R?" V 6980 5800 50  0000 C CNN
+F 1 "1k" V 6900 5800 50  0000 C CNN
+F 2 "" V 6830 5800 30  0000 C CNN
+F 3 "" H 6900 5800 30  0000 C CNN
+	1    6900 5800
+	1    0    0    -1
+$EndComp
+$Comp
+L GND #PWR?
+U 1 1 57759291
+P 6900 6000
+F 0 "#PWR?" H 6900 5750 50  0001 C CNN
+F 1 "GND" H 6900 5850 50  0000 C CNN
+F 2 "" H 6900 6000 60  0000 C CNN
+F 3 "" H 6900 6000 60  0000 C CNN
+	1    6900 6000
+	1    0    0    -1
+$EndComp
+Wire Wire Line
+	6950 5600 6900 5600
+Wire Wire Line
+	6900 5600 6900 5650
+Wire Wire Line
+	6900 5950 6900 6000
+Text HLabel 6950 5600 2    60   Input ~ 0
+E78
+Text HLabel 6950 4200 2    60   Input ~ 0
+E45
+Text HLabel 6950 2800 2    60   Input ~ 0
+E36
+Text HLabel 6950 1400 2    60   Input ~ 0
+E12
 $EndSCHEMATC

Commit message: v4.0
Parts:
- removed JP? (x2): Jumper_NO_Small, symbol Jumper_NO_Small
- C17, C53, C54, C55, C56: renamed from C?; footprint (none) -> Capacitors_SMD:C_0603
- J3: renamed from J?; value RJ45sh_LEDS -> RJ45_LED; footprint (none) -> stmbl:RJ45_LED; symbol RJ45sh_LEDS -> RJ45_LED
- R101, R102, R103, R104, R17, R18, R31, R62, R63, R64, R65, R66, R67, R68, R69, R70, R71, R72, R73: renamed from R?; footprint (none) -> Resistors_SMD:R_0603
- T26, T27, T28, T29: renamed from T?; footprint (none) -> Measurement_Points:Measurement_Point_Round-SMD-Pad_Small
- U10, U11, U8, U9: renamed from U?; footprint SO-8 -> Power_Integrations:SO-8
Connections:
- wire segments 154 -> 150

Commit message: v4.0
Parts:
- added C?: 100n, Capacitors_SMD:C_0603, symbol C
- added L?: 220R 700mA, symbol INDUCTOR
Connections:
- net +5V: now also C?.1, L?.2; no longer C53.1, C54.1, C55.1, C56.1, R62.1, R65.1, R68.1, R71.1, U10.8 (VCC), U11.8 (VCC), U8.8 (VCC), U9.8 (VCC)
- net GND: now also C?.2
- new net: C53.1, C54.1, C55.1, C56.1, L?.1, R62.1, R65.1, R68.1, R71.1, U10.8 (VCC), U11.8 (VCC), U8.8 (VCC), U9.8 (VCC)

Commit message: v4.0
Parts:
- added P15: CONN_01X02, stmbl:akl182-2, symbol CONN_01X02
- L7: renamed from L?; value 220R 700mA -> 220r 700mA
- gave numbers to parts that had none: 1
Connections:
- net at J3.4, R69.2, R70.1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: now also P15.1 (P1)
- net at J3.5, R68.2, R69.1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: now also P15.2 (P2)
- net +5V renamed +5F
Changed lines of the file:
@@
 LIBS:conn
 LIBS:power
+LIBS:74xgxx
+LIBS:74xx
+LIBS:ac-dc
+LIBS:actel
+LIBS:adc-dac
+LIBS:Altera
+LIBS:analog_devices
+LIBS:analog_switches
+LIBS:atmel
+LIBS:audio
+LIBS:brooktre
+LIBS:cmos_ieee
+LIBS:cmos4000
+LIBS:contrib
+LIBS:cypress
+LIBS:dc-dc
+LIBS:device
+LIBS:digital-audio
+LIBS:diode
+LIBS:display
+LIBS:dsp
+LIBS:elec-unifil
+LIBS:ESD_Protection
+LIBS:ftdi
+LIBS:gennum
+LIBS:graphic
+LIBS:hc11
+LIBS:intel
+LIBS:interface
+LIBS:ir
+LIBS:Lattice
+LIBS:linear
+LIBS:logo
+LIBS:maxim
+LIBS:memory
+LIBS:microchip_dspic33dsc
+LIBS:microchip_pic10mcu
+LIBS:microchip_pic12mcu
+LIBS:microchip_pic16mcu
+LIBS:microchip_pic18mcu
+LIBS:microchip_pic32mcu
+LIBS:microchip
+LIBS:microcontrollers
+LIBS:motor_drivers
+LIBS:motorola
+LIBS:msp430
+LIBS:nordicsemi
+LIBS:nxp_armmcu
+LIBS:onsemi
+LIBS:opto
+LIBS:Oscillators
+LIBS:philips
+LIBS:Power_Management
+LIBS:powerint
+LIBS:pspice
+LIBS:references
+LIBS:regul
+LIBS:relays
+LIBS:rfcom
+LIBS:sensors
+LIBS:silabs
+LIBS:siliconi
+LIBS:stm8
+LIBS:supertex
+LIBS:switches
+LIBS:texas
+LIBS:transf
+LIBS:ttl_ieee
+LIBS:valves
+LIBS:video
+LIBS:Xicor
+LIBS:xilinx
+LIBS:Zilog
 LIBS:stmbl_4.0-cache
 EELAYER 25 0
@@
 $Descr A4 11693 8268
 encoding utf-8
-Sheet 10 15
+Sheet 10 14
 Title ""
 Date ""
@@
 $EndComp
 $Comp
-L GND #PWR96
+L GND #PWR077
 U 1 1 565DD8E9
 P 5450 1900
-F 0 "#PWR96" H 5450 1650 50  0001 C CNN
+F 0 "#PWR077" H 5450 1650 50  0001 C CNN
 F 1 "GND" H 5450 1750 50  0000 C CNN
 F 2 "" H 5450 1900 60  0000 C CNN
@@
 $EndComp
 $Comp
-L GND #PWR98
+L GND #PWR078
 U 1 1 565DDCB0
 P 5450 3300
-F 0 "#PWR98" H 5450 3050 50  0001 C CNN
+F 0 "#PWR078" H 5450 3050 50  0001 C CNN
 F 1 "GND" H 5450 3150 50  0000 C CNN
 F 2 "" H 5450 3300 60  0000 C CNN
@@
 $EndComp
 $Comp
-L GND #PWR100
+L GND #PWR079
 U 1 1 565DDF1B
 P 5450 4700
-F 0 "#PWR100" H 5450 4450 50  0001 C CNN
+F 0 "#PWR079" H 5450 4450 50  0001 C CNN
 F 1 "GND" H 5450 4550 50  0000 C CNN
 F 2 "" H 5450 4700 60  0000 C CNN
@@
 $EndComp
 $Comp
-L GND #PWR102
+L GND #PWR080
 U 1 1 565DDF51
 P 5450 6100
-F 0 "#PWR102" H 5450 5850 50  0001 C CNN
+F 0 "#PWR080" H 5450 5850 50  0001 C CNN
 F 1 "GND" H 5450 5950 50  0000 C CNN
 F 2 "" H 5450 6100 60  0000 C CNN
@@
 $EndComp
 $Comp
-L GND #PWR51
+L GND #PWR081
 U 1 1 565DE705
 P 3000 4550
-F 0 "#PWR51" H 3000 4300 50  0001 C CNN
+F 0 "#PWR081" H 3000 4300 50  0001 C CNN
 F 1 "GND" H 3000 4400 50  0000 C CNN
 F 2 "" H 3000 4550 60  0000 C CNN
@@
 $EndComp
 $Comp
-L GND #PWR35
+L GND #PWR082
 U 1 1 565DE73D
 P 2450 3950
-F 0 "#PWR35" H 2450 3700 50  0001 C CNN
+F 0 "#PWR082" H 2450 3700 50  0001 C CNN
 F 1 "GND" H 2450 3800 50  0000 C CNN
 F 2 "" H 2450 3950 60  0000 C CNN
@@
 $EndComp
 $Comp
-L GND #PWR34
+L GND #PWR083
 U 1 1 565DE775
 P 2450 3250
-F 0 "#PWR34" H 2450 3000 50  0001 C CNN
+F 0 "#PWR083" H 2450 3000 50  0001 C CNN
 F 1 "GND" H 2450 3100 50  0000 C CNN
 F 2 "" H 2450 3250 60  0000 C CNN
@@
 $EndComp
 $Comp
-L GND #PWR115
+L GND #PWR084
 U 1 1 57758BC5
 P 6900 1800
-F 0 "#PWR115" H 6900 1550 50  0001 C CNN
+F 0 "#PWR084" H 6900 1550 50  0001 C CNN
 F 1 "GND" H 6900 1650 50  0000 C CNN
 F 2 "" H 6900 1800 60  0000 C CNN
@@
 $EndComp
 $Comp
-L GND #PWR116
+L GND #PWR085
 U 1 1 57758FA1
 P 6900 3200
-F 0 "#PWR116" H 6900 2950 50  0001 C CNN
+F 0 "#PWR085" H 6900 2950 50  0001 C CNN
 F 1 "GND" H 6900 3050 50  0000 C CNN
 F 2 "" H 6900 3200 60  0000 C CNN
@@
 $EndComp
 $Comp
-L GND #PWR117
+L GND #PWR086
 U 1 1 577591B7
 P 6900 4600
-F 0 "#PWR117" H 6900 4350 50  0001 C CNN
+F 0 "#PWR086" H 6900 4350 50  0001 C CNN
 F 1 "GND" H 6900 4450 50  0000 C CNN
 F 2 "" H 6900 4600 60  0000 C CNN
@@
 $EndComp
 $Comp
-L GND #PWR118
+L GND #PWR087
 U 1 1 57759291
 P 6900 6000
-F 0 "#PWR118" H 6900 5750 50  0001 C CNN
+F 0 "#PWR087" H 6900 5750 50  0001 C CNN
 F 1 "GND" H 6900 5850 50  0000 C CNN
 F 2 "" H 6900 6000 60  0000 C CNN
@@
 E12
 $Comp
-L +5V #PWR?
-U 1 1 57AD7E38
-P 8100 850
-F 0 "#PWR?" H 8100 700 50  0001 C CNN
-F 1 "+5V" H 8100 990 50  0000 C CNN
-F 2 "" H 8100 850 50  0000 C CNN
-F 3 "" H 8100 850 50  0000 C CNN
-	1    8100 850
-	1    0    0    -1
-$EndComp
-$Comp
-L INDUCTOR L?
+L INDUCTOR L7
 U 1 1 57AD7F96
 P 7700 950
-F 0 "L?" V 7650 950 50  0000 C CNN
-F 1 "220R 700mA" V 7800 950 50  0000 C CNN
-F 2 "" H 7700 950 50  0000 C CNN
+F 0 "L7" V 7650 950 50  0000 C CNN
+F 1 "220r 700mA" V 7800 950 50  0000 C CNN
+F 2 "" H 7700 950 50  0001 C CNN
 F 3 "" H 7700 950 50  0000 C CNN
 	1    7700 950
@@
 $EndComp
 $Comp
-L C C?
+L C C112
 U 1 1 57AD80BE
 P 8100 1200
-F 0 "C?" H 8125 1300 50  0000 L CNN
+F 0 "C112" H 8125 1300 50  0000 L CNN
 F 1 "100n" H 8125 1100 50  0000 L CNN
 F 2 "Capacitors_SMD:C_0603" H 8138 1050 30  0001 C CNN
@@
 	1    8100 1200
 	1    0    0    -1
+$EndComp
+$Comp
+L GND #PWR088
+U 1 1 57AD9057
+P 8100 1450
+F 0 "#PWR088" H 8100 1200 50  0001 C CNN
+F 1 "GND" H 8100 1300 50  0000 C CNN
+F 2 "" H 8100 1450 60  0000 C CNN
+F 3 "" H 8100 1450 60  0000 C CNN
+	1    8100 1450
+	1    0    0    -1
+$EndComp
+$Comp
+L CONN_01X02 P15
+U 1 1 57B3D62F
+P 4400 4200
+F 0 "P15" H 4400 4350 50  0000 C CNN
+F 1 "CONN_01X02" V 4500 4200 50  0000 C CNN
+F 2 "stmbl:akl182-2" H 4400 4200 60  0001 C CNN
+F 3 "" H 4400 4200 60  0000 C CNN
+	1    4400 4200
+	-1   0    0    1
 $EndComp
 Wire Wire Line
@@
 Connection ~ 7300 2350
 Connection ~ 6500 2350
-$Comp
-L GND #PWR?
-U 1 1 57AD9057
-P 8100 1450
-F 0 "#PWR?" H 8100 1200 50  0001 C CNN
-F 1 "GND" H 8100 1300 50  0000 C CNN
-F 2 "" H 8100 1450 60  0000 C CNN
-F 3 "" H 8100 1450 60  0000 C CNN
-	1    8100 1450
-	1    0    0    -1
-$EndComp
 Wire Wire Line
 	8100 1350 8100 1450
+Wire Wire Line
+	4600 4150 4700 4150
+Wire Wire Line
+	4700 4150 4700 4050
+Connection ~ 4700 4050
+Wire Wire Line
+	4600 4250 4700 4250
+Wire Wire Line
+	4700 4250 4700 4350
+Connection ~ 4700 4350
+$Comp
+L +5F #PWR089
+U 1 1 57D6FF89
+P 8100 850
+F 0 "#PWR089" H 8100 700 50  0001 C CNN
+F 1 "+5F" H 8100 990 50  0000 C CNN
+F 2 "" H 8100 850 50  0000 C CNN
+F 3 "" H 8100 850 50  0000 C CNN
+	1    8100 850
+	1    0    0    -1
+$EndComp
 $EndSCHEMATC

Commit message: v4.0
Parts:
- L7: footprint (none) -> Resistors_SMD:R_0603
- U10, U11, U8, U9: footprint Power_Integrations:SO-8 -> SMD_Packages:SOIC-8-N
Changed lines of the file:
@@
 F 0 "U8" H 5150 1750 50  0000 L CNN
 F 1 "SN65176B" H 5550 1750 50  0000 L CNN
-F 2 "Power_Integrations:SO-8" H 5450 1400 50  0000 C CIN
+F 2 "SMD_Packages:SOIC-8-N" H 5450 1400 50  0000 C CIN
 F 3 "" H 5450 1400 60  0000 C CNN
 	1    5450 1400
@@
 $EndComp
 $Comp
-L GND #PWR077
+L GND #PWR076
 U 1 1 565DD8E9
 P 5450 1900
-F 0 "#PWR077" H 5450 1650 50  0001 C CNN
+F 0 "#PWR076" H 5450 1650 50  0001 C CNN
 F 1 "GND" H 5450 1750 50  0000 C CNN
 F 2 "" H 5450 1900 60  0000 C CNN
@@
 F 0 "U9" H 5150 3150 50  0000 L CNN
 F 1 "SN65176B" H 5550 3150 50  0000 L CNN
-F 2 "Power_Integrations:SO-8" H 5450 2800 50  0000 C CIN
+F 2 "SMD_Packages:SOIC-8-N" H 5450 2800 50  0000 C CIN
 F 3 "" H 5450 2800 60  0000 C CNN
 	1    5450 2800
@@
 $EndComp
 $Comp
-L GND #PWR078
+L GND #PWR077
 U 1 1 565DDCB0
 P 5450 3300
-F 0 "#PWR078" H 5450 3050 50  0001 C CNN
+F 0 "#PWR077" H 5450 3050 50  0001 C CNN
 F 1 "GND" H 5450 3150 50  0000 C CNN
 F 2 "" H 5450 3300 60  0000 C CNN
@@
 F 0 "U10" H 5150 4550 50  0000 L CNN
 F 1 "SN65176B" H 5550 4550 50  0000 L CNN
-F 2 "Power_Integrations:SO-8" H 5450 4200 50  0000 C CIN
+F 2 "SMD_Packages:SOIC-8-N" H 5450 4200 50  0000 C CIN
 F 3 "" H 5450 4200 60  0000 C CNN
 	1    5450 4200
@@
 $EndComp
 $Comp
-L GND #PWR079
+L GND #PWR078
 U 1 1 565DDF1B
 P 5450 4700
-F 0 "#PWR079" H 5450 4450 50  0001 C CNN
+F 0 "#PWR078" H 5450 4450 50  0001 C CNN
 F 1 "GND" H 5450 4550 50  0000 C CNN
 F 2 "" H 5450 4700 60  0000 C CNN
@@
 F 0 "U11" H 5150 5950 50  0000 L CNN
 F 1 "SN65176B" H 5550 5950 50  0000 L CNN
-F 2 "Power_Integrations:SO-8" H 5450 5600 50  0000 C CIN
+F 2 "SMD_Packages:SOIC-8-N" H 5450 5600 50  0000 C CIN
 F 3 "" H 5450 5600 60  0000 C CNN
 	1    5450 5600
@@
 $EndComp
 $Comp
-L GND #PWR080
+L GND #PWR079
 U 1 1 565DDF51
 P 5450 6100
-F 0 "#PWR080" H 5450 5850 50  0001 C CNN
+F 0 "#PWR079" H 5450 5850 50  0001 C CNN
 F 1 "GND" H 5450 5950 50  0000 C CNN
 F 2 "" H 5450 6100 60  0000 C CNN
@@
 $EndComp
 $Comp
-L GND #PWR081
+L GND #PWR080
 U 1 1 565DE705
 P 3000 4550
-F 0 "#PWR081" H 3000 4300 50  0001 C CNN
+F 0 "#PWR080" H 3000 4300 50  0001 C CNN
 F 1 "GND" H 3000 4400 50  0000 C CNN
 F 2 "" H 3000 4550 60  0000 C CNN
@@
 $EndComp
 $Comp
-L GND #PWR082
+L GND #PWR081
 U 1 1 565DE73D
 P 2450 3950
-F 0 "#PWR082" H 2450 3700 50  0001 C CNN
+F 0 "#PWR081" H 2450 3700 50  0001 C CNN
 F 1 "GND" H 2450 3800 50  0000 C CNN
 F 2 "" H 2450 3950 60  0000 C CNN
@@
 $EndComp
 $Comp
-L GND #PWR083
+L GND #PWR082
 U 1 1 565DE775
 P 2450 3250
-F 0 "#PWR083" H 2450 3000 50  0001 C CNN
+F 0 "#PWR082" H 2450 3000 50  0001 C CNN
 F 1 "GND" H 2450 3100 50  0000 C CNN
 F 2 "" H 2450 3250 60  0000 C CNN
@@
 $EndComp
 $Comp
-L GND #PWR084
+L GND #PWR083
 U 1 1 57758BC5
 P 6900 1800
-F 0 "#PWR084" H 6900 1550 50  0001 C CNN
+F 0 "#PWR083" H 6900 1550 50  0001 C CNN
 F 1 "GND" H 6900 1650 50  0000 C CNN
 F 2 "" H 6900 1800 60  0000 C CNN
@@
 $EndComp
 $Comp
-L GND #PWR085
+L GND #PWR084
 U 1 1 57758FA1
 P 6900 3200
-F 0 "#PWR085" H 6900 2950 50  0001 C CNN
+F 0 "#PWR084" H 6900 2950 50  0001 C CNN
 F 1 "GND" H 6900 3050 50  0000 C CNN
 F 2 "" H 6900 3200 60  0000 C CNN
@@
 $EndComp
 $Comp
-L GND #PWR086
+L GND #PWR085
 U 1 1 577591B7
 P 6900 4600
-F 0 "#PWR086" H 6900 4350 50  0001 C CNN
+F 0 "#PWR085" H 6900 4350 50  0001 C CNN
 F 1 "GND" H 6900 4450 50  0000 C CNN
 F 2 "" H 6900 4600 60  0000 C CNN
@@
 $EndComp
 $Comp
-L GND #PWR087
+L GND #PWR086
 U 1 1 57759291
 P 6900 6000
-F 0 "#PWR087" H 6900 5750 50  0001 C CNN
+F 0 "#PWR086" H 6900 5750 50  0001 C CNN
 F 1 "GND" H 6900 5850 50  0000 C CNN
 F 2 "" H 6900 6000 60  0000 C CNN
@@
 F 0 "L7" V 7650 950 50  0000 C CNN
 F 1 "220r 700mA" V 7800 950 50  0000 C CNN
-F 2 "" H 7700 950 50  0001 C CNN
+F 2 "Resistors_SMD:R_0603" H 7700 950 50  0001 C CNN
 F 3 "" H 7700 950 50  0000 C CNN
 	1    7700 950
@@
 $EndComp
 $Comp
-L GND #PWR088
+L GND #PWR087
 U 1 1 57AD9057
 P 8100 1450
-F 0 "#PWR088" H 8100 1200 50  0001 C CNN
+F 0 "#PWR087" H 8100 1200 50  0001 C CNN
 F 1 "GND" H 8100 1300 50  0000 C CNN
 F 2 "" H 8100 1450 60  0000 C CNN
@@
 Connection ~ 4700 4350
 $Comp
-L +5F #PWR089
+L +5F #PWR088
 U 1 1 57D6FF89
 P 8100 850
-F 0 "#PWR089" H 8100 700 50  0001 C CNN
+F 0 "#PWR088" H 8100 700 50  0001 C CNN
 F 1 "+5F" H 8100 990 50  0000 C CNN
 F 2 "" H 8100 850 50  0000 C CNN

Commit message: v4.0
Parts:
- U10, U11, U8, U9: footprint SMD_Packages:SOIC-8-N -> stmbl:SOIC-8-N
Changed lines of the file:
@@
 F 0 "U8" H 5150 1750 50  0000 L CNN
 F 1 "SN65176B" H 5550 1750 50  0000 L CNN
-F 2 "SMD_Packages:SOIC-8-N" H 5450 1400 50  0000 C CIN
+F 2 "stmbl:SOIC-8-N" H 5450 1400 50  0000 C CIN
 F 3 "" H 5450 1400 60  0000 C CNN
 	1    5450 1400
@@
 $EndComp
 $Comp
-L GND #PWR076
+L GND #PWR081
 U 1 1 565DD8E9
 P 5450 1900
-F 0 "#PWR076" H 5450 1650 50  0001 C CNN
+F 0 "#PWR081" H 5450 1650 50  0001 C CNN
 F 1 "GND" H 5450 1750 50  0000 C CNN
 F 2 "" H 5450 1900 60  0000 C CNN
@@
 F 0 "U9" H 5150 3150 50  0000 L CNN
 F 1 "SN65176B" H 5550 3150 50  0000 L CNN
-F 2 "SMD_Packages:SOIC-8-N" H 5450 2800 50  0000 C CIN
+F 2 "stmbl:SOIC-8-N" H 5450 2800 50  0000 C CIN
 F 3 "" H 5450 2800 60  0000 C CNN
 	1    5450 2800
@@
 $EndComp
 $Comp
-L GND #PWR077
+L GND #PWR082
 U 1 1 565DDCB0
 P 5450 3300
-F 0 "#PWR077" H 5450 3050 50  0001 C CNN
+F 0 "#PWR082" H 5450 3050 50  0001 C CNN
 F 1 "GND" H 5450 3150 50  0000 C CNN
 F 2 "" H 5450 3300 60  0000 C CNN
@@
 F 0 "U10" H 5150 4550 50  0000 L CNN
 F 1 "SN65176B" H 5550 4550 50  0000 L CNN
-F 2 "SMD_Packages:SOIC-8-N" H 5450 4200 50  0000 C CIN
+F 2 "stmbl:SOIC-8-N" H 5450 4200 50  0000 C CIN
 F 3 "" H 5450 4200 60  0000 C CNN
 	1    5450 4200
@@
 $EndComp
 $Comp
-L GND #PWR078
+L GND #PWR083
 U 1 1 565DDF1B
 P 5450 4700
-F 0 "#PWR078" H 5450 4450 50  0001 C CNN
+F 0 "#PWR083" H 5450 4450 50  0001 C CNN
 F 1 "GND" H 5450 4550 50  0000 C CNN
 F 2 "" H 5450 4700 60  0000 C CNN
@@
 F 0 "U11" H 5150 5950 50  0000 L CNN
 F 1 "SN65176B" H 5550 5950 50  0000 L CNN
-F 2 "SMD_Packages:SOIC-8-N" H 5450 5600 50  0000 C CIN
+F 2 "stmbl:SOIC-8-N" H 5450 5600 50  0000 C CIN
 F 3 "" H 5450 5600 60  0000 C CNN
 	1    5450 5600
@@
 $EndComp
 $Comp
-L GND #PWR079
+L GND #PWR084
 U 1 1 565DDF51
 P 5450 6100
-F 0 "#PWR079" H 5450 5850 50  0001 C CNN
+F 0 "#PWR084" H 5450 5850 50  0001 C CNN
 F 1 "GND" H 5450 5950 50  0000 C CNN
 F 2 "" H 5450 6100 60  0000 C CNN
@@
 $EndComp
 $Comp
-L GND #PWR080
+L GND #PWR085
 U 1 1 565DE705
 P 3000 4550
-F 0 "#PWR080" H 3000 4300 50  0001 C CNN
+F 0 "#PWR085" H 3000 4300 50  0001 C CNN
 F 1 "GND" H 3000 4400 50  0000 C CNN
 F 2 "" H 3000 4550 60  0000 C CNN
@@
 $EndComp
 $Comp
-L GND #PWR081
+L GND #PWR086
 U 1 1 565DE73D
 P 2450 3950
-F 0 "#PWR081" H 2450 3700 50  0001 C CNN
+F 0 "#PWR086" H 2450 3700 50  0001 C CNN
 F 1 "GND" H 2450 3800 50  0000 C CNN
 F 2 "" H 2450 3950 60  0000 C CNN
@@
 $EndComp
 $Comp
-L GND #PWR082
+L GND #PWR087
 U 1 1 565DE775
 P 2450 3250
-F 0 "#PWR082" H 2450 3000 50  0001 C CNN
+F 0 "#PWR087" H 2450 3000 50  0001 C CNN
 F 1 "GND" H 2450 3100 50  0000 C CNN
 F 2 "" H 2450 3250 60  0000 C CNN
@@
 $EndComp
 $Comp
-L GND #PWR083
+L GND #PWR088
 U 1 1 57758BC5
 P 6900 1800
-F 0 "#PWR083" H 6900 1550 50  0001 C CNN
+F 0 "#PWR088" H 6900 1550 50  0001 C CNN
 F 1 "GND" H 6900 1650 50  0000 C CNN
 F 2 "" H 6900 1800 60  0000 C CNN
@@
 $EndComp
 $Comp
-L GND #PWR084
+L GND #PWR089
 U 1 1 57758FA1
 P 6900 3200
-F 0 "#PWR084" H 6900 2950 50  0001 C CNN
+F 0 "#PWR089" H 6900 2950 50  0001 C CNN
 F 1 "GND" H 6900 3050 50  0000 C CNN
 F 2 "" H 6900 3200 60  0000 C CNN
@@
 $EndComp
 $Comp
-L GND #PWR085
+L GND #PWR090
 U 1 1 577591B7
 P 6900 4600
-F 0 "#PWR085" H 6900 4350 50  0001 C CNN
+F 0 "#PWR090" H 6900 4350 50  0001 C CNN
 F 1 "GND" H 6900 4450 50  0000 C CNN
 F 2 "" H 6900 4600 60  0000 C CNN
@@
 $EndComp
 $Comp
-L GND #PWR086
+L GND #PWR091
 U 1 1 57759291
 P 6900 6000
-F 0 "#PWR086" H 6900 5750 50  0001 C CNN
+F 0 "#PWR091" H 6900 5750 50  0001 C CNN
 F 1 "GND" H 6900 5850 50  0000 C CNN
 F 2 "" H 6900 6000 60  0000 C CNN
@@
 $EndComp
 $Comp
-L GND #PWR087
+L GND #PWR092
 U 1 1 57AD9057
 P 8100 1450
-F 0 "#PWR087" H 8100 1200 50  0001 C CNN
+F 0 "#PWR092" H 8100 1200 50  0001 C CNN
 F 1 "GND" H 8100 1300 50  0000 C CNN
 F 2 "" H 8100 1450 60  0000 C CNN
@@
 Connection ~ 4700 4350
 $Comp
-L +5F #PWR088
+L +5F #PWR093
 U 1 1 57D6FF89
 P 8100 850
-F 0 "#PWR088" H 8100 700 50  0001 C CNN
+F 0 "#PWR093" H 8100 700 50  0001 C CNN
 F 1 "+5F" H 8100 990 50  0000 C CNN
 F 2 "" H 8100 850 50  0000 C CNN
