File: hw/kicad/v4.0/cmd.sch (KiCad schematic (older format))
At the start: 36 parts, among them J3 RJ45_LED, P15 CONN_01X02, T26 testpoint, T27 testpoint, T28 testpoint, T29 testpoint, U10 SN65176B, U11 SN65176B, U8 SN65176B, U9 SN65176B

Commit message: v4.0
Parts:
- R17, R18: value 470 -> 560
Changed lines of the file:
@@
 $EndComp
 $Comp
-L GND #PWR081
+L GND #PWR080
 U 1 1 565DD8E9
 P 5450 1900
-F 0 "#PWR081" H 5450 1650 50  0001 C CNN
+F 0 "#PWR080" H 5450 1650 50  0001 C CNN
 F 1 "GND" H 5450 1750 50  0000 C CNN
 F 2 "" H 5450 1900 60  0000 C CNN
@@
 $EndComp
 $Comp
-L GND #PWR082
+L GND #PWR081
 U 1 1 565DDCB0
 P 5450 3300
-F 0 "#PWR082" H 5450 3050 50  0001 C CNN
+F 0 "#PWR081" H 5450 3050 50  0001 C CNN
 F 1 "GND" H 5450 3150 50  0000 C CNN
 F 2 "" H 5450 3300 60  0000 C CNN
@@
 $EndComp
 $Comp
-L GND #PWR083
+L GND #PWR082
 U 1 1 565DDF1B
 P 5450 4700
-F 0 "#PWR083" H 5450 4450 50  0001 C CNN
+F 0 "#PWR082" H 5450 4450 50  0001 C CNN
 F 1 "GND" H 5450 4550 50  0000 C CNN
 F 2 "" H 5450 4700 60  0000 C CNN
@@
 $EndComp
 $Comp
-L GND #PWR084
+L GND #PWR083
 U 1 1 565DDF51
 P 5450 6100
-F 0 "#PWR084" H 5450 5850 50  0001 C CNN
+F 0 "#PWR083" H 5450 5850 50  0001 C CNN
 F 1 "GND" H 5450 5950 50  0000 C CNN
 F 2 "" H 5450 6100 60  0000 C CNN
@@
 $EndComp
 $Comp
-L GND #PWR085
+L GND #PWR084
 U 1 1 565DE705
 P 3000 4550
-F 0 "#PWR085" H 3000 4300 50  0001 C CNN
+F 0 "#PWR084" H 3000 4300 50  0001 C CNN
 F 1 "GND" H 3000 4400 50  0000 C CNN
 F 2 "" H 3000 4550 60  0000 C CNN
@@
 $EndComp
 $Comp
-L GND #PWR086
+L GND #PWR085
 U 1 1 565DE73D
 P 2450 3950
-F 0 "#PWR086" H 2450 3700 50  0001 C CNN
+F 0 "#PWR085" H 2450 3700 50  0001 C CNN
 F 1 "GND" H 2450 3800 50  0000 C CNN
 F 2 "" H 2450 3950 60  0000 C CNN
@@
 $EndComp
 $Comp
-L GND #PWR087
+L GND #PWR086
 U 1 1 565DE775
 P 2450 3250
-F 0 "#PWR087" H 2450 3000 50  0001 C CNN
+F 0 "#PWR086" H 2450 3000 50  0001 C CNN
 F 1 "GND" H 2450 3100 50  0000 C CNN
 F 2 "" H 2450 3250 60  0000 C CNN
@@
 P 2300 3100
 F 0 "R17" V 2380 3100 50  0000 C CNN
-F 1 "470" V 2300 3100 50  0000 C CNN
+F 1 "560" V 2300 3100 50  0000 C CNN
 F 2 "Resistors_SMD:R_0603" V 2230 3100 30  0001 C CNN
 F 3 "" H 2300 3100 30  0000 C CNN
@@
 P 2300 3800
 F 0 "R18" V 2380 3800 50  0000 C CNN
-F 1 "470" V 2300 3800 50  0000 C CNN
+F 1 "560" V 2300 3800 50  0000 C CNN
 F 2 "Resistors_SMD:R_0603" V 2230 3800 30  0001 C CNN
 F 3 "" H 2300 3800 30  0000 C CNN
@@
 $EndComp
 $Comp
-L GND #PWR088
+L GND #PWR087
 U 1 1 57758BC5
 P 6900 1800
-F 0 "#PWR088" H 6900 1550 50  0001 C CNN
+F 0 "#PWR087" H 6900 1550 50  0001 C CNN
 F 1 "GND" H 6900 1650 50  0000 C CNN
 F 2 "" H 6900 1800 60  0000 C CNN
@@
 $EndComp
 $Comp
-L GND #PWR089
+L GND #PWR088
 U 1 1 57758FA1
 P 6900 3200
-F 0 "#PWR089" H 6900 2950 50  0001 C CNN
+F 0 "#PWR088" H 6900 2950 50  0001 C CNN
 F 1 "GND" H 6900 3050 50  0000 C CNN
 F 2 "" H 6900 3200 60  0000 C CNN
@@
 $EndComp
 $Comp
-L GND #PWR090
+L GND #PWR089
 U 1 1 577591B7
 P 6900 4600
-F 0 "#PWR090" H 6900 4350 50  0001 C CNN
+F 0 "#PWR089" H 6900 4350 50  0001 C CNN
 F 1 "GND" H 6900 4450 50  0000 C CNN
 F 2 "" H 6900 4600 60  0000 C CNN
@@
 $EndComp
 $Comp
-L GND #PWR091
+L GND #PWR090
 U 1 1 57759291
 P 6900 6000
-F 0 "#PWR091" H 6900 5750 50  0001 C CNN
+F 0 "#PWR090" H 6900 5750 50  0001 C CNN
 F 1 "GND" H 6900 5850 50  0000 C CNN
 F 2 "" H 6900 6000 60  0000 C CNN
@@
 $EndComp
 $Comp
-L GND #PWR092
+L GND #PWR091
 U 1 1 57AD9057
 P 8100 1450
-F 0 "#PWR092" H 8100 1200 50  0001 C CNN
+F 0 "#PWR091" H 8100 1200 50  0001 C CNN
 F 1 "GND" H 8100 1300 50  0000 C CNN
 F 2 "" H 8100 1450 60  0000 C CNN
@@
 Connection ~ 4700 4350
 $Comp
-L +5F #PWR093
+L +5F #PWR092
 U 1 1 57D6FF89
 P 8100 850
-F 0 "#PWR093" H 8100 700 50  0001 C CNN
+F 0 "#PWR092" H 8100 700 50  0001 C CNN
 F 1 "+5F" H 8100 990 50  0000 C CNN
 F 2 "" H 8100 850 50  0000 C CNN
