File: hw/kicad/v4.0/io.sch (KiCad schematic (older format))
At the start: 27 parts

Commit message: v4.0
Parts:
- removed JP?: JUMPER3, symbol JUMPER3
- removed P?: CONN_02X10, symbol CONN_02X10
- added P10: CONN_02X07, Socket_Strips:Socket_Strip_Angled_2x07, symbol CONN_02X07
- C66, C67, C68: renamed from C?; footprint (none) -> Capacitors_SMD:C_0603
- D2, D3, D5, D7: renamed from D?; footprint (none) -> Diodes_SMD:SOD-123
- P5, P9: renamed from P?; footprint (none) -> stmbl:akl182-6
- P7: renamed from P?; footprint (none) -> Pin_Headers:Pin_Header_Straight_1x03
- Q1, Q2, Q3, Q4: renamed from Q?; footprint SOT-23 -> TO_SOT_Packages_SMD:SOT-23
- R10, R11, R12, R13, R14, R40, R45, R9: renamed from R?; footprint (none) -> Resistors_SMD:R_0603
- U22, U23, U24: renamed from U?; footprint (none) -> TO_SOT_Packages_SMD:SOT-23-6
Connections:
- net labels removed: +12V, I2C_SCL, I2C_SDA, IO_IN2, IO_IN3
- wire segments 66 -> 62

Commit message: v4.0
Parts:
- added C52, C59: 1n, Capacitors_SMD:C_0603, symbol C
- added R105, R108, R119, R99: 1k, Resistors_SMD:R_0603, symbol R
- added R106, R98: 10k, Resistors_SMD:R_0603, symbol R
- added T20, T30: testpoint, Measurement_Points:Measurement_Point_Round-SMD-Pad_Small, symbol testpoint
Connections:
- net +3V3: now also R105.1, R119.1
- net GND: now also C52.2, C59.2, R108.2, R99.2
- new net A_IO0: R98.1
- new net A_IO0_: C52.1, R105.2, R98.2, R99.1, T20.1
- new net A_IO1: R106.1
- new net A_IO1_: C59.1, R106.2, R108.1, R119.2, T30.1

Commit message: v4.0
Parts:
- removed T20, T30: testpoint, Measurement_Points:Measurement_Point_Round-SMD-Pad_Small, symbol testpoint
- added JP? (x2): Jumper_NO_Small, symbol Jumper_NO_Small
Connections:
- net +24V: now also JP?.1; no longer D7.1 (K), P7.1 (P1)
- new net: D7.1 (K), JP?.2, JP?.2, P7.1 (P1)
- new net +12V: JP?.1
Changed lines of the file:
@@
 LIBS:stm32
 LIBS:conn
+LIBS:power
 LIBS:stmbl_4.0-cache
 EELAYER 25 0
@@
 $Descr A4 11693 8268
 encoding utf-8
-Sheet 14 14
+Sheet 14 15
 Title ""
 Date ""
@@
 $EndComp
 Wire Wire Line
-	1600 1900 1800 1900
+	1600 1900 1700 1900
+Wire Wire Line
+	1700 1900 1800 1900
 Wire Wire Line
 	1700 2000 1700 1900
@@
 	1700 2400 2100 2400
 Wire Wire Line
-	2100 2050 2100 2500
+	2100 2050 2100 2400
+Wire Wire Line
+	2100 2400 2100 2500
 $Comp
 L GND #PWR27
@@
 $EndComp
 Wire Wire Line
-	2100 1450 2100 1650
+	2100 1450 2100 1550
+Wire Wire Line
+	2100 1550 2100 1650
 $Comp
 L +24V #PWR26
@@
 $EndComp
 Wire Wire Line
-	2100 950  2100 1150
+	2100 950  2100 1050
+Wire Wire Line
+	2100 1050 2100 1150
 Wire Wire Line
 	1300 1900 1200 1900
@@
 $EndComp
 Wire Wire Line
-	1600 3900 1800 3900
+	1600 3900 1700 3900
+Wire Wire Line
+	1700 3900 1800 3900
 Wire Wire Line
 	1700 4000 1700 3900
@@
 	1700 4400 2100 4400
 Wire Wire Line
-	2100 4050 2100 4500
+	2100 4050 2100 4400
+Wire Wire Line
+	2100 4400 2100 4500
 $Comp
 L GND #PWR29
@@
 $EndComp
 Wire Wire Line
-	2100 3450 2100 3650
+	2100 3450 2100 3550
+Wire Wire Line
+	2100 3550 2100 3650
 $Comp
 L +24V #PWR28
@@
 $EndComp
 Wire Wire Line
-	2100 2950 2100 3150
+	2100 2950 2100 3050
+Wire Wire Line
+	2100 3050 2100 3150
 Wire Wire Line
 	1300 3900 1200 3900
@@
 $EndComp
 Wire Wire Line
-	1600 5900 1800 5900
+	1600 5900 1700 5900
+Wire Wire Line
+	1700 5900 1800 5900
 Wire Wire Line
 	1700 6000 1700 5900
@@
 	1700 6400 2100 6400
 Wire Wire Line
-	2100 6050 2100 6500
+	2100 6050 2100 6400
+Wire Wire Line
+	2100 6400 2100 6500
 $Comp
 L GND #PWR31
@@
 $EndComp
 Wire Wire Line
-	2100 5450 2100 5650
+	2100 5450 2100 5550
+Wire Wire Line
+	2100 5550 2100 5650
 $Comp
 L +24V #PWR30
@@
 $EndComp
 Wire Wire Line
-	2100 4950 2100 5150
+	2100 4950 2100 5050
+Wire Wire Line
+	2100 5050 2100 5150
 Wire Wire Line
 	1300 5900 1200 5900
@@
 $EndComp
 Wire Wire Line
-	4300 3900 4500 3900
+	4300 3900 4400 3900
+Wire Wire Line
+	4400 3900 4500 3900
 Wire Wire Line
 	4400 4000 4400 3900
@@
 	4400 4400 4800 4400
 Wire Wire Line
-	4800 4050 4800 4500
+	4800 4050 4800 4400
+Wire Wire Line
+	4800 4400 4800 4500
 $Comp
 L GND #PWR80
@@
 $EndComp
 Wire Wire Line
-	4800 3450 4800 3650
+	4800 3450 4800 3550
+Wire Wire Line
+	4800 3550 4800 3650
 $Comp
 L +24V #PWR79
 U 1 1 57014DBB
-P 4800 2950
-F 0 "#PWR79" H 4800 2800 50  0001 C CNN
-F 1 "+24V" H 4800 3090 50  0000 C CNN
-F 2 "" H 4800 2950 50  0000 C CNN
-F 3 "" H 4800 2950 50  0000 C CNN
-	1    4800 2950
-	1    0    0    -1
-$EndComp
-Wire Wire Line
-	4800 2950 4800 3150
+P 4800 2650
+F 0 "#PWR79" H 4800 2500 50  0001 C CNN
+F 1 "+24V" H 4800 2790 50  0000 C CNN
+F 2 "" H 4800 2650 50  0000 C CNN
+F 3 "" H 4800 2650 50  0000 C CNN
+	1    4800 2650
+	1    0    0    -1
+$EndComp
+Wire Wire Line
+	4800 2950 4800 3050
+Wire Wire Line
+	4800 3050 4800 3150
 Wire Wire Line
 	4000 3900 3900 3900
@@
 Wire Wire Line
 	5100 3050 4800 3050
+Wire Wire Line
+	4800 3050 4550 3050
 Connection ~ 4800 3050
 Wire Wire Line
@@
 	1    0    0    -1
 $EndComp
-Text HLabel 9650 2600 0    60   Input ~ 0
+Text HLabel 9750 2600 0    60   Input ~ 0
 A_IO1_
 Text HLabel 8950 2100 0    60   Input ~ 0
@@
 	1    0    0    -1
 $EndComp
-Text HLabel 8850 2600 0    60   Input ~ 0
+Text HLabel 8950 2600 0    60   Input ~ 0
 A_IO0_
 $Comp
@@
 	1    0    0    -1
 $EndComp
-$Comp
-L testpoint T20
-U 1 1 5777ECCC
-P 8750 2800
-F 0 "T20" H 8750 2900 60  0000 C CNN
-F 1 "testpoint" H 8750 2700 60  0000 C CNN
-F 2 "Measurement_Points:Measurement_Point_Round-SMD-Pad_Small" H 8750 2800 60  0001 C CNN
-F 3 "" H 8750 2800 60  0000 C CNN
-	1    8750 2800
-	-1   0    0    1
-$EndComp
 Wire Wire Line
 	9750 2100 9850 2100
@@
 	9850 2100 9850 2200
 Wire Wire Line
-	9850 2500 9850 2700
-Wire Wire Line
-	10050 2500 10050 2700
-Wire Wire Line
-	9650 2600 10050 2600
+	9850 2500 9850 2600
+Wire Wire Line
+	9850 2600 9850 2700
+Wire Wire Line
+	10050 2500 10050 2600
+Wire Wire Line
+	10050 2600 10050 2700
+Wire Wire Line
+	9750 2600 9750 2600
+Wire Wire Line
+	9750 2600 9850 2600
+Wire Wire Line
+	9850 2600 10050 2600
 Connection ~ 9850 2600
 Wire Wire Line
-	9850 3000 9850 3200
+	9850 3000 9850 3100
+Wire Wire Line
+	9850 3100 9850 3200
 Wire Wire Line
 	10050 2100 10050 2200
@@
 	9050 2100 9050 2200
 Wire Wire Line
-	9050 2500 9050 2700
-Wire Wire Line
-	9250 2500 9250 2700
+	9050 2500 9050 2600
+Wire Wire Line
+	9050 2600 9050 2700
+Wire Wire Line
+	9250 2500 9250 2600
+Wire Wire Line
+	9250 2600 9250 2700
 Connection ~ 9050 2600
 Wire Wire Line
-	9050 3000 9050 3200
+	9050 3000 9050 3100
+Wire Wire Line
+	9050 3100 9050 3200
 Wire Wire Line
 	9250 2100 9250 2200
@@
 	9250 3100 9050 3100
 Connection ~ 9050 3100
-$Comp
-L testpoint T30
-U 1 1 5777ECEA
-P 9550 2800
-F 0 "T30" H 9550 2900 60  0000 C CNN
-F 1 "testpoint" H 9550 2700 60  0000 C CNN
-F 2 "Measurement_Points:Measurement_Point_Round-SMD-Pad_Small" H 9550 2800 60  0001 C CNN
-F 3 "" H 9550 2800 60  0000 C CNN
-	1    9550 2800
-	-1   0    0    1
-$EndComp
-Wire Wire Line
-	8850 2600 9250 2600
-Wire Wire Line
-	8950 2800 8950 2600
-Connection ~ 8950 2600
-Wire Wire Line
-	9750 2600 9750 2800
-Connection ~ 9750 2600
+Wire Wire Line
+	8950 2600 9050 2600
+Wire Wire Line
+	9050 2600 9250 2600
+$Comp
+L Jumper_NO_Small JP?
+U 1 1 57AF943B
+P 4550 2850
+F 0 "JP?" H 4550 2930 50  0000 C CNN
+F 1 "Jumper_NO_Small" H 4560 2790 50  0001 C CNN
+F 2 "" H 4550 2850 50  0000 C CNN
+F 3 "" H 4550 2850 50  0000 C CNN
+	1    4550 2850
+	0    1    1    0
+$EndComp
+$Comp
+L Jumper_NO_Small JP?
+U 1 1 57AF94D3
+P 4800 2850
+F 0 "JP?" H 4800 2930 50  0000 C CNN
+F 1 "Jumper_NO_Small" H 4810 2790 50  0001 C CNN
+F 2 "" H 4800 2850 50  0000 C CNN
+F 3 "" H 4800 2850 50  0000 C CNN
+	1    4800 2850
+	0    1    1    0
+$EndComp
+$Comp
+L +12V #PWR?
+U 1 1 57AF9557
+P 4550 2650
+F 0 "#PWR?" H 4550 2500 50  0001 C CNN
+F 1 "+12V" H 4550 2790 50  0000 C CNN
+F 2 "" H 4550 2650 50  0000 C CNN
+F 3 "" H 4550 2650 50  0000 C CNN
+	1    4550 2650
+	1    0    0    -1
+$EndComp
+Wire Wire Line
+	4550 3050 4550 2950
+Wire Wire Line
+	4550 2650 4550 2750
+Wire Wire Line
+	4800 2650 4800 2750
 $EndSCHEMATC

Commit message: v4.0
Parts:
- gave numbers to parts that had none: 2
Connections:
- net A_IO0_ is gone; now on net IO_IN0: C52.1, R105.2, R98.2, R99.1
- net A_IO1_ is gone; now on net IO_IN1: C59.1, R106.2, R108.1, R119.2
- net IO_IN0: no longer P9.2 (P2)
- net IO_IN1: no longer P9.5 (P5)
- net A_IO0: no longer names the net of R98.1
- net A_IO0: now also P9.2 (P2)
- net A_IO1: no longer names the net of R106.1
- net A_IO1: now also P9.5 (P5)
Other:
- moved on the sheet: P9

Commit message: v4.0
Parts:
- removed JP3, JP4: Jumper_NO_Small, symbol Jumper_NO_Small
- added JP3: JUMPER3, symbol JUMPER3
Connections:
- net +12V: now also JP3.1
- net +24V: now also JP3.3
- net +3V3: now also C66.1, C67.1, C68.1, U22.5 (VBUS), U23.5 (VBUS), U24.5 (VBUS)
- net GND: now also C66.2, C67.2, C68.2, U22.2 (GND), U23.2 (GND), U24.2 (GND)
- net at D7.1 (K), P7.1 (P1): now also JP3.2
Other:
- moved on the sheet: C66, C67, C68, U22, U23, U24
