File: hw/kicad/v4.0/supply.sch (KiCad schematic (older format))
At the start: 16 parts

Commit message: v4.0
Parts:
- C18, C8: renamed from C?; footprint (none) -> Capacitors_SMD:C_0805
- C35, C50: renamed from C?; footprint (none) -> Capacitors_SMD:C_0603
- P3: renamed from P?; footprint (none) -> stmbl:akl182-2
- R60, R74: renamed from R?; footprint (none) -> Resistors_SMD:R_0603
- T11, T12, T4: renamed from T?; footprint (none) -> Measurement_Points:Measurement_Point_Round-SMD-Pad_Small
- U2: renamed from U?; footprint (none) -> stmbl:SOT-223
- gave numbers to parts that had none: 5
Changed lines of the file:
@@
 LIBS:transistors
 LIBS:stm32
-LIBS:texas
-LIBS:diode
-LIBS:opto
-LIBS:display
-LIBS:device
+LIBS:conn
 LIBS:stmbl_4.0-cache
 EELAYER 25 0
@@
 $EndDescr
 $Comp
-L lmr1420X IC?
+L lmr1420X IC1
 U 1 1 565A1FC6
 P 4300 2300
-F 0 "IC?" H 4100 2550 60  0000 C CNN
+F 0 "IC1" H 4100 2550 60  0000 C CNN
 F 1 "lmr1420X" H 4250 2050 60  0000 C CNN
-F 2 "" H 4200 2300 60  0000 C CNN
+F 2 "" H 4200 2300 60  0001 C CNN
 F 3 "" H 4200 2300 60  0000 C CNN
 	1    4300 2300
@@
 $EndComp
 $Comp
-L C C?
+L C C50
 U 1 1 566068C0
 P 6050 2550
-F 0 "C?" H 6075 2650 50  0000 L CNN
+F 0 "C50" H 6075 2650 50  0000 L CNN
 F 1 "47µ" H 6075 2450 50  0000 L CNN
-F 2 "" H 6088 2400 30  0000 C CNN
+F 2 "Capacitors_SMD:C_0603" H 6088 2400 30  0001 C CNN
 F 3 "" H 6050 2550 60  0000 C CNN
 F 4 "6.3V" H 6050 2550 60  0001 C CNN "Voltage"
@@
 $EndComp
 $Comp
-L R R?
+L R R74
 U 1 1 5660690B
 P 5100 2400
-F 0 "R?" V 5180 2400 50  0000 C CNN
+F 0 "R74" V 5180 2400 50  0000 C CNN
 F 1 "5.6k" V 5100 2400 50  0000 C CNN
-F 2 "" V 5030 2400 30  0000 C CNN
+F 2 "Resistors_SMD:R_0603" V 5030 2400 30  0001 C CNN
 F 3 "" H 5100 2400 30  0000 C CNN
 	1    5100 2400
@@
 $EndComp
 $Comp
-L R R?
+L R R60
 U 1 1 56606967
 P 4850 2650
-F 0 "R?" V 4930 2650 50  0000 C CNN
+F 0 "R60" V 4930 2650 50  0000 C CNN
 F 1 "1k" V 4850 2650 50  0000 C CNN
-F 2 "" V 4780 2650 30  0000 C CNN
+F 2 "Resistors_SMD:R_0603" V 4780 2650 30  0001 C CNN
 F 3 "" H 4850 2650 30  0000 C CNN
 	1    4850 2650
@@
 $EndComp
 $Comp
-L D_Schottky D?
+L D_Schottky D9
 U 1 1 566069A3
 P 5450 2650
-F 0 "D?" H 5450 2750 50  0000 C CNN
+F 0 "D9" H 5450 2750 50  0000 C CNN
 F 1 "60V 1A" H 5450 2550 50  0000 C CNN
-F 2 "" H 5450 2650 60  0000 C CNN
+F 2 "" H 5450 2650 60  0001 C CNN
 F 3 "" H 5450 2650 60  0000 C CNN
 	1    5450 2650
@@
 $EndComp
 $Comp
-L C C?
+L C C35
 U 1 1 56606BAA
 P 5000 2200
-F 0 "C?" H 5025 2300 50  0000 L CNN
+F 0 "C35" H 5025 2300 50  0000 L CNN
 F 1 "0.22µ 16V" H 5025 2100 50  0000 L CNN
-F 2 "" H 5038 2050 30  0000 C CNN
+F 2 "Capacitors_SMD:C_0603" H 5038 2050 30  0001 C CNN
 F 3 "" H 5000 2200 60  0000 C CNN
 	1    5000 2200
@@
 $EndComp
 $Comp
-L INDUCTOR L?
+L INDUCTOR L1
 U 1 1 56606C2D
 P 5750 2200
-F 0 "L?" V 5700 2200 50  0000 C CNN
+F 0 "L1" V 5700 2200 50  0000 C CNN
 F 1 "15µH 1.5A" V 5850 2200 50  0000 C CNN
-F 2 "" H 5750 2200 60  0000 C CNN
+F 2 "" H 5750 2200 60  0001 C CNN
 F 3 "" H 5750 2200 60  0000 C CNN
 	1    5750 2200
@@
 $EndComp
 $Comp
-L LM7812 U?
+L LM7812 U2
 U 1 1 566074A9
 P 2900 4950
-F 0 "U?" H 3050 4754 60  0000 C CNN
+F 0 "U2" H 3050 4754 60  0000 C CNN
 F 1 "zldo1117" H 2900 5150 60  0000 C CNN
-F 2 "" H 2900 4950 60  0000 C CNN
+F 2 "stmbl:SOT-223" H 2900 4950 60  0001 C CNN
 F 3 "" H 2900 4950 60  0000 C CNN
 	1    2900 4950
@@
 $EndComp
 $Comp
-L C C?
+L C C18
 U 1 1 566075DC
 P 3400 5250
-F 0 "C?" H 3425 5350 50  0000 L CNN
+F 0 "C18" H 3425 5350 50  0000 L CNN
 F 1 "4.7µ" H 3425 5150 50  0000 L CNN
-F 2 "" H 3438 5100 30  0000 C CNN
+F 2 "Capacitors_SMD:C_0805" H 3438 5100 30  0001 C CNN
 F 3 "" H 3400 5250 60  0000 C CNN
 F 4 "16V" H 3400 5250 60  0001 C CNN "Voltage"
@@
 $EndComp
 $Comp
-L C C?
+L C C8
 U 1 1 566076FA
 P 2400 5250
-F 0 "C?" H 2425 5350 50  0000 L CNN
+F 0 "C8" H 2425 5350 50  0000 L CNN
 F 1 "4.7µ" H 2425 5150 50  0000 L CNN
-F 2 "" H 2438 5100 30  0000 C CNN
+F 2 "Capacitors_SMD:C_0805" H 2438 5100 30  0001 C CNN
 F 3 "" H 2400 5250 60  0000 C CNN
 F 4 "16V" H 2400 5250 60  0001 C CNN "Voltage"
@@
 	3400 4800 3400 5100
 $Comp
-L +5V #PWR?
+L +5V #PWR20
 U 1 1 5660786F
 P 1900 4800
-F 0 "#PWR?" H 1900 4650 50  0001 C CNN
+F 0 "#PWR20" H 1900 4650 50  0001 C CNN
 F 1 "+5V" H 1900 4940 50  0000 C CNN
 F 2 "" H 1900 4800 60  0000 C CNN
@@
 $EndComp
 $Comp
-L +3.3V #PWR?
+L +3.3V #PWR51
 U 1 1 566078DE
 P 3400 4800
-F 0 "#PWR?" H 3400 4650 50  0001 C CNN
+F 0 "#PWR51" H 3400 4650 50  0001 C CNN
 F 1 "+3.3V" H 3400 4940 50  0000 C CNN
 F 2 "" H 3400 4800 60  0000 C CNN
@@
 Connection ~ 3400 4900
 $Comp
-L GND #PWR?
+L GND #PWR33
 U 1 1 5660843E
 P 2500 2500
-F 0 "#PWR?" H 2500 2250 50  0001 C CNN
+F 0 "#PWR33" H 2500 2250 50  0001 C CNN
 F 1 "GND" H 2500 2350 50  0000 C CNN
 F 2 "" H 2500 2500 60  0000 C CNN
@@
 $EndComp
 $Comp
-L +24V #PWR?
+L +24V #PWR32
 U 1 1 56608476
 P 2500 2200
-F 0 "#PWR?" H 2500 2050 50  0001 C CNN
+F 0 "#PWR32" H 2500 2050 50  0001 C CNN
 F 1 "+24V" H 2500 2340 50  0000 C CNN
 F 2 "" H 2500 2200 60  0000 C CNN
@@
 	2500 2400 2500 2500
 $Comp
-L ZENER D?
+L ZENER D6
 U 1 1 56694BC4
 P 2150 5200
-F 0 "D?" H 2150 5300 50  0000 C CNN
+F 0 "D6" H 2150 5300 50  0000 C CNN
 F 1 "5V" H 2150 5100 50  0000 C CNN
-F 2 "" H 2150 5200 60  0000 C CNN
+F 2 "" H 2150 5200 60  0001 C CNN
 F 3 "" H 2150 5200 60  0000 C CNN
 	1    2150 5200
@@
 	2150 5400 2150 5500
 $Comp
-L CONN_01X02 P?
+L CONN_01X02 P3
 U 1 1 566CDEAC
 P 2200 2350
-F 0 "P?" H 2200 2500 50  0000 C CNN
+F 0 "P3" H 2200 2500 50  0000 C CNN
 F 1 "CONN_01X02" V 2300 2350 50  0000 C CNN
-F 2 "" H 2200 2350 60  0000 C CNN
+F 2 "stmbl:akl182-2" H 2200 2350 60  0001 C CNN
 F 3 "" H 2200 2350 60  0000 C CNN
 	1    2200 2350
@@
 $EndComp
 $Comp
-L testpoint T?
+L testpoint T4
 U 1 1 56819741
 P 2150 4700
-F 0 "T?" H 2150 4800 60  0000 C CNN
+F 0 "T4" H 2150 4800 60  0000 C CNN
 F 1 "testpoint" H 2150 4600 60  0000 C CNN
-F 2 "" H 2150 4700 60  0000 C CNN
+F 2 "Measurement_Points:Measurement_Point_Round-SMD-Pad_Small" H 2150 4700 60  0001 C CNN
 F 3 "" H 2150 4700 60  0000 C CNN
 	1    2150 4700
@@
 $EndComp
 $Comp
-L testpoint T?
+L testpoint T11
 U 1 1 568197A1
 P 3650 4700
-F 0 "T?" H 3650 4800 60  0000 C CNN
+F 0 "T11" H 3650 4800 60  0000 C CNN
 F 1 "testpoint" H 3650 4600 60  0000 C CNN
-F 2 "" H 3650 4700 60  0000 C CNN
+F 2 "Measurement_Points:Measurement_Point_Round-SMD-Pad_Small" H 3650 4700 60  0001 C CNN
 F 3 "" H 3650 4700 60  0000 C CNN
 	1    3650 4700
@@
 $EndComp
 $Comp
-L testpoint T?
+L testpoint T12
 U 1 1 5682CF3A
 P 3700 5500
-F 0 "T?" H 3700 5600 60  0000 C CNN
+F 0 "T12" H 3700 5600 60  0000 C CNN
 F 1 "testpoint" H 3700 5400 60  0000 C CNN
-F 2 "" H 3700 5500 60  0000 C CNN
+F 2 "Measurement_Points:Measurement_Point_Round-SMD-Pad_Small" H 3700 5500 60  0001 C CNN
 F 3 "" H 3700 5500 60  0000 C CNN
 	1    3700 5500
@@
 $EndComp
 $Comp
-L lm25011 U?
+L lm25011 U4
 U 1 1 570D946D
 P 4350 1550
-F 0 "U?" H 4350 2003 60  0000 C CNN
+F 0 "U4" H 4350 2003 60  0000 C CNN
 F 1 "lm25011" H 4350 1897 60  0000 C CNN
-F 2 "" H 4350 1550 60  0000 C CNN
+F 2 "" H 4350 1550 60  0001 C CNN
 F 3 "" H 4350 1550 60  0000 C CNN
 	1    4350 1550
@@
 	1900 4900 2500 4900
 $Comp
-L GND #PWR?
+L GND #PWR21
 U 1 1 57744A84
 P 1900 5550
-F 0 "#PWR?" H 1900 5300 50  0001 C CNN
+F 0 "#PWR21" H 1900 5300 50  0001 C CNN
 F 1 "GND" H 1900 5400 50  0000 C CNN
 F 2 "" H 1900 5550 60  0000 C CNN

Commit message: v4.0
Parts:
- removed D6: 5V, symbol ZENER
Connections:
- wire segments 30 -> 28
Changed lines of the file:
@@
 Wire Wire Line
 	2500 2400 2500 2500
-$Comp
-L ZENER D6
-U 1 1 56694BC4
-P 2150 5200
-F 0 "D6" H 2150 5300 50  0000 C CNN
-F 1 "5V" H 2150 5100 50  0000 C CNN
-F 2 "" H 2150 5200 60  0001 C CNN
-F 3 "" H 2150 5200 60  0000 C CNN
-	1    2150 5200
-	0    1    1    0
-$EndComp
-Wire Wire Line
-	2150 5000 2150 4900
 Connection ~ 2150 4900
-Wire Wire Line
-	2150 5400 2150 5500
 $Comp
 L CONN_01X02 P3
@@
 Wire Wire Line
 	1900 5500 3500 5500
-Connection ~ 2150 5500
 Connection ~ 2400 5500
 Connection ~ 2900 5500

Commit message: v4.0
Parts:
- removed IC1: lmr1420X, symbol lmr1420X
- removed U4: lm25011, symbol lm25011
- added R97: 100k, Resistors_SMD:R_0603, symbol R
- added U4: ACT4088, TO_SOT_Packages_SMD:SOT-23-6, symbol ACT4088
- C35: value 0.22µ 16V -> 22n 16V
- C50: value 47µ -> 22µ
- D9: value 60V 1A -> B240A 60V 1A
- L1: value 15µH 1.5A -> 4.7µH 1.5A
- R60: value 1k -> 10k
- R74: value 5.6k -> 100k
Connections:
- wire segments 28 -> 35
- no-connect marks 0 -> 1
Other:
- moved on the sheet: C35, C50, D9, L1, R74
Changed lines of the file:
@@
 $EndDescr
-$Comp
-L lmr1420X IC1
-U 1 1 565A1FC6
-P 4300 2300
-F 0 "IC1" H 4100 2550 60  0000 C CNN
-F 1 "lmr1420X" H 4250 2050 60  0000 C CNN
-F 2 "" H 4200 2300 60  0001 C CNN
-F 3 "" H 4200 2300 60  0000 C CNN
-	1    4300 2300
-	1    0    0    -1
-$EndComp
 $Comp
 L C C50
 U 1 1 566068C0
-P 6050 2550
-F 0 "C50" H 6075 2650 50  0000 L CNN
-F 1 "47µ" H 6075 2450 50  0000 L CNN
-F 2 "Capacitors_SMD:C_0603" H 6088 2400 30  0001 C CNN
-F 3 "" H 6050 2550 60  0000 C CNN
-F 4 "6.3V" H 6050 2550 60  0001 C CNN "Voltage"
-	1    6050 2550
+P 6150 2550
+F 0 "C50" H 6175 2650 50  0000 L CNN
+F 1 "22µ" H 6175 2450 50  0000 L CNN
+F 2 "Capacitors_SMD:C_0603" H 6188 2400 30  0001 C CNN
+F 3 "" H 6150 2550 60  0000 C CNN
+F 4 "6.3V" H 6150 2550 60  0001 C CNN "Voltage"
+	1    6150 2550
 	1    0    0    -1
 $EndComp
@@
 L R R74
 U 1 1 5660690B
-P 5100 2400
-F 0 "R74" V 5180 2400 50  0000 C CNN
-F 1 "5.6k" V 5100 2400 50  0000 C CNN
-F 2 "Resistors_SMD:R_0603" V 5030 2400 30  0001 C CNN
-F 3 "" H 5100 2400 30  0000 C CNN
-	1    5100 2400
+P 5150 2400
+F 0 "R74" V 5230 2400 50  0000 C CNN
+F 1 "100k" V 5150 2400 50  0000 C CNN
+F 2 "Resistors_SMD:R_0603" V 5080 2400 30  0001 C CNN
+F 3 "" H 5150 2400 30  0000 C CNN
+	1    5150 2400
 	0    1    1    0
 $EndComp
@@
 P 4850 2650
 F 0 "R60" V 4930 2650 50  0000 C CNN
-F 1 "1k" V 4850 2650 50  0000 C CNN
+F 1 "10k" V 4850 2650 50  0000 C CNN
 F 2 "Resistors_SMD:R_0603" V 4780 2650 30  0001 C CNN
 F 3 "" H 4850 2650 30  0000 C CNN
@@
 L D_Schottky D9
 U 1 1 566069A3
-P 5450 2650
-F 0 "D9" H 5450 2750 50  0000 C CNN
-F 1 "60V 1A" H 5450 2550 50  0000 C CNN
-F 2 "" H 5450 2650 60  0001 C CNN
-F 3 "" H 5450 2650 60  0000 C CNN
-	1    5450 2650
+P 5550 2650
+F 0 "D9" H 5550 2750 50  0000 C CNN
+F 1 "B240A 60V 1A" H 5550 2550 50  0000 C CNN
+F 2 "" H 5550 2650 60  0001 C CNN
+F 3 "" H 5550 2650 60  0000 C CNN
+	1    5550 2650
 	0    1    1    0
 $EndComp
@@
 L C C35
 U 1 1 56606BAA
-P 5000 2200
-F 0 "C35" H 5025 2300 50  0000 L CNN
-F 1 "0.22µ 16V" H 5025 2100 50  0000 L CNN
-F 2 "Capacitors_SMD:C_0603" H 5038 2050 30  0001 C CNN
-F 3 "" H 5000 2200 60  0000 C CNN
-	1    5000 2200
+P 5000 2100
+F 0 "C35" H 5025 2200 50  0000 L CNN
+F 1 "22n 16V" H 5025 2000 50  0000 L CNN
+F 2 "Capacitors_SMD:C_0603" H 5038 1950 30  0001 C CNN
+F 3 "" H 5000 2100 60  0000 C CNN
+	1    5000 2100
 	0    -1   -1   0
 $EndComp
@@
 L INDUCTOR L1
 U 1 1 56606C2D
-P 5750 2200
-F 0 "L1" V 5700 2200 50  0000 C CNN
-F 1 "15µH 1.5A" V 5850 2200 50  0000 C CNN
-F 2 "" H 5750 2200 60  0001 C CNN
-F 3 "" H 5750 2200 60  0000 C CNN
-	1    5750 2200
+P 5850 2100
+F 0 "L1" V 5800 2100 50  0000 C CNN
+F 1 "4.7µH 1.5A" V 5950 2100 50  0000 C CNN
+F 2 "" H 5850 2100 60  0001 C CNN
+F 3 "" H 5850 2100 60  0000 C CNN
+	1    5850 2100
 	0    -1   -1   0
 $EndComp
@@
 $EndComp
 Wire Wire Line
-	4750 2200 4850 2200
-Wire Wire Line
-	5150 2200 5450 2200
-Wire Wire Line
-	5450 2200 5450 2500
-Wire Wire Line
-	6050 2200 6050 2400
-Wire Wire Line
-	6050 2400 5250 2400
-Wire Wire Line
-	6050 2800 6050 2700
-Connection ~ 6050 2400
-Wire Wire Line
-	4950 2400 4750 2400
+	4750 2100 4850 2100
+Wire Wire Line
+	5150 2100 5550 2100
+Wire Wire Line
+	5550 2100 5550 2500
+Wire Wire Line
+	6150 2100 6150 2400
+Wire Wire Line
+	6150 2400 5300 2400
+Wire Wire Line
+	6150 2800 6150 2700
+Connection ~ 6150 2400
+Wire Wire Line
+	4750 2400 5000 2400
 Wire Wire Line
 	4850 2500 4850 2400
 Connection ~ 4850 2400
 Wire Wire Line
-	3850 2400 3850 2800
-Wire Wire Line
-	3100 2200 3850 2200
-Wire Wire Line
-	3850 2300 3750 2300
-Wire Wire Line
-	3750 2300 3750 2200
-Connection ~ 3750 2200
-Wire Wire Line
-	4750 2300 5250 2300
-Wire Wire Line
-	5250 2300 5250 2200
-Connection ~ 5250 2200
+	4750 2250 5250 2250
+Wire Wire Line
+	5250 2250 5250 2100
+Connection ~ 5250 2100
 Wire Wire Line
 	3400 5500 3400 5400
@@
 	2400 5400 2400 5500
 Wire Wire Line
-	2900 5200 2900 5500
-Wire Wire Line
-	2400 5100 2400 4900
+	2900 5500 2900 5200
+Wire Wire Line
+	2400 4900 2400 5100
 Connection ~ 2400 4900
 Wire Wire Line
@@
 	3400 4800 3400 5100
 $Comp
-L +5V #PWR20
+L +5V #PWR24
 U 1 1 5660786F
 P 1900 4800
-F 0 "#PWR20" H 1900 4650 50  0001 C CNN
+F 0 "#PWR24" H 1900 4650 50  0001 C CNN
 F 1 "+5V" H 1900 4940 50  0000 C CNN
 F 2 "" H 1900 4800 60  0000 C CNN
@@
 $EndComp
 $Comp
-L +3.3V #PWR51
+L +3.3V #PWR55
 U 1 1 566078DE
 P 3400 4800
-F 0 "#PWR51" H 3400 4650 50  0001 C CNN
+F 0 "#PWR55" H 3400 4650 50  0001 C CNN
 F 1 "+3.3V" H 3400 4940 50  0000 C CNN
 F 2 "" H 3400 4800 60  0000 C CNN
@@
 	1    0    0    -1
 $EndComp
-Connection ~ 6050 2200
+Connection ~ 6150 2100
 Wire Wire Line
 	1900 4800 1900 4900
 Connection ~ 3400 4900
 $Comp
-L GND #PWR33
+L GND #PWR37
 U 1 1 5660843E
 P 2500 2500
-F 0 "#PWR33" H 2500 2250 50  0001 C CNN
+F 0 "#PWR37" H 2500 2250 50  0001 C CNN
 F 1 "GND" H 2500 2350 50  0000 C CNN
 F 2 "" H 2500 2500 60  0000 C CNN
@@
 $EndComp
 $Comp
-L +24V #PWR32
+L +24V #PWR36
 U 1 1 56608476
 P 2500 2200
-F 0 "#PWR32" H 2500 2050 50  0001 C CNN
+F 0 "#PWR36" H 2500 2050 50  0001 C CNN
 F 1 "+24V" H 2500 2340 50  0000 C CNN
 F 2 "" H 2500 2200 60  0000 C CNN
@@
 	1    0    0    -1
 $EndComp
-$Comp
-L lm25011 U4
-U 1 1 570D946D
-P 4350 1550
-F 0 "U4" H 4350 2003 60  0000 C CNN
-F 1 "lm25011" H 4350 1897 60  0000 C CNN
-F 2 "" H 4350 1550 60  0001 C CNN
-F 3 "" H 4350 1550 60  0000 C CNN
-	1    4350 1550
-	1    0    0    -1
-$EndComp
 Wire Wire Line
 	1900 4900 2500 4900
 $Comp
-L GND #PWR21
+L GND #PWR25
 U 1 1 57744A84
 P 1900 5550
-F 0 "#PWR21" H 1900 5300 50  0001 C CNN
+F 0 "#PWR25" H 1900 5300 50  0001 C CNN
 F 1 "GND" H 1900 5400 50  0000 C CNN
 F 2 "" H 1900 5550 60  0000 C CNN
@@
 Connection ~ 2900 5500
 Connection ~ 3400 5500
+$Comp
+L ACT4088 U4
+U 1 1 5776D958
+P 4350 2250
+F 0 "U4" H 4200 2500 60  0000 C CNN
+F 1 "ACT4088" H 4350 2000 60  0000 C CNN
+F 2 "TO_SOT_Packages_SMD:SOT-23-6" H 4350 2250 60  0001 C CNN
+F 3 "" H 4350 2250 60  0000 C CNN
+	1    4350 2250
+	1    0    0    -1
+$EndComp
+$Comp
+L GND #PWR60
+U 1 1 5776DE81
+P 3850 2900
+F 0 "#PWR60" H 3850 2650 50  0001 C CNN
+F 1 "GND" H 3850 2750 50  0000 C CNN
+F 2 "" H 3850 2900 60  0000 C CNN
+F 3 "" H 3850 2900 60  0000 C CNN
+	1    3850 2900
+	1    0    0    -1
+$EndComp
+Wire Wire Line
+	6150 2800 3850 2800
+Wire Wire Line
+	3850 2400 3850 2900
+Wire Wire Line
+	3950 2400 3850 2400
+Connection ~ 3850 2800
+$Comp
+L +24V #PWR59
+U 1 1 5776DF85
+P 3850 2000
+F 0 "#PWR59" H 3850 1850 50  0001 C CNN
+F 1 "+24V" H 3850 2140 50  0000 C CNN
+F 2 "" H 3850 2000 60  0000 C CNN
+F 3 "" H 3850 2000 60  0000 C CNN
+	1    3850 2000
+	1    0    0    -1
+$EndComp
+Wire Wire Line
+	3850 2000 3850 2100
+Wire Wire Line
+	3850 2100 3950 2100
+$Comp
+L R R97
+U 1 1 5776E176
+P 5150 2550
+F 0 "R97" V 5230 2550 50  0000 C CNN
+F 1 "100k" V 5150 2550 50  0000 C CNN
+F 2 "Resistors_SMD:R_0603" V 5080 2550 30  0001 C CNN
+F 3 "" H 5150 2550 30  0000 C CNN
+	1    5150 2550
+	0    1    1    0
+$EndComp
+Wire Wire Line
+	5000 2550 4950 2550
+Wire Wire Line
+	4950 2550 4950 2400
+Connection ~ 4950 2400
+Wire Wire Line
+	5300 2550 5350 2550
+Wire Wire Line
+	5350 2550 5350 2400
+Connection ~ 5350 2400
+NoConn ~ 3950 2250
+$Comp
+L +5V #PWR114
+U 1 1 5776E9E0
+P 6250 2000
+F 0 "#PWR114" H 6250 1850 50  0001 C CNN
+F 1 "+5V" H 6250 2140 50  0000 C CNN
+F 2 "" H 6250 2000 50  0000 C CNN
+F 3 "" H 6250 2000 50  0000 C CNN
+	1    6250 2000
+	1    0    0    -1
+$EndComp
+Wire Wire Line
+	6150 2100 6250 2100
+Wire Wire Line
+	6250 2100 6250 2000
+Connection ~ 5550 2100
+Connection ~ 5550 2800
+Connection ~ 4850 2800
 $EndSCHEMATC

Commit message: v4.0
Parts:
- removed C35: 22n 16V, Capacitors_SMD:C_0603, symbol C
- removed C50: 22µ, Capacitors_SMD:C_0603, symbol C
- removed D9: B240A 60V 1A, symbol D_Schottky
- removed L1: 4.7µH 1.5A, symbol INDUCTOR
- removed R60: 10k, Resistors_SMD:R_0603, symbol R
- removed R74, R97: 100k, Resistors_SMD:R_0603, symbol R
- removed T11, T12, T4: testpoint, Measurement_Points:Measurement_Point_Round-SMD-Pad_Small, symbol testpoint
- removed U4: ACT4088, TO_SOT_Packages_SMD:SOT-23-6, symbol ACT4088
- added C? (x3): 10µ, Capacitors_SMD:C_0603, symbol C
- added C? (x13): 100n, Capacitors_SMD:C_0603, symbol C
- added D? (x2): B240A 60V 1A, symbol D_Schottky
- added L? (x2): 4.7µH 1.5A, symbol INDUCTOR
- added R? (x4): 100k, Resistors_SMD:R_0603, symbol R
- added R?: 3.9k, Resistors_SMD:R_0603, symbol R
- added R?: 10k, Resistors_SMD:R_0603, symbol R
- added U? (x2): ACT4088, TO_SOT_Packages_SMD:SOT-23-6, symbol ACT4088
Connections:
- net +24V: now also C?.1, C?.1, C?.1, C?.1, C?.1, C?.1, C?.1, U?.2 (IN), U?.2 (IN)
- net +3V3: now also C?.1
- net +5V: now also C?.1, C?.1, C?.1, C?.1, L?.2, R?.1, R?.1
- net GND: now also C?.2, C?.2, C?.2, C?.2, C?.2, C?.2, C?.2, C?.2, C?.2, C?.2, C?.2, C?.2, C?.2, C?.2, D?.2 (A), D?.2 (A), R?.2, R?.2, U?.5 (GND), U?.5 (GND)
- new net: R?.1, R?.2, R?.2, U?.4 (FB) (x2)
- new net: C?.2, D?.1 (K), L?.1, U?.1 (SW) (x2)
- new net: C?.1, U?.6 (BST) (x2)
- new net +12V: C?.1, C?.1, L?.2, R?.1, R?.1
- no-connect marks 1 -> 2
Other:
- moved on the sheet: C8, U2

Commit message: v4.0
Parts:
- added C120, C121, C122: 100n, Capacitors_SMD:C_0603, symbol C
- added C123, C124: 10µ, Capacitors_SMD:C_1206, symbol C
- added D13: B240A 60V 1A, symbol D_Schottky
- added L12: 4.7µH 1.5A, symbol INDUCTOR
- added R132: 10k, Resistors_SMD:R_0603, symbol R
- added R133, R134: 100k, Resistors_SMD:R_0603, symbol R
- added U28: ACT4088, TO_SOT_Packages_SMD:SOT-23-6, symbol ACT4088
- C109, C110, C111: renamed from C?; footprint Capacitors_SMD:C_0603 -> Capacitors_SMD:C_1206
- gave numbers to parts that had none: 25
Connections:
- net +24V: now also C120.1, U28.2 (IN)
- net GND: now also C120.2, C122.2, C123.2, C124.2, D13.2 (A), R132.2, U28.5 (GND)
- net EN_12V: now reaches U27.3 (EN)
- new net: R132.1, R133.2, R134.2, U28.4 (FB)
- new net: C121.2, D13.1 (K), L12.1, U28.1 (SW)
- new net: C121.1, U28.6 (BST)
- new net +5F: C122.1, C123.1, C124.1, L12.2, R133.1, R134.1
- new net EN_5V: U28.3 (EN)
- no-connect marks 2 -> 1
Other:
- note added: "CPU, IO and analog"
- note added: "FB and FAN"
- note added: "FB and RS485"
- moved on the sheet: C100, C101, C102, C104, C97, C98, P3
