File: hw/kicad/v4.0/supply.sch (KiCad schematic (older format))
At the start: 43 parts, among them P3 CONN_01X02, U13 ACT4088, U2 zldo1117, U27 ACT4088, U28 ACT4088

Commit message: v4.0
Parts:
- added JP?: Jumper_NO_Small, symbol Jumper_NO_Small
- U2: symbol LM7812 -> zldo1117
Connections:
- net +5F: now also JP?.1
- net +5V: now also JP?.2
Changed lines of the file:
@@
 $EndDescr
 $Comp
-L LM7812 U2
+L zldo1117 U2
 U 1 1 566074A9
 P 2700 4950
@@
 	3400 4800 3400 5100
 $Comp
-L +5V #PWR061
+L +5V #PWR060
 U 1 1 5660786F
 P 1900 4800
-F 0 "#PWR061" H 1900 4650 50  0001 C CNN
+F 0 "#PWR060" H 1900 4650 50  0001 C CNN
 F 1 "+5V" H 1900 4940 50  0000 C CNN
 F 2 "" H 1900 4800 60  0000 C CNN
@@
 $EndComp
 $Comp
-L +3.3V #PWR062
+L +3.3V #PWR061
 U 1 1 566078DE
 P 3400 4800
-F 0 "#PWR062" H 3400 4650 50  0001 C CNN
+F 0 "#PWR061" H 3400 4650 50  0001 C CNN
 F 1 "+3.3V" H 3400 4940 50  0000 C CNN
 F 2 "" H 3400 4800 60  0000 C CNN
@@
 Connection ~ 3400 4900
 $Comp
-L GND #PWR063
+L GND #PWR062
 U 1 1 5660843E
 P 2250 3400
-F 0 "#PWR063" H 2250 3150 50  0001 C CNN
+F 0 "#PWR062" H 2250 3150 50  0001 C CNN
 F 1 "GND" H 2250 3250 50  0000 C CNN
 F 2 "" H 2250 3400 60  0000 C CNN
@@
 $EndComp
 $Comp
-L +24V #PWR064
+L +24V #PWR063
 U 1 1 56608476
 P 2650 2900
-F 0 "#PWR064" H 2650 2750 50  0001 C CNN
+F 0 "#PWR063" H 2650 2750 50  0001 C CNN
 F 1 "+24V" H 2650 3040 50  0000 C CNN
 F 2 "" H 2650 2900 60  0000 C CNN
@@
 	1900 4900 2300 4900
 $Comp
-L GND #PWR065
+L GND #PWR064
 U 1 1 57744A84
 P 1900 5550
-F 0 "#PWR065" H 1900 5300 50  0001 C CNN
+F 0 "#PWR064" H 1900 5300 50  0001 C CNN
 F 1 "GND" H 1900 5400 50  0000 C CNN
 F 2 "" H 1900 5550 60  0000 C CNN
@@
 Connection ~ 6600 4800
 $Comp
-L GND #PWR066
+L GND #PWR065
 U 1 1 57AD27D2
 P 4300 5600
-F 0 "#PWR066" H 4300 5350 50  0001 C CNN
+F 0 "#PWR065" H 4300 5350 50  0001 C CNN
 F 1 "GND" H 4300 5450 50  0000 C CNN
 F 2 "" H 4300 5600 60  0000 C CNN
@@
 Connection ~ 4300 5500
 $Comp
-L +24V #PWR067
+L +24V #PWR066
 U 1 1 57AD27DC
 P 4300 4700
-F 0 "#PWR067" H 4300 4550 50  0001 C CNN
+F 0 "#PWR066" H 4300 4550 50  0001 C CNN
 F 1 "+24V" H 4300 4840 50  0000 C CNN
 F 2 "" H 4300 4700 60  0000 C CNN
@@
 $EndComp
 $Comp
-L GND #PWR068
+L GND #PWR067
 U 1 1 57AD3DDA
 P 4300 3800
-F 0 "#PWR068" H 4300 3550 50  0001 C CNN
+F 0 "#PWR067" H 4300 3550 50  0001 C CNN
 F 1 "GND" H 4300 3650 50  0000 C CNN
 F 2 "" H 4300 3800 60  0000 C CNN
@@
 Connection ~ 4300 3700
 $Comp
-L +24V #PWR069
+L +24V #PWR068
 U 1 1 57AD3DE4
 P 4300 2900
-F 0 "#PWR069" H 4300 2750 50  0001 C CNN
+F 0 "#PWR068" H 4300 2750 50  0001 C CNN
 F 1 "+24V" H 4300 3040 50  0000 C CNN
 F 2 "" H 4300 2900 60  0000 C CNN
@@
 NoConn ~ 4400 3150
 $Comp
-L +5V #PWR070
+L +5V #PWR069
 U 1 1 57AD3DF9
 P 6700 2900
-F 0 "#PWR070" H 6700 2750 50  0001 C CNN
+F 0 "#PWR069" H 6700 2750 50  0001 C CNN
 F 1 "+5V" H 6700 3040 50  0000 C CNN
 F 2 "" H 6700 2900 50  0000 C CNN
@@
 	6600 3000 6700 3000
 $Comp
-L +12V #PWR071
+L +12V #PWR070
 U 1 1 57AD61BC
 P 6700 4700
-F 0 "#PWR071" H 6700 4550 50  0001 C CNN
+F 0 "#PWR070" H 6700 4550 50  0001 C CNN
 F 1 "+12V" H 6700 4840 50  0000 C CNN
 F 2 "" H 6700 4700 50  0000 C CNN
@@
 $EndComp
 $Comp
-L GND #PWR072
+L GND #PWR071
 U 1 1 57B218AB
 P 2650 3400
-F 0 "#PWR072" H 2650 3150 50  0001 C CNN
+F 0 "#PWR071" H 2650 3150 50  0001 C CNN
 F 1 "GND" H 2650 3250 50  0000 C CNN
 F 2 "" H 2650 3400 60  0000 C CNN
@@
 $EndComp
 $Comp
-L +24V #PWR073
+L +24V #PWR072
 U 1 1 57B21AA8
 P 2250 3100
-F 0 "#PWR073" H 2250 2950 50  0001 C CNN
+F 0 "#PWR072" H 2250 2950 50  0001 C CNN
 F 1 "+24V" H 2250 3240 50  0000 C CNN
 F 2 "" H 2250 3100 60  0000 C CNN
@@
 $EndComp
 $Comp
-L GND #PWR074
+L GND #PWR073
 U 1 1 57D63C3E
 P 4300 2300
-F 0 "#PWR074" H 4300 2050 50  0001 C CNN
+F 0 "#PWR073" H 4300 2050 50  0001 C CNN
 F 1 "GND" H 4300 2150 50  0000 C CNN
 F 2 "" H 4300 2300 60  0000 C CNN
@@
 Connection ~ 4300 2200
 $Comp
-L +24V #PWR075
+L +24V #PWR074
 U 1 1 57D63C47
 P 4300 1400
-F 0 "#PWR075" H 4300 1250 50  0001 C CNN
+F 0 "#PWR074" H 4300 1250 50  0001 C CNN
 F 1 "+24V" H 4300 1540 50  0000 C CNN
 F 2 "" H 4300 1400 60  0000 C CNN
@@
 Connection ~ 6600 2200
 $Comp
-L +5F #PWR076
+L +5F #PWR075
 U 1 1 57D6418F
 P 6700 1400
-F 0 "#PWR076" H 6700 1250 50  0001 C CNN
+F 0 "#PWR075" H 6700 1250 50  0001 C CNN
 F 1 "+5F" H 6700 1540 50  0000 C CNN
 F 2 "" H 6700 1400 50  0000 C CNN
@@
 Text Notes 6850 1300 0    60   ~ 0
 FB and RS485
+$Comp
+L Jumper_NO_Small JP?
+U 1 1 57D95B7C
+P 8400 1800
+F 0 "JP?" H 8400 1880 50  0000 C CNN
+F 1 "Jumper_NO_Small" H 8410 1740 50  0001 C CNN
+F 2 "" H 8400 1800 50  0000 C CNN
+F 3 "" H 8400 1800 50  0000 C CNN
+	1    8400 1800
+	1    0    0    -1
+$EndComp
+$Comp
+L +5F #PWR?
+U 1 1 57D95C13
+P 8200 1700
+F 0 "#PWR?" H 8200 1550 50  0001 C CNN
+F 1 "+5F" H 8200 1840 50  0000 C CNN
+F 2 "" H 8200 1700 50  0000 C CNN
+F 3 "" H 8200 1700 50  0000 C CNN
+	1    8200 1700
+	1    0    0    -1
+$EndComp
+$Comp
+L +5V #PWR?
+U 1 1 57D95CA2
+P 8600 1700
+F 0 "#PWR?" H 8600 1550 50  0001 C CNN
+F 1 "+5V" H 8600 1840 50  0000 C CNN
+F 2 "" H 8600 1700 50  0000 C CNN
+F 3 "" H 8600 1700 50  0000 C CNN
+	1    8600 1700
+	1    0    0    -1
+$EndComp
+Wire Wire Line
+	8600 1700 8600 1800
+Wire Wire Line
+	8600 1800 8500 1800
+Wire Wire Line
+	8300 1800 8200 1800
+Wire Wire Line
+	8200 1800 8200 1700
 $EndSCHEMATC

Commit message: v4.0
Parts:
- gave numbers to parts that had none: 1
Changed lines of the file:
@@
 	3400 4800 3400 5100
 $Comp
-L +5V #PWR060
+L +5V #PWR063
 U 1 1 5660786F
 P 1900 4800
-F 0 "#PWR060" H 1900 4650 50  0001 C CNN
+F 0 "#PWR063" H 1900 4650 50  0001 C CNN
 F 1 "+5V" H 1900 4940 50  0000 C CNN
 F 2 "" H 1900 4800 60  0000 C CNN
@@
 $EndComp
 $Comp
-L +3.3V #PWR061
+L +3.3V #PWR064
 U 1 1 566078DE
 P 3400 4800
-F 0 "#PWR061" H 3400 4650 50  0001 C CNN
+F 0 "#PWR064" H 3400 4650 50  0001 C CNN
 F 1 "+3.3V" H 3400 4940 50  0000 C CNN
 F 2 "" H 3400 4800 60  0000 C CNN
@@
 Connection ~ 3400 4900
 $Comp
-L GND #PWR062
+L GND #PWR065
 U 1 1 5660843E
 P 2250 3400
-F 0 "#PWR062" H 2250 3150 50  0001 C CNN
+F 0 "#PWR065" H 2250 3150 50  0001 C CNN
 F 1 "GND" H 2250 3250 50  0000 C CNN
 F 2 "" H 2250 3400 60  0000 C CNN
@@
 $EndComp
 $Comp
-L +24V #PWR063
+L +24V #PWR066
 U 1 1 56608476
 P 2650 2900
-F 0 "#PWR063" H 2650 2750 50  0001 C CNN
+F 0 "#PWR066" H 2650 2750 50  0001 C CNN
 F 1 "+24V" H 2650 3040 50  0000 C CNN
 F 2 "" H 2650 2900 60  0000 C CNN
@@
 	1900 4900 2300 4900
 $Comp
-L GND #PWR064
+L GND #PWR067
 U 1 1 57744A84
 P 1900 5550
-F 0 "#PWR064" H 1900 5300 50  0001 C CNN
+F 0 "#PWR067" H 1900 5300 50  0001 C CNN
 F 1 "GND" H 1900 5400 50  0000 C CNN
 F 2 "" H 1900 5550 60  0000 C CNN
@@
 Connection ~ 6600 4800
 $Comp
-L GND #PWR065
+L GND #PWR068
 U 1 1 57AD27D2
 P 4300 5600
-F 0 "#PWR065" H 4300 5350 50  0001 C CNN
+F 0 "#PWR068" H 4300 5350 50  0001 C CNN
 F 1 "GND" H 4300 5450 50  0000 C CNN
 F 2 "" H 4300 5600 60  0000 C CNN
@@
 Connection ~ 4300 5500
 $Comp
-L +24V #PWR066
+L +24V #PWR069
 U 1 1 57AD27DC
 P 4300 4700
-F 0 "#PWR066" H 4300 4550 50  0001 C CNN
+F 0 "#PWR069" H 4300 4550 50  0001 C CNN
 F 1 "+24V" H 4300 4840 50  0000 C CNN
 F 2 "" H 4300 4700 60  0000 C CNN
@@
 $EndComp
 $Comp
-L GND #PWR067
+L GND #PWR070
 U 1 1 57AD3DDA
 P 4300 3800
-F 0 "#PWR067" H 4300 3550 50  0001 C CNN
+F 0 "#PWR070" H 4300 3550 50  0001 C CNN
 F 1 "GND" H 4300 3650 50  0000 C CNN
 F 2 "" H 4300 3800 60  0000 C CNN
@@
 Connection ~ 4300 3700
 $Comp
-L +24V #PWR068
+L +24V #PWR071
 U 1 1 57AD3DE4
 P 4300 2900
-F 0 "#PWR068" H 4300 2750 50  0001 C CNN
+F 0 "#PWR071" H 4300 2750 50  0001 C CNN
 F 1 "+24V" H 4300 3040 50  0000 C CNN
 F 2 "" H 4300 2900 60  0000 C CNN
@@
 NoConn ~ 4400 3150
 $Comp
-L +5V #PWR069
+L +5V #PWR072
 U 1 1 57AD3DF9
 P 6700 2900
-F 0 "#PWR069" H 6700 2750 50  0001 C CNN
+F 0 "#PWR072" H 6700 2750 50  0001 C CNN
 F 1 "+5V" H 6700 3040 50  0000 C CNN
 F 2 "" H 6700 2900 50  0000 C CNN
@@
 	6600 3000 6700 3000
 $Comp
-L +12V #PWR070
+L +12V #PWR073
 U 1 1 57AD61BC
 P 6700 4700
-F 0 "#PWR070" H 6700 4550 50  0001 C CNN
+F 0 "#PWR073" H 6700 4550 50  0001 C CNN
 F 1 "+12V" H 6700 4840 50  0000 C CNN
 F 2 "" H 6700 4700 50  0000 C CNN
@@
 $EndComp
 $Comp
-L GND #PWR071
+L GND #PWR074
 U 1 1 57B218AB
 P 2650 3400
-F 0 "#PWR071" H 2650 3150 50  0001 C CNN
+F 0 "#PWR074" H 2650 3150 50  0001 C CNN
 F 1 "GND" H 2650 3250 50  0000 C CNN
 F 2 "" H 2650 3400 60  0000 C CNN
@@
 $EndComp
 $Comp
-L +24V #PWR072
+L +24V #PWR075
 U 1 1 57B21AA8
 P 2250 3100
-F 0 "#PWR072" H 2250 2950 50  0001 C CNN
+F 0 "#PWR075" H 2250 2950 50  0001 C CNN
 F 1 "+24V" H 2250 3240 50  0000 C CNN
 F 2 "" H 2250 3100 60  0000 C CNN
@@
 $EndComp
 $Comp
-L GND #PWR073
+L GND #PWR076
 U 1 1 57D63C3E
 P 4300 2300
-F 0 "#PWR073" H 4300 2050 50  0001 C CNN
+F 0 "#PWR076" H 4300 2050 50  0001 C CNN
 F 1 "GND" H 4300 2150 50  0000 C CNN
 F 2 "" H 4300 2300 60  0000 C CNN
@@
 Connection ~ 4300 2200
 $Comp
-L +24V #PWR074
+L +24V #PWR077
 U 1 1 57D63C47
 P 4300 1400
-F 0 "#PWR074" H 4300 1250 50  0001 C CNN
+F 0 "#PWR077" H 4300 1250 50  0001 C CNN
 F 1 "+24V" H 4300 1540 50  0000 C CNN
 F 2 "" H 4300 1400 60  0000 C CNN
@@
 Connection ~ 6600 2200
 $Comp
-L +5F #PWR075
+L +5F #PWR078
 U 1 1 57D6418F
 P 6700 1400
-F 0 "#PWR075" H 6700 1250 50  0001 C CNN
+F 0 "#PWR078" H 6700 1250 50  0001 C CNN
 F 1 "+5F" H 6700 1540 50  0000 C CNN
 F 2 "" H 6700 1400 50  0000 C CNN
@@
 FB and RS485
 $Comp
-L Jumper_NO_Small JP?
+L Jumper_NO_Small JP4
 U 1 1 57D95B7C
 P 8400 1800
-F 0 "JP?" H 8400 1880 50  0000 C CNN
+F 0 "JP4" H 8400 1880 50  0000 C CNN
 F 1 "Jumper_NO_Small" H 8410 1740 50  0001 C CNN
-F 2 "" H 8400 1800 50  0000 C CNN
+F 2 "" H 8400 1800 50  0001 C CNN
 F 3 "" H 8400 1800 50  0000 C CNN
 	1    8400 1800
@@
 $EndComp
 $Comp
-L +5F #PWR?
+L +5F #PWR079
 U 1 1 57D95C13
 P 8200 1700
-F 0 "#PWR?" H 8200 1550 50  0001 C CNN
+F 0 "#PWR079" H 8200 1550 50  0001 C CNN
 F 1 "+5F" H 8200 1840 50  0000 C CNN
 F 2 "" H 8200 1700 50  0000 C CNN
@@
 $EndComp
 $Comp
-L +5V #PWR?
+L +5V #PWR080
 U 1 1 57D95CA2
 P 8600 1700
-F 0 "#PWR?" H 8600 1550 50  0001 C CNN
+F 0 "#PWR080" H 8600 1550 50  0001 C CNN
 F 1 "+5V" H 8600 1840 50  0000 C CNN
 F 2 "" H 8600 1700 50  0000 C CNN

Commit message: v4.0
Parts:
- removed R120, R134, R74: 100k, Resistors_SMD:R_0603, symbol R
- D12, D13, D9: footprint (none) -> Diodes_SMD:SMA_Standard
- L12, L5, L6: footprint (none) -> stmbl:SMD_INDUCTOR_32x25
- R133, R60, R97: value 100k -> 50k
Changed lines of the file:
@@
 	3400 4800 3400 5100
 $Comp
-L +5V #PWR063
+L +5V #PWR062
 U 1 1 5660786F
 P 1900 4800
-F 0 "#PWR063" H 1900 4650 50  0001 C CNN
+F 0 "#PWR062" H 1900 4650 50  0001 C CNN
 F 1 "+5V" H 1900 4940 50  0000 C CNN
 F 2 "" H 1900 4800 60  0000 C CNN
@@
 $EndComp
 $Comp
-L +3.3V #PWR064
+L +3.3V #PWR063
 U 1 1 566078DE
 P 3400 4800
-F 0 "#PWR064" H 3400 4650 50  0001 C CNN
+F 0 "#PWR063" H 3400 4650 50  0001 C CNN
 F 1 "+3.3V" H 3400 4940 50  0000 C CNN
 F 2 "" H 3400 4800 60  0000 C CNN
@@
 Connection ~ 3400 4900
 $Comp
-L GND #PWR065
+L GND #PWR064
 U 1 1 5660843E
 P 2250 3400
-F 0 "#PWR065" H 2250 3150 50  0001 C CNN
+F 0 "#PWR064" H 2250 3150 50  0001 C CNN
 F 1 "GND" H 2250 3250 50  0000 C CNN
 F 2 "" H 2250 3400 60  0000 C CNN
@@
 $EndComp
 $Comp
-L +24V #PWR066
+L +24V #PWR065
 U 1 1 56608476
 P 2650 2900
-F 0 "#PWR066" H 2650 2750 50  0001 C CNN
+F 0 "#PWR065" H 2650 2750 50  0001 C CNN
 F 1 "+24V" H 2650 3040 50  0000 C CNN
 F 2 "" H 2650 2900 60  0000 C CNN
@@
 	1900 4900 2300 4900
 $Comp
-L GND #PWR067
+L GND #PWR066
 U 1 1 57744A84
 P 1900 5550
-F 0 "#PWR067" H 1900 5300 50  0001 C CNN
+F 0 "#PWR066" H 1900 5300 50  0001 C CNN
 F 1 "GND" H 1900 5400 50  0000 C CNN
 F 2 "" H 1900 5550 60  0000 C CNN
@@
 P 5600 5100
 F 0 "R97" V 5680 5100 50  0000 C CNN
-F 1 "100k" V 5600 5100 50  0000 C CNN
+F 1 "50k" V 5600 5100 50  0000 C CNN
 F 2 "Resistors_SMD:R_0603" V 5530 5100 30  0001 C CNN
 F 3 "" H 5600 5100 30  0000 C CNN
@@
 F 0 "D12" H 6000 5450 50  0000 C CNN
 F 1 "B240A 60V 1A" H 6000 5250 50  0000 C CNN
-F 2 "" H 6000 5350 60  0001 C CNN
+F 2 "Diodes_SMD:SMA_Standard" H 6000 5350 60  0001 C CNN
 F 3 "" H 6000 5350 60  0000 C CNN
 	1    6000 5350
@@
 F 0 "L6" V 6250 4800 50  0000 C CNN
 F 1 "4.7µH 1.5A" V 6400 4800 50  0000 C CNN
-F 2 "" H 6300 4800 60  0001 C CNN
+F 2 "stmbl:SMD_INDUCTOR_32x25" H 6300 4800 60  0001 C CNN
 F 3 "" H 6300 4800 60  0000 C CNN
 	1    6300 4800
@@
 Connection ~ 6600 4800
 $Comp
-L GND #PWR068
+L GND #PWR067
 U 1 1 57AD27D2
 P 4300 5600
-F 0 "#PWR068" H 4300 5350 50  0001 C CNN
+F 0 "#PWR067" H 4300 5350 50  0001 C CNN
 F 1 "GND" H 4300 5450 50  0000 C CNN
 F 2 "" H 4300 5600 60  0000 C CNN
@@
 Connection ~ 4300 5500
 $Comp
-L +24V #PWR069
+L +24V #PWR068
 U 1 1 57AD27DC
 P 4300 4700
-F 0 "#PWR069" H 4300 4550 50  0001 C CNN
+F 0 "#PWR068" H 4300 4550 50  0001 C CNN
 F 1 "+24V" H 4300 4840 50  0000 C CNN
 F 2 "" H 4300 4700 60  0000 C CNN
@@
 Wire Wire Line
 	3700 4800 4400 4800
-$Comp
-L R R120
-U 1 1 57AD27E4
-P 5600 5250
-F 0 "R120" V 5680 5250 50  0000 C CNN
-F 1 "100k" V 5600 5250 50  0000 C CNN
-F 2 "Resistors_SMD:R_0603" V 5530 5250 30  0001 C CNN
-F 3 "" H 5600 5250 30  0000 C CNN
-	1    5600 5250
-	0    1    1    0
-$EndComp
-Wire Wire Line
-	5450 5250 5400 5250
-Wire Wire Line
-	5400 5250 5400 5100
-Connection ~ 5400 5100
-Wire Wire Line
-	5750 5250 5800 5250
-Wire Wire Line
-	5800 5250 5800 5100
-Connection ~ 5800 5100
 Wire Wire Line
 	6600 4800 6700 4800
@@
 P 5600 3300
 F 0 "R60" V 5680 3300 50  0000 C CNN
-F 1 "100k" V 5600 3300 50  0000 C CNN
+F 1 "50k" V 5600 3300 50  0000 C CNN
 F 2 "Resistors_SMD:R_0603" V 5530 3300 30  0001 C CNN
 F 3 "" H 5600 3300 30  0000 C CNN
@@
 F 0 "D9" H 6000 3650 50  0000 C CNN
 F 1 "B240A 60V 1A" H 6000 3450 50  0000 C CNN
-F 2 "" H 6000 3550 60  0001 C CNN
+F 2 "Diodes_SMD:SMA_Standard" H 6000 3550 60  0001 C CNN
 F 3 "" H 6000 3550 60  0000 C CNN
 	1    6000 3550
@@
 F 0 "L5" V 6250 3000 50  0000 C CNN
 F 1 "4.7µH 1.5A" V 6400 3000 50  0000 C CNN
-F 2 "" H 6300 3000 60  0001 C CNN
+F 2 "stmbl:SMD_INDUCTOR_32x25" H 6300 3000 60  0001 C CNN
 F 3 "" H 6300 3000 60  0000 C CNN
 	1    6300 3000
@@
 $EndComp
 $Comp
-L GND #PWR070
+L GND #PWR069
 U 1 1 57AD3DDA
 P 4300 3800
-F 0 "#PWR070" H 4300 3550 50  0001 C CNN
+F 0 "#PWR069" H 4300 3550 50  0001 C CNN
 F 1 "GND" H 4300 3650 50  0000 C CNN
 F 2 "" H 4300 3800 60  0000 C CNN
@@
 Connection ~ 4300 3700
 $Comp
-L +24V #PWR071
+L +24V #PWR070
 U 1 1 57AD3DE4
 P 4300 2900
-F 0 "#PWR071" H 4300 2750 50  0001 C CNN
+F 0 "#PWR070" H 4300 2750 50  0001 C CNN
 F 1 "+24V" H 4300 3040 50  0000 C CNN
 F 2 "" H 4300 2900 60  0000 C CNN
@@
 Wire Wire Line
 	4100 3000 4400 3000
-$Comp
-L R R74
-U 1 1 57AD3DEC
-P 5600 3450
-F 0 "R74" V 5680 3450 50  0000 C CNN
-F 1 "100k" V 5600 3450 50  0000 C CNN
-F 2 "Resistors_SMD:R_0603" V 5530 3450 30  0001 C CNN
-F 3 "" H 5600 3450 30  0000 C CNN
-	1    5600 3450
-	0    1    1    0
-$EndComp
-Wire Wire Line
-	5450 3450 5400 3450
-Wire Wire Line
-	5400 3450 5400 3300
-Connection ~ 5400 3300
-Wire Wire Line
-	5750 3450 5800 3450
-Wire Wire Line
-	5800 3450 5800 3300
-Connection ~ 5800 3300
 NoConn ~ 4400 3150
 $Comp
-L +5V #PWR072
+L +5V #PWR071
 U 1 1 57AD3DF9
 P 6700 2900
-F 0 "#PWR072" H 6700 2750 50  0001 C CNN
+F 0 "#PWR071" H 6700 2750 50  0001 C CNN
 F 1 "+5V" H 6700 3040 50  0000 C CNN
 F 2 "" H 6700 2900 50  0000 C CNN
@@
 	6600 3000 6700 3000
 $Comp
-L +12V #PWR073
+L +12V #PWR072
 U 1 1 57AD61BC
 P 6700 4700
-F 0 "#PWR073" H 6700 4550 50  0001 C CNN
+F 0 "#PWR072" H 6700 4550 50  0001 C CNN
 F 1 "+12V" H 6700 4840 50  0000 C CNN
 F 2 "" H 6700 4700 50  0000 C CNN
@@
 $EndComp
 $Comp
-L GND #PWR074
+L GND #PWR073
 U 1 1 57B218AB
 P 2650 3400
-F 0 "#PWR074" H 2650 3150 50  0001 C CNN
+F 0 "#PWR073" H 2650 3150 50  0001 C CNN
 F 1 "GND" H 2650 3250 50  0000 C CNN
 F 2 "" H 2650 3400 60  0000 C CNN
@@
 $EndComp
 $Comp
-L +24V #PWR075
+L +24V #PWR074
 U 1 1 57B21AA8
 P 2250 3100
-F 0 "#PWR075" H 2250 2950 50  0001 C CNN
+F 0 "#PWR074" H 2250 2950 50  0001 C CNN
 F 1 "+24V" H 2250 3240 50  0000 C CNN
 F 2 "" H 2250 3100 60  0000 C CNN
@@
 P 5600 1800
 F 0 "R133" V 5680 1800 50  0000 C CNN
-F 1 "100k" V 5600 1800 50  0000 C CNN
+F 1 "50k" V 5600 1800 50  0000 C CNN
 F 2 "Resistors_SMD:R_0603" V 5530 1800 30  0001 C CNN
 F 3 "" H 5600 1800 30  0000 C CNN
@@
 F 0 "D13" H 6000 2150 50  0000 C CNN
 F 1 "B240A 60V 1A" H 6000 1950 50  0000 C CNN
-F 2 "" H 6000 2050 60  0001 C CNN
+F 2 "Diodes_SMD:SMA_Standard" H 6000 2050 60  0001 C CNN
 F 3 "" H 6000 2050 60  0000 C CNN
 	1    6000 2050
@@
 F 0 "L12" V 6250 1500 50  0000 C CNN
 F 1 "4.7µH 1.5A" V 6400 1500 50  0000 C CNN
-F 2 "" H 6300 1500 60  0001 C CNN
+F 2 "stmbl:SMD_INDUCTOR_32x25" H 6300 1500 60  0001 C CNN
 F 3 "" H 6300 1500 60  0000 C CNN
 	1    6300 1500
@@
 $EndComp
 $Comp
-L GND #PWR076
+L GND #PWR075
 U 1 1 57D63C3E
 P 4300 2300
-F 0 "#PWR076" H 4300 2050 50  0001 C CNN
+F 0 "#PWR075" H 4300 2050 50  0001 C CNN
 F 1 "GND" H 4300 2150 50  0000 C CNN
 F 2 "" H 4300 2300 60  0000 C CNN
@@
 Connection ~ 4300 2200
 $Comp
-L +24V #PWR077
+L +24V #PWR076
 U 1 1 57D63C47
 P 4300 1400
-F 0 "#PWR077" H 4300 1250 50  0001 C CNN
+F 0 "#PWR076" H 4300 1250 50  0001 C CNN
 F 1 "+24V" H 4300 1540 50  0000 C CNN
 F 2 "" H 4300 1400 60  0000 C CNN
@@
 Wire Wire Line
 	3800 1500 4400 1500
-$Comp
-L R R134
-U 1 1 57D63C4F
-P 5600 1950
-F 0 "R134" V 5680 1950 50  0000 C CNN
-F 1 "100k" V 5600 1950 50  0000 C CNN
-F 2 "Resistors_SMD:R_0603" V 5530 1950 30  0001 C CNN
-F 3 "" H 5600 1950 30  0000 C CNN
-	1    5600 1950
-	0    1    1    0
-$EndComp
-Wire Wire Line
-	5450 1950 5400 1950
-Wire Wire Line
-	5400 1950 5400 1800
-Connection ~ 5400 1800
-Wire Wire Line
-	5750 1950 5800 1950
-Wire Wire Line
-	5800 1950 5800 1800
-Connection ~ 5800 1800
 Wire Wire Line
 	6700 1500 6700 1400
@@
 Connection ~ 6600 2200
 $Comp
-L +5F #PWR078
+L +5F #PWR077
 U 1 1 57D6418F
 P 6700 1400
-F 0 "#PWR078" H 6700 1250 50  0001 C CNN
+F 0 "#PWR077" H 6700 1250 50  0001 C CNN
 F 1 "+5F" H 6700 1540 50  0000 C CNN
 F 2 "" H 6700 1400 50  0000 C CNN
@@
 $EndComp
 $Comp
-L +5F #PWR079
+L +5F #PWR078
 U 1 1 57D95C13
 P 8200 1700
-F 0 "#PWR079" H 8200 1550 50  0001 C CNN
+F 0 "#PWR078" H 8200 1550 50  0001 C CNN
 F 1 "+5F" H 8200 1840 50  0000 C CNN
 F 2 "" H 8200 1700 50  0000 C CNN
@@
 $EndComp
 $Comp
-L +5V #PWR080
+L +5V #PWR079
 U 1 1 57D95CA2
 P 8600 1700
-F 0 "#PWR080" H 8600 1550 50  0001 C CNN
+F 0 "#PWR079" H 8600 1550 50  0001 C CNN
 F 1 "+5V" H 8600 1840 50  0000 C CNN
 F 2 "" H 8600 1700 50  0000 C CNN
