File: hw/kicad/v4.0/f4.sch (KiCad schematic (older format))
At the start: 32 parts, among them P1 USB_OTG, U1 USBLC6-4SC6, U26 STM32F405VG, Y2 8M

Commit message: v4.0
Parts:
- removed C91: 100n, Capacitors_SMD:C_0603, symbol C
- C1, C119, C16, C29, C31, C32, C64, C65, C77, C80, C81, C84, C85, C86, C87, C88, C89, C90: footprint Capacitors_SMD:C_0603 -> stmbl:C_0603
- L3, R1, R116, R117, R121, R122, R61: footprint Resistors_SMD:R_0603 -> stmbl:R_0603

Commit message: v4.0
Parts:
- added R15, R16: 22, stmbl:R_0603, symbol R
Connections:
- net at U1.3 (I/O2), U26.70 (PA11/USART1_CTS/CAN1_RX/TIM1_CH4_/OTG_FS_DM/EVENTOUT): now also R15.1; no longer P1.2 (D-)
- net at U1.1 (I/O1), U26.71 (PA12/USART1_RTS/CAN1_TX/TIM1_ETR/OTG_FS_DP/EVENTOUT): now also R16.1; no longer P1.3 (D+)
- new net: P1.2 (D-), R15.2
- new net: P1.3 (D+), R16.2
Changed lines of the file:
@@
 $EndComp
 $Comp
-L GND #PWR0139
+L GND #PWR0140
 U 1 1 565FE0C3
 P 4400 4000
-F 0 "#PWR0139" H 4400 3750 50  0001 C CNN
+F 0 "#PWR0140" H 4400 3750 50  0001 C CNN
 F 1 "GND" H 4400 3850 50  0000 C CNN
 F 2 "" H 4400 4000 60  0000 C CNN
@@
 $EndComp
 $Comp
-L GND #PWR0140
+L GND #PWR0141
 U 1 1 565FE0E1
 P 4400 3400
-F 0 "#PWR0140" H 4400 3150 50  0001 C CNN
+F 0 "#PWR0141" H 4400 3150 50  0001 C CNN
 F 1 "GND" H 4400 3250 50  0000 C CNN
 F 2 "" H 4400 3400 60  0000 C CNN
@@
 $EndComp
 $Comp
-L GND #PWR0141
+L GND #PWR0142
 U 1 1 565FE268
 P 10600 8600
-F 0 "#PWR0141" H 10600 8350 50  0001 C CNN
+F 0 "#PWR0142" H 10600 8350 50  0001 C CNN
 F 1 "GND" H 10600 8450 50  0000 C CNN
 F 2 "" H 10600 8600 60  0000 C CNN
@@
 $EndComp
 $Comp
-L GND #PWR0142
+L GND #PWR0143
 U 1 1 565FE28C
 P 10400 8600
-F 0 "#PWR0142" H 10400 8350 50  0001 C CNN
+F 0 "#PWR0143" H 10400 8350 50  0001 C CNN
 F 1 "GND" H 10400 8450 50  0000 C CNN
 F 2 "" H 10400 8600 60  0000 C CNN
@@
 $EndComp
 $Comp
-L GND #PWR0143
+L GND #PWR0144
 U 1 1 565FE2A9
 P 10200 8600
-F 0 "#PWR0143" H 10200 8350 50  0001 C CNN
+F 0 "#PWR0144" H 10200 8350 50  0001 C CNN
 F 1 "GND" H 10200 8450 50  0000 C CNN
 F 2 "" H 10200 8600 60  0000 C CNN
@@
 $EndComp
 $Comp
-L GND #PWR0144
+L GND #PWR0145
 U 1 1 565FE2C6
 P 10000 8600
-F 0 "#PWR0144" H 10000 8350 50  0001 C CNN
+F 0 "#PWR0145" H 10000 8350 50  0001 C CNN
 F 1 "GND" H 10000 8450 50  0000 C CNN
 F 2 "" H 10000 8600 60  0000 C CNN
@@
 $EndComp
 $Comp
-L GND #PWR0145
+L GND #PWR0146
 U 1 1 565FE2E3
 P 9800 8600
-F 0 "#PWR0145" H 9800 8350 50  0001 C CNN
+F 0 "#PWR0146" H 9800 8350 50  0001 C CNN
 F 1 "GND" H 9800 8450 50  0000 C CNN
 F 2 "" H 9800 8600 60  0000 C CNN
@@
 $EndComp
 $Comp
-L GND #PWR0146
+L GND #PWR0147
 U 1 1 565FE300
 P 11100 9000
-F 0 "#PWR0146" H 11100 8750 50  0001 C CNN
+F 0 "#PWR0147" H 11100 8750 50  0001 C CNN
 F 1 "GND" H 11100 8850 50  0000 C CNN
 F 2 "" H 11100 9000 60  0000 C CNN
@@
 $EndComp
 $Comp
-L GND #PWR0147
+L GND #PWR0148
 U 1 1 565FE31D
 P 11600 9000
-F 0 "#PWR0147" H 11600 8750 50  0001 C CNN
+F 0 "#PWR0148" H 11600 8750 50  0001 C CNN
 F 1 "GND" H 11600 8850 50  0000 C CNN
 F 2 "" H 11600 9000 60  0000 C CNN
@@
 $EndComp
 $Comp
-L +3.3V #PWR0148
+L +3.3V #PWR0149
 U 1 1 565FEC9D
 P 11800 2300
-F 0 "#PWR0148" H 11800 2150 50  0001 C CNN
+F 0 "#PWR0149" H 11800 2150 50  0001 C CNN
 F 1 "+3.3V" H 11800 2440 50  0000 C CNN
 F 2 "" H 11800 2300 60  0000 C CNN
@@
 $EndComp
 $Comp
-L GND #PWR0149
+L GND #PWR0150
 U 1 1 565FECDB
 P 11400 1900
-F 0 "#PWR0149" H 11400 1650 50  0001 C CNN
+F 0 "#PWR0150" H 11400 1650 50  0001 C CNN
 F 1 "GND" H 11400 1750 50  0000 C CNN
 F 2 "" H 11400 1900 60  0000 C CNN
@@
 $EndComp
 $Comp
-L GND #PWR0150
+L GND #PWR0151
 U 1 1 565FED17
 P 10900 1900
-F 0 "#PWR0150" H 10900 1650 50  0001 C CNN
+F 0 "#PWR0151" H 10900 1650 50  0001 C CNN
 F 1 "GND" H 10900 1750 50  0000 C CNN
 F 2 "" H 10900 1900 60  0000 C CNN
@@
 $EndComp
 $Comp
-L GND #PWR0151
+L GND #PWR0152
 U 1 1 565FED4C
 P 10600 1900
-F 0 "#PWR0151" H 10600 1650 50  0001 C CNN
+F 0 "#PWR0152" H 10600 1650 50  0001 C CNN
 F 1 "GND" H 10600 1750 50  0000 C CNN
 F 2 "" H 10600 1900 60  0000 C CNN
@@
 $EndComp
 $Comp
-L GND #PWR0152
+L GND #PWR0153
 U 1 1 565FED81
 P 10300 1900
-F 0 "#PWR0152" H 10300 1650 50  0001 C CNN
+F 0 "#PWR0153" H 10300 1650 50  0001 C CNN
 F 1 "GND" H 10300 1750 50  0000 C CNN
 F 2 "" H 10300 1900 60  0000 C CNN
@@
 $EndComp
 $Comp
-L GND #PWR0153
+L GND #PWR0154
 U 1 1 565FEDB6
 P 10000 1900
-F 0 "#PWR0153" H 10000 1650 50  0001 C CNN
+F 0 "#PWR0154" H 10000 1650 50  0001 C CNN
 F 1 "GND" H 10000 1750 50  0000 C CNN
 F 2 "" H 10000 1900 60  0000 C CNN
@@
 $EndComp
 $Comp
-L GND #PWR0154
+L GND #PWR0155
 U 1 1 565FEDEB
 P 9700 1900
-F 0 "#PWR0154" H 9700 1650 50  0001 C CNN
+F 0 "#PWR0155" H 9700 1650 50  0001 C CNN
 F 1 "GND" H 9700 1750 50  0000 C CNN
 F 2 "" H 9700 1900 60  0000 C CNN
@@
 $EndComp
 $Comp
-L GND #PWR0155
+L GND #PWR0156
 U 1 1 565FEE20
 P 9400 1900
-F 0 "#PWR0155" H 9400 1650 50  0001 C CNN
+F 0 "#PWR0156" H 9400 1650 50  0001 C CNN
 F 1 "GND" H 9400 1750 50  0000 C CNN
 F 2 "" H 9400 1900 60  0000 C CNN
@@
 $EndComp
 $Comp
-L GND #PWR0156
+L GND #PWR0157
 U 1 1 565FF1AF
 P 8400 1900
-F 0 "#PWR0156" H 8400 1650 50  0001 C CNN
+F 0 "#PWR0157" H 8400 1650 50  0001 C CNN
 F 1 "GND" H 8400 1750 50  0000 C CNN
 F 2 "" H 8400 1900 60  0000 C CNN
@@
 	5100 4800 5200 4800
 Wire Wire Line
-	4800 3400 5000 3400
-Wire Wire Line
-	5000 3400 5200 3400
-Wire Wire Line
-	4800 4000 5000 4000
-Wire Wire Line
-	5000 4000 5200 4000
+	4800 3400 5200 3400
+Wire Wire Line
+	4800 4000 5200 4000
 Wire Wire Line
 	5000 3850 5000 4000
@@
 	9800 8500 9800 8600
 Wire Wire Line
-	11400 2300 11400 2400
-Wire Wire Line
-	11400 2400 11400 2500
-Wire Wire Line
-	10900 2300 10900 2400
-Wire Wire Line
-	10900 2400 10900 2500
-Wire Wire Line
-	10600 2300 10600 2400
-Wire Wire Line
-	10600 2400 10600 2500
-Wire Wire Line
-	10300 2300 10300 2400
-Wire Wire Line
-	10300 2400 10300 2500
-Wire Wire Line
-	10000 2300 10000 2400
-Wire Wire Line
-	10000 2400 10000 2500
-Wire Wire Line
-	9700 2300 9700 2400
-Wire Wire Line
-	9700 2400 9700 2500
-Wire Wire Line
-	9400 2300 9400 2400
-Wire Wire Line
-	9400 2400 9400 2500
-Wire Wire Line
-	9200 2400 9400 2400
-Wire Wire Line
-	9400 2400 9700 2400
-Wire Wire Line
-	9700 2400 10000 2400
-Wire Wire Line
-	10000 2400 10300 2400
-Wire Wire Line
-	10300 2400 10600 2400
-Wire Wire Line
-	10600 2400 10900 2400
-Wire Wire Line
-	10900 2400 11400 2400
-Wire Wire Line
-	11400 2400 11800 2400
+	11400 2300 11400 2500
+Wire Wire Line
+	10900 2300 10900 2500
+Wire Wire Line
+	10600 2300 10600 2500
+Wire Wire Line
+	10300 2300 10300 2500
+Wire Wire Line
+	10000 2300 10000 2500
+Wire Wire Line
+	9700 2300 9700 2500
+Wire Wire Line
+	9400 2300 9400 2500
+Wire Wire Line
+	9200 2400 11800 2400
 Connection ~ 9700 2400
 Connection ~ 9400 2400
@@
 	9400 2000 9400 1900
 Wire Wire Line
-	8400 2300 8400 2400
-Wire Wire Line
-	8400 2400 8400 2500
+	8400 2300 8400 2500
 Wire Wire Line
 	8400 2000 8400 1900
@@
 	7900 2500 7900 2400
 Wire Wire Line
-	7900 2400 8100 2400
-Wire Wire Line
-	8100 2400 8400 2400
-Wire Wire Line
-	8400 2400 8600 2400
+	7900 2400 8600 2400
 Connection ~ 8400 2400
 Wire Wire Line
@@
 	4600 2700 4600 2600
 Wire Wire Line
-	4500 3200 4600 3200
-Wire Wire Line
-	4600 3200 5200 3200
+	4500 3200 5200 3200
 Wire Wire Line
 	4600 3200 4600 3000
@@
 	15300 5400 15200 5400
 Wire Wire Line
-	650  6800 750  6800
-Wire Wire Line
-	750  6800 850  6800
+	650  6800 850  6800
 Wire Wire Line
 	750  6900 750  6800
@@
 	750  6400 750  6500
 Wire Wire Line
-	650  6500 750  6500
-Wire Wire Line
-	750  6500 850  6500
+	650  6500 850  6500
 Connection ~ 750  6500
 Wire Wire Line
@@
 	7850 8800 7850 8900
 Wire Wire Line
-	7850 9200 7850 9300
-Wire Wire Line
-	7850 9300 7850 9400
-Wire Wire Line
-	7850 9700 7850 9800
-Wire Wire Line
-	7850 9800 7850 9900
+	7850 9200 7850 9400
+Wire Wire Line
+	7850 9700 7850 9900
 Wire Wire Line
 	8950 8800 8950 8900
 Wire Wire Line
-	8950 9200 8950 9300
-Wire Wire Line
-	8950 9300 8950 9400
-Wire Wire Line
-	8950 9700 8950 9800
-Wire Wire Line
-	8950 9800 8950 9900
-Wire Wire Line
-	8850 9300 8950 9300
-Wire Wire Line
-	8950 9300 9150 9300
+	8950 9200 8950 9400
+Wire Wire Line
+	8950 9700 8950 9900
+Wire Wire Line
+	8850 9300 9150 9300
 Connection ~ 8950 9300
 Wire Wire Line
-	7750 9300 7850 9300
-Wire Wire Line
-	7850 9300 8050 9300
+	7750 9300 8050 9300
 Connection ~ 7850 9300
 Wire Wire Line
@@
 	4850 2900 4850 3000
 Wire Wire Line
-	4850 3000 5100 3000
-Wire Wire Line
-	5100 3000 5200 3000
+	4850 3000 5200 3000
 Wire Wire Line
 	5100 2900 5100 3000
@@
 	5100 2600 5100 2700
 Wire Wire Line
-	1150 6000 1750 6000
-Wire Wire Line
-	1750 6000 5200 6000
-Wire Wire Line
-	1150 5900 1350 5900
-Wire Wire Line
-	1350 5900 5200 5900
+	1550 6000 5200 6000
 Wire Wire Line
 	1750 6450 1750 6000
 Connection ~ 1750 6000
-Wire Wire Line
-	1750 6650 1350 6650
-Wire Wire Line
-	1350 6650 1350 5900
-Connection ~ 1350 5900
 Wire Wire Line
 	1650 6550 1750 6550
@@
 Wire Wire Line
 	15300 4400 15200 4400
+$Comp
+L R R16
+U 1 1 57F851F7
+P 1400 6000
+F 0 "R16" V 1480 6000 50  0000 C CNN
+F 1 "22" V 1400 6000 50  0000 C CNN
+F 2 "stmbl:R_0603" V 1330 6000 30  0001 C CNN
+F 3 "" H 1400 6000 30  0000 C CNN
+	1    1400 6000
+	0    1    1    0
+$EndComp
+Wire Wire Line
+	1250 6000 1150 6000
+$Comp
+L R R15
+U 1 1 57F85A1B
+P 1400 5900
+F 0 "R15" V 1480 5900 50  0000 C CNN
+F 1 "22" V 1400 5900 50  0000 C CNN
+F 2 "stmbl:R_0603" V 1330 5900 30  0001 C CNN
+F 3 "" H 1400 5900 30  0000 C CNN
+	1    1400 5900
+	0    1    1    0
+$EndComp
+Wire Wire Line
+	1750 6650 1350 6650
+Wire Wire Line
+	1350 6650 1350 6400
+Wire Wire Line
+	1350 6400 1650 6400
+Wire Wire Line
+	1650 6400 1650 5900
+Connection ~ 1650 5900
+Wire Wire Line
+	1550 5900 5200 5900
+Wire Wire Line
+	1250 5900 1150 5900
 $EndSCHEMATC

Commit message: v4.0
Connections:
- net IO_RX: no longer names the net of U26.87 (PD6/FSMC_NWAIT/USART2_RX/EVENTOUT)
- net IO_TX: no longer names the net of U26.86 (PD5/FSMC_NWE/USART2_TX/EVENTOUT)
Changed lines of the file:
@@
 $Descr A3 16535 11693
 encoding utf-8
-Sheet 13 14
+Sheet 14 14
 Title ""
 Date ""
@@
 $EndComp
 $Comp
-L GND #PWR0140
+L GND #PWR0178
 U 1 1 565FE0C3
 P 4400 4000
-F 0 "#PWR0140" H 4400 3750 50  0001 C CNN
+F 0 "#PWR0178" H 4400 3750 50  0001 C CNN
 F 1 "GND" H 4400 3850 50  0000 C CNN
 F 2 "" H 4400 4000 60  0000 C CNN
@@
 $EndComp
 $Comp
-L GND #PWR0141
+L GND #PWR0179
 U 1 1 565FE0E1
 P 4400 3400
-F 0 "#PWR0141" H 4400 3150 50  0001 C CNN
+F 0 "#PWR0179" H 4400 3150 50  0001 C CNN
 F 1 "GND" H 4400 3250 50  0000 C CNN
 F 2 "" H 4400 3400 60  0000 C CNN
@@
 $EndComp
 $Comp
-L GND #PWR0142
+L GND #PWR0180
 U 1 1 565FE268
 P 10600 8600
-F 0 "#PWR0142" H 10600 8350 50  0001 C CNN
+F 0 "#PWR0180" H 10600 8350 50  0001 C CNN
 F 1 "GND" H 10600 8450 50  0000 C CNN
 F 2 "" H 10600 8600 60  0000 C CNN
@@
 $EndComp
 $Comp
-L GND #PWR0143
+L GND #PWR0181
 U 1 1 565FE28C
 P 10400 8600
-F 0 "#PWR0143" H 10400 8350 50  0001 C CNN
+F 0 "#PWR0181" H 10400 8350 50  0001 C CNN
 F 1 "GND" H 10400 8450 50  0000 C CNN
 F 2 "" H 10400 8600 60  0000 C CNN
@@
 $EndComp
 $Comp
-L GND #PWR0144
+L GND #PWR0182
 U 1 1 565FE2A9
 P 10200 8600
-F 0 "#PWR0144" H 10200 8350 50  0001 C CNN
+F 0 "#PWR0182" H 10200 8350 50  0001 C CNN
 F 1 "GND" H 10200 8450 50  0000 C CNN
 F 2 "" H 10200 8600 60  0000 C CNN
@@
 $EndComp
 $Comp
-L GND #PWR0145
+L GND #PWR0183
 U 1 1 565FE2C6
 P 10000 8600
-F 0 "#PWR0145" H 10000 8350 50  0001 C CNN
+F 0 "#PWR0183" H 10000 8350 50  0001 C CNN
 F 1 "GND" H 10000 8450 50  0000 C CNN
 F 2 "" H 10000 8600 60  0000 C CNN
@@
 $EndComp
 $Comp
-L GND #PWR0146
+L GND #PWR0184
 U 1 1 565FE2E3
 P 9800 8600
-F 0 "#PWR0146" H 9800 8350 50  0001 C CNN
+F 0 "#PWR0184" H 9800 8350 50  0001 C CNN
 F 1 "GND" H 9800 8450 50  0000 C CNN
 F 2 "" H 9800 8600 60  0000 C CNN
@@
 $EndComp
 $Comp
-L GND #PWR0147
+L GND #PWR0185
 U 1 1 565FE300
 P 11100 9000
-F 0 "#PWR0147" H 11100 8750 50  0001 C CNN
+F 0 "#PWR0185" H 11100 8750 50  0001 C CNN
 F 1 "GND" H 11100 8850 50  0000 C CNN
 F 2 "" H 11100 9000 60  0000 C CNN
@@
 $EndComp
 $Comp
-L GND #PWR0148
+L GND #PWR0186
 U 1 1 565FE31D
 P 11600 9000
-F 0 "#PWR0148" H 11600 8750 50  0001 C CNN
+F 0 "#PWR0186" H 11600 8750 50  0001 C CNN
 F 1 "GND" H 11600 8850 50  0000 C CNN
 F 2 "" H 11600 9000 60  0000 C CNN
@@
 $EndComp
 $Comp
-L +3.3V #PWR0149
+L +3.3V #PWR0187
 U 1 1 565FEC9D
 P 11800 2300
-F 0 "#PWR0149" H 11800 2150 50  0001 C CNN
+F 0 "#PWR0187" H 11800 2150 50  0001 C CNN
 F 1 "+3.3V" H 11800 2440 50  0000 C CNN
 F 2 "" H 11800 2300 60  0000 C CNN
@@
 $EndComp
 $Comp
-L GND #PWR0150
+L GND #PWR0188
 U 1 1 565FECDB
 P 11400 1900
-F 0 "#PWR0150" H 11400 1650 50  0001 C CNN
+F 0 "#PWR0188" H 11400 1650 50  0001 C CNN
 F 1 "GND" H 11400 1750 50  0000 C CNN
 F 2 "" H 11400 1900 60  0000 C CNN
@@
 $EndComp
 $Comp
-L GND #PWR0151
+L GND #PWR0189
 U 1 1 565FED17
 P 10900 1900
-F 0 "#PWR0151" H 10900 1650 50  0001 C CNN
+F 0 "#PWR0189" H 10900 1650 50  0001 C CNN
 F 1 "GND" H 10900 1750 50  0000 C CNN
 F 2 "" H 10900 1900 60  0000 C CNN
@@
 $EndComp
 $Comp
-L GND #PWR0152
+L GND #PWR0190
 U 1 1 565FED4C
 P 10600 1900
-F 0 "#PWR0152" H 10600 1650 50  0001 C CNN
+F 0 "#PWR0190" H 10600 1650 50  0001 C CNN
 F 1 "GND" H 10600 1750 50  0000 C CNN
 F 2 "" H 10600 1900 60  0000 C CNN
@@
 $EndComp
 $Comp
-L GND #PWR0153
+L GND #PWR0191
 U 1 1 565FED81
 P 10300 1900
-F 0 "#PWR0153" H 10300 1650 50  0001 C CNN
+F 0 "#PWR0191" H 10300 1650 50  0001 C CNN
 F 1 "GND" H 10300 1750 50  0000 C CNN
 F 2 "" H 10300 1900 60  0000 C CNN
@@
 $EndComp
 $Comp
-L GND #PWR0154
+L GND #PWR0192
 U 1 1 565FEDB6
 P 10000 1900
-F 0 "#PWR0154" H 10000 1650 50  0001 C CNN
+F 0 "#PWR0192" H 10000 1650 50  0001 C CNN
 F 1 "GND" H 10000 1750 50  0000 C CNN
 F 2 "" H 10000 1900 60  0000 C CNN
@@
 $EndComp
 $Comp
-L GND #PWR0155
+L GND #PWR0193
 U 1 1 565FEDEB
 P 9700 1900
-F 0 "#PWR0155" H 9700 1650 50  0001 C CNN
+F 0 "#PWR0193" H 9700 1650 50  0001 C CNN
 F 1 "GND" H 9700 1750 50  0000 C CNN
 F 2 "" H 9700 1900 60  0000 C CNN
@@
 $EndComp
 $Comp
-L GND #PWR0156
+L GND #PWR0194
 U 1 1 565FEE20
 P 9400 1900
-F 0 "#PWR0156" H 9400 1650 50  0001 C CNN
+F 0 "#PWR0194" H 9400 1650 50  0001 C CNN
 F 1 "GND" H 9400 1750 50  0000 C CNN
 F 2 "" H 9400 1900 60  0000 C CNN
@@
 $EndComp
 $Comp
-L GND #PWR0157
+L GND #PWR0195
 U 1 1 565FF1AF
 P 8400 1900
-F 0 "#PWR0157" H 8400 1650 50  0001 C CNN
+F 0 "#PWR0195" H 8400 1650 50  0001 C CNN
 F 1 "GND" H 8400 1750 50  0000 C CNN
 F 2 "" H 8400 1900 60  0000 C CNN
@@
 $EndComp
 $Comp
-L GND #PWR0158
+L GND #PWR0196
 U 1 1 565FFB31
 P 4600 2600
-F 0 "#PWR0158" H 4600 2350 50  0001 C CNN
+F 0 "#PWR0196" H 4600 2350 50  0001 C CNN
 F 1 "GND" H 4600 2450 50  0000 C CNN
 F 2 "" H 4600 2600 60  0000 C CNN
@@
 Text HLabel 4500 3200 0    60   Input ~ 0
 NRST
-Text HLabel 15300 5300 2    60   Input ~ 0
-IO_TX
-Text HLabel 15300 5400 2    60   Input ~ 0
-IO_RX
 $Comp
 L USB_OTG P1
@@
 $EndComp
 $Comp
-L GND #PWR0159
+L GND #PWR0197
 U 1 1 56602FE1
 P 750 6900
-F 0 "#PWR0159" H 750 6650 50  0001 C CNN
+F 0 "#PWR0197" H 750 6650 50  0001 C CNN
 F 1 "GND" H 750 6750 50  0000 C CNN
 F 2 "" H 750 6900 60  0000 C CNN
@@
 $EndComp
 $Comp
-L GND #PWR0160
+L GND #PWR0198
 U 1 1 56603874
 P 1250 6300
-F 0 "#PWR0160" H 1250 6050 50  0001 C CNN
+F 0 "#PWR0198" H 1250 6050 50  0001 C CNN
 F 1 "GND" H 1250 6150 50  0000 C CNN
 F 2 "" H 1250 6300 60  0000 C CNN
@@
 IO_OUT1
 $Comp
-L GND #PWR0161
+L GND #PWR0199
 U 1 1 5667D307
 P 1650 6550
-F 0 "#PWR0161" H 1650 6300 50  0001 C CNN
+F 0 "#PWR0199" H 1650 6300 50  0001 C CNN
 F 1 "GND" H 1650 6400 50  0000 C CNN
 F 2 "" H 1650 6550 60  0000 C CNN
@@
 $EndComp
 $Comp
-L +3.3V #PWR0162
+L +3.3V #PWR0200
 U 1 1 5667D40D
 P 4400 6450
-F 0 "#PWR0162" H 4400 6300 50  0001 C CNN
+F 0 "#PWR0200" H 4400 6300 50  0001 C CNN
 F 1 "+3.3V" H 4400 6590 50  0000 C CNN
 F 2 "" H 4400 6450 60  0000 C CNN
@@
 $EndComp
 $Comp
-L GND #PWR0163
+L GND #PWR0201
 U 1 1 5668EC91
 P 7850 9900
-F 0 "#PWR0163" H 7850 9650 50  0001 C CNN
+F 0 "#PWR0201" H 7850 9650 50  0001 C CNN
 F 1 "GND" H 7850 9750 50  0000 C CNN
 F 2 "" H 7850 9900 60  0000 C CNN
@@
 $EndComp
 $Comp
-L GND #PWR0164
+L GND #PWR0202
 U 1 1 5668F551
 P 8950 9900
-F 0 "#PWR0164" H 8950 9650 50  0001 C CNN
+F 0 "#PWR0202" H 8950 9650 50  0001 C CNN
 F 1 "GND" H 8950 9750 50  0000 C CNN
 F 2 "" H 8950 9900 60  0000 C CNN
@@
 $EndComp
 $Comp
-L GND #PWR0165
+L GND #PWR0203
 U 1 1 566A9D9E
 P 4850 2500
-F 0 "#PWR0165" H 4850 2250 50  0001 C CNN
+F 0 "#PWR0203" H 4850 2250 50  0001 C CNN
 F 1 "GND" H 4850 2350 50  0000 C CNN
 F 2 "" H 4850 2500 60  0000 C CNN
@@
 $EndComp
 $Comp
-L +3.3V #PWR0166
+L +3.3V #PWR0204
 U 1 1 566A9F89
 P 5100 2600
-F 0 "#PWR0166" H 5100 2450 50  0001 C CNN
+F 0 "#PWR0204" H 5100 2450 50  0001 C CNN
 F 1 "+3.3V" H 5100 2740 50  0000 C CNN
 F 2 "" H 5100 2600 60  0000 C CNN
@@
 $EndComp
 $Comp
-L GND #PWR0167
+L GND #PWR0205
 U 1 1 56667EDB
 P 3050 7050
-F 0 "#PWR0167" H 3050 6800 50  0001 C CNN
+F 0 "#PWR0205" H 3050 6800 50  0001 C CNN
 F 1 "GND" H 3050 6900 50  0000 C CNN
 F 2 "" H 3050 7050 60  0000 C CNN
@@
 $EndComp
 $Comp
-L +3.3V #PWR0168
+L +3.3V #PWR0206
 U 1 1 566680A9
 P 2550 7050
-F 0 "#PWR0168" H 2550 6900 50  0001 C CNN
+F 0 "#PWR0206" H 2550 6900 50  0001 C CNN
 F 1 "+3.3V" H 2550 7190 50  0000 C CNN
 F 2 "" H 2550 7050 60  0000 C CNN
@@
 	5100 6200 5200 6200
 Wire Wire Line
-	15300 5300 15200 5300
-Wire Wire Line
-	15300 5400 15200 5400
-Wire Wire Line
 	650  6800 850  6800
 Wire Wire Line
@@
 $EndComp
 $Comp
-L +5V #PWR0169
+L +5V #PWR0207
 U 1 1 56A313ED
 P 1550 5700
-F 0 "#PWR0169" H 1550 5550 50  0001 C CNN
+F 0 "#PWR0207" H 1550 5550 50  0001 C CNN
 F 1 "+5V" H 1568 5874 50  0000 C CNN
 F 2 "" H 1550 5700 50  0000 C CNN
@@
 	1550 5800 1550 5700
 $Comp
-L +24V #PWR0170
+L +24V #PWR0208
 U 1 1 56FF1B13
 P 7850 8800
-F 0 "#PWR0170" H 7850 8650 50  0001 C CNN
+F 0 "#PWR0208" H 7850 8650 50  0001 C CNN
 F 1 "+24V" H 7868 8974 50  0000 C CNN
 F 2 "" H 7850 8800 50  0000 C CNN
@@
 $EndComp
 $Comp
-L +5V #PWR0171
+L +5V #PWR0209
 U 1 1 56FF1E56
 P 8950 8800
-F 0 "#PWR0171" H 8950 8650 50  0001 C CNN
+F 0 "#PWR0209" H 8950 8650 50  0001 C CNN
 F 1 "+5V" H 8968 8974 50  0000 C CNN
 F 2 "" H 8950 8800 50  0000 C CNN
@@
 	8100 1900 8100 2000
 $Comp
-L GND #PWR0172
+L GND #PWR0210
 U 1 1 57B0781F
 P 8100 1900
-F 0 "#PWR0172" H 8100 1650 50  0001 C CNN
+F 0 "#PWR0210" H 8100 1650 50  0001 C CNN
 F 1 "GND" H 8100 1750 50  0000 C CNN
 F 2 "" H 8100 1900 60  0000 C CNN
@@
 	-1   0    0    1
 $EndComp
-Text HLabel 1500 8800 0    60   Input ~ 0
+Text HLabel 1500 9300 0    60   Input ~ 0
 EN_5V
-Text HLabel 1500 8900 0    60   Input ~ 0
+Text HLabel 1500 9400 0    60   Input ~ 0
 EN_12V
 Text HLabel 3950 6450 2    60   Input ~ 0
@@
 Wire Wire Line
 	1250 5900 1150 5900
+Text HLabel 1500 8400 0    60   Input ~ 0
+IO_L0
+Text HLabel 1500 8500 0    60   Input ~ 0
+IO_L1
+Text HLabel 1500 8600 0    60   Input ~ 0
+IO_GREEN
+Text HLabel 1500 8700 0    60   Input ~ 0
+IO_YELLOW
+Text HLabel 1500 8800 0    60   Input ~ 0
+IO_RED
 $EndSCHEMATC

Commit message: v4.0
Parts:
- removed JP2: Jumper_NO_Small, symbol Jumper_NO_Small
- removed R15, R16: 22, stmbl:R_0603, symbol R
- added D21: D, Diodes_SMD:SMA_Standard, symbol D
Connections:
- net +5V: now also D21.1 (K)
- net at U1.3 (I/O2), U26.70 (PA11/USART1_CTS/CAN1_RX/TIM1_CH4_/OTG_FS_DM/EVENTOUT): now also P1.2 (D-)
- net at U1.1 (I/O1), U26.71 (PA12/USART1_RTS/CAN1_TX/TIM1_ETR/OTG_FS_DP/EVENTOUT): now also P1.3 (D+)
- net at P1.1 (VCC): now also D21.2 (A)

Commit message: v4.0
Parts:
- added C61, C66, C67: C, stmbl:C_0603, symbol C
- added U20, U22, U23: USBLC6-4SC6, TO_SOT_Packages_SMD:SOT-23-6, symbol USBLC6-4SC6
- JP9: footprint (none) -> stmbl:SOLDER_JUMPER
Connections:
- net +3V3: now also C61.1, C66.1, C67.1, U20.5 (VBUS), U22.5 (VBUS), U23.5 (VBUS)
- net CAN_RX: now also U22.6 (I/O4)
- net CAN_TX: now also U22.4 (I/O3)
- net CMD_12: now also U22.3 (I/O2)
- net CMD_36: now also U20.4 (I/O3)
- net CMD_45: now also U22.1 (I/O1)
- net FB0_V: now also U23.6 (I/O4); no longer U1.6 (I/O4)
- net FB1_V: now also U23.4 (I/O3); no longer U1.4 (I/O3)
- net GND: now also C61.2, C66.2, C67.2, U20.2 (GND), U22.2 (GND), U23.2 (GND)
- net HV_RX: now also U1.4 (I/O3)
- net HV_TX: now also U1.6 (I/O4)
- net IO_AIN0: now also U23.1 (I/O1)
- net IO_AIN1: now also U23.3 (I/O2)
- net NRST: now also U20.1 (I/O1)
- net SWCLK: now also U20.6 (I/O4)
- net SWDIO: now also U20.3 (I/O2)
