File: hw/kicad/v4.0/f4.sch (KiCad schematic (older format))
At the start: 37 parts, among them P1 USB_OTG, U1 USBLC6-4SC6, U20 USBLC6-4SC6, U22 USBLC6-4SC6, U23 USBLC6-4SC6, U26 STM32F405VG, Y2 8M

Commit message: v4.0 mapping
Parts:
- C61, C66, C67: value C -> 100n
Connections:
- net CAN_RX: now also U26.81 (PD0/FSMC_D2/CAN1_RX/EVENTOUT); no longer U26.95 (PB8/TIM4_CH3/SDIO_D4/TIM10_CH1/I2C1_SCL/CAN1_RX/EVENTOUT)
- net CAN_TX: now also U26.82 (PD1/FSMC_D3/CAN1_TX/EVENTOUT); no longer U26.96 (PB9/SPI2_NSS/I2S2_WS/TIM4_CH4/TIM11_CH1/SDIO_D5/I2C1_SDA/CAN1_TX/EVENTOUT)
- net CMD_12E: now also U26.92 (PB6/I2C1_SCL/TIM4_CH1/CAN2_TX/USART1_TX/EVENTOUT)
- net CMD_36E: now also U26.93 (PB7/I2C1_SDA/FSMC_NL/USART1_RX/TIM4_CH2/EVENTOUT)
- net CMD_45E: now also U26.96 (PB9/SPI2_NSS/I2S2_WS/TIM4_CH4/TIM11_CH1/SDIO_D5/I2C1_SDA/CAN1_TX/EVENTOUT)
- net CMD_78: now also U26.95 (PB8/TIM4_CH3/SDIO_D4/TIM10_CH1/I2C1_SCL/CAN1_RX/EVENTOUT)
- net CMD_78E: now also U26.37 (PB2/BOOT1/EVENTOUT)
- net CMD_L1: now also U26.35 (PB0/TIM3_CH3/TIM8_CH2N/OTG_HS_ULPI_D1/TIM1_CH2N/EVENTOUT)
- net CMD_L2: now also U26.36 (PB1/TIM3_CH4/TIM8_CH3N/OTG_HS_ULPI_D2/OTG_HS_INTN/TIM1_CH3N/EVENTOUT)
- net EN_12V: now also U26.8 (PC14/OSC32_IN/EVENTOUT)
- net EN_5V: now also U26.7 (PC13/EVENTOUT)
- net FB0_12E: now also U26.58 (PD11/FSMC_CLE/FSMC_A16/USART3_CTS/EVENTOUT)
- net FB0_36E: now also U26.57 (PD10/FSMC_D15/USART3_CK/EVENTOUT)
- net FB0_C: now also U26.32 (PA7/SPI1_MOSI/TIM8_CH1N/TIM14_CH1/TIM3_CH2/TIM1_CH1N/EVENTOUT)
- net FB0_L1: now also U26.55 (PD8/FSMC_D13/USART3_TX/EVENTOUT)
- net FB0_L2: now also U26.56 (PD9/FSMC_D14/USART3_RX/EVENTOUT)
- net FB0_S: now also U26.31 (PA6/SPI1_MISO/TIM8_BKIN/TIM13_CH1/TIM3_CH1/TIM1_BKIN/EVENTOUT)
- net FB0_V: now also U26.18 (PC3/SPI2_MOSI/I2S2_SD/OTG_HS_ULPI_NXT/EVENTOUT)
- net FB1_12E: now also U26.41 (PE10/FSMC_D7/TIM1_CH2N/EVENTOUT)
- net FB1_36E: now also U26.43 (PE12/FSMC_D9/TIM1_CH3N/EVENTOUT)
- net FB1_C: now also U26.30 (PA5/SPI1_SCK/OTG_HS_ULPI_CK/TIM2_CH1_ETR/TIM8_CHIN/EVENTOUT)
- net FB1_L1: now also U26.38 (PE7/FSMC_D4/TIM1_ETR/EVENTOUT)
- net FB1_L2: now also U26.39 (PE8/FSMC_D5/TIM1_CH1N/EVENTOUT)
- net FB1_S: now also U26.29 (PA4/SPI1_NSS/SPI3_NSS/USART2_CK/OTG_HS_SOF/I2S3_WS/EVENTOUT)
- net FB1_V: now also U26.17 (PC2/SPI2_MISO/OTG_HS_ULPI_DIR/I2S2ext_SD/EVENTOUT)
- net HV_RX: now also U26.26 (PA3/USART2_RX/TIM5_CH4/TIM9_CH2/TIM2_CH4/OTG_HS_ULPI_D0/EVENTOUT); no longer U26.24 (PA1/USART2_RTS/UART4_RX/TIM5_CH2/TIMM2_CH2/EVENTOUT)
- net HV_TX: now also U26.25 (PA2/USART2_TX/TIM5_CH3/TIM9_CH1/TIM2_CH3/EVENTOUT); no longer U26.23 (PA0/WKUP/USART2_CTS/UART4_TX/TIM2_CH1_ETR/TIM5_CH1/TIM8_ETR/EVENTOUT)
- net IO_AIN0: now also U26.15 (PC0/OTG_HS_ULPI_STP/EVENTOUT)
- net IO_AIN1: now also U26.16 (PC1/_EVENTOUT)
- net IO_BRAKE: now also U26.5 (PE6/TRACED3_/_FSMC_A22/TIM9_CH2/EVENTOUT)
- net IO_FAN: now also U26.2 (PE3/TRACED0/FSMC_A19/EVENTOUT)
- net IO_GREEN: now also U26.86 (PD5/FSMC_NWE/USART2_TX/EVENTOUT)
- net IO_L0: now also U26.98 (PE1/FSMC_NBL1/EVENTOUT)
- net IO_L1: now also U26.97 (PE0/TIM4_ETR/FSMC_NBL0/EVENTOUT)
- net IO_OUT0: now also U26.3 (PE4/TRACED1/FSMC_A20/EVENTOUT)
- net IO_OUT1: now also U26.4 (PE5/TRACED2/FSMC_A21/TIM9_CH1/EVENTOUT)
- net IO_RED: now also U26.84 (PD3/FSMC_CLK/USART2_CTS/EVENTOUT)
- net IO_YELLOW: now also U26.85 (PD4/FSMC_NOE/USART2_RTS/EVENTOUT)
- net A_24V_ renamed A_24V
- net A_24V: now also U26.24 (PA1/USART2_RTS/UART4_RX/TIM5_CH2/TIMM2_CH2/EVENTOUT)
- net A_5V_ renamed A_5V
Other:
- moved on the sheet: C81, R121, R122

Commit message: v4.0
Parts:
- added R153: 1k, stmbl:R_0603, symbol R
Connections:
- net CAN_RX: now also U20.6 (I/O4); no longer U22.6 (I/O4)
- net CAN_TX: now also U20.4 (I/O3); no longer U22.4 (I/O3)
- net CMD_36: now also U22.6 (I/O4); no longer U20.4 (I/O3)
- net NRST: now also U22.4 (I/O3); no longer U20.1 (I/O1)
- net SWCLK: now also U20.1 (I/O1); no longer U20.6 (I/O4)
- net at C32.1, Y2.2: now also R153.2; no longer U26.13 (PH1/OSC_OUT/EVENTOUT)
- net IO_BRAKE renamed IO_OUT2
- new net: R153.1, U26.13 (PH1/OSC_OUT/EVENTOUT)
Other:
- moved on the sheet: C31, C32, Y2
Changed lines of the file:
@@
 L Crystal Y2
 U 1 1 565FDF0A
-P 5000 3700
-F 0 "Y2" H 5000 3850 50  0000 C CNN
-F 1 "8M" H 5000 3550 50  0000 C CNN
-F 2 "stmbl:Crystal_SMD_0603_4Pads" H 5000 3700 60  0001 C CNN
-F 3 "" H 5000 3700 60  0000 C CNN
-	1    5000 3700
+P 4700 3700
+F 0 "Y2" H 4700 3850 50  0000 C CNN
+F 1 "8M" H 4700 3550 50  0000 C CNN
+F 2 "stmbl:Crystal_SMD_0603_4Pads" H 4700 3700 60  0001 C CNN
+F 3 "" H 4700 3700 60  0000 C CNN
+	1    4700 3700
 	0    1    1    0
 $EndComp
@@
 L C C31
 U 1 1 565FDF4E
-P 4650 3400
-F 0 "C31" H 4675 3500 50  0000 L CNN
-F 1 "18p" H 4675 3300 50  0000 L CNN
-F 2 "stmbl:C_0603" H 4688 3250 30  0001 C CNN
-F 3 "" H 4650 3400 60  0000 C CNN
-	1    4650 3400
+P 4350 3400
+F 0 "C31" H 4375 3500 50  0000 L CNN
+F 1 "18p" H 4375 3300 50  0000 L CNN
+F 2 "stmbl:C_0603" H 4388 3250 30  0001 C CNN
+F 3 "" H 4350 3400 60  0000 C CNN
+	1    4350 3400
 	0    1    1    0
 $EndComp
@@
 L C C32
 U 1 1 565FDFAD
-P 4650 4000
-F 0 "C32" H 4675 4100 50  0000 L CNN
-F 1 "18p" H 4675 3900 50  0000 L CNN
-F 2 "stmbl:C_0603" H 4688 3850 30  0001 C CNN
-F 3 "" H 4650 4000 60  0000 C CNN
-	1    4650 4000
+P 4350 4000
+F 0 "C32" H 4375 4100 50  0000 L CNN
+F 1 "18p" H 4375 3900 50  0000 L CNN
+F 2 "stmbl:C_0603" H 4388 3850 30  0001 C CNN
+F 3 "" H 4350 4000 60  0000 C CNN
+	1    4350 4000
 	0    1    1    0
 $EndComp
@@
 L GND #PWR0167
 U 1 1 565FE0C3
-P 4400 4000
-F 0 "#PWR0167" H 4400 3750 50  0001 C CNN
-F 1 "GND" H 4400 3850 50  0000 C CNN
-F 2 "" H 4400 4000 60  0000 C CNN
-F 3 "" H 4400 4000 60  0000 C CNN
-	1    4400 4000
+P 4100 4000
+F 0 "#PWR0167" H 4100 3750 50  0001 C CNN
+F 1 "GND" H 4100 3850 50  0000 C CNN
+F 2 "" H 4100 4000 60  0000 C CNN
+F 3 "" H 4100 4000 60  0000 C CNN
+	1    4100 4000
 	0    1    1    0
 $EndComp
@@
 L GND #PWR0168
 U 1 1 565FE0E1
-P 4400 3400
-F 0 "#PWR0168" H 4400 3150 50  0001 C CNN
-F 1 "GND" H 4400 3250 50  0000 C CNN
-F 2 "" H 4400 3400 60  0000 C CNN
-F 3 "" H 4400 3400 60  0000 C CNN
-	1    4400 3400
+P 4100 3400
+F 0 "#PWR0168" H 4100 3150 50  0001 C CNN
+F 1 "GND" H 4100 3250 50  0000 C CNN
+F 2 "" H 4100 3400 60  0000 C CNN
+F 3 "" H 4100 3400 60  0000 C CNN
+	1    4100 3400
 	0    1    1    0
 $EndComp
@@
 IO_FAN
 Text HLabel 15300 3600 2    60   Input ~ 0
-IO_BRAKE
+IO_OUT2
 Text HLabel 15300 3400 2    60   Input ~ 0
 IO_OUT0
@@
 	5100 5000 5200 5000
 Wire Wire Line
-	4800 3400 5200 3400
-Wire Wire Line
-	4800 4000 5200 4000
-Wire Wire Line
-	5000 3850 5000 4000
-Connection ~ 5000 4000
-Wire Wire Line
-	5000 3550 5000 3400
-Connection ~ 5000 3400
-Wire Wire Line
-	4500 3400 4400 3400
-Wire Wire Line
-	4500 4000 4400 4000
+	4500 3400 5200 3400
+Wire Wire Line
+	4500 4000 4800 4000
+Wire Wire Line
+	4700 4000 4700 3850
+Connection ~ 4700 4000
+Wire Wire Line
+	4700 3550 4700 3400
+Connection ~ 4700 3400
+Wire Wire Line
+	4200 3400 4100 3400
+Wire Wire Line
+	4200 4000 4100 4000
 Wire Wire Line
 	11600 8500 11600 8600
@@
 Text HLabel 1650 2050 0    60   Input ~ 0
 SWDIO
-Text HLabel 3950 1850 2    60   Input ~ 0
+Text HLabel 1650 1850 0    60   Input ~ 0
 SWCLK
-Text HLabel 3950 2050 2    60   Input ~ 0
+Text HLabel 3950 2550 2    60   Input ~ 0
 IO_SPI_CK
 Text HLabel 1650 2550 0    60   Input ~ 0
@@
 Text HLabel 1650 2750 0    60   Input ~ 0
 IO_SPI_MISO
-Text HLabel 3950 2550 2    60   Input ~ 0
+Text HLabel 3950 1850 2    60   Input ~ 0
 CAN_RX
+Text HLabel 3950 2050 2    60   Input ~ 0
+CAN_TX
 Text HLabel 3950 2750 2    60   Input ~ 0
-CAN_TX
-Text HLabel 1650 1850 0    60   Input ~ 0
 NRST
 Text HLabel 3450 10050 0    60   Input ~ 0
@@
 Wire Wire Line
 	15350 6900 15200 6900
+$Comp
+L R R153
+U 1 1 582C978B
+P 4950 4000
+F 0 "R153" V 5030 4000 50  0000 C CNN
+F 1 "1k" V 4950 4000 50  0000 C CNN
+F 2 "stmbl:R_0603" V 4880 4000 30  0001 C CNN
+F 3 "" H 4950 4000 30  0000 C CNN
+	1    4950 4000
+	0    1    1    0
+$EndComp
+Wire Wire Line
+	5100 4000 5200 4000
 $EndSCHEMATC
