File: hw/kicad/v4.0/f3.sch (KiCad schematic (older format))
At the start: 28 parts, among them P12 CONN_01X04, T1 testpoint, T44 testpoint, T45 testpoint, T46 testpoint, U20 USBLC6-4SC6, U21 USBLC6-4SC6, U25 STM32F303CBTx, U29 USBLC6-4SC6, Y1 8M

Commit message: v4.0
Other:
- moved on the sheet: R8

Commit message: v4.0
Parts:
- C10, C128, C2, C5, C6, C61, C7, C78, C79, C82, C83, C9: footprint Capacitors_SMD:C_0603 -> stmbl:C_0603
- L1, R129, R2, R8: footprint Resistors_SMD:R_0603 -> stmbl:R_0603
Changed lines of the file:
@@
 F 0 "C78" H 9625 950 50  0000 L CNN
 F 1 "100n" H 9625 750 50  0000 L CNN
-F 2 "Capacitors_SMD:C_0603" H 9638 700 30  0001 C CNN
+F 2 "stmbl:C_0603" H 9638 700 30  0001 C CNN
 F 3 "" H 9600 850 60  0000 C CNN
 	1    9600 850
@@
 F 0 "C79" H 9725 950 50  0000 L CNN
 F 1 "100n" H 9725 750 50  0000 L CNN
-F 2 "Capacitors_SMD:C_0603" H 9738 700 30  0001 C CNN
+F 2 "stmbl:C_0603" H 9738 700 30  0001 C CNN
 F 3 "" H 9700 850 60  0000 C CNN
 	1    9700 850
@@
 F 0 "C82" H 9825 950 50  0000 L CNN
 F 1 "100n" H 9825 750 50  0000 L CNN
-F 2 "Capacitors_SMD:C_0603" H 9838 700 30  0001 C CNN
+F 2 "stmbl:C_0603" H 9838 700 30  0001 C CNN
 F 3 "" H 9800 850 60  0000 C CNN
 	1    9800 850
@@
 F 0 "C83" H 9925 950 50  0000 L CNN
 F 1 "100n" H 9925 750 50  0000 L CNN
-F 2 "Capacitors_SMD:C_0603" H 9938 700 30  0001 C CNN
+F 2 "stmbl:C_0603" H 9938 700 30  0001 C CNN
 F 3 "" H 9900 850 60  0000 C CNN
 	1    9900 850
@@
 F 0 "C5" H 1975 2200 50  0000 L CNN
 F 1 "18p" H 1975 2000 50  0000 L CNN
-F 2 "Capacitors_SMD:C_0603" H 1988 1950 30  0001 C CNN
+F 2 "stmbl:C_0603" H 1988 1950 30  0001 C CNN
 F 3 "" H 1950 2100 60  0000 C CNN
 	1    1950 2100
@@
 F 0 "C6" H 1975 2500 50  0000 L CNN
 F 1 "18p" H 1975 2300 50  0000 L CNN
-F 2 "Capacitors_SMD:C_0603" H 1988 2250 30  0001 C CNN
+F 2 "stmbl:C_0603" H 1988 2250 30  0001 C CNN
 F 3 "" H 1950 2400 60  0000 C CNN
 	1    1950 2400
@@
 F 0 "C2" H 1125 2350 50  0000 L CNN
 F 1 "100n" H 1125 2150 50  0000 L CNN
-F 2 "Capacitors_SMD:C_0603" H 1138 2100 30  0001 C CNN
+F 2 "stmbl:C_0603" H 1138 2100 30  0001 C CNN
 F 3 "" H 1100 2250 60  0000 C CNN
 	1    1100 2250
@@
 F 0 "C7" H 2175 1700 50  0000 L CNN
 F 1 "100n" H 2175 1500 50  0000 L CNN
-F 2 "Capacitors_SMD:C_0603" H 2188 1450 30  0001 C CNN
+F 2 "stmbl:C_0603" H 2188 1450 30  0001 C CNN
 F 3 "" H 2150 1600 60  0000 C CNN
 	1    2150 1600
@@
 F 0 "C61" H 7575 5900 50  0000 L CNN
 F 1 "100n" H 7575 5700 50  0000 L CNN
-F 2 "Capacitors_SMD:C_0603" H 7588 5650 30  0001 C CNN
+F 2 "stmbl:C_0603" H 7588 5650 30  0001 C CNN
 F 3 "" H 7550 5800 60  0000 C CNN
 	1    7550 5800
@@
 F 0 "R2" V 880 2050 50  0000 C CNN
 F 1 "1k" V 800 2050 50  0000 C CNN
-F 2 "Resistors_SMD:R_0603" V 730 2050 30  0001 C CNN
+F 2 "stmbl:R_0603" V 730 2050 30  0001 C CNN
 F 3 "" H 800 2050 30  0000 C CNN
 	1    800  2050
@@
 F 0 "R129" V 17530 4500 50  0000 C CNN
 F 1 "1k" V 17450 4500 50  0000 C CNN
-F 2 "Resistors_SMD:R_0603" V 17380 4500 30  0001 C CNN
+F 2 "stmbl:R_0603" V 17380 4500 30  0001 C CNN
 F 3 "" H 17450 4500 30  0000 C CNN
 	1    17450 4500
@@
 F 0 "R8" V 18130 3700 50  0000 C CNN
 F 1 "560" V 18050 3700 50  0000 C CNN
-F 2 "Resistors_SMD:R_0603" V 17980 3700 30  0001 C CNN
+F 2 "stmbl:R_0603" V 17980 3700 30  0001 C CNN
 F 3 "" H 18050 3700 30  0000 C CNN
 	1    18050 3700
@@
 F 0 "L1" V 10250 1100 50  0000 C CNN
 F 1 "220r 700mA" V 10400 1100 50  0000 C CNN
-F 2 "Resistors_SMD:R_0603" H 10300 1100 50  0001 C CNN
+F 2 "stmbl:R_0603" H 10300 1100 50  0001 C CNN
 F 3 "" H 10300 1100 50  0000 C CNN
 	1    10300 1100
@@
 F 0 "C10" H 10725 1000 50  0000 L CNN
 F 1 "100n" H 10725 800 50  0000 L CNN
-F 2 "Capacitors_SMD:C_0603" H 10738 750 30  0001 C CNN
+F 2 "stmbl:C_0603" H 10738 750 30  0001 C CNN
 F 3 "" H 10700 900 60  0000 C CNN
 	1    10700 900
@@
 F 0 "C9" H 7175 5900 50  0000 L CNN
 F 1 "100n" H 7175 5700 50  0000 L CNN
-F 2 "Capacitors_SMD:C_0603" H 7188 5650 30  0001 C CNN
+F 2 "stmbl:C_0603" H 7188 5650 30  0001 C CNN
 F 3 "" H 7150 5800 60  0000 C CNN
 	1    7150 5800
@@
 F 0 "C128" H 2775 5750 50  0000 L CNN
 F 1 "100n" H 2775 5550 50  0000 L CNN
-F 2 "Capacitors_SMD:C_0603" H 2788 5500 30  0001 C CNN
+F 2 "stmbl:C_0603" H 2788 5500 30  0001 C CNN
 F 3 "" H 2750 5650 60  0000 C CNN
 	1    2750 5650

Commit message: v4.0
Parts:
- R8: value 560 -> 470
Changed lines of the file:
@@
 P 18050 3700
 F 0 "R8" V 18130 3700 50  0000 C CNN
-F 1 "560" V 18050 3700 50  0000 C CNN
+F 1 "470" V 18050 3700 50  0000 C CNN
 F 2 "stmbl:R_0603" V 17980 3700 30  0001 C CNN
 F 3 "" H 18050 3700 30  0000 C CNN

Commit message: v4.0
Parts:
- removed C61: 100n, stmbl:C_0603, symbol C
- removed U20: USBLC6-4SC6, TO_SOT_Packages_SMD:SOT-23-6, symbol USBLC6-4SC6
- JP1: footprint (none) -> stmbl:SOLDER_JUMPER
Changed lines of the file:
@@
 A_T_HV
-$Comp
-L USBLC6-4SC6 U20
-U 1 1 566A7439
-P 9400 5800
-F 0 "U20" H 8701 6148 50  0000 C CNN
-F 1 "USBLC6-4SC6" H 9400 6050 50  0000 C CNN
-F 2 "TO_SOT_Packages_SMD:SOT-23-6" H 9400 5800 60  0001 C CNN
-F 3 "" H 9400 5800 60  0000 C CNN
-F 4 "TRANSIENT VOLTAGE SUPPRESSOR" H 9400 5550 50  0000 C CNN "Description"
-	1    9400 5800
-	1    0    0    -1
-$EndComp
-Text HLabel 8150 5700 0    60   Input ~ 0
-A_U
-Text HLabel 8150 5900 0    60   Input ~ 0
-A_V
-Text HLabel 10650 5700 2    60   Input ~ 0
-A_W
-Text HLabel 10650 5900 2    60   Input ~ 0
-A_HV
-$Comp
-L GNDPWR #PWR020
-U 1 1 566A7681
-P 8250 6100
-F 0 "#PWR020" H 8250 5900 50  0001 C CNN
-F 1 "GNDPWR" H 8250 5970 50  0000 C CNN
-F 2 "" H 8250 6050 60  0000 C CNN
-F 3 "" H 8250 6050 60  0000 C CNN
-	1    8250 6100
-	1    0    0    -1
-$EndComp
-$Comp
-L +3.3VP #PWR021
-U 1 1 566A76B0
-P 10550 5500
-F 0 "#PWR021" H 10700 5450 50  0001 C CNN
-F 1 "+3.3VP" H 10550 5600 50  0000 C CNN
-F 2 "" H 10550 5500 60  0000 C CNN
-F 3 "" H 10550 5500 60  0000 C CNN
-	1    10550 5500
-	1    0    0    -1
-$EndComp
-$Comp
-L C C61
-U 1 1 566A7777
-P 7550 5800
-F 0 "C61" H 7575 5900 50  0000 L CNN
-F 1 "100n" H 7575 5700 50  0000 L CNN
-F 2 "stmbl:C_0603" H 7588 5650 30  0001 C CNN
-F 3 "" H 7550 5800 60  0000 C CNN
-	1    7550 5800
-	1    0    0    -1
-$EndComp
-$Comp
-L GNDPWR #PWR022
-U 1 1 566A77FF
-P 7550 6100
-F 0 "#PWR022" H 7550 5900 50  0001 C CNN
-F 1 "GNDPWR" H 7550 5970 50  0000 C CNN
-F 2 "" H 7550 6050 60  0000 C CNN
-F 3 "" H 7550 6050 60  0000 C CNN
-	1    7550 6100
-	1    0    0    -1
-$EndComp
-$Comp
-L +3.3VP #PWR023
-U 1 1 566A7831
-P 7550 5500
-F 0 "#PWR023" H 7700 5450 50  0001 C CNN
-F 1 "+3.3VP" H 7550 5600 50  0000 C CNN
-F 2 "" H 7550 5500 60  0000 C CNN
-F 3 "" H 7550 5500 60  0000 C CNN
-	1    7550 5500
-	1    0    0    -1
-$EndComp
 $Comp
 L R R2
@@
 $EndComp
 $Comp
-L GNDPWR #PWR024
+L GNDPWR #PWR020
 U 1 1 566A7E7E
 P 800 2300
-F 0 "#PWR024" H 800 2100 50  0001 C CNN
+F 0 "#PWR020" H 800 2100 50  0001 C CNN
 F 1 "GNDPWR" H 800 2170 50  0000 C CNN
 F 2 "" H 800 2250 60  0000 C CNN
@@
 $EndComp
 $Comp
-L +3.3VP #PWR025
+L +3.3VP #PWR021
 U 1 1 566A7F0A
 P 800 1400
-F 0 "#PWR025" H 950 1350 50  0001 C CNN
+F 0 "#PWR021" H 950 1350 50  0001 C CNN
 F 1 "+3.3VP" H 800 1500 50  0000 C CNN
 F 2 "" H 800 1400 60  0000 C CNN
@@
 F 0 "JP1" H 800 1680 50  0000 C CNN
 F 1 "Jumper_NO_Small" H 810 1540 50  0001 C CNN
-F 2 "" H 800 1600 60  0001 C CNN
+F 2 "stmbl:SOLDER_JUMPER" H 800 1600 60  0001 C CNN
 F 3 "" H 800 1600 60  0000 C CNN
 	1    800  1600
@@
 $EndComp
 $Comp
-L GNDPWR #PWR026
+L GNDPWR #PWR022
 U 1 1 56821409
 P 8250 6800
-F 0 "#PWR026" H 8250 6600 50  0001 C CNN
+F 0 "#PWR022" H 8250 6600 50  0001 C CNN
 F 1 "GNDPWR" H 8250 6670 50  0000 C CNN
 F 2 "" H 8250 6750 60  0000 C CNN
@@
 $EndComp
 $Comp
-L +3.3VP #PWR027
+L +3.3VP #PWR023
 U 1 1 56821444
 P 10550 6400
-F 0 "#PWR027" H 10700 6350 50  0001 C CNN
+F 0 "#PWR023" H 10700 6350 50  0001 C CNN
 F 1 "+3.3VP" H 10550 6500 50  0000 C CNN
 F 2 "" H 10550 6400 60  0000 C CNN
@@
 $EndComp
 $Comp
-L +3.3VP #PWR028
+L +3.3VP #PWR024
 U 1 1 57B2E8A4
 P 10950 1000
-F 0 "#PWR028" H 11100 950 50  0001 C CNN
+F 0 "#PWR024" H 11100 950 50  0001 C CNN
 F 1 "+3.3VP" H 10950 1100 50  0000 C CNN
 F 2 "" H 10950 1000 60  0000 C CNN
@@
 $EndComp
 $Comp
-L GNDPWR #PWR029
+L GNDPWR #PWR025
 U 1 1 57B30D4B
 P 7150 6100
-F 0 "#PWR029" H 7150 5900 50  0001 C CNN
+F 0 "#PWR025" H 7150 5900 50  0001 C CNN
 F 1 "GNDPWR" H 7150 5970 50  0000 C CNN
 F 2 "" H 7150 6050 60  0000 C CNN
@@
 $EndComp
 $Comp
-L +3.3VP #PWR030
+L +3.3VP #PWR026
 U 1 1 57B30D51
 P 7150 5500
-F 0 "#PWR030" H 7300 5450 50  0001 C CNN
+F 0 "#PWR026" H 7300 5450 50  0001 C CNN
 F 1 "+3.3VP" H 7150 5600 50  0000 C CNN
 F 2 "" H 7150 5500 60  0000 C CNN
@@
 $EndComp
 $Comp
-L GNDPWR #PWR031
+L GNDPWR #PWR027
 U 1 1 57DF4034
 P 2750 5950
-F 0 "#PWR031" H 2750 5750 50  0001 C CNN
+F 0 "#PWR027" H 2750 5750 50  0001 C CNN
 F 1 "GNDPWR" H 2750 5820 50  0000 C CNN
 F 2 "" H 2750 5900 60  0000 C CNN
@@
 $EndComp
 $Comp
-L +3.3VP #PWR032
+L +3.3VP #PWR028
 U 1 1 57DF403A
 P 2750 5350
-F 0 "#PWR032" H 2900 5300 50  0001 C CNN
+F 0 "#PWR028" H 2900 5300 50  0001 C CNN
 F 1 "+3.3VP" H 2750 5450 50  0000 C CNN
 F 2 "" H 2750 5350 60  0000 C CNN
@@
 IO_RX
 $Comp
-L GNDPWR #PWR033
+L GNDPWR #PWR029
 U 1 1 57F61589
 P 18300 3700
-F 0 "#PWR033" H 18300 3500 50  0001 C CNN
+F 0 "#PWR029" H 18300 3500 50  0001 C CNN
 F 1 "GNDPWR" H 18300 3570 50  0000 C CNN
 F 2 "" H 18300 3650 60  0000 C CNN
@@
 	800  1800 2500 1800
 Wire Wire Line
-	7550 6100 7550 5950
-Wire Wire Line
-	7550 5650 7550 5500
-Wire Wire Line
-	8250 5800 8350 5800
-Wire Wire Line
-	8250 6100 8250 5800
-Wire Wire Line
-	10550 5800 10550 5500
-Wire Wire Line
-	10450 5800 10550 5800
-Wire Wire Line
-	10450 5900 10650 5900
-Wire Wire Line
-	10450 5700 10650 5700
-Wire Wire Line
-	8150 5900 8350 5900
-Wire Wire Line
-	8150 5700 8350 5700
-Wire Wire Line
 	18050 4100 18600 4100

Commit message: v4.0
Parts:
- added P11: USB_OTG, stmbl:USB_Micro-B_10103594-0001LF, symbol USB_OTG
- added P7: CONN_01X03, Pin_Headers:Pin_Header_Straight_1x03, symbol CONN_01X03
- added R150: 1.5k, stmbl:R_0603, symbol R
- added R151, R152: 22, stmbl:R_0603, symbol R
Connections:
- net +3.3VP: now also U29.5 (VBUS), R150.2
- net A_HV: now also U25.25 (PB12/ADC4_IN3/COMP3_INM/I2C2_SMBA/I2S2_WS/OPAMP4_VOUT/SPI2_NSS/TIM1_BKIN/TSC_G6_IO2/USART3_CK)
- net A_IU: now also U25.18 (PB0/ADC3_IN12/COMP4_INP/OPAMP2_VINP/OPAMP2_VINP_SEC/OPAMP3_VINP/OPAMP3_VINP_SEC/TIM1_CH2N/TIM3_CH3/TIM8_CH2N/TSC_G3_IO2)
- net A_IV: now also U25.17 (ADC2_IN4/COMP2_INP/COMP2_OUT/OPAMP1_VINP/OPAMP1_VINP_SEC/OPAMP2_VINP/OPAMP2_VINP_SEC/SPI1_MOSI/TIM17_CH1/TIM1_CH1N/TIM3_CH2/TIM8_CH1N/TSC_G2_IO4/PA7)
- net A_IW: now also U25.11 (ADC1_IN2/COMP1_INP/OPAMP1_VINP/OPAMP1_VINP_SEC/OPAMP3_VINP/OPAMP3_VINP_SEC/RTC_REFIN/TIM15_CH1N/TIM2_CH2/TSC_G1_IO2/USART2_DE/USART2_RTS/PA1)
- net A_T_HV: now also U25.27 (PB14/ADC4_IN4/COMP3_INP/I2S2_ext_SD/OPAMP2_VINP/OPAMP2_VINP_SEC/SPI2_MISO/TIM15_CH1/TIM1_CH2N/TSC_G6_IO4/USART3_DE/USART3_RTS)
- net A_T_MOT: now also U25.28 (PB15/ADC1_EXTI15/ADC2_EXTI15/ADC4_IN5/COMP6_INM/I2S2_SD/RTC_REFIN/SPI2_MOSI/TIM15_CH1N/TIM15_CH2/TIM1_CH3N)
- net A_U: now also U25.26 (PB13/ADC3_IN5/COMP5_INP/I2S2_CK/OPAMP3_VINP/OPAMP3_VINP_SEC/OPAMP4_VINP/OPAMP4_VINP_SEC/SPI2_SCK/TIM1_CH1N/TSC_G6_IO3/USART3_CTS)
- net A_V: now also U25.15 (ADC2_IN2/COMP1_INM/COMP2_INM/COMP3_INM/COMP4_INM/COMP5_INM/COMP6_INM/COMP7_INM/DAC_OUT2/OPAMP1_VINP/OPAMP1_VINP_SEC/OPAMP2_VINM/OPAMP2_VINM_SEC/OPAMP3_VINP/OPAMP3_VINP_SEC/SPI1_SCK/TIM2_CH1/TIM2_ETR/TSC_G2_IO2/PA5)
- net A_W: now also U25.13 (ADC1_IN4/COMP2_INP/OPAMP1_VINM/OPAMP1_VINM_SEC/OPAMP1_VINP/OPAMP1_VINP_SEC/TIM15_CH2/TIM2_CH4/TSC_G1_IO4/USART2_RX/PA3)
- net GNDPWR: now also U29.2 (GND), P11.5 (GND), P11.6 (shield), P7.1 (P1)
- net IO_RX: now also U29.4 (I/O3), P7.2 (P2)
- net IO_TX: now also U29.6 (I/O4), P7.3 (P3)
- net NRST: now also U21.6 (I/O4)
- net SWCLK: now also U21.3 (I/O2)
- net SWDIO: now also U21.1 (I/O1)
- net USB_DM: now also U29.1 (I/O1), R151.1
- net USB_DP: now also U29.3 (I/O2), R152.1
- new net: P11.2 (D-), R151.2
- new net: P11.3 (D+), R150.1, R152.2
Other:
- moved on the sheet: C128, C9, U29

Commit message: v4.0
Parts:
- D1: footprint LEDs:LED-0603 -> LEDs:LED-0805
Changed lines of the file:
@@
 F 0 "D1" H 17600 3800 50  0000 C CNN
 F 1 "LED" H 17600 3600 50  0000 C CNN
-F 2 "LEDs:LED-0603" H 17600 3700 50  0001 C CNN
+F 2 "LEDs:LED-0805" H 17600 3700 50  0001 C CNN
 F 3 "" H 17600 3700 50  0000 C CNN
 	1    17600 3700

Commit message: v4.0
Parts:
- added R118: 1k, stmbl:R_0603, symbol R
Connections:
- net at C6.1, Y1.2: now also R118.2; no longer U25.6 (PF1/I2C2_SCL/RCC_OSC_OUT)
- new net: R118.1, U25.6 (PF1/I2C2_SCL/RCC_OSC_OUT)
Other:
- moved on the sheet: C5, C6, Y1
Changed lines of the file:
@@
 L Crystal Y1
 U 1 1 56631593
-P 2200 2250
-F 0 "Y1" H 2200 2400 50  0000 C CNN
-F 1 "8M" H 2200 2100 50  0000 C CNN
-F 2 "stmbl:Crystal_SMD_0603_4Pads" H 2200 2250 60  0001 C CNN
-F 3 "" H 2200 2250 60  0000 C CNN
-	1    2200 2250
+P 1900 2250
+F 0 "Y1" H 1900 2400 50  0000 C CNN
+F 1 "8M" H 1900 2100 50  0000 C CNN
+F 2 "stmbl:Crystal_SMD_0603_4Pads" H 1900 2250 60  0001 C CNN
+F 3 "" H 1900 2250 60  0000 C CNN
+	1    1900 2250
 	0    1    1    0
 $EndComp
@@
 L GNDPWR #PWR014
 U 1 1 566315E8
-P 1700 2100
-F 0 "#PWR014" H 1700 1900 50  0001 C CNN
-F 1 "GNDPWR" H 1700 1970 50  0000 C CNN
-F 2 "" H 1700 2050 60  0000 C CNN
-F 3 "" H 1700 2050 60  0000 C CNN
-	1    1700 2100
+P 1400 2100
+F 0 "#PWR014" H 1400 1900 50  0001 C CNN
+F 1 "GNDPWR" H 1400 1970 50  0000 C CNN
+F 2 "" H 1400 2050 60  0000 C CNN
+F 3 "" H 1400 2050 60  0000 C CNN
+	1    1400 2100
 	0    1    1    0
 $EndComp
@@
 L C C5
 U 1 1 56631605
-P 1950 2100
-F 0 "C5" H 1975 2200 50  0000 L CNN
-F 1 "18p" H 1975 2000 50  0000 L CNN
-F 2 "stmbl:C_0603" H 1988 1950 30  0001 C CNN
-F 3 "" H 1950 2100 60  0000 C CNN
-	1    1950 2100
+P 1650 2100
+F 0 "C5" H 1675 2200 50  0000 L CNN
+F 1 "18p" H 1675 2000 50  0000 L CNN
+F 2 "stmbl:C_0603" H 1688 1950 30  0001 C CNN
+F 3 "" H 1650 2100 60  0000 C CNN
+	1    1650 2100
 	0    1    1    0
 $EndComp
@@
 L GNDPWR #PWR015
 U 1 1 5663163A
-P 1700 2400
-F 0 "#PWR015" H 1700 2200 50  0001 C CNN
-F 1 "GNDPWR" H 1700 2270 50  0000 C CNN
-F 2 "" H 1700 2350 60  0000 C CNN
-F 3 "" H 1700 2350 60  0000 C CNN
-	1    1700 2400
+P 1400 2400
+F 0 "#PWR015" H 1400 2200 50  0001 C CNN
+F 1 "GNDPWR" H 1400 2270 50  0000 C CNN
+F 2 "" H 1400 2350 60  0000 C CNN
+F 3 "" H 1400 2350 60  0000 C CNN
+	1    1400 2400
 	0    1    1    0
 $EndComp
@@
 L C C6
 U 1 1 566316C7
-P 1950 2400
-F 0 "C6" H 1975 2500 50  0000 L CNN
-F 1 "18p" H 1975 2300 50  0000 L CNN
-F 2 "stmbl:C_0603" H 1988 2250 30  0001 C CNN
-F 3 "" H 1950 2400 60  0000 C CNN
-	1    1950 2400
+P 1650 2400
+F 0 "C6" H 1675 2500 50  0000 L CNN
+F 1 "18p" H 1675 2300 50  0000 L CNN
+F 2 "stmbl:C_0603" H 1688 2250 30  0001 C CNN
+F 3 "" H 1650 2400 60  0000 C CNN
+	1    1650 2400
 	0    1    1    0
 $EndComp
@@
 Wire Wire Line
 	1100 2000 2500 2000
-Connection ~ 2200 2100
+Connection ~ 1900 2100
 Wire Wire Line
 	2400 2100 2400 2200
 Wire Wire Line
 	2400 2200 2500 2200
-Connection ~ 2200 2400
+Connection ~ 1900 2400
 Wire Wire Line
 	2400 2300 2500 2300
@@
 	2400 2400 2400 2300
 Wire Wire Line
-	2100 2400 2400 2400
-Wire Wire Line
-	2100 2100 2400 2100
-Wire Wire Line
-	1700 2100 1800 2100
-Wire Wire Line
-	1700 2400 1800 2400
+	1800 2400 2000 2400
+Wire Wire Line
+	1800 2100 2400 2100
+Wire Wire Line
+	1400 2100 1500 2100
+Wire Wire Line
+	1400 2400 1500 2400
 Connection ~ 1100 2000
 Wire Wire Line
@@
 Wire Wire Line
 	2350 4400 2500 4400
+$Comp
+L R R118
+U 1 1 582CAB11
+P 2150 2400
+F 0 "R118" V 2230 2400 50  0000 C CNN
+F 1 "1k" V 2150 2400 50  0000 C CNN
+F 2 "stmbl:R_0603" V 2080 2400 30  0001 C CNN
+F 3 "" H 2150 2400 30  0000 C CNN
+	1    2150 2400
+	0    1    1    0
+$EndComp
+Wire Wire Line
+	2300 2400 2400 2400
 $EndSCHEMATC

Commit message: v4.0
Parts:
- D1: value LED -> red
Changed lines of the file:
@@
 P 17600 3700
 F 0 "D1" H 17600 3800 50  0000 C CNN
-F 1 "LED" H 17600 3600 50  0000 C CNN
+F 1 "red" H 17600 3600 50  0000 C CNN
 F 2 "LEDs:LED-0805" H 17600 3700 50  0001 C CNN
 F 3 "" H 17600 3700 50  0000 C CNN
