File: hw/kicad/v4.0/ctrl.sch (KiCad schematic (older format))
At the start: 2 parts, among them P14 CONN_01X04, U32 non_plated

Commit message: v4.0
Changed lines of the file:
@@
 F1 "supply.sch" 60
 F2 "EN_5V" I R 2900 4100 60
-F3 "EN_12V" I R 2900 4200 60
 $EndSheet
 $Sheet
@@
 Wire Wire Line
 	2900 4100 3100 4100
-Wire Wire Line
-	2900 4200 3100 4200
 $Sheet
 S 3100 700  1400 3800
@@
 F49 "IO_AIN1" I L 3100 2100 60
 F50 "EN_5V" I L 3100 4100 60
-F51 "EN_12V" I L 3100 4200 60
-F52 "IO_L0" I L 3100 1400 60
-F53 "IO_L1" I L 3100 1500 60
-F54 "IO_GREEN" I L 3100 1100 60
-F55 "IO_YELLOW" I L 3100 1200 60
-F56 "IO_RED" I L 3100 1300 60
-$EndSheet
-Wire Wire Line
+F51 "IO_L0" I L 3100 1400 60
+F52 "IO_L1" I L 3100 1500 60
+F53 "IO_GREEN" I L 3100 1100 60
+F54 "IO_YELLOW" I L 3100 1200 60
+F55 "IO_RED" I L 3100 1300 60
+$EndSheet
+Wire Wire Line

Commit message: v4.0
Parts:
- added LOGO1: OPEN_HARDWARE_1, Symbols:Symbol_OSHW-Logo_SilkScreen, symbol OPEN_HARDWARE_1
- P14: footprint Pin_Headers:Pin_Header_Angled_1x04 -> stmbl:Pin_Header_Angled_1x04
Changed lines of the file:
@@
 	1600 1800 1650 1800
 $Comp
-L +3.3V #PWR063
+L +3.3V #PWR63
 U 1 1 578427DC
 P 1650 1550
-F 0 "#PWR063" H 1650 1400 50  0001 C CNN
+F 0 "#PWR63" H 1650 1400 50  0001 C CNN
 F 1 "+3.3V" H 1650 1690 50  0000 C CNN
 F 2 "" H 1650 1550 50  0000 C CNN
@@
 	1650 1600 1600 1600
 $Comp
-L GND #PWR064
+L GND #PWR64
 U 1 1 57848EA2
 P 1650 1950
-F 0 "#PWR064" H 1650 1700 50  0001 C CNN
+F 0 "#PWR64" H 1650 1700 50  0001 C CNN
 F 1 "GND" H 1650 1800 50  0000 C CNN
 F 2 "" H 1650 1950 50  0000 C CNN
@@
 F 0 "P14" H 1400 2000 50  0000 C CNN
 F 1 "CONN_01X04" V 1500 1750 50  0000 C CNN
-F 2 "Pin_Headers:Pin_Header_Angled_1x04" H 1400 1750 50  0001 C CNN
+F 2 "stmbl:Pin_Header_Angled_1x04" H 1400 1750 50  0001 C CNN
 F 3 "" H 1400 1750 50  0000 C CNN
 	1    1400 1750
@@
 	1    0    0    -1
 $EndComp
+$Comp
+L OPEN_HARDWARE_1 LOGO1
+U 1 1 58341DA7
+P 2400 5400
+F 0 "LOGO1" H 2400 5675 50  0000 C CNN
+F 1 "OPEN_HARDWARE_1" H 2400 5175 50  0000 C CNN
+F 2 "Symbols:Symbol_OSHW-Logo_SilkScreen" H 2400 5400 60  0001 C CNN
+F 3 "" H 2400 5400 60  0001 C CNN
+	1    2400 5400
+	1    0    0    -1
+$EndComp

Commit message: stmbl 4.2 wip
Parts:
- LOGO1: symbol OPEN_HARDWARE_1 -> stmbl1:OPEN_HARDWARE_1
- P14: symbol CONN_01X04 -> stmbl1:CONN_01X04
- U32: symbol non_plated -> stmbl1:non_plated
Changed lines of the file:
@@
-EESchema Schematic File Version 2
-LIBS:transistors
-LIBS:stm32
-LIBS:conn
-LIBS:power
-LIBS:74xgxx
-LIBS:74xx
-LIBS:ac-dc
-LIBS:actel
-LIBS:adc-dac
-LIBS:Altera
-LIBS:analog_devices
-LIBS:analog_switches
-LIBS:atmel
-LIBS:audio
-LIBS:brooktre
-LIBS:cmos_ieee
-LIBS:cmos4000
-LIBS:contrib
-LIBS:cypress
-LIBS:dc-dc
-LIBS:device
-LIBS:digital-audio
-LIBS:diode
-LIBS:display
-LIBS:dsp
-LIBS:elec-unifil
-LIBS:ESD_Protection
-LIBS:ftdi
-LIBS:gennum
-LIBS:graphic
-LIBS:hc11
-LIBS:intel
-LIBS:interface
-LIBS:ir
-LIBS:Lattice
-LIBS:linear
-LIBS:logo
-LIBS:maxim
-LIBS:memory
-LIBS:microchip_dspic33dsc
-LIBS:microchip_pic10mcu
-LIBS:microchip_pic12mcu
-LIBS:microchip_pic16mcu
-LIBS:microchip_pic18mcu
-LIBS:microchip_pic32mcu
-LIBS:microchip
-LIBS:microcontrollers
-LIBS:motor_drivers
-LIBS:motorola
-LIBS:msp430
-LIBS:nordicsemi
-LIBS:nxp_armmcu
-LIBS:onsemi
-LIBS:opto
-LIBS:Oscillators
-LIBS:philips
-LIBS:Power_Management
-LIBS:powerint
-LIBS:pspice
-LIBS:references
-LIBS:regul
-LIBS:relays
-LIBS:rfcom
-LIBS:sensors
-LIBS:silabs
-LIBS:siliconi
-LIBS:stm8
-LIBS:supertex
-LIBS:switches
-LIBS:texas
-LIBS:transf
-LIBS:ttl_ieee
-LIBS:valves
-LIBS:video
-LIBS:Xicor
-LIBS:xilinx
-LIBS:Zilog
+EESchema Schematic File Version 4
 LIBS:stmbl_4.0-cache
-EELAYER 25 0
+EELAYER 26 0
 EELAYER END
 $Descr A4 11693 8268
@@
 	1600 1800 1650 1800
 $Comp
-L +3.3V #PWR070
+L stmbl1:+3.3V #PWR070
 U 1 1 578427DC
 P 1650 1550
@@
 	1650 1600 1600 1600
 $Comp
-L GND #PWR071
+L stmbl1:GND #PWR071
 U 1 1 57848EA2
 P 1650 1950
@@
 	1650 1900 1650 1950
 $Comp
-L CONN_01X04 P14
+L stmbl1:CONN_01X04 P14
 U 1 1 57AEB2FC
 P 1400 1750
@@
 	3100 1750 2900 1750
 $Comp
-L non_plated U32
+L stmbl1:non_plated U32
 U 1 1 5830D361
 P 6450 1250
@@
 $EndComp
 $Comp
-L OPEN_HARDWARE_1 LOGO1
+L stmbl1:OPEN_HARDWARE_1 LOGO1
 U 1 1 58341DA7
 P 2400 5400

Commit message: stmbl 4.2
Parts:
- LOGO1: footprint Symbols:Symbol_OSHW-Logo_SilkScreen -> stmbl:Symbol_OSHW-Logo_SilkScreen
Changed lines of the file:
@@
 F 0 "LOGO1" H 2400 5675 50  0000 C CNN
 F 1 "OPEN_HARDWARE_1" H 2400 5175 50  0000 C CNN
-F 2 "Symbols:Symbol_OSHW-Logo_SilkScreen" H 2400 5400 60  0001 C CNN
+F 2 "stmbl:Symbol_OSHW-Logo_SilkScreen" H 2400 5400 60  0001 C CNN
 F 3 "" H 2400 5400 60  0001 C CNN
 	1    2400 5400

Commit message: stmbl 4.2 bom
Parts:
- P14: Manufacturer No (none) -> (none); Source (none) -> (none); Voltage (none) -> (none)
Changed lines of the file:
@@
 F 2 "stmbl:Pin_Header_Angled_1x04" H 1400 1750 50  0001 C CNN
 F 3 "" H 1400 1750 50  0000 C CNN
+F 4 " " H 1400 1750 50  0001 C CNN "Manufacturer No"
+F 5 " " H 1400 1750 50  0001 C CNN "Voltage"
+F 6 " " H 1400 1750 50  0001 C CNN "Source"
 	1    1400 1750
 	-1   0    0    1
