File: hw/kicad/v4.0/stmbl_4.0.sch (KiCad schematic (older format))
At the start: 2 parts

Commit message: v4.0
Connections:
- net hv/RX is gone; now on net ctrl/TX: P?.3 (P3)
- net hv/TX is gone; now on net ctrl/RX: P?.2 (P2)
Changed lines of the file:
@@
 LIBS:transistors
 LIBS:stm32
-LIBS:stmbl_3.4-cache
+LIBS:texas
+LIBS:diode
+LIBS:opto
+LIBS:display
+LIBS:device
+LIBS:stmbl_4.0-cache
 EELAYER 25 0
 EELAYER END
@@
 $EndComp
 Wire Wire Line
-	6250 2500 6500 2500
+	4950 2500 6500 2500
 Wire Wire Line
-	6250 2600 6500 2600
+	4950 2600 6500 2600
 Wire Wire Line
-	6250 2700 6350 2700
+	5100 2700 6350 2700
 Wire Wire Line
 	6350 2700 6350 2800
 Wire Wire Line
-	6250 2400 6350 2400
+	5100 2400 6350 2400
 Wire Wire Line
 	6350 2400 6350 2300
@@
 	5100 2300 5100 2400
 Wire Wire Line
-	5100 2400 5200 2400
-Wire Wire Line
-	5200 2700 5100 2700
-Wire Wire Line
 	5100 2700 5100 2800
-Wire Wire Line
-	4950 2500 5200 2500
-Wire Wire Line
-	4950 2600 5200 2600
+Connection ~ 6250 2400
+Connection ~ 5200 2400
+Connection ~ 6250 2500
+Connection ~ 5200 2500
+Connection ~ 6250 2600
+Connection ~ 5200 2600
+Connection ~ 6250 2700
+Connection ~ 5200 2700
 $EndSCHEMATC

Commit message: v4.0
Parts:
- P13: renamed from P?; footprint (none) -> Pin_Headers:Pin_Header_Angled_2x02
- P14: renamed from P?; footprint (none) -> Pin_Headers:Pin_Header_Straight_2x02
Changed lines of the file:
@@
 LIBS:transistors
 LIBS:stm32
-LIBS:texas
-LIBS:diode
-LIBS:opto
-LIBS:display
-LIBS:device
+LIBS:conn
 LIBS:stmbl_4.0-cache
 EELAYER 25 0
@@
 $EndSheet
 $Comp
-L CONN_01X04 P?
+L CONN_01X04 P13
 U 1 1 566A9008
 P 5400 2550
-F 0 "P?" H 5400 2800 50  0000 C CNN
+F 0 "P13" H 5400 2800 50  0000 C CNN
 F 1 "CONN_01X04" V 5500 2550 50  0000 C CNN
-F 2 "" H 5400 2550 60  0000 C CNN
+F 2 "Pin_Headers:Pin_Header_Angled_2x02" H 5400 2550 60  0001 C CNN
 F 3 "" H 5400 2550 60  0000 C CNN
 	1    5400 2550
@@
 $EndComp
 $Comp
-L CONN_01X04 P?
+L CONN_01X04 P14
 U 1 1 566A906D
 P 6050 2550
-F 0 "P?" H 6050 2800 50  0000 C CNN
+F 0 "P14" H 6050 2800 50  0000 C CNN
 F 1 "CONN_01X04" V 6150 2550 50  0000 C CNN
-F 2 "" H 6050 2550 60  0000 C CNN
+F 2 "Pin_Headers:Pin_Header_Straight_2x02" H 6050 2550 60  0001 C CNN
 F 3 "" H 6050 2550 60  0000 C CNN
 	1    6050 2550
@@
 $EndComp
 $Comp
-L GND #PWR?
+L GND #PWR184
 U 1 1 566A90FF
 P 6350 2800
-F 0 "#PWR?" H 6350 2550 50  0001 C CNN
+F 0 "#PWR184" H 6350 2550 50  0001 C CNN
 F 1 "GND" H 6350 2650 50  0000 C CNN
 F 2 "" H 6350 2800 60  0000 C CNN
@@
 $EndComp
 $Comp
-L GND #PWR?
+L GND #PWR182
 U 1 1 566A912B
 P 5100 2800
-F 0 "#PWR?" H 5100 2550 50  0001 C CNN
+F 0 "#PWR182" H 5100 2550 50  0001 C CNN
 F 1 "GND" H 5100 2650 50  0000 C CNN
 F 2 "" H 5100 2800 60  0000 C CNN
@@
 $EndComp
 $Comp
-L +3.3V #PWR?
+L +3.3V #PWR181
 U 1 1 566A9173
 P 5100 2300
-F 0 "#PWR?" H 5100 2150 50  0001 C CNN
+F 0 "#PWR181" H 5100 2150 50  0001 C CNN
 F 1 "+3.3V" H 5100 2440 50  0000 C CNN
 F 2 "" H 5100 2300 60  0000 C CNN
@@
 $EndComp
 $Comp
-L +3.3V #PWR?
+L +3.3V #PWR183
 U 1 1 566A919F
 P 6350 2300
-F 0 "#PWR?" H 6350 2150 50  0001 C CNN
+F 0 "#PWR183" H 6350 2150 50  0001 C CNN
 F 1 "+3.3V" H 6350 2440 50  0000 C CNN
 F 2 "" H 6350 2300 60  0000 C CNN

Commit message: v4.0
Parts:
- removed P13: CONN_01X04, Pin_Headers:Pin_Header_Angled_2x02, symbol CONN_01X04
- removed P14: CONN_01X04, Pin_Headers:Pin_Header_Straight_2x02, symbol CONN_01X04
Changed lines of the file:
@@
 LIBS:stm32
 LIBS:conn
+LIBS:power
 LIBS:stmbl_4.0-cache
 EELAYER 25 0
@@
 $Descr A4 11693 8268
 encoding utf-8
-Sheet 1 14
+Sheet 1 15
 Title ""
 Date ""
@@
 $EndDescr
 $Sheet
-S 6500 2300 600  500
+S 5500 2300 600  500
 U 5659094D
 F0 "hv" 60
 F1 "hv.sch" 60
-F2 "TX" I L 6500 2500 60
-F3 "RX" I L 6500 2600 60
+F2 "TX" I L 5500 2500 60
+F3 "RX" I L 5500 2600 60
 $EndSheet
 $Sheet
@@
 F3 "RX" I R 4950 2500 60
 $EndSheet
-$Comp
-L CONN_01X04 P13
-U 1 1 566A9008
-P 5400 2550
-F 0 "P13" H 5400 2800 50  0000 C CNN
-F 1 "CONN_01X04" V 5500 2550 50  0000 C CNN
-F 2 "Pin_Headers:Pin_Header_Angled_2x02" H 5400 2550 60  0001 C CNN
-F 3 "" H 5400 2550 60  0000 C CNN
-	1    5400 2550
-	1    0    0    -1
-$EndComp
-$Comp
-L CONN_01X04 P14
-U 1 1 566A906D
-P 6050 2550
-F 0 "P14" H 6050 2800 50  0000 C CNN
-F 1 "CONN_01X04" V 6150 2550 50  0000 C CNN
-F 2 "Pin_Headers:Pin_Header_Straight_2x02" H 6050 2550 60  0001 C CNN
-F 3 "" H 6050 2550 60  0000 C CNN
-	1    6050 2550
-	-1   0    0    -1
-$EndComp
-$Comp
-L GND #PWR4
-U 1 1 566A90FF
-P 6350 2800
-F 0 "#PWR4" H 6350 2550 50  0001 C CNN
-F 1 "GND" H 6350 2650 50  0000 C CNN
-F 2 "" H 6350 2800 60  0000 C CNN
-F 3 "" H 6350 2800 60  0000 C CNN
-	1    6350 2800
-	1    0    0    -1
-$EndComp
-$Comp
-L GND #PWR2
-U 1 1 566A912B
-P 5100 2800
-F 0 "#PWR2" H 5100 2550 50  0001 C CNN
-F 1 "GND" H 5100 2650 50  0000 C CNN
-F 2 "" H 5100 2800 60  0000 C CNN
-F 3 "" H 5100 2800 60  0000 C CNN
-	1    5100 2800
-	1    0    0    -1
-$EndComp
-$Comp
-L +3.3V #PWR1
-U 1 1 566A9173
-P 5100 2300
-F 0 "#PWR1" H 5100 2150 50  0001 C CNN
-F 1 "+3.3V" H 5100 2440 50  0000 C CNN
-F 2 "" H 5100 2300 60  0000 C CNN
-F 3 "" H 5100 2300 60  0000 C CNN
-	1    5100 2300
-	1    0    0    -1
-$EndComp
-$Comp
-L +3.3V #PWR3
-U 1 1 566A919F
-P 6350 2300
-F 0 "#PWR3" H 6350 2150 50  0001 C CNN
-F 1 "+3.3V" H 6350 2440 50  0000 C CNN
-F 2 "" H 6350 2300 60  0000 C CNN
-F 3 "" H 6350 2300 60  0000 C CNN
-	1    6350 2300
-	1    0    0    -1
-$EndComp
 Wire Wire Line
-	4950 2500 6500 2500
+	4950 2500 5500 2500
 Wire Wire Line
-	4950 2600 6500 2600
-Wire Wire Line
-	5100 2700 6350 2700
-Wire Wire Line
-	6350 2700 6350 2800
-Wire Wire Line
-	5100 2400 6350 2400
-Wire Wire Line
-	6350 2400 6350 2300
-Wire Wire Line
-	5100 2300 5100 2400
-Wire Wire Line
-	5100 2700 5100 2800
-Connection ~ 6250 2400
-Connection ~ 5200 2400
-Connection ~ 6250 2500
-Connection ~ 5200 2500
-Connection ~ 6250 2600
-Connection ~ 5200 2600
-Connection ~ 6250 2700
-Connection ~ 5200 2700
+	4950 2600 5500 2600
 $EndSCHEMATC

Commit message: v4.0
Changed lines of the file:
@@
 LIBS:conn
 LIBS:power
+LIBS:74xgxx
+LIBS:74xx
+LIBS:ac-dc
+LIBS:actel
+LIBS:adc-dac
+LIBS:Altera
+LIBS:analog_devices
+LIBS:analog_switches
+LIBS:atmel
+LIBS:audio
+LIBS:brooktre
+LIBS:cmos_ieee
+LIBS:cmos4000
+LIBS:contrib
+LIBS:cypress
+LIBS:dc-dc
+LIBS:device
+LIBS:digital-audio
+LIBS:diode
+LIBS:display
+LIBS:dsp
+LIBS:elec-unifil
+LIBS:ESD_Protection
+LIBS:ftdi
+LIBS:gennum
+LIBS:graphic
+LIBS:hc11
+LIBS:intel
+LIBS:interface
+LIBS:ir
+LIBS:Lattice
+LIBS:linear
+LIBS:logo
+LIBS:maxim
+LIBS:memory
+LIBS:microchip_dspic33dsc
+LIBS:microchip_pic10mcu
+LIBS:microchip_pic12mcu
+LIBS:microchip_pic16mcu
+LIBS:microchip_pic18mcu
+LIBS:microchip_pic32mcu
+LIBS:microchip
+LIBS:microcontrollers
+LIBS:motor_drivers
+LIBS:motorola
+LIBS:msp430
+LIBS:nordicsemi
+LIBS:nxp_armmcu
+LIBS:onsemi
+LIBS:opto
+LIBS:Oscillators
+LIBS:philips
+LIBS:Power_Management
+LIBS:powerint
+LIBS:pspice
+LIBS:references
+LIBS:regul
+LIBS:relays
+LIBS:rfcom
+LIBS:sensors
+LIBS:silabs
+LIBS:siliconi
+LIBS:stm8
+LIBS:supertex
+LIBS:switches
+LIBS:texas
+LIBS:transf
+LIBS:ttl_ieee
+LIBS:valves
+LIBS:video
+LIBS:Xicor
+LIBS:xilinx
+LIBS:Zilog
 LIBS:stmbl_4.0-cache
 EELAYER 25 0
@@
 $Descr A4 11693 8268
 encoding utf-8
-Sheet 1 15
+Sheet 1 14
 Title ""
 Date ""
@@
 F0 "hv" 60
 F1 "hv.sch" 60
-F2 "TX" I L 5500 2500 60
-F3 "RX" I L 5500 2600 60
+F2 "TX" I L 5500 2600 60
+F3 "RX" I L 5500 2500 60
 $EndSheet
 $Sheet

Commit message: stmbl 4.2 wip
Parts:
- added U33, U34, U35, U36, U37, U39: non_plated, stmbl:non_plated_1mm, symbol stmbl1:non_plated
Changed lines of the file:
@@
-EESchema Schematic File Version 2
-LIBS:transistors
-LIBS:stm32
-LIBS:conn
-LIBS:power
-LIBS:74xgxx
-LIBS:74xx
-LIBS:ac-dc
-LIBS:actel
-LIBS:adc-dac
-LIBS:Altera
-LIBS:analog_devices
-LIBS:analog_switches
-LIBS:atmel
-LIBS:audio
-LIBS:brooktre
-LIBS:cmos_ieee
-LIBS:cmos4000
-LIBS:contrib
-LIBS:cypress
-LIBS:dc-dc
-LIBS:device
-LIBS:digital-audio
-LIBS:diode
-LIBS:display
-LIBS:dsp
-LIBS:elec-unifil
-LIBS:ESD_Protection
-LIBS:ftdi
-LIBS:gennum
-LIBS:graphic
-LIBS:hc11
-LIBS:intel
-LIBS:interface
-LIBS:ir
-LIBS:Lattice
-LIBS:linear
-LIBS:logo
-LIBS:maxim
-LIBS:memory
-LIBS:microchip_dspic33dsc
-LIBS:microchip_pic10mcu
-LIBS:microchip_pic12mcu
-LIBS:microchip_pic16mcu
-LIBS:microchip_pic18mcu
-LIBS:microchip_pic32mcu
-LIBS:microchip
-LIBS:microcontrollers
-LIBS:motor_drivers
-LIBS:motorola
-LIBS:msp430
-LIBS:nordicsemi
-LIBS:nxp_armmcu
-LIBS:onsemi
-LIBS:opto
-LIBS:Oscillators
-LIBS:philips
-LIBS:Power_Management
-LIBS:powerint
-LIBS:pspice
-LIBS:references
-LIBS:regul
-LIBS:relays
-LIBS:rfcom
-LIBS:sensors
-LIBS:silabs
-LIBS:siliconi
-LIBS:stm8
-LIBS:supertex
-LIBS:switches
-LIBS:texas
-LIBS:transf
-LIBS:ttl_ieee
-LIBS:valves
-LIBS:video
-LIBS:Xicor
-LIBS:xilinx
-LIBS:Zilog
+EESchema Schematic File Version 4
 LIBS:stmbl_4.0-cache
-EELAYER 25 0
+EELAYER 26 0
 EELAYER END
 $Descr A4 11693 8268
@@
 Wire Wire Line
 	4950 2600 5500 2600
+$Comp
+L stmbl1:non_plated U33
+U 1 1 5AC37C2D
+P 4600 4100
+F 0 "U33" H 4600 3750 60  0000 C CNN
+F 1 "non_plated" H 4650 4350 60  0000 C CNN
+F 2 "stmbl:non_plated_1mm" H 4600 4100 60  0001 C CNN
+F 3 "" H 4600 4100 60  0001 C CNN
+	1    4600 4100
+	1    0    0    -1
+$EndComp
+$Comp
+L stmbl1:non_plated U35
+U 1 1 5AC37C5C
+P 5200 4100
+F 0 "U35" H 5200 3750 60  0000 C CNN
+F 1 "non_plated" H 5250 4350 60  0000 C CNN
+F 2 "stmbl:non_plated_1mm" H 5200 4100 60  0001 C CNN
+F 3 "" H 5200 4100 60  0001 C CNN
+	1    5200 4100
+	1    0    0    -1
+$EndComp
+$Comp
+L stmbl1:non_plated U34
+U 1 1 5AC37CB2
+P 4600 4800
+F 0 "U34" H 4600 4450 60  0000 C CNN
+F 1 "non_plated" H 4650 5050 60  0000 C CNN
+F 2 "stmbl:non_plated_1mm" H 4600 4800 60  0001 C CNN
+F 3 "" H 4600 4800 60  0001 C CNN
+	1    4600 4800
+	1    0    0    -1
+$EndComp
+$Comp
+L stmbl1:non_plated U36
+U 1 1 5AC37CB8
+P 5200 4800
+F 0 "U36" H 5200 4450 60  0000 C CNN
+F 1 "non_plated" H 5250 5050 60  0000 C CNN
+F 2 "stmbl:non_plated_1mm" H 5200 4800 60  0001 C CNN
+F 3 "" H 5200 4800 60  0001 C CNN
+	1    5200 4800
+	1    0    0    -1
+$EndComp
+$Comp
+L stmbl1:non_plated U37
+U 1 1 5AC37D5D
+P 5750 4100
+F 0 "U37" H 5750 3750 60  0000 C CNN
+F 1 "non_plated" H 5800 4350 60  0000 C CNN
+F 2 "stmbl:non_plated_1mm" H 5750 4100 60  0001 C CNN
+F 3 "" H 5750 4100 60  0001 C CNN
+	1    5750 4100
+	1    0    0    -1
+$EndComp
+$Comp
+L stmbl1:non_plated U39
+U 1 1 5AC37D64
+P 5750 4800
+F 0 "U39" H 5750 4450 60  0000 C CNN
+F 1 "non_plated" H 5800 5050 60  0000 C CNN
+F 2 "stmbl:non_plated_1mm" H 5750 4800 60  0001 C CNN
+F 3 "" H 5750 4800 60  0001 C CNN
+	1    5750 4800
+	1    0    0    -1
+$EndComp
 $EndSCHEMATC

Commit message: stmbl 4.2 bom
Parts:
- removed U33, U34, U35, U36, U37, U39: non_plated, stmbl:non_plated_1mm, symbol stmbl1:non_plated
Changed lines of the file:
@@
 Wire Wire Line
 	4950 2600 5500 2600
-$Comp
-L stmbl1:non_plated U33
-U 1 1 5AC37C2D
-P 4600 4100
-F 0 "U33" H 4600 3750 60  0000 C CNN
-F 1 "non_plated" H 4650 4350 60  0000 C CNN
-F 2 "stmbl:non_plated_1mm" H 4600 4100 60  0001 C CNN
-F 3 "" H 4600 4100 60  0001 C CNN
-	1    4600 4100
-	1    0    0    -1
-$EndComp
-$Comp
-L stmbl1:non_plated U35
-U 1 1 5AC37C5C
-P 5200 4100
-F 0 "U35" H 5200 3750 60  0000 C CNN
-F 1 "non_plated" H 5250 4350 60  0000 C CNN
-F 2 "stmbl:non_plated_1mm" H 5200 4100 60  0001 C CNN
-F 3 "" H 5200 4100 60  0001 C CNN
-	1    5200 4100
-	1    0    0    -1
-$EndComp
-$Comp
-L stmbl1:non_plated U34
-U 1 1 5AC37CB2
-P 4600 4800
-F 0 "U34" H 4600 4450 60  0000 C CNN
-F 1 "non_plated" H 4650 5050 60  0000 C CNN
-F 2 "stmbl:non_plated_1mm" H 4600 4800 60  0001 C CNN
-F 3 "" H 4600 4800 60  0001 C CNN
-	1    4600 4800
-	1    0    0    -1
-$EndComp
-$Comp
-L stmbl1:non_plated U36
-U 1 1 5AC37CB8
-P 5200 4800
-F 0 "U36" H 5200 4450 60  0000 C CNN
-F 1 "non_plated" H 5250 5050 60  0000 C CNN
-F 2 "stmbl:non_plated_1mm" H 5200 4800 60  0001 C CNN
-F 3 "" H 5200 4800 60  0001 C CNN
-	1    5200 4800
-	1    0    0    -1
-$EndComp
-$Comp
-L stmbl1:non_plated U37
-U 1 1 5AC37D5D
-P 5750 4100
-F 0 "U37" H 5750 3750 60  0000 C CNN
-F 1 "non_plated" H 5800 4350 60  0000 C CNN
-F 2 "stmbl:non_plated_1mm" H 5750 4100 60  0001 C CNN
-F 3 "" H 5750 4100 60  0001 C CNN
-	1    5750 4100
-	1    0    0    -1
-$EndComp
-$Comp
-L stmbl1:non_plated U39
-U 1 1 5AC37D64
-P 5750 4800
-F 0 "U39" H 5750 4450 60  0000 C CNN
-F 1 "non_plated" H 5800 5050 60  0000 C CNN
-F 2 "stmbl:non_plated_1mm" H 5750 4800 60  0001 C CNN
-F 3 "" H 5750 4800 60  0001 C CNN
-	1    5750 4800
-	1    0    0    -1
-$EndComp
 $EndSCHEMATC
