File: hw/kicad/bob/db25_bob_v2/led.sch (KiCad schematic (older format))
At the start: 40 parts, among them U20 74HC595, U21 74HC595, U22 74HC595, U23 74HC595, U24 74HC595, U25 74HC595, U26 74HC595, U27 74HC595

Commit message: More routing + schematic changes
Parts:
- removed U22, U23, U25, U26, U27: 74HC595, SMD_Packages:SO-16-N, symbol 74HC595
Changed lines of the file:
@@
-$EndComp
-$Comp
-L 74HC595 U23
-U 1 1 57450DF6
-P 7400 4800
-F 0 "U23" H 7400 5566 50  0000 C CNN
-F 1 "74HC595" H 7400 5475 50  0000 C CNN
-F 2 "SMD_Packages:SO-16-N" H 7400 4800 50  0001 C CNN
-F 3 "" H 7400 4800 50  0000 C CNN
-	1    7400 4800
-	1    0    0    -1
 $EndComp
 $Comp
@@
 	1    0    0    -1
 $EndComp
-$Comp
-L 74HC595 U25
-U 1 1 574511F5
-P 9300 2500
-F 0 "U25" H 9300 3266 50  0000 C CNN
-F 1 "74HC595" H 9300 3175 50  0000 C CNN
-F 2 "SMD_Packages:SO-16-N" H 9300 2500 50  0001 C CNN
-F 3 "" H 9300 2500 50  0000 C CNN
-	1    9300 2500
-	1    0    0    -1
-$EndComp
-$Comp
-L 74HC595 U27
-U 1 1 574511FB
-P 9300 4800
-F 0 "U27" H 9300 5566 50  0000 C CNN
-F 1 "74HC595" H 9300 5475 50  0000 C CNN
-F 2 "SMD_Packages:SO-16-N" H 9300 4800 50  0001 C CNN
-F 3 "" H 9300 4800 50  0000 C CNN
-	1    9300 4800
-	1    0    0    -1
-$EndComp
-$Comp
-L 74HC595 U22
-U 1 1 574514E5
-P 7400 3650
-F 0 "U22" H 7400 4416 50  0000 C CNN
-F 1 "74HC595" H 7400 4325 50  0000 C CNN
-F 2 "SMD_Packages:SO-16-N" H 7400 3650 50  0001 C CNN
-F 3 "" H 7400 3650 50  0000 C CNN
-	1    7400 3650
-	1    0    0    -1
-$EndComp
-$Comp
-L 74HC595 U26
-U 1 1 574514EB
-P 9300 3650
-F 0 "U26" H 9300 4416 50  0000 C CNN
-F 1 "74HC595" H 9300 4325 50  0000 C CNN
-F 2 "SMD_Packages:SO-16-N" H 9300 3650 50  0001 C CNN
-F 3 "" H 9300 3650 50  0000 C CNN
-	1    9300 3650
-	1    0    0    -1
-$EndComp

Commit message: More stuff.
Parts:
- removed D10, D11, D12, D13, D14, D15, D16, D17, D18, D19, D20, D21, D22, D23, D24, D25, D26, D27, D28, D29, D3, D30, D31, D32, D33, D34, D4, D5, D6, D7, D8, D9: Led_x2, LEDs:LED_0805, symbol Led_x2
- removed U24: 74HC595, SMD_Packages:SO-16-N, symbol 74HC595
- added D31, D32, D33, D34, D35, D36, D37, D38, D39, D40, D41, D42, D43, D44, D45, D46, D47, D48, D49, D50, D51, D52, D53, D54, D55, D56, D57, D58, D59, D60, D61, D62: LED, LEDs:LED_0603, symbol LED
