File: hw/kicad/bob/db25_bob_v2/db25_bob_v2.kicad_pcb (KiCad board)
At the start: 2 copper layers, 100 x 100 mm, 94 parts, among them J1 RJ45, J2 RJ45, J3 RJ45, J4 RJ45, J5 RJ45, J6 RJ45, J7 RJ45, J8 RJ45, P1 CONN_01X08, P2 CONN_01X08, P3 CONN_01X08, P4 CONN_01X08, P5 CONN_01X08, P6 CONN_01X08, P7 CONN_01X08, P8 CONN_01X08, U1 STM32F303CBTx, U10 ADM4857, U11 ADuM1201WT, U12 ADM4857, U13 ADuM1201WT, U14 ADM4857, U15 ADuM1201WT, U16 ADM4857, U17 ADuM1201WT, U18 NCV7608, U19 NCV7608, U2 ADM4857, U20 74HC595, U21 74HC595, U22 74HC595, U23 74HC595, U24 74HC595, U25 74HC595, U26 74HC595, U27 74HC595, U28 ADuM1201WT, U3 ADuM1201WT, U4 ADM4857, U5 ADuM1201WT, U6 ADM4857, U7 ADuM1201WT, U8 ADM4857, U9 ADuM1201WT

Commit message: More routing + schematic changes
Parts:
- added C1: C, Capacitors_SMD:C_1206, B.Cu at (163.8, 68.2)
- added J9: DB25, Connect:DB25FD, F.Cu at (102.0, 98.7)
- U1: moved to B.Cu
- moved C9 82.6 mm to (39.6, 110.7)
- moved D1 82.6 mm to (38.6, 113.1)
- moved D2 82.6 mm to (41.3, 115.5)
- moved R2 82.6 mm to (40.0, 107.6)
- moved JP2 44.5 mm to (190.0, 91.6)
- moved JP1 31.1 mm to (197.6, 93.6)
- moved U28 20.0 mm to (226.1, 122.1)
- moved U1 14.6 mm to (118.6, 100.3), turned to 90 degrees
Connections:
- net IN10 renamed AIN10
- net IN11 renamed AIN11
- net IN12 renamed AIN12
- net IN13 renamed AIN13
- net IN14 renamed AIN14
- net IN15 renamed AIN15
- net IN16 renamed AESTOP
- net IN8 renamed AIN8
- net IN9 renamed AIN9
- C3 pad 1: 5V8 -> 5V3
- C3 pad 2: GND8 -> GND3
- C4 pad 1: 5V2 -> 5V5
- C4 pad 2: GND2 -> GND5
- C5 pad 1: 5V3 -> 5V8
- C5 pad 2: GND3 -> GND8
- C6 pad 1: 5V4 -> 5V2
- C6 pad 2: GND4 -> GND2
- C7 pad 1: 5V5 -> 5V4
- C7 pad 2: GND5 -> GND4
- J2 pad 9: GND1 -> Net-(J2-Pad9)
- J3 pad 7: 5V8 -> 5V3
- J3 pad 8: GND8 -> GND3
- J4 pad 7: 5V2 -> 5V5
- J4 pad 8: GND2 -> GND5
- J4 pad 9: GND2 -> Net-(J4-Pad9)
- J5 pad 7: 5V3 -> 5V8
- J5 pad 8: GND3 -> GND8
- J5 pad 9: GND3 -> Net-(J5-Pad9)
- J6 pad 7: 5V4 -> 5V2
- J6 pad 8: GND4 -> GND2
- J6 pad 9: GND4 -> Net-(J6-Pad9)
- J7 pad 7: 5V5 -> 5V4
- J7 pad 8: GND5 -> GND4
- J7 pad 9: GND5 -> Net-(J7-Pad9)
- J8 pad 9: GND6 -> Net-(J8-Pad9)
- P1 pad 2: IN7 -> AIN7
- P1 pad 3: IN6 -> AIN6
- P1 pad 4: IN5 -> AIN5
- P1 pad 5: IN4 -> AIN4
- P1 pad 6: IN3 -> AIN3
- P1 pad 7: IN2 -> AIN2
- P1 pad 8: IN1 -> AIN1
- U1 pad 29: Net-(U1-Pad29) -> PWM1
- U1 pad 30: Net-(U1-Pad30) -> PWM2
- U1 pad 31: Net-(U1-Pad31) -> PWM3
- U1 pad 32: Net-(U1-Pad32) -> PWM4
- U1 pad 33: Net-(U1-Pad33) -> PWM5
- U1 pad 34: Net-(U1-Pad34) -> PWM6
- U1 pad 37: Net-(U1-Pad37) -> PWM7
- U1 pad 38: Net-(U1-Pad38) -> PWM8
- U1 pad 39: Net-(U1-Pad39) -> SCK
- U1 pad 40: Net-(U1-Pad40) -> MOSI
- U1 pad 41: Net-(U1-Pad41) -> MISO
- U10 pad 1: 5V3 -> 5V8
- U10 pad 4: GND3 -> GND8
- U11 pad 2: OUT2 -> OUT7
- U11 pad 3: IN2 -> IN7
- U11 pad 5: GND3 -> GND8
- U11 pad 8: 5V3 -> 5V8
- U12 pad 1: 5V4 -> 5V2
- U12 pad 4: GND4 -> GND2
- U13 pad 2: OUT3 -> OUT1
- U13 pad 3: IN3 -> IN1
- U13 pad 5: GND4 -> GND2
- U13 pad 8: 5V4 -> 5V2
- U14 pad 1: 5V5 -> 5V4
- U14 pad 4: GND5 -> GND4
- U15 pad 2: OUT4 -> OUT3
- U15 pad 3: IN4 -> IN3
- U15 pad 5: GND5 -> GND4
- U15 pad 8: 5V5 -> 5V4
- U18 pad 6: SCLK -> SCK
- U18 pad 7: SI1 -> MOSI
- U19 pad 6: SCLK -> SCK
- U19 pad 9: SO2 -> MISO
- U6 pad 1: 5V8 -> 5V3
- U6 pad 4: GND8 -> GND3
- U7 pad 2: OUT7 -> OUT2
- U7 pad 3: IN7 -> IN2
- U7 pad 5: GND8 -> GND3
- U7 pad 8: 5V8 -> 5V3
- U8 pad 1: 5V2 -> 5V5
- U8 pad 4: GND2 -> GND5
- U9 pad 2: OUT1 -> OUT4
- U9 pad 3: IN1 -> IN4
- U9 pad 5: GND2 -> GND5
- U9 pad 8: 5V2 -> 5V5
Routing:
- net OUT7: track 4.19 -> 99.5 mm
- net IN7: track 0.00 -> 92.1 mm
- net OUT6: track 11.3 -> 96.3 mm
- net IN6: track 0.00 -> 81.3 mm
- net OUT5: track 12.2 -> 79.5 mm
- net IN5: track 0.00 -> 63.4 mm
- net OUT4: track 6.00 -> 62.2 mm
- net IN4: track 0.00 -> 53.7 mm
- net IN3: track 0.00 -> 37.6 mm
- net OUT3: track 4.18 -> 41.4 mm
- net SO1: track 0.00 -> 33.5 mm
- net SCK: track 0.00 -> 32.6 mm, vias 0 -> 2
- net IN2: track 0.00 -> 30.4 mm
- net GND2: track 52.8 -> 23.0 mm
- net OUT2: track 12.3 -> 42.0 mm
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
Commit message: More stuff.
Parts:
- removed REF** (x4): MountingHole_3.2mm_M3_ISO7380, Mounting_Holes:MountingHole_3.2mm_M3_ISO7380
- removed U22, U23, U24, U25, U26, U27: 74HC595, SMD_Packages:SO-16-N
- added C10: C, Capacitors_SMD:C_0603, B.Cu at (163.5, 106.5)
- added C11: C, Capacitors_SMD:C_0603, B.Cu at (138.2, 106.5)
- added C12: C, Capacitors_SMD:C_0603, B.Cu at (167.0, 106.5)
- added C13: C, Capacitors_SMD:C_0603, B.Cu at (141.8, 106.5)
- added C14: C, Capacitors_SMD:C_0603, B.Cu at (170.5, 106.5)
- added C15: C, Capacitors_SMD:C_0603, B.Cu at (145.2, 106.5)
- added C16: C, Capacitors_SMD:C_0603, B.Cu at (174.0, 106.6)
- added C17: C, Capacitors_SMD:C_0603, B.Cu at (148.8, 106.5)
- added C18: C, Capacitors_SMD:C_0603, B.Cu at (177.5, 106.5)
- added C19: C, Capacitors_SMD:C_0603, B.Cu at (152.2, 106.5)
- added C20: C, Capacitors_SMD:C_0603, B.Cu at (181.0, 106.5)
- added C21: C, Capacitors_SMD:C_0603, B.Cu at (155.8, 106.5)
- added C22: C, Capacitors_SMD:C_0603, B.Cu at (184.5, 106.5)
- added C23: C, Capacitors_SMD:C_0603, B.Cu at (159.2, 106.5)
- added D35: LED, LEDs:LED_0603, F.Cu at (90.7, 178.8)
- added D36: LED, LEDs:LED_0603, F.Cu at (83.8, 183.8)
- added D37: LED, LEDs:LED_0603, F.Cu at (87.2, 178.8)
- added D38: LED, LEDs:LED_0603, F.Cu at (90.7, 173.7)
- added D39: LED, LEDs:LED_0603, F.Cu at (83.8, 178.8)
- added D40: LED, LEDs:LED_0603, F.Cu at (80.3, 183.8)
- added D41: LED, LEDs:LED_0603, F.Cu at (87.2, 173.7)
- added D42: LED, LEDs:LED_0603, F.Cu at (80.3, 173.7)
- added D43: LED, LEDs:LED_0603, F.Cu at (59.6, 178.8)
- added D44: LED, LEDs:LED_0603, F.Cu at (63.1, 173.7)
- added D45: LED, LEDs:LED_0603, F.Cu at (59.6, 183.8)
- added D46: LED, LEDs:LED_0603, F.Cu at (66.5, 173.7)
- added D47: LED, LEDs:LED_0603, F.Cu at (63.1, 178.8)
- added D48: LED, LEDs:LED_0603, F.Cu at (66.5, 178.8)
- added D49: LED, LEDs:LED_0603, F.Cu at (63.1, 183.8)
- added D50: LED, LEDs:LED_0603, F.Cu at (66.5, 183.8)
- added D51: LED, LEDs:LED_0603, F.Cu at (83.8, 173.7)
- added D52: LED, LEDs:LED_0603, F.Cu at (80.3, 178.8)
- added D53: LED, LEDs:LED_0603, F.Cu at (73.4, 183.8)
- added D54: LED, LEDs:LED_0603, F.Cu at (76.9, 178.8)
- added D55: LED, LEDs:LED_0603, F.Cu at (70.0, 183.8)
- added D56: LED, LEDs:LED_0603, F.Cu at (59.6, 173.7)
- added D57: LED, LEDs:LED_0603, F.Cu at (73.4, 178.8)
- added D58: LED, LEDs:LED_0603, F.Cu at (76.9, 173.7)
- added D59: LED, LEDs:LED_0603, F.Cu at (70.0, 178.8)
- added D60: LED, LEDs:LED_0603, F.Cu at (76.9, 183.8)
- added D61: LED, LEDs:LED_0603, F.Cu at (73.4, 173.7)
- added D62: LED, LEDs:LED_0603, F.Cu at (70.0, 173.7)
- added R10: R, Resistors_SMD:R_0805, B.Cu at (140.0, 106.5)
- added R11: R, Resistors_SMD:R_1206, B.Cu at (169.5, 110.5)
- added R12: R, Resistors_SMD:R_0805, B.Cu at (168.8, 106.5)
- added R13: R, Resistors_SMD:R_1206, B.Cu at (144.2, 110.5)
- added R14: R, Resistors_SMD:R_0805, B.Cu at (143.5, 106.5)
- added R15: R, Resistors_SMD:R_1206, B.Cu at (173.0, 110.5)
- added R16: R, Resistors_SMD:R_0805, B.Cu at (172.2, 106.5)
- added R17: R, Resistors_SMD:R_1206, B.Cu at (147.8, 110.5)
- added R18: R, Resistors_SMD:R_0805, B.Cu at (147.0, 106.5)
- added R19: R, Resistors_SMD:R_1206, B.Cu at (176.5, 110.5)
- added R20: R, Resistors_SMD:R_0805, B.Cu at (175.8, 106.5)
- added R21: R, Resistors_SMD:R_1206, B.Cu at (151.2, 110.5)
- added R22: R, Resistors_SMD:R_0805, B.Cu at (150.5, 106.5)
- added R23: R, Resistors_SMD:R_1206, B.Cu at (180.0, 110.5)
- added R24: R, Resistors_SMD:R_0805, B.Cu at (179.2, 106.5)
- added R25: R, Resistors_SMD:R_1206, B.Cu at (154.8, 110.5)
- added R26: R, Resistors_SMD:R_0805, B.Cu at (154.0, 106.5)
- added R27: R, Resistors_SMD:R_1206, B.Cu at (183.5, 110.5)
- added R28: R, Resistors_SMD:R_0805, B.Cu at (182.8, 106.5)
- added R29: R, Resistors_SMD:R_1206, B.Cu at (158.2, 110.5)
- added R3: R, Resistors_SMD:R_1206, B.Cu at (162.5, 110.5)
- added R30: R, Resistors_SMD:R_0805, B.Cu at (157.5, 106.5)
- added R4: R, Resistors_SMD:R_0805, B.Cu at (161.8, 106.5)
- added R5: R, Resistors_SMD:R_1206, B.Cu at (137.2, 110.5)
- added R6: R, Resistors_SMD:R_0805, B.Cu at (136.5, 106.5)
- added R7: R, Resistors_SMD:R_1206, B.Cu at (166.0, 110.5)
- added R8: R, Resistors_SMD:R_0805, B.Cu at (165.2, 106.5)
- added R9: R, Resistors_SMD:R_1206, B.Cu at (140.8, 110.5)
- C9: footprint Capacitors_SMD:C_0805 -> Capacitors_SMD:C_0603
- D10, D11, D12, D13, D14, D15, D16, D17, D18, D19, D20, D21, D22, D23, D24, D25, D26, D27, D28, D29, D3, D30, D4, D5, D6, D7, D8, D9: value Led_x2 -> D; footprint LEDs:LED_0805 -> Diodes_SMD:MiniMELF_Standard
- D31, D32, D33, D34: value Led_x2 -> LED; footprint LEDs:LED_0805 -> LEDs:LED_0603
- R2: footprint Resistors_SMD:R_1206 -> Resistors_SMD:R_0805
- moved C9 95.2 mm to (134.8, 106.5), turned to 90 degrees
- moved R2 93.0 mm to (133.0, 106.5), turned to 90 degrees
- moved D1 34.9 mm to (73.3, 116.5)
- moved D2 33.8 mm to (74.9, 119.7)
- moved JP1 25.8 mm to (181.2, 73.7)
- moved R1 24.5 mm to (133.8, 110.5), turned to 270 degrees
- moved JP2 22.1 mm to (177.0, 73.8)
- moved U1 8.84 mm to (122.2, 92.2)
- moved P1 1.25 mm to (133.7, 114.3)
- moved P3 1.25 mm to (162.5, 114.3)
- moved P7 0.82 mm to (162.2, 99.8)
- moved P8 0.75 mm to (133.7, 99.8)
- moved P2 0.50 mm to (133.7, 122.5)
- moved P4 0.50 mm to (162.5, 122.5)
Connections:
- net OUT10 renamed SSOUT10
- net OUT11 renamed SSOUT11
- net OUT12 renamed SSOUT12
- net OUT13 renamed SSOUT13
- net OUT14 renamed SSOUT14
- net OUT15 renamed SSOUT15
- net OUT16 renamed SSOUT16
- net OUT8 renamed SSOUT8
- net OUT9 renamed SSOUT9
- D10 pad 1: Net-(D10-Pad1) -> IN3_ADC
- D10 pad 2: Net-(D10-Pad2) -> GND
- D11 pad 1: Net-(D11-Pad1) -> +3V3
- D11 pad 2: GND -> IN11_ADC
- D12 pad 1: Net-(D12-Pad1) -> IN11_ADC
- D12 pad 2: Net-(D12-Pad2) -> GND
- D13 pad 1: Net-(D13-Pad1) -> +3V3
- D13 pad 2: Net-(D13-Pad2) -> IN4_ADC
- D14 pad 1: Net-(D14-Pad1) -> IN4_ADC
- D14 pad 2: Net-(D14-Pad2) -> GND
- D15 pad 1: Net-(D15-Pad1) -> +3V3
- D15 pad 2: Net-(D15-Pad2) -> IN12_ADC
- D16 pad 1: Net-(D16-Pad1) -> IN12_ADC
- D16 pad 2: Net-(D16-Pad2) -> GND
- D17 pad 1: Net-(D17-Pad1) -> +3V3
- D17 pad 2: Net-(D17-Pad2) -> IN5_ADC
- D18 pad 1: Net-(D18-Pad1) -> IN5_ADC
- D18 pad 2: Net-(D18-Pad2) -> GND
- D19 pad 1: Net-(D19-Pad1) -> +3V3
- D19 pad 2: GND -> IN13_ADC
- D20 pad 1: Net-(D20-Pad1) -> IN13_ADC
- D20 pad 2: Net-(D20-Pad2) -> GND
- D21 pad 1: Net-(D21-Pad1) -> +3V3
- D21 pad 2: Net-(D21-Pad2) -> IN6_ADC
- D22 pad 1: Net-(D22-Pad1) -> IN6_ADC
- D22 pad 2: Net-(D22-Pad2) -> GND
- D23 pad 1: Net-(D23-Pad1) -> +3V3
- D23 pad 2: Net-(D23-Pad2) -> IN14_ADC
- D24 pad 1: Net-(D24-Pad1) -> IN14_ADC
- D24 pad 2: Net-(D24-Pad2) -> GND
- D25 pad 1: Net-(D25-Pad1) -> +3V3
- D25 pad 2: Net-(D25-Pad2) -> IN7_ADC
- D26 pad 1: Net-(D26-Pad1) -> IN7_ADC
- D26 pad 2: Net-(D26-Pad2) -> GND
- D27 pad 1: Net-(D27-Pad1) -> +3V3
- D27 pad 2: GND -> IN15_ADC
- D28 pad 1: Net-(D28-Pad1) -> IN15_ADC
- D28 pad 2: Net-(D28-Pad2) -> GND
- D29 pad 1: Net-(D29-Pad1) -> +3V3
- D29 pad 2: Net-(D29-Pad2) -> IN18ADC
- D3 pad 1: Net-(D3-Pad1) -> +3V3
- D3 pad 2: GND -> IN9_ADC
- D30 pad 1: Net-(D30-Pad1) -> IN18ADC
- D30 pad 2: Net-(D30-Pad2) -> GND
- D4 pad 1: Net-(D4-Pad1) -> IN9_ADC
- D4 pad 2: Net-(D4-Pad2) -> GND
- D5 pad 1: Net-(D5-Pad1) -> +3V3
- D5 pad 2: Net-(D5-Pad2) -> IN2_ADC
- D6 pad 1: Net-(D6-Pad1) -> IN2_ADC
- D6 pad 2: Net-(D6-Pad2) -> GND
- D7 pad 1: Net-(D7-Pad1) -> +3V3
- D7 pad 2: Net-(D7-Pad2) -> IN10_ADC
- D8 pad 1: Net-(D8-Pad1) -> IN10_ADC
- D8 pad 2: Net-(D8-Pad2) -> GND
- D9 pad 1: Net-(D9-Pad1) -> +3V3
- D9 pad 2: Net-(D9-Pad2) -> IN3_ADC
- P1 pad 1: AIN8 -> AIN1
- P1 pad 2: AIN7 -> AIN2
- P1 pad 3: AIN6 -> AIN3
- P1 pad 4: AIN5 -> AIN4
- P1 pad 5: AIN4 -> AIN5
- P1 pad 6: AIN3 -> AIN6
- P1 pad 7: AIN2 -> AIN7
- P1 pad 8: AIN1 -> AIN8
- P3 pad 1: AESTOP -> AIN9
- P3 pad 2: AIN15 -> AIN10
- P3 pad 3: AIN14 -> AIN11
- P3 pad 4: AIN13 -> AIN12
- P3 pad 5: AIN12 -> AIN13
- P3 pad 6: AIN11 -> AIN14
- P3 pad 7: AIN10 -> AIN15
- P3 pad 8: AIN9 -> AESTOP
- P5 pad 1: OUT1 -> SSOUT1
- P5 pad 2: OUT2 -> SSOUT2
- P5 pad 3: OUT3 -> SSOUT3
- P5 pad 4: OUT4 -> SSOUT4
- P5 pad 5: OUT5 -> SSOUT5
- P5 pad 6: OUT6 -> SSOUT6
- P5 pad 7: OUT7 -> SSOUT7
- R1 pad 2: IN1 -> AIN1
- U18 pad 12: OUT5 -> SSOUT5
- U18 pad 13: OUT6 -> SSOUT6
- U18 pad 16: OUT7 -> SSOUT7
- U18 pad 2: OUT2 -> SSOUT2
- U18 pad 26: OUT4 -> SSOUT4
- U18 pad 27: OUT3 -> SSOUT3
- U18 pad 3: OUT1 -> SSOUT1
Routing:
- net OUT1: track 35.2 -> 15.4 mm
- net SSOUT1: track 0.00 -> 19.8 mm
- net SSOUT2: track 0.00 -> 12.3 mm
- net OUT2: track 42.0 -> 29.7 mm
- net OUT5: track 79.5 -> 67.3 mm, vias 1 -> 0
- net SSOUT5: track 0.00 -> 12.2 mm, vias 0 -> 1
- net OUT6: track 96.3 -> 84.9 mm, vias 1 -> 0
- net SSOUT6: track 0.00 -> 11.3 mm, vias 0 -> 1
- net SSOUT4: track 0.00 -> 6.00 mm
- net OUT4: track 62.2 -> 56.2 mm
- net GND5: track 42.0 -> 36.8 mm
- net Net-(J4-Pad9): track 1.77 -> 6.93 mm
- net Net-(J2-Pad9): track 1.77 -> 6.93 mm
- net GND1: track 42.0 -> 36.8 mm
- net SSOUT7: track 0.00 -> 4.19 mm
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
Commit message: Wip
Parts:
- removed D1, D10, D11, D12, D13, D14, D15, D16, D17, D18, D19, D2, D20, D21, D22, D23, D24, D25, D26, D27, D28, D29, D30, D4, D5, D6, D7, D8, D9: D, Diodes_SMD:MiniMELF_Standard
- added J10: RJ45-TRANSFO, rj45_MHRJJ88NFVS:MHRJJ88NFVS, F.Cu at (143.1, 120.5)
- added U22: DP83848C, Housings_QFP:LQFP-48_7x7mm_Pitch0.5mm, B.Cu at (143.6, 100.2)
- P1, P2, P3, P4, P5, P6, P7, P8: footprint Terminal_Blocks:TerminalBlock_Pheonix_PT-3.5mm_8pol -> Terminal_Blocks:TerminalBlock_Pheonix_MPT-2.54mm_8pol
- R1, R11, R13, R15, R17, R19, R21, R23, R25, R27, R29, R3, R5, R7, R9: footprint Resistors_SMD:R_1206 -> Resistors_SMD:R_0805
- U1: value STM32F303CBTx -> STM32F407VG; footprint Housings_QFP:LQFP-48_7x7mm_Pitch0.5mm -> Housings_QFP:TQFP-100_14x14mm_Pitch0.5mm
- moved C10 119.2 mm to (47.5, 79.1)
- moved C11 119.2 mm to (22.2, 79.1)
- moved C12 119.2 mm to (51.0, 79.1)
- moved C13 119.2 mm to (25.8, 79.1)
- moved C14 119.2 mm to (54.5, 79.1)
- moved C16 119.2 mm to (58.0, 79.2)
- moved C17 119.2 mm to (32.8, 79.1)
- moved C18 119.2 mm to (61.5, 79.1)
- moved C19 119.2 mm to (36.2, 79.1)
- moved C20 119.2 mm to (65.0, 79.1)
- moved C21 119.2 mm to (39.8, 79.1)
- moved C22 119.2 mm to (68.5, 79.1)
- moved C23 119.2 mm to (43.2, 79.1)
- moved C9 119.2 mm to (18.8, 79.1)
- moved R10 119.2 mm to (24.0, 79.1)
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Connections:
- U1 pad 16: Net-(U1-Pad16) -> mdc
- U1 pad 17: Net-(U1-Pad17) -> tx_d2
- U1 pad 18: Net-(U1-Pad18) -> tx_clk
- U1 pad 24: Net-(U1-Pad24) -> rx_clk
- U1 pad 25: Net-(U1-Pad25) -> mdio
- U1 pad 26: Net-(U1-Pad26) -> col
- U1 pad 29: PWM1 -> Net-(U1-Pad29)
- U1 pad 30: PWM2 -> Net-(U1-Pad30)
- U1 pad 31: PWM3 -> Net-(U1-Pad31)
- U1 pad 32: PWM4 -> rx_dv
- U1 pad 33: PWM5 -> rx_d0
- U1 pad 34: PWM6 -> rx_d1
- U1 pad 35: Net-(U1-Pad35) -> rx_d2
- U1 pad 36: Net-(U1-Pad36) -> rx_d3
- U1 pad 37: PWM7 -> Net-(U1-Pad37)
- U1 pad 38: PWM8 -> Net-(U1-Pad38)
- U1 pad 39: SCK -> Net-(U1-Pad39)
- U1 pad 40: MOSI -> Net-(U1-Pad40)
- U1 pad 41: MISO -> Net-(U1-Pad41)
- U1 pad 48: Net-(U1-Pad48) -> tx_en
Routing:
- net (no net): track 0.00 -> 268.8 mm, vias 0 -> 21
- net SO1: track 33.5 -> 0.00 mm
- net SCK: track 32.6 -> 0.00 mm, vias 2 -> 0
- net +24V: track 38.1 -> 8.38 mm, vias 14 -> 0
- net rx_d3: track 0.00 -> 22.8 mm, vias 0 -> 2
- net rx_d2: track 0.00 -> 22.1 mm, vias 0 -> 2
- net rx_d1: track 0.00 -> 20.7 mm, vias 0 -> 2
- net rx_d0: track 0.00 -> 19.8 mm, vias 0 -> 2
- net T+: track 0.00 -> 12.7 mm
- net T-: track 0.00 -> 11.4 mm
- net R+: track 0.00 -> 8.88 mm, vias 0 -> 1
- net R-: track 0.00 -> 7.46 mm
- net SSOUT1: track 19.8 -> 14.1 mm, vias 0 -> 1
- net SSOUT9: track 19.8 -> 14.3 mm, vias 0 -> 1
- net SSOUT8: track 12.2 -> 7.03 mm, vias 0 -> 1
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- added copper zone on B.Cu, net +24V
