File: hw/kicad/bob/db25_bob_v2/stm32.sch (KiCad schematic (older format))
At the start: 10 parts, among them P1 CONN_01X08, P2 CONN_01X08, P3 CONN_01X08, P4 CONN_01X08, U1 STM32F303CBTx

Commit message: More routing + schematic changes
Parts:
- added C? (x14): C, Capacitors_SMD:C_0805, symbol C-RESCUE-db25_bob_v2
- added D? (x28): D, Diodes_SMD:MiniMELF_Standard, symbol D
- added R? (x28): R, Resistors_SMD:R_1206, symbol R-RESCUE-db25_bob_v2
Connections:
- net +3V3: now also D?.1 (K), D?.1 (K), D?.1 (K), D?.1 (K), D?.1 (K), D?.1 (K), D?.1 (K), D?.1 (K), D?.1 (K), D?.1 (K), D?.1 (K), D?.1 (K), D?.1 (K), D?.1 (K)
- net GND: now also C?.2, C?.2, C?.2, C?.2, C?.2, C?.2, C?.2, C?.2, C?.2, C?.2, C?.2, C?.2, C?.2, C?.2, D?.2 (A), D?.2 (A), D?.2 (A), D?.2 (A), D?.2 (A), D?.2 (A), D?.2 (A), D?.2 (A), D?.2 (A), D?.2 (A), D?.2 (A), D?.2 (A), D?.2 (A), D?.2 (A), R?.2, R?.2, R?.2, R?.2, R?.2, R?.2, R?.2, R?.2, R?.2, R?.2, R?.2, R?.2, R?.2, R?.2
- net IN1: no longer P1.8 (P8)
- net PWM1: now reaches U1.29 (COMP3_OUT/I2C2_SMBA/I2S2_MCK/RCC_MCO/TIM1_CH1/TIM4_ETR/USART1_CK/PA8)
- net PWM2: now reaches U1.30 (COMP5_OUT/DAC_EXTI9/I2C2_SCL/I2S3_MCK/TIM15_BKIN/TIM1_CH2/TIM2_CH3/TSC_G4_IO1/USART1_TX/PA9)
- net PWM3: now reaches U1.31 (COMP6_OUT/I2C2_SDA/TIM17_BKIN/TIM1_CH3/TIM2_CH4/TIM8_BKIN/TSC_G4_IO2/USART1_RX/PA10)
- net PWM4: now reaches U1.32 (ADC1_EXTI11/ADC2_EXTI11/CAN_RX/COMP1_OUT/TIM1_BKIN2/TIM1_CH1N/TIM1_CH4/TIM4_CH1/USART1_CTS/USB_DM/PA11)
- net PWM5: now reaches U1.33 (CAN_TX/COMP2_OUT/TIM16_CH1/TIM1_CH2N/TIM1_ETR/TIM4_CH2/USART1_DE/USART1_RTS/USB_DP/PA12)
- net PWM6: now reaches U1.34 (IR_OUT/SYS_JTMS-SWDIO/TIM16_CH1N/TIM4_CH3/TSC_G4_IO3/USART3_CTS/PA13)
- net PWM7: now reaches U1.37 (I2C1_SDA/SYS_JTCK-SWCLK/TIM1_BKIN/TIM8_CH2/TSC_G4_IO4/USART2_TX/PA14)
- net PWM8: now reaches U1.38 (ADC1_EXTI15/ADC2_EXTI15/I2C1_SCL/I2S3_WS/SPI1_NSS/SPI3_NSS/SYS_JTDI/TIM1_BKIN/TIM2_CH1/TIM2_ETR/TIM8_CH1/USART2_RX/PA15)
- net SCK: now reaches U1.39 (PB3/I2S3_CK/SPI1_SCK/SPI3_SCK/SYS_JTDO-TRACESWO/TIM2_CH2/TIM3_ETR/TIM4_ETR/TIM8_CH1N/TSC_G5_IO1/USART2_TX)
- net MOSI: now reaches U1.40 (PB4/I2S3_ext_SD/SPI1_MISO/SPI3_MISO/SYS_NJTRST/TIM16_CH1/TIM17_BKIN/TIM3_CH1/TIM8_CH2N/TSC_G5_IO2/USART2_RX)
- net MISO: now reaches U1.41 (PB5/I2C1_SMBA/I2S3_SD/SPI1_MOSI/SPI3_MOSI/TIM16_BKIN/TIM17_CH1/TIM3_CH2/TIM8_CH3N/USART2_CK)
- net IN10 renamed AIN10
- net AIN10: now also R?.2
- net IN11 renamed AIN11
- net AIN11: now also R?.2
- net IN12 renamed AIN12
- net AIN12: now also R?.2
- net IN13 renamed AIN13
- net AIN13: now also R?.2
- net IN14 renamed AIN14
- net AIN14: now also R?.2
- net IN15 renamed AIN15
- net AIN15: now also R?.2
- net IN16 renamed AESTOP
- net IN2 renamed AIN2
- net AIN2: now also R?.2
- net IN3 renamed AIN3
- net AIN3: now also R?.2
- net IN4 renamed AIN4
- net AIN4: now also R?.2
- net IN5 renamed AIN5
- net AIN5: now also R?.2
- net IN6 renamed AIN6
- net AIN6: now also R?.2
- net IN7 renamed AIN7
- net AIN7: now also R?.2
- net IN8 renamed AIN8
- net AIN8: now also R?.2
- net IN9 renamed AIN9
- net AIN9: now also R?.2
- new net AIN1: P1.8 (P8)
- new net IN10_ADC: C?.1, D?.1 (K), D?.2 (A), R?.1, R?.1
- new net IN11_ADC: C?.1, D?.1 (K), D?.2 (A), R?.1, R?.1
- new net IN12_ADC: C?.1, D?.1 (K), D?.2 (A), R?.1, R?.1
- new net IN13_ADC: C?.1, D?.1 (K), D?.2 (A), R?.1, R?.1
- new net IN14_ADC: C?.1, D?.1 (K), D?.2 (A), R?.1, R?.1
- new net IN15_ADC: C?.1, D?.1 (K), D?.2 (A), R?.1, R?.1
- new net IN18ADC: C?.1, D?.1 (K), D?.2 (A), R?.1, R?.1
- new net IN2_ADC: C?.1, D?.1 (K), D?.2 (A), R?.1, R?.1
- new net IN3_ADC: C?.1, D?.1 (K), D?.2 (A), R?.1, R?.1
- new net IN4_ADC: C?.1, D?.1 (K), D?.2 (A), R?.1, R?.1
- new net IN5_ADC: C?.1, D?.1 (K), D?.2 (A), R?.1, R?.1
- new net IN6_ADC: C?.1, D?.1 (K), D?.2 (A), R?.1, R?.1
- new net IN7_ADC: C?.1, D?.1 (K), D?.2 (A), R?.1, R?.1
- new net IN9_ADC: C?.1, D?.1 (K), D?.2 (A), R?.1, R?.1
Other:
- moved on the sheet: C9, D1, D2, P1, P2, P3, P4, R1, R2

Commit message: More stuff.
Parts:
- removed D1, D2, D? (x27): D, Diodes_SMD:MiniMELF_Standard, symbol D
- C10, C11, C12, C13, C14, C15, C16, C17, C18, C19, C20, C21, C22, C23: renamed from C?; footprint Capacitors_SMD:C_0805 -> Capacitors_SMD:C_0603
- C9: footprint Capacitors_SMD:C_0805 -> Capacitors_SMD:C_0603
- R10, R12, R14, R16, R18, R20, R22, R24, R26, R28, R30, R4, R6, R8: renamed from R?; footprint Resistors_SMD:R_1206 -> Resistors_SMD:R_0805
- R2: footprint Resistors_SMD:R_1206 -> Resistors_SMD:R_0805
- gave numbers to parts that had none: 15
Connections:
- net IN1 is gone; now on net AIN1: R1.2
- net AESTOP: now also P3.8 (P8); no longer P3.1 (P1)
- net AIN1: now also P1.1 (P1); no longer P1.8 (P8)
- net AIN10: now also P3.2 (P2); no longer P3.7 (P7)
- net AIN11: now also P3.3 (P3); no longer P3.6 (P6)
- net AIN12: now also P3.4 (P4); no longer P3.5 (P5)
- net AIN13: now also P3.5 (P5); no longer P3.4 (P4)
- net AIN14: now also P3.6 (P6); no longer P3.3 (P3)
- net AIN15: now also P3.7 (P7); no longer P3.2 (P2)
- net AIN2: now also P1.2 (P2); no longer P1.7 (P7)
- net AIN3: now also P1.3 (P3); no longer P1.6 (P6)
- net AIN4: now also P1.4 (P4); no longer P1.5 (P5)
- net AIN5: now also P1.5 (P5); no longer P1.4 (P4)
- net AIN6: now also P1.6 (P6); no longer P1.3 (P3)
- net AIN7: now also P1.7 (P7); no longer P1.2 (P2)
- net AIN8: now also P1.8 (P8); no longer P1.1 (P1)
- net AIN9: now also P3.1 (P1); no longer P3.8 (P8)

Commit message: Wip
Parts:
- removed U1: STM32F303CBTx, Housings_QFP:LQFP-48_7x7mm_Pitch0.5mm, symbol STM32F303CBTx
- added J10: RJ45-TRANSFO, rj45_MHRJJ88NFVS:MHRJJ88NFVS, symbol RJ45-TRANSFO
- added U1: STM32F407VG, Housings_QFP:TQFP-100_14x14mm_Pitch0.5mm, symbol STM32F407VG
- added U22: DP83848C, Housings_QFP:LQFP-48_7x7mm_Pitch0.5mm, symbol DP83848C
- P1, P2, P3, P4: footprint Terminal_Blocks:TerminalBlock_Pheonix_PT-3.5mm_8pol -> Terminal_Blocks:TerminalBlock_Pheonix_MPT-2.54mm_8pol
- R1, R11, R13, R15, R17, R19, R21, R23, R25, R27, R29, R3, R5, R7, R9: footprint Resistors_SMD:R_1206 -> Resistors_SMD:R_0805
Connections:
- net labels added: R+, R-, T+, T-, col, mdc, mdio, rx_clk, rx_d0, rx_d1, rx_d2, rx_d3, rx_dv, tx_clk, tx_d0, tx_d1, tx_d2, tx_d3, tx_en
- wire segments 139 -> 176
Other:
- moved on the sheet: C10, C11, C12, C13, C14, C15, C16, C17, C18, C19, C20, C21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
