File: hw/kicad/bob/ethernet_bob/io_base/opto_in.sch (KiCad schematic (older format))
At the start: 51 parts, among them P1 CONN_01X08, P2 CONN_01X08, P3 CONN_01X08, P4 CONN_01X08, P5 CONN_01X08, P6 CONN_01X08, U1 OPTO-TRANSISTOR-4, U2 OPTO-TRANSISTOR-4, U3 VN808, U4 VN808

Commit message: WIP
Parts:
- added D13, D14, D15, D16, D17, D18, D19, D20, D21, D22, D23, D24, D25, D26, D27, D28: LED, LEDs:LED_0603, symbol LED
- added R25, R26, R27, R28, R29, R30, R31, R32, R33, R34, R35, R36, R37, R38, R39, R40: R, stmbl:R_0603, symbol R
- D1, D2, D3, D4, D5, D6, D7, D8: footprint (none) -> LEDs:LED_0603
- D10, D11, D12, D9: renamed from D?; footprint (none) -> LEDs:LED_0603
- P1, P2: footprint (none) -> Terminal_Blocks:TerminalBlock_Pheonix_PT-3.5mm_8pol
- P3: renamed from P?; footprint (none) -> Terminal_Blocks:TerminalBlock_Pheonix_PT-3.5mm_8pol
- P4: renamed from P3; footprint (none) -> Terminal_Blocks:TerminalBlock_Pheonix_PT-3.5mm_8pol
- P5: renamed from P4; footprint (none) -> Terminal_Blocks:TerminalBlock_Pheonix_PT-3.5mm_8pol
- P6: renamed from P5; footprint (none) -> Terminal_Blocks:TerminalBlock_Pheonix_PT-3.5mm_8pol
- P7: renamed from P6; footprint (none) -> Terminal_Blocks:TerminalBlock_Pheonix_PT-3.5mm_8pol
- R1, R2, R3, R4, R5, R6, R7, R8: footprint (none) -> stmbl:R_0603
- R10, R11, R12, R21, R22, R23, R24, R9: renamed from R?; footprint (none) -> stmbl:R_0603
- R13: renamed from R9; footprint (none) -> stmbl:R_0603
- R14: renamed from R10; footprint (none) -> stmbl:R_0603
- R15: renamed from R11; footprint (none) -> stmbl:R_0603
- R16: renamed from R12; footprint (none) -> stmbl:R_0603
- R17: renamed from R13; footprint (none) -> stmbl:R_0603
- R18: renamed from R14; footprint (none) -> stmbl:R_0603
- R19: renamed from R15; footprint (none) -> stmbl:R_0603
- R20: renamed from R16; footprint (none) -> stmbl:R_0603
- U1, U2: footprint (none) -> Housings_DIP:DIP-16_W7.62mm
- U3: renamed from U?; footprint (none) -> Housings_DIP:DIP-16_W7.62mm
- U4: renamed from U3; footprint (none) -> io_base:POWERSO36
- U5: renamed from U4; footprint (none) -> io_base:POWERSO36
Connections:
- net labels added: PO1, PO10, PO11, PO12, PO13, PO14, PO15, PO16, PO2, PO3, PO4, PO5, PO6, PO7, PO8, PO9
- wire segments 166 -> 265
