File: hw/kicad/bob/ethernet_bob/io_base/plug.sch (KiCad schematic (older format))
At the start: 2 parts

Commit message: WIP
Parts:
- P8, P9: renamed from P?; footprint (none) -> Socket_Strips:Socket_Strip_Straight_2x25
Changed lines of the file:
@@
 LIBS:valves
 LIBS:vn808
+LIBS:74xgxx
+LIBS:ac-dc
+LIBS:actel
+LIBS:allegro
+LIBS:Altera
+LIBS:analog_devices
+LIBS:battery_management
+LIBS:bbd
+LIBS:brooktre
+LIBS:cmos_ieee
+LIBS:dc-dc
+LIBS:diode
+LIBS:elec-unifil
+LIBS:ESD_Protection
+LIBS:ftdi
+LIBS:gennum
+LIBS:graphic
+LIBS:hc11
+LIBS:ir
+LIBS:Lattice
+LIBS:logo
+LIBS:maxim
+LIBS:mechanical
+LIBS:microchip_dspic33dsc
+LIBS:microchip_pic10mcu
+LIBS:microchip_pic12mcu
+LIBS:microchip_pic16mcu
+LIBS:microchip_pic18mcu
+LIBS:microchip_pic32mcu
+LIBS:motor_drivers
+LIBS:motors
+LIBS:msp430
+LIBS:nordicsemi
+LIBS:nxp_armmcu
+LIBS:onsemi
+LIBS:Oscillators
+LIBS:powerint
+LIBS:Power_Management
+LIBS:pspice
+LIBS:references
+LIBS:relays
+LIBS:rfcom
+LIBS:sensors
+LIBS:silabs
+LIBS:stm8
+LIBS:stm32
+LIBS:supertex
+LIBS:switches
+LIBS:transf
+LIBS:ttl_ieee
+LIBS:video
+LIBS:wiznet
+LIBS:Worldsemi
+LIBS:Xicor
+LIBS:zetex
+LIBS:Zilog
+LIBS:stmbl_4.0-cache
 LIBS:io_base-cache
 EELAYER 25 0
@@
 $EndDescr
 $Comp
-L CONN_02X25 P?
+L CONN_02X25 P8
 U 1 1 5841CC38
 P 3150 2450
-F 0 "P?" H 3150 3865 50  0000 C CNN
+F 0 "P8" H 3150 3865 50  0000 C CNN
 F 1 "CONN_02X25" H 3150 3774 50  0000 C CNN
-F 2 "" H 3150 1700 50  0000 C CNN
+F 2 "Socket_Strips:Socket_Strip_Straight_2x25" H 3150 1700 50  0001 C CNN
 F 3 "" H 3150 1700 50  0000 C CNN
 	1    3150 2450
@@
 $EndComp
 $Comp
-L CONN_02X25 P?
+L CONN_02X25 P9
 U 1 1 5841CD0D
 P 3150 5350
-F 0 "P?" H 3150 6765 50  0000 C CNN
+F 0 "P9" H 3150 6765 50  0000 C CNN
 F 1 "CONN_02X25" H 3150 6674 50  0000 C CNN
-F 2 "" H 3150 4600 50  0000 C CNN
+F 2 "Socket_Strips:Socket_Strip_Straight_2x25" H 3150 4600 50  0001 C CNN
 F 3 "" H 3150 4600 50  0000 C CNN
 	1    3150 5350
@@
 $EndComp
 $Comp
-L GND #PWR?
+L GND #PWR010
 U 1 1 5841CE73
 P 3500 4150
-F 0 "#PWR?" H 3500 3900 50  0001 C CNN
+F 0 "#PWR010" H 3500 3900 50  0001 C CNN
 F 1 "GND" V 3505 4022 50  0000 R CNN
 F 2 "" H 3500 4150 50  0000 C CNN
@@
 $EndComp
 $Comp
-L GND #PWR?
+L GND #PWR011
 U 1 1 5841CE91
 P 2800 4150
-F 0 "#PWR?" H 2800 3900 50  0001 C CNN
+F 0 "#PWR011" H 2800 3900 50  0001 C CNN
 F 1 "GND" V 2805 4022 50  0000 R CNN
 F 2 "" H 2800 4150 50  0000 C CNN
@@
 $EndComp
 $Comp
-L +5V #PWR?
+L +5V #PWR012
 U 1 1 5841CEAC
 P 3500 4250
-F 0 "#PWR?" H 3500 4100 50  0001 C CNN
+F 0 "#PWR012" H 3500 4100 50  0001 C CNN
 F 1 "+5V" V 3515 4378 50  0000 L CNN
 F 2 "" H 3500 4250 50  0000 C CNN
@@
 $EndComp
 $Comp
-L +5V #PWR?
+L +5V #PWR013
 U 1 1 5841CECC
 P 2800 4250
-F 0 "#PWR?" H 2800 4100 50  0001 C CNN
+F 0 "#PWR013" H 2800 4100 50  0001 C CNN
 F 1 "+5V" V 2815 4378 50  0000 L CNN
 F 2 "" H 2800 4250 50  0000 C CNN
@@
 $EndComp
 $Comp
-L +3V3 #PWR?
+L +3V3 #PWR014
 U 1 1 5841CEE7
 P 3500 4350
-F 0 "#PWR?" H 3500 4200 50  0001 C CNN
+F 0 "#PWR014" H 3500 4200 50  0001 C CNN
 F 1 "+3V3" V 3515 4478 50  0000 L CNN
 F 2 "" H 3500 4350 50  0000 C CNN
@@
 $EndComp
 $Comp
-L +3V3 #PWR?
+L +3V3 #PWR015
 U 1 1 5841CF01
 P 2800 4350
-F 0 "#PWR?" H 2800 4200 50  0001 C CNN
+F 0 "#PWR015" H 2800 4200 50  0001 C CNN
 F 1 "+3V3" V 2815 4478 50  0000 L CNN
 F 2 "" H 2800 4350 50  0000 C CNN
@@
 	3400 4150 3500 4150
 $Comp
-L +3V3 #PWR?
+L +3V3 #PWR016
 U 1 1 5841CF51
 P 3500 5150
-F 0 "#PWR?" H 3500 5000 50  0001 C CNN
+F 0 "#PWR016" H 3500 5000 50  0001 C CNN
 F 1 "+3V3" V 3515 5278 50  0000 L CNN
 F 2 "" H 3500 5150 50  0000 C CNN
@@
 	3400 5150 3500 5150
 $Comp
-L GND #PWR?
+L GND #PWR017
 U 1 1 5841CFAC
 P 3500 6550
-F 0 "#PWR?" H 3500 6300 50  0001 C CNN
+F 0 "#PWR017" H 3500 6300 50  0001 C CNN
 F 1 "GND" V 3505 6422 50  0000 R CNN
 F 2 "" H 3500 6550 50  0000 C CNN
@@
 $EndComp
 $Comp
-L GND #PWR?
+L GND #PWR018
 U 1 1 5841CFED
 P 2800 6550
-F 0 "#PWR?" H 2800 6300 50  0001 C CNN
+F 0 "#PWR018" H 2800 6300 50  0001 C CNN
 F 1 "GND" V 2805 6422 50  0000 R CNN
 F 2 "" H 2800 6550 50  0000 C CNN
@@
 	3400 6550 3500 6550
 $Comp
-L GND #PWR?
+L GND #PWR019
 U 1 1 5841D0A7
 P 3500 3650
-F 0 "#PWR?" H 3500 3400 50  0001 C CNN
+F 0 "#PWR019" H 3500 3400 50  0001 C CNN
 F 1 "GND" V 3505 3522 50  0000 R CNN
 F 2 "" H 3500 3650 50  0000 C CNN
@@
 $EndComp
 $Comp
-L GND #PWR?
+L GND #PWR020
 U 1 1 5841D0B8
 P 2800 3650
-F 0 "#PWR?" H 2800 3400 50  0001 C CNN
+F 0 "#PWR020" H 2800 3400 50  0001 C CNN
 F 1 "GND" V 2805 3522 50  0000 R CNN
 F 2 "" H 2800 3650 50  0000 C CNN
@@
 	3400 3650 3500 3650
 $Comp
-L GND #PWR?
+L GND #PWR021
 U 1 1 5841D13C
 P 2800 2350
-F 0 "#PWR?" H 2800 2100 50  0001 C CNN
+F 0 "#PWR021" H 2800 2100 50  0001 C CNN
 F 1 "GND" V 2805 2222 50  0000 R CNN
 F 2 "" H 2800 2350 50  0000 C CNN
@@
 	2800 2350 2900 2350
 $Comp
-L GND #PWR?
+L GND #PWR022
 U 1 1 5841D180
 P 2800 1250
-F 0 "#PWR?" H 2800 1000 50  0001 C CNN
+F 0 "#PWR022" H 2800 1000 50  0001 C CNN
 F 1 "GND" V 2805 1122 50  0000 R CNN
 F 2 "" H 2800 1250 50  0000 C CNN
@@
 $EndComp
 $Comp
-L GND #PWR?
+L GND #PWR023
 U 1 1 5841D191
 P 3500 1250
-F 0 "#PWR?" H 3500 1000 50  0001 C CNN
+F 0 "#PWR023" H 3500 1000 50  0001 C CNN
 F 1 "GND" V 3505 1122 50  0000 R CNN
 F 2 "" H 3500 1250 50  0000 C CNN
@@
 	3400 1250 3500 1250
 $Comp
-L GND #PWR?
+L GND #PWR024
 U 1 1 5841D1CD
 P 2800 1450
-F 0 "#PWR?" H 2800 1200 50  0001 C CNN
+F 0 "#PWR024" H 2800 1200 50  0001 C CNN
 F 1 "GND" V 2805 1322 50  0000 R CNN
 F 2 "" H 2800 1450 50  0000 C CNN
@@
 	2800 1450 2900 1450
 $Comp
-L +3V3 #PWR?
+L +3V3 #PWR025
 U 1 1 5841D252
 P 3500 1350
-F 0 "#PWR?" H 3500 1200 50  0001 C CNN
+F 0 "#PWR025" H 3500 1200 50  0001 C CNN
 F 1 "+3V3" V 3515 1478 50  0000 L CNN
 F 2 "" H 3500 1350 50  0000 C CNN
@@
 $EndComp
 $Comp
-L +3V3 #PWR?
+L +3V3 #PWR026
 U 1 1 5841D2C9
 P 2800 1350
-F 0 "#PWR?" H 2800 1200 50  0001 C CNN
+F 0 "#PWR026" H 2800 1200 50  0001 C CNN
 F 1 "+3V3" V 2815 1478 50  0000 L CNN
 F 2 "" H 2800 1350 50  0000 C CNN
