File: hw/kicad/bob/ethernet_bob/io_base/io_base.kicad_pcb (KiCad board)
At the start: 2 copper layers, 99.9 x 99.9 mm, 0 parts

Commit message: WIP
Parts:
- added C1: 100n, stmbl:C_0603, F.Cu at (182.7, 92.2)
- added C10: 10µ, stmbl:C_1206, F.Cu at (168.2, 67.2)
- added C2: 100n, stmbl:C_0603, F.Cu at (182.1, 63.6)
- added C3: 100n, stmbl:C_0603, F.Cu at (177.3, 63.6)
- added C4: 100n, stmbl:C_0603, F.Cu at (182.9, 68.7)
- added C5: 100n, stmbl:C_0603, F.Cu at (172.6, 62.5)
- added C6: 100n, stmbl:C_0603, F.Cu at (178.1, 67.9)
- added C7: 100n, stmbl:C_0603, F.Cu at (181.2, 73.0)
- added C8: 100n, stmbl:C_0603, F.Cu at (167.8, 62.5)
- added C9: 10µ, stmbl:C_1206, F.Cu at (176.1, 72.6)
- added D1: LED, LEDs:LED_0603, F.Cu at (141.2, 75.1)
- added D10: LED, LEDs:LED_0603, F.Cu at (78.3, 75.1)
- added D11: LED, LEDs:LED_0603, F.Cu at (73.2, 75.1)
- added D12: LED, LEDs:LED_0603, F.Cu at (68.1, 75.1)
- added D13: LED, LEDs:LED_0603, F.Cu at (119.4, 96.3)
- added D14: LED, LEDs:LED_0603, F.Cu at (119.4, 97.8)
- added D15: LED, LEDs:LED_0603, F.Cu at (119.4, 99.3)
- added D16: LED, LEDs:LED_0603, F.Cu at (119.4, 100.8)
- added D17: LED, LEDs:LED_0603, F.Cu at (119.4, 102.3)
- added D18: LED, LEDs:LED_0603, F.Cu at (119.4, 103.9)
- added D19: LED, LEDs:LED_0603, F.Cu at (119.4, 105.4)
- added D2: LED, LEDs:LED_0603, F.Cu at (136.1, 75.1)
- added D20: LED, LEDs:LED_0603, F.Cu at (119.4, 106.9)
- added D21: LED, LEDs:LED_0603, F.Cu at (119.5, 125.2)
- added D22: LED, LEDs:LED_0603, F.Cu at (119.5, 126.7)
- added D23: LED, LEDs:LED_0603, F.Cu at (119.5, 128.3)
- added D24: LED, LEDs:LED_0603, F.Cu at (119.5, 129.8)
- added D25: LED, LEDs:LED_0603, F.Cu at (119.5, 131.3)
- added D26: LED, LEDs:LED_0603, F.Cu at (119.5, 132.8)
- added D27: LED, LEDs:LED_0603, F.Cu at (119.5, 134.4)
- added D28: LED, LEDs:LED_0603, F.Cu at (119.5, 135.8)
- added D29: B240A, Diodes_SMD:SMA_Standard, F.Cu at (170.3, 80.4)
- added D3: LED, LEDs:LED_0603, F.Cu at (131.0, 75.1)
- added D4: LED, LEDs:LED_0603, F.Cu at (125.9, 75.1)
- added D5: LED, LEDs:LED_0603, F.Cu at (112.1, 75.1)
- added D6: LED, LEDs:LED_0603, F.Cu at (107.1, 75.1)
- added D7: LED, LEDs:LED_0603, F.Cu at (102.0, 75.1)
- added D8: LED, LEDs:LED_0603, F.Cu at (96.9, 75.1)
- added D9: LED, LEDs:LED_0603, F.Cu at (83.4, 75.1)
- added L1: 4.7µH 1.5A, stmbl:SMD_INDUCTOR_32x25, F.Cu at (179.2, 79.6)
- added P1: CONN_01X08, Terminal_Blocks:TerminalBlock_Pheonix_PT-3.5mm_8pol, F.Cu at (120.0, 53.6)
- added P10: CONN_01X02, stmbl:akl182-2, F.Cu at (154.2, 58.2)
- added P2: CONN_01X08, Terminal_Blocks:TerminalBlock_Pheonix_PT-3.5mm_8pol, F.Cu at (91.0, 53.6)
- added P3: CONN_01X08, Terminal_Blocks:TerminalBlock_Pheonix_PT-3.5mm_8pol, F.Cu at (62.2, 53.6)
- added P4: CONN_01X08, Terminal_Blocks:TerminalBlock_Pheonix_PT-3.5mm_8pol, F.Cu at (144.7, 89.3)
- added P5: CONN_01X08, Terminal_Blocks:TerminalBlock_Pheonix_PT-3.5mm_8pol, F.Cu at (144.7, 118.4)
- added P6: CONN_01X08, Terminal_Blocks:TerminalBlock_Pheonix_PT-3.5mm_8pol, F.Cu at (151.8, 113.7)
- added P7: CONN_01X08, Terminal_Blocks:TerminalBlock_Pheonix_PT-3.5mm_8pol, F.Cu at (151.8, 142.9)
- added P8: CONN_02X25, Socket_Strips:Socket_Strip_Straight_2x25, F.Cu at (112.3, 143.3)
- added P9: CONN_02X25, Socket_Strips:Socket_Strip_Straight_2x25, F.Cu at (61.2, 143.3)
- added R1: R, stmbl:R_0603, F.Cu at (144.5, 59.9)
- added R10: R, stmbl:R_0603, F.Cu at (79.8, 60.0)
- added R11: R, stmbl:R_0603, F.Cu at (72.8, 60.0)
- added R12: R, stmbl:R_0603, F.Cu at (65.8, 60.0)
- added R13: R, stmbl:R_0603, F.Cu at (142.0, 77.4)
- added R14: R, stmbl:R_0603, F.Cu at (136.9, 77.4)
- added R15: R, stmbl:R_0603, F.Cu at (131.8, 77.4)
- added R16: R, stmbl:R_0603, F.Cu at (126.7, 77.4)
- added R17: R, stmbl:R_0603, F.Cu at (112.9, 77.4)
- added R18: R, stmbl:R_0603, F.Cu at (107.9, 77.4)
- added R19: R, stmbl:R_0603, F.Cu at (102.8, 77.3)
- added R2: R, stmbl:R_0603, F.Cu at (137.5, 60.0)
- added R20: R, stmbl:R_0603, F.Cu at (97.7, 77.3)
- added R21: R, stmbl:R_0603, F.Cu at (84.2, 77.4)
- added R22: R, stmbl:R_0603, F.Cu at (79.1, 77.4)
- added R23: R, stmbl:R_0603, F.Cu at (74.0, 77.4)
- added R24: R, stmbl:R_0603, F.Cu at (68.9, 77.4)
- added R25: R, stmbl:R_0603, F.Cu at (122.1, 96.3)
- added R26: R, stmbl:R_0603, F.Cu at (122.1, 97.8)
- added R27: R, stmbl:R_0603, F.Cu at (122.1, 99.3)
- added R28: R, stmbl:R_0603, F.Cu at (122.1, 100.8)
- added R29: R, stmbl:R_0603, F.Cu at (122.1, 102.3)
- added R3: R, stmbl:R_0603, F.Cu at (130.5, 60.0)
- added R30: R, stmbl:R_0603, F.Cu at (122.1, 103.9)
- added R31: R, stmbl:R_0603, F.Cu at (122.1, 105.4)
- added R32: R, stmbl:R_0603, F.Cu at (122.1, 106.9)
- added R33: R, stmbl:R_0603, F.Cu at (122.2, 125.2)
- added R34: R, stmbl:R_0603, F.Cu at (122.2, 126.7)
- added R35: R, stmbl:R_0603, F.Cu at (122.2, 128.3)
- added R36: R, stmbl:R_0603, F.Cu at (122.2, 129.8)
- added R37: R, stmbl:R_0603, F.Cu at (122.2, 131.3)
- added R38: R, stmbl:R_0603, F.Cu at (122.2, 132.8)
- added R39: R, stmbl:R_0603, F.Cu at (122.2, 134.4)
- added R4: R, stmbl:R_0603, F.Cu at (123.5, 60.0)
- added R40: R, stmbl:R_0603, F.Cu at (122.2, 135.8)
- added R41: 10k, stmbl:R_0603, F.Cu at (173.4, 68.0)
- added R42: 50k, stmbl:R_0603, F.Cu at (182.7, 88.3)
- added R5: R, stmbl:R_0603, F.Cu at (115.5, 60.0)
- added R6: R, stmbl:R_0603, F.Cu at (108.5, 60.0)
- added R7: R, stmbl:R_0603, F.Cu at (101.5, 60.0)
- added R8: R, stmbl:R_0603, F.Cu at (94.5, 60.0)
- added R9: R, stmbl:R_0603, F.Cu at (86.8, 60.0)
- added U1: OPTO-TRANSISTOR-4, Housings_DIP:DIP-16_W7.62mm, F.Cu at (141.2, 64.3)
- added U2: OPTO-TRANSISTOR-4, Housings_DIP:DIP-16_W7.62mm, F.Cu at (112.1, 64.0)
- added U3: OPTO-TRANSISTOR-4, Housings_DIP:DIP-16_W7.62mm, F.Cu at (83.4, 64.0)
- added U4: VN808, io_base:POWERSO36, F.Cu at (131.9, 101.5)
- added U5: VN808, io_base:POWERSO36, F.Cu at (131.9, 130.6)
- added U6: ACT4088, TO_SOT_Packages_SMD:SOT-23-6, F.Cu at (169.4, 73.2)
Routing:
- net Net-(P1-Pad1): track 0.00 -> 12.1 mm
- net Net-(P3-Pad1): track 0.00 -> 11.8 mm
- net Net-(P2-Pad1): track 0.00 -> 11.8 mm
- net PO16: track 0.00 -> 11.7 mm
- net Net-(P1-Pad7): track 0.00 -> 11.7 mm
- net PO8: track 0.00 -> 11.6 mm
- net Net-(P3-Pad7): track 0.00 -> 11.4 mm
- net Net-(P2-Pad7): track 0.00 -> 11.4 mm
- net Net-(P1-Pad3): track 0.00 -> 11.3 mm
- net Net-(P3-Pad3): track 0.00 -> 11.0 mm
- net Net-(P2-Pad3): track 0.00 -> 11.0 mm
- net PO1: track 0.00 -> 10.9 mm
- net Net-(P1-Pad5): track 0.00 -> 10.9 mm
- net PO9: track 0.00 -> 10.8 mm
- net Net-(P3-Pad5): track 0.00 -> 10.6 mm
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
Commit message: WIP
Routing:
- net +3V3: track 0.00 -> 92.1 mm
- net OUT16: track 0.00 -> 75.3 mm, vias 0 -> 3
- net OUT15: track 0.00 -> 73.5 mm, vias 0 -> 3
- net OUT8: track 0.00 -> 68.9 mm
- net OUT14: track 0.00 -> 67.9 mm, vias 0 -> 3
- net OUT2: track 0.00 -> 67.6 mm, vias 0 -> 2
- net OUT4: track 0.00 -> 66.8 mm, vias 0 -> 2
- net OUT6: track 0.00 -> 66.7 mm, vias 0 -> 2
- net OUT1: track 0.00 -> 65.6 mm, vias 0 -> 2
- net OUT13: track 0.00 -> 65.5 mm, vias 0 -> 3
- net OUT7: track 0.00 -> 63.9 mm, vias 0 -> 2
- net OUT3: track 0.00 -> 63.6 mm, vias 0 -> 2
- net OUT5: track 0.00 -> 62.9 mm, vias 0 -> 2
- net OUT11: track 0.00 -> 58.2 mm, vias 0 -> 3
- net OUT12: track 0.00 -> 57.3 mm, vias 0 -> 3
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Other:
- board text added: "BOTANYDIVING"
