File: hw/kicad/stmsp/io.sch (KiCad schematic (older format))
At the start: 28 parts, among them Q1 Q_NJFET_GSD, Q2 Q_NJFET_GSD, U1 USBLC6-4SC6, U10 USBLC6-4SC6

Commit message: stmsp
Parts:
- removed C30, C5: C, stmbl:C_0603, symbol C
- removed U1, U10: USBLC6-4SC6, stmbl:SOT-23-6, symbol USBLC6-4SC6
Connections:
- net AIN0 is gone; now on net IN0: R37.1
- net AIN1 is gone; now on net IN1: R40.1
- net AIN2 is gone; now on net IN2: R43.1
- net IN0: no longer C31.1, R37.2, R38.1, R39.2
- net IN1: no longer C32.1, R40.2, R41.1, R42.2
- net IN2: no longer C33.1, R43.2, R44.1, R45.2
- new net I0: C31.1, R37.2, R38.1, R39.2
- new net I1: C32.1, R40.2, R41.1, R42.2
- new net I2: C33.1, R43.2, R44.1, R45.2
Other:
- note added: "IRLML0060TRPBF"
Changed lines of the file:
@@
 EESchema Schematic File Version 2
-LIBS:stmsp-rescue
+LIBS:stmbl
 LIBS:transistors
 LIBS:stm32
@@
 LIBS:video
 LIBS:Xicor
-LIBS:xilinx
-LIBS:Zilog
-LIBS:stmbl
 LIBS:stmsp-cache
 EELAYER 26 0
@@
 $Descr A4 11693 8268
 encoding utf-8
-Sheet 7 7
+Sheet 7 9
 Title ""
 Date ""
@@
 $EndDescr
 $Comp
-L USBLC6-4SC6 U10
-U 1 1 59235FEA
-P 5700 3650
-F 0 "U10" H 5001 3998 50  0000 C CNN
-F 1 "USBLC6-4SC6" H 5700 3900 50  0000 C CNN
-F 2 "stmbl:SOT-23-6" H 5700 3650 60  0001 C CNN
-F 3 "" H 5700 3650 60  0000 C CNN
-F 4 "TRANSIENT VOLTAGE SUPPRESSOR" H 5700 3400 50  0000 C CNN "Description"
-	1    5700 3650
-	1    0    0    -1
-$EndComp
-$Comp
 L R R40
 U 1 1 59236B6A
@@
 Connection ~ 8050 1950
 $Comp
-L +3.3V #PWR042
+L +3.3V #PWR052
 U 1 1 59236E8B
 P 8300 1450
-F 0 "#PWR042" H 8300 1300 50  0001 C CNN
+F 0 "#PWR052" H 8300 1300 50  0001 C CNN
 F 1 "+3.3V" H 8300 1590 50  0000 C CNN
 F 2 "" H 8300 1450 50  0000 C CNN
@@
 	8300 2350 8300 2550
 $Comp
-L GND #PWR043
+L GND #PWR053
 U 1 1 59236F1D
 P 8300 2550
-F 0 "#PWR043" H 8300 2300 50  0001 C CNN
+F 0 "#PWR053" H 8300 2300 50  0001 C CNN
 F 1 "GND" H 8300 2400 50  0000 C CNN
 F 2 "" H 8300 2550 50  0000 C CNN
@@
 	8050 1450 7950 1450
 Text HLabel 7950 1450 0    60   Input ~ 0
-AIN1
+IN1
 Text HLabel 8400 1950 2    60   Input ~ 0
-IN1
-Text HLabel 4550 3550 0    60   Input ~ 0
-IN0
-Wire Wire Line
-	4550 3550 4650 3550
-$Comp
-L C C30
-U 1 1 592371B8
-P 7250 3650
-F 0 "C30" H 7275 3750 50  0000 L CNN
-F 1 "C" H 7275 3550 50  0000 L CNN
-F 2 "stmbl:C_0603" H 7288 3500 50  0001 C CNN
-F 3 "" H 7250 3650 50  0000 C CNN
-	1    7250 3650
-	1    0    0    -1
-$EndComp
-$Comp
-L +3.3V #PWR044
-U 1 1 59237267
-P 7250 3400
-F 0 "#PWR044" H 7250 3250 50  0001 C CNN
-F 1 "+3.3V" H 7250 3540 50  0000 C CNN
-F 2 "" H 7250 3400 50  0000 C CNN
-F 3 "" H 7250 3400 50  0000 C CNN
-	1    7250 3400
-	1    0    0    -1
-$EndComp
-$Comp
-L GND #PWR045
-U 1 1 592372E0
-P 7250 3900
-F 0 "#PWR045" H 7250 3650 50  0001 C CNN
-F 1 "GND" H 7250 3750 50  0000 C CNN
-F 2 "" H 7250 3900 50  0000 C CNN
-F 3 "" H 7250 3900 50  0000 C CNN
-	1    7250 3900
-	1    0    0    -1
-$EndComp
-Wire Wire Line
-	7250 3400 7250 3500
-Wire Wire Line
-	7250 3800 7250 3900
-$Comp
-L GND #PWR046
-U 1 1 592373AB
-P 4550 3650
-F 0 "#PWR046" H 4550 3400 50  0001 C CNN
-F 1 "GND" H 4550 3500 50  0000 C CNN
-F 2 "" H 4550 3650 50  0000 C CNN
-F 3 "" H 4550 3650 50  0000 C CNN
-	1    4550 3650
-	0    1    1    0
-$EndComp
-Wire Wire Line
-	4550 3650 4650 3650
-$Comp
-L +3.3V #PWR047
-U 1 1 5923743F
-P 6850 3650
-F 0 "#PWR047" H 6850 3500 50  0001 C CNN
-F 1 "+3.3V" H 6850 3790 50  0000 C CNN
-F 2 "" H 6850 3650 50  0000 C CNN
-F 3 "" H 6850 3650 50  0000 C CNN
-	1    6850 3650
-	0    1    1    0
-$EndComp
-Wire Wire Line
-	6750 3650 6850 3650
+I1
 $Comp
 L R R43
@@
 Connection ~ 8900 1950
 $Comp
-L +3.3V #PWR048
+L +3.3V #PWR054
 U 1 1 59237877
 P 9150 1450
-F 0 "#PWR048" H 9150 1300 50  0001 C CNN
+F 0 "#PWR054" H 9150 1300 50  0001 C CNN
 F 1 "+3.3V" H 9150 1590 50  0000 C CNN
 F 2 "" H 9150 1450 50  0000 C CNN
@@
 	9150 2350 9150 2550
 $Comp
-L GND #PWR049
+L GND #PWR055
 U 1 1 59237881
 P 9150 2550
-F 0 "#PWR049" H 9150 2300 50  0001 C CNN
+F 0 "#PWR055" H 9150 2300 50  0001 C CNN
 F 1 "GND" H 9150 2400 50  0000 C CNN
 F 2 "" H 9150 2550 50  0000 C CNN
@@
 	8900 1450 8800 1450
 Text HLabel 8800 1450 0    60   Input ~ 0
-AIN2
+IN2
 Text HLabel 9250 1950 2    60   Input ~ 0
-IN2
+I2
 $Comp
 L R R37
@@
 Connection ~ 7200 1950
 $Comp
-L +3.3V #PWR050
+L +3.3V #PWR056
 U 1 1 5923794F
 P 7450 1450
-F 0 "#PWR050" H 7450 1300 50  0001 C CNN
+F 0 "#PWR056" H 7450 1300 50  0001 C CNN
 F 1 "+3.3V" H 7450 1590 50  0000 C CNN
 F 2 "" H 7450 1450 50  0000 C CNN
@@
 	7450 2350 7450 2550
 $Comp
-L GND #PWR051
+L GND #PWR057
 U 1 1 59237959
 P 7450 2550
-F 0 "#PWR051" H 7450 2300 50  0001 C CNN
+F 0 "#PWR057" H 7450 2300 50  0001 C CNN
 F 1 "GND" H 7450 2400 50  0000 C CNN
 F 2 "" H 7450 2550 50  0000 C CNN
@@
 	7200 1450 7100 1450
 Text HLabel 7100 1450 0    60   Input ~ 0
-AIN0
+IN0
 Text HLabel 7550 1950 2    60   Input ~ 0
-IN0
-Text HLabel 4550 3750 0    60   Input ~ 0
-IN1
-Wire Wire Line
-	4550 3750 4650 3750
-Text HLabel 6850 3550 2    60   Input ~ 0
-IN1
-Wire Wire Line
-	6850 3550 6750 3550
+I0
 $Comp
 L R R35
@@
 	5100 2250 5100 2650
 $Comp
-L VPP #PWR052
+L VPP #PWR058
 U 1 1 59238B56
 P 5100 1250
-F 0 "#PWR052" H 5100 1100 50  0001 C CNN
+F 0 "#PWR058" H 5100 1100 50  0001 C CNN
 F 1 "VPP" H 5100 1400 50  0000 C CNN
 F 2 "" H 5100 1250 50  0000 C CNN
@@
 Connection ~ 5100 2550
 $Comp
-L GND #PWR053
+L GND #PWR059
 U 1 1 59238DA9
 P 5100 2650
-F 0 "#PWR053" H 5100 2400 50  0001 C CNN
+F 0 "#PWR059" H 5100 2400 50  0001 C CNN
 F 1 "GND" H 5100 2500 50  0000 C CNN
 F 2 "" H 5100 2650 50  0000 C CNN
@@
 	2800 2250 2800 2650
 $Comp
-L VPP #PWR054
+L VPP #PWR060
 U 1 1 5923AA35
 P 2800 1250
-F 0 "#PWR054" H 2800 1100 50  0001 C CNN
+F 0 "#PWR060" H 2800 1100 50  0001 C CNN
 F 1 "VPP" H 2800 1400 50  0000 C CNN
 F 2 "" H 2800 1250 50  0000 C CNN
@@
 Connection ~ 2800 2550
 $Comp
-L GND #PWR055
+L GND #PWR061
 U 1 1 5923AA3F
 P 2800 2650
-F 0 "#PWR055" H 2800 2400 50  0001 C CNN
+F 0 "#PWR061" H 2800 2400 50  0001 C CNN
 F 1 "GND" H 2800 2500 50  0000 C CNN
 F 2 "" H 2800 2650 50  0000 C CNN
@@
 	2150 1850 2150 1750
 Connection ~ 2150 1750
-$Comp
-L USBLC6-4SC6 U1
-U 1 1 5923B2F2
-P 5700 4600
-F 0 "U1" H 5001 4948 50  0000 C CNN
-F 1 "USBLC6-4SC6" H 5700 4850 50  0000 C CNN
-F 2 "stmbl:SOT-23-6" H 5700 4600 60  0001 C CNN
-F 3 "" H 5700 4600 60  0000 C CNN
-F 4 "TRANSIENT VOLTAGE SUPPRESSOR" H 5700 4350 50  0000 C CNN "Description"
-	1    5700 4600
-	1    0    0    -1
-$EndComp
-Text HLabel 4550 4500 0    60   Input ~ 0
-SWCLK
-Wire Wire Line
-	4550 4500 4650 4500
-$Comp
-L C C5
-U 1 1 5923B2FA
-P 7250 4600
-F 0 "C5" H 7275 4700 50  0000 L CNN
-F 1 "C" H 7275 4500 50  0000 L CNN
-F 2 "stmbl:C_0603" H 7288 4450 50  0001 C CNN
-F 3 "" H 7250 4600 50  0000 C CNN
-	1    7250 4600
-	1    0    0    -1
-$EndComp
-$Comp
-L +3.3V #PWR056
-U 1 1 5923B300
-P 7250 4350
-F 0 "#PWR056" H 7250 4200 50  0001 C CNN
-F 1 "+3.3V" H 7250 4490 50  0000 C CNN
-F 2 "" H 7250 4350 50  0000 C CNN
-F 3 "" H 7250 4350 50  0000 C CNN
-	1    7250 4350
-	1    0    0    -1
-$EndComp
-$Comp
-L GND #PWR057
-U 1 1 5923B306
-P 7250 4850
-F 0 "#PWR057" H 7250 4600 50  0001 C CNN
-F 1 "GND" H 7250 4700 50  0000 C CNN
-F 2 "" H 7250 4850 50  0000 C CNN
-F 3 "" H 7250 4850 50  0000 C CNN
-	1    7250 4850
-	1    0    0    -1
-$EndComp
-Wire Wire Line
-	7250 4350 7250 4450
-Wire Wire Line
-	7250 4750 7250 4850
-$Comp
-L GND #PWR058
-U 1 1 5923B30E
-P 4550 4600
-F 0 "#PWR058" H 4550 4350 50  0001 C CNN
-F 1 "GND" H 4550 4450 50  0000 C CNN
-F 2 "" H 4550 4600 50  0000 C CNN
-F 3 "" H 4550 4600 50  0000 C CNN
-	1    4550 4600
-	0    1    1    0
-$EndComp
-Wire Wire Line
-	4550 4600 4650 4600
-$Comp
-L +3.3V #PWR059
-U 1 1 5923B315
-P 6850 4600
-F 0 "#PWR059" H 6850 4450 50  0001 C CNN
-F 1 "+3.3V" H 6850 4740 50  0000 C CNN
-F 2 "" H 6850 4600 50  0000 C CNN
-F 3 "" H 6850 4600 50  0000 C CNN
-	1    6850 4600
-	0    1    1    0
-$EndComp
-Wire Wire Line
-	6750 4600 6850 4600
-Text HLabel 4550 4700 0    60   Input ~ 0
-SWDIO
-Wire Wire Line
-	4550 4700 4650 4700
-Text HLabel 6850 4500 2    60   Input ~ 0
-USBDP
-Wire Wire Line
-	6850 4500 6750 4500
-Text HLabel 6850 3750 2    60   Input ~ 0
-NRST
-Wire Wire Line
-	6850 3750 6750 3750
-Text HLabel 6850 4700 2    60   Input ~ 0
-USBDP
-Wire Wire Line
-	6850 4700 6750 4700
+Text Notes 3100 1750 0    60   ~ 0
+IRLML0060TRPBF
 $EndSCHEMATC
