File: hw/kicad/stmsp/sensor.sch (KiCad schematic (older format))
At the start: 3 parts, among them U7 TLE5012

Commit message: stmsp
Parts:
- added U10: TLE5012, stmbl:SOIC-8-N, symbol TLE5012
Connections:
- net CSQ: now also U10.3 (CSQ)
- net DATA: now also U10.4 (DATA)
- net GND: now also U10.1 (CLK), U10.7 (GND)
- net SCK: now also U10.2 (SCK)
- net at C27.1, JP2.2, U7.6 (VCC): now also U10.6 (VCC)
Changed lines of the file:
@@
 EESchema Schematic File Version 2
-LIBS:stmsp-rescue
+LIBS:stmbl
 LIBS:transistors
 LIBS:stm32
@@
 LIBS:video
 LIBS:Xicor
-LIBS:xilinx
-LIBS:Zilog
-LIBS:stmbl
 LIBS:stmsp-cache
 EELAYER 26 0
@@
 $Descr A4 11693 8268
 encoding utf-8
-Sheet 5 7
+Sheet 4 10
 Title ""
 Date ""
@@
 $EndComp
 $Comp
-L GND #PWR032
+L GND #PWR029
 U 1 1 5923BFBE
 P 5450 3350
-F 0 "#PWR032" H 5450 3100 50  0001 C CNN
+F 0 "#PWR029" H 5450 3100 50  0001 C CNN
 F 1 "GND" H 5450 3200 50  0000 C CNN
 F 2 "" H 5450 3350 50  0000 C CNN
@@
 	4550 3150 4650 3150
 $Comp
-L GND #PWR033
+L GND #PWR030
 U 1 1 5923C005
 P 5000 3750
-F 0 "#PWR033" H 5000 3500 50  0001 C CNN
+F 0 "#PWR030" H 5000 3500 50  0001 C CNN
 F 1 "GND" H 5000 3600 50  0000 C CNN
 F 2 "" H 5000 3750 50  0000 C CNN
@@
 	5000 3550 5000 3750
 $Comp
-L +5V #PWR034
+L +5V #PWR031
 U 1 1 5923C047
 P 4650 2550
-F 0 "#PWR034" H 4650 2400 50  0001 C CNN
+F 0 "#PWR031" H 4650 2400 50  0001 C CNN
 F 1 "+5V" H 4650 2690 50  0000 C CNN
 F 2 "" H 4650 2550 50  0000 C CNN
@@
 	5000 2750 5000 2950
 $Comp
-L +3.3V #PWR035
+L +3.3V #PWR032
 U 1 1 5923C08F
 P 5350 2550
-F 0 "#PWR035" H 5350 2400 50  0001 C CNN
+F 0 "#PWR032" H 5350 2400 50  0001 C CNN
 F 1 "+3.3V" H 5350 2690 50  0000 C CNN
 F 2 "" H 5350 2550 50  0000 C CNN
@@
 	5350 2650 5350 2550
 Wire Wire Line
-	5950 3200 5950 2850
-Wire Wire Line
-	5950 2850 5000 2850
+	5950 2850 5950 3200
+Wire Wire Line
+	3350 2850 5950 2850
 Connection ~ 5000 2850
 Wire Wire Line
-	5000 3650 5950 3650
+	3350 3650 5950 3650
 Wire Wire Line
 	5950 3650 5950 3500
 Connection ~ 5000 3650
+$Comp
+L TLE5012 U10
+U 1 1 5945AC83
+P 3350 3250
+F 0 "U10" H 3150 3500 60  0000 C CNN
+F 1 "TLE5012" H 3600 3000 60  0000 C CNN
+F 2 "stmbl:SOIC-8-N" H 3300 3250 60  0001 C CNN
+F 3 "" H 3300 3250 60  0001 C CNN
+	1    3350 3250
+	-1   0    0    -1
+$EndComp
+Text HLabel 3800 3150 2    60   Input ~ 0
+CSQ
+Text HLabel 3800 3250 2    60   Input ~ 0
+SCK
+Text HLabel 3800 3350 2    60   Input ~ 0
+DATA
+Wire Wire Line
+	3800 3350 3700 3350
+Wire Wire Line
+	3800 3250 3700 3250
+Wire Wire Line
+	3800 3150 3700 3150
+Wire Wire Line
+	3350 3650 3350 3550
+Wire Wire Line
+	3350 2850 3350 2950
+$Comp
+L GND #PWR033
+U 1 1 5945AE01
+P 2900 3350
+F 0 "#PWR033" H 2900 3100 50  0001 C CNN
+F 1 "GND" H 2900 3200 50  0000 C CNN
+F 2 "" H 2900 3350 50  0000 C CNN
+F 3 "" H 2900 3350 50  0000 C CNN
+	1    2900 3350
+	0    1    1    0
+$EndComp
+Wire Wire Line
+	2900 3350 3000 3350
 $EndSCHEMATC
