File: hw/kicad/stmsp/stmsp.kicad_pcb (KiCad board)
At the start: 4 copper layers, 42 x 42 mm, 127 parts, among them J1 CONN_02X05, P1 USB_OTG, P2 CONN_01X04, P3 CONN_01X04, P4 CONN_01X02, P5 CONN_01X06, P6 CONN_01X02, Q1 Q_NJFET_GSD, Q2 Q_NJFET_GSD, U1 USBLC6-4SC6, U10 TLE5012, U2 L6206Q, U3 STM32F303CBTx, U4 USBLC6-4SC6, U5 MCP16331, U6 MIC55, U7 TLE5012, U8 SN65176B, U9 SN65176B, Y1 8M

Commit message: stmsp
Parts:
- added R43: 470, stmbl:R_0603, F.Cu at (73.2, 75.8)
- added T1: testpoint, stmbl:Measurement_Point_Round-SMD-Pad_Small, F.Cu at (59.1, 95.6)
- added T2: testpoint, stmbl:Measurement_Point_Round-SMD-Pad_Small, F.Cu at (59.1, 102.7)
- added T3: testpoint, stmbl:Measurement_Point_Round-SMD-Pad_Small, F.Cu at (66.2, 95.6)
- added T4: testpoint, stmbl:Measurement_Point_Round-SMD-Pad_Small, B.Cu at (55.0, 78.5)
- added T5: testpoint, stmbl:Measurement_Point_Round-SMD-Pad_Small, B.Cu at (55.0, 80.2)
- U6: value MIC55 -> MIC5504-3.3YM5
- moved C37 0.75 mm to (69.8, 76.0)
- moved U4 0.75 mm to (66.5, 76.0)
- moved R26 0.50 mm to (90.2, 59.5)
- moved JP2 0.35 mm to (64.8, 71.8)
- moved C36 0.25 mm to (63.2, 74.0)
- moved C4 0.25 mm to (70.8, 78.5)
Connections:
- U3 pad 16: (no net) -> Net-(T3-Pad1)
- U3 pad 19: (no net) -> Net-(T1-Pad1)
- U3 pad 25: (no net) -> Net-(T2-Pad1)
- U3 pad 41: /MOSI -> Net-(R43-Pad1)
Routing:
- net +5V: track 36.2 -> 106.2 mm, vias 1 -> 8
- net /TEMP: track 3.85 -> 32.0 mm
- net /DCLINK: track 5.31 -> 30.4 mm
- net GND: track 106.0 -> 126.6 mm, vias 58 -> 80
- net Net-(C27-Pad1): track 9.03 -> 22.0 mm, vias 1 -> 2
- net VPP: track 34.3 -> 43.7 mm
- net /MOSI: track 21.2 -> 11.8 mm
- net Net-(R25-Pad2): track 0.00 -> 5.13 mm
- net Net-(P1-Pad3): track 2.85 -> 6.06 mm, vias 0 -> 1
- net +3V3: track 106.0 -> 109.1 mm, vias 14 -> 15
- net Net-(C24-Pad1): track 0.00 -> 3.09 mm
- net Net-(P1-Pad2): track 1.64 -> 4.64 mm, vias 0 -> 1
- net Net-(R43-Pad1): track 0.00 -> 1.75 mm
- net /SWDIO: track 22.2 -> 23.8 mm
- net /ENA: track 28.5 -> 27.3 mm
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- added copper zone on F.Cu, net +3V3
- added copper zone on F.Cu, net +5V
- added copper zone on F.Cu, net Net-(C24-Pad2)

Commit message: stmsp
Parts:
- added REF**: Fiducial_1mm_Dia_2.54mm_Outer_CopperTop, stmbl:Fiducial_1mm_Outer_CopperTop, F.Cu at (57.5, 57.5)
- added REF**: Fiducial_1mm_Dia_2.54mm_Outer_CopperTop, stmbl:Fiducial_1mm_Outer_CopperTop, F.Cu at (90.0, 85.0)
- T1, T2, T3: moved to B.Cu
- moved T2 34.8 mm to (80.0, 75.0)
- moved T1 28.4 mm to (80.0, 76.5)
- moved T3 22.4 mm to (80.0, 78.0)
Routing:
- net GND: track 126.6 -> 165.5 mm, vias 80 -> 125
- net Net-(T2-Pad1): track 0.00 -> 4.91 mm, vias 0 -> 1
- net Net-(T1-Pad1): track 0.00 -> 4.76 mm, vias 0 -> 1
- net Net-(T3-Pad1): track 0.00 -> 4.60 mm, vias 0 -> 1
- net /DCLINK: track 30.4 -> 31.5 mm
- net /BEMF_1A: track 23.2 -> 24.2 mm
- net Net-(R12-Pad2): track 41.2 -> 41.9 mm

Commit message: stmsp
Parts:
- moved T5 0.25 mm to (55.0, 80.5)
Changed lines of the file:
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@@
     (thickness 1.6)
     (drawings 16)
-    (tracks 1234)
+    (tracks 1235)
     (zones 0)
     (modules 135)
@@
   )
   (module stmbl:Measurement_Point_Round-SMD-Pad_Small (layer B.Cu)
-    (at 55 80.25)
+    (at 55 80.5)
     (descr "Mesurement Point, Round, SMD Pad, DM 1.5mm,")
     (tags "Mesurement Point, Round, SMD Pad, DM 1.5mm,")
@@
   (segment (start 56.5 78.5) (end 56.15 78.85) (width 0.2) (layer F.Cu) (net 4) (status 10))
   (segment (start 56.15 78.85) (end 55 78.85) (width 0.2) (layer F.Cu) (net 4) (status 20))
+  (segment (start 55 80.25) (end 55.25 80.5) (width 0.2) (layer B.Cu) (net 5))
+  (segment (start 55.25 80.5) (end 56.5 80.5) (width 0.2) (layer B.Cu) (net 5))
+  (segment (start 56.5 80.5) (end 57.25 79.75) (width 0.2) (layer B.Cu) (net 5))
   (segment (start 57.25 79.75) (end 56.5 79.75) (width 0.2) (layer F.Cu) (net 5))
-  (segment (start 55 80.25) (end 56.75 80.25) (width 0.2) (layer B.Cu) (net 5))
-  (segment (start 56.75 80.25) (end 57.25 79.75) (width 0.2) (layer B.Cu) (net 5))
   (via (at 57.25 79.75) (size 0.6) (drill 0.3) (layers F.Cu B.Cu) (net 5))
   (segment (start 56.5 81) (end 56.5 79.75) (width 0.2) (layer F.Cu) (net 5) (status 30))

Commit message: stmsp
Parts:
- C26: value 10u -> 22u
- C34, C35, C6: value C -> 18p
- R12, R8: value 0.015 -> 0.02
- R32, R37: value 1k -> 1.5k
- R46, R47, R48: value R -> 3.9k
- R49, R50, R51: value R -> 120
- moved R3 0.75 mm to (58.0, 81.0)
- moved R4 0.75 mm to (58.0, 78.5)
- moved R5 0.75 mm to (58.0, 79.8)
- moved P1 0.50 mm to (52.8, 79.5)
- moved T4 0.50 mm to (55.5, 78.5)
- moved T5 0.50 mm to (55.5, 80.5)
- moved D7 0.25 mm to (76.0, 91.0)
- moved D8 0.25 mm to (80.0, 91.0)
- moved D9 0.25 mm to (84.0, 91.0)
- moved R52 0.25 mm to (76.0, 89.5)
- moved R53 0.25 mm to (80.0, 89.5)
- moved R54 0.25 mm to (83.2, 89.5)
- moved Y1 0.25 mm to (77.5, 86.8)
Routing:
- net +5V: track 106.3 -> 16.4 mm, vias 8 -> 9
- net +3V3: track 109.1 -> 47.6 mm, vias 15 -> 19
- net Net-(C13-Pad1): track 24.0 -> 9.79 mm
- net GND: track 165.5 -> 175.1 mm, vias 125 -> 131
- net VPP: track 43.7 -> 47.5 mm, vias 8 -> 14
- added copper zone on In2.Cu, net +3V3
- added copper zone on In2.Cu, net +5V
- added copper zone on In2.Cu, net Net-(C13-Pad1)
- removed copper zone on In2.Cu, net GND
Other:
- outline, holes or cut-outs redrawn

Commit message: stmsp
Routing:
- added copper zone on In2.Cu, net GND
Changed lines of the file:
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@@
   (segment (start 86 74) (end 86.75 74) (width 0.2) (layer F.Cu) (net 77))
   (segment (start 86 74) (end 84.35 74) (width 0.2) (layer F.Cu) (net 77))
-  (segment (start 84.5 72) (end 84.5 72.75) (width 0.2) (layer B.Cu) (net 77))
+  (segment (start 84.5 72) (end 84.5 72.75) (width 0.2) (layer F.Cu) (net 77))
   (via (at 84.5 72.75) (size 0.6) (drill 0.3) (layers F.Cu B.Cu) (net 77))
   (segment (start 84.5 71.25) (end 84.5 72) (width 0.2) (layer F.Cu) (net 77))
   (via (at 84.5 72) (size 0.6) (drill 0.3) (layers F.Cu B.Cu) (net 77))
-  (segment (start 85.25 71.25) (end 84.5 71.25) (width 0.2) (layer B.Cu) (net 77))
+  (segment (start 85.25 71.25) (end 84.5 71.25) (width 0.2) (layer F.Cu) (net 77))
   (via (at 84.5 71.25) (size 0.6) (drill 0.3) (layers F.Cu B.Cu) (net 77))
   (segment (start 85.25 72) (end 85.25 71.25) (width 0.2) (layer F.Cu) (net 77))
   (via (at 85.25 71.25) (size 0.6) (drill 0.3) (layers F.Cu B.Cu) (net 77))
-  (segment (start 85.25 72.75) (end 85.25 72) (width 0.2) (layer B.Cu) (net 77))
+  (segment (start 85.25 72.75) (end 85.25 72) (width 0.2) (layer F.Cu) (net 77))
   (via (at 85.25 72) (size 0.6) (drill 0.3) (layers F.Cu B.Cu) (net 77))
   (segment (start 88.1 71.6) (end 86.95 72.75) (width 0.2) (layer F.Cu) (net 77))
@@
     )
   )
-  (zone (net 0) (net_name "") (layer In1.Cu) (hatch edge 0.508)
-    (connect_pads yes (clearance 0.2))
-    (min_thickness 0.2)
-    (keepout (tracks not_allowed) (vias not_allowed) (copperpour not_allowed))
-    (fill yes (arc_segments 16) (thermal_gap 0.2) (thermal_bridge_width 0.25))
-    (polygon
-      (pts
-        (xy 85.75 66)
-      )
-    )
-  )
   (zone (net 10) (net_name +5V) (layer F.Cu) (hatch edge 0.508)
     (priority 1)
@@
       )
     )
+  )
+  (zone (net 7) (net_name GND) (layer In1.Cu) (hatch edge 0.508)
+    (connect_pads yes (clearance 0.25))
+    (min_thickness 0.25)
+    (fill yes (arc_segments 16) (thermal_gap 0.508) (thermal_bridge_width 0.508))
+    (polygon
+      (pts
+        (xy 63 55.75) (xy 69 55.75) (xy 69 61.75) (xy 63 61.75)
+      )
+    )
+  )
+  (zone (net 7) (net_name GND) (layer In2.Cu) (hatch edge 0.508)
+    (connect_pads yes (clearance 0.25))
+    (min_thickness 0.25)
+    (fill yes (arc_segments 16) (thermal_gap 0.508) (thermal_bridge_width 0.508))
+    (polygon
+      (pts
+        (xy 63.25 50) (xy 68.75 50) (xy 68.75 61.75) (xy 63.25 61.75)
+      )
+    )
+  )
+  (zone (net 0) (net_name "") (layer In2.Cu) (hatch edge 0.508)
+    (connect_pads yes (clearance 0.25))
+    (min_thickness 0.25)
+    (keepout (tracks allowed) (vias allowed) (copperpour not_allowed))
+    (fill yes (arc_segments 16) (thermal_gap 0.508) (thermal_bridge_width 0.508))
+    (polygon
+      (pts
+        (xy 65.75 53.25) (xy 65.5 53.5) (xy 65.5 54) (xy 65.75 54.25) (xy 66.25 54.25)
+        (xy 66.5 54) (xy 66.5 53.5) (xy 66.25 53.25)
+      )
+    )
+  )
+  (zone (net 0) (net_name "") (layer B.Cu) (hatch edge 0.508)
+    (connect_pads yes (clearance 0.25))
+    (min_thickness 0.25)
+    (keepout (tracks allowed) (vias allowed) (copperpour not_allowed))
+    (fill yes (arc_segments 16) (thermal_gap 0.508) (thermal_bridge_width 0.508))
+    (polygon
+      (pts
+        (xy 65.75 53.25) (xy 65.5 53.5) (xy 65.5 54) (xy 65.75 54.25) (xy 66.25 54.25)
+        (xy 66.5 54) (xy 66.5 53.5) (xy 66.25 53.25)
+      )
+    )

Commit message: stmsp
Parts:
- moved R46 0.25 mm to (89.8, 76.5)
- moved R47 0.25 mm to (89.8, 75.2)
- moved R48 0.25 mm to (89.8, 79.0)
- moved R49 0.25 mm to (89.8, 77.8)
- moved R50 0.25 mm to (89.8, 74.0)
- moved R51 0.25 mm to (89.8, 80.2)
Routing:
- net GND: track 175.1 -> 177.3 mm, vias 131 -> 132
- net Net-(R12-Pad2): track 41.9 -> 42.5 mm

Commit message: stmsp
Routing:
- net Net-(C27-Pad1): track 22.0 -> 23.0 mm
- net /SCK: track 14.7 -> 15.6 mm
- net /MOSI: track 11.8 -> 12.7 mm
- added copper zone on B.Cu, net /CSQ
- added copper zone on B.Cu, net /MOSI
- added copper zone on B.Cu, net /SCK
- added copper zone on B.Cu, net Net-(C27-Pad1)
Changed lines of the file:
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@@
     (thickness 1.6)
     (drawings 20)
-    (tracks 1234)
+    (tracks 1238)
     (zones 0)
     (modules 135)
@@
   (segment (start 85 63.5) (end 85 62.4) (width 0.2) (layer F.Cu) (net 16) (status 30))
   (segment (start 85 62.4) (end 85.2 62.2) (width 0.2) (layer F.Cu) (net 16) (status 30))
+  (segment (start 70 71.5) (end 70 72.5) (width 0.2) (layer B.Cu) (net 17))
   (segment (start 62.5 69.75) (end 62.5 70) (width 0.2) (layer F.Cu) (net 17))
   (segment (start 62.5 70) (end 63 70.5) (width 0.2) (layer F.Cu) (net 17))
@@
   (segment (start 69.25 83.25) (end 68.095 82.095) (width 0.2) (layer F.Cu) (net 60) (status 20))
   (segment (start 68.095 82.095) (end 68.095 81.75) (width 0.2) (layer F.Cu) (net 60) (status 30))
+  (segment (start 73.75 72.905) (end 74.475 72.905) (width 0.2) (layer B.Cu) (net 61))
+  (segment (start 74.475 72.905) (end 74.57 73) (width 0.2) (layer B.Cu) (net 61))
   (segment (start 72.5 75.75) (end 71.75 75.75) (width 0.2) (layer F.Cu) (net 61))
   (segment (start 71.75 75.75) (end 71.75 74) (width 0.2) (layer B.Cu) (net 61))
@@
   (segment (start 68.75 73) (end 68.655 72.905) (width 0.2) (layer F.Cu) (net 61) (status 30))
   (segment (start 68.655 72.905) (end 68.25 72.905) (width 0.2) (layer F.Cu) (net 61) (status 30))
+  (segment (start 73.75 70.365) (end 74.635 70.365) (width 0.2) (layer B.Cu) (net 62))
   (segment (start 69.75 70.25) (end 70.5 69.5) (width 0.2) (layer B.Cu) (net 62))
   (segment (start 70.5 69.5) (end 72.5 69.5) (width 0.2) (layer B.Cu) (net 62))
@@
       )
     )
+  )
+  (zone (net 61) (net_name /MOSI) (layer B.Cu) (hatch edge 0.508)
+    (priority 1)
+    (connect_pads yes (clearance 0.25))
+    (min_thickness 0.254)
+    (fill yes (arc_segments 16) (thermal_gap 0.508) (thermal_bridge_width 0.508))
+    (polygon
+      (pts
+        (xy 74.25 72.5) (xy 74.5 72.25) (xy 75.75 72.25) (xy 76 72.5) (xy 76 73.25)
+        (xy 75.75 73.5) (xy 74.5 73.5) (xy 74.25 73.25)
+      )
+    )
+  )
+  (zone (net 63) (net_name /CSQ) (layer B.Cu) (hatch edge 0.508)
+    (priority 1)
+    (connect_pads yes (clearance 0.25))
+    (min_thickness 0.254)
+    (fill yes (arc_segments 16) (thermal_gap 0.508) (thermal_bridge_width 0.508))
+    (polygon
+      (pts
+        (xy 71.5 71.25) (xy 71.75 71) (xy 73 71) (xy 73.25 71.25) (xy 73.25 72)
+        (xy 73 72.25) (xy 71.75 72.25) (xy 71.5 72)
+      )
+    )
+  )
+  (zone (net 62) (net_name /SCK) (layer B.Cu) (hatch edge 0.508)
+    (priority 1)
+    (connect_pads yes (clearance 0.25))
+    (min_thickness 0.254)
+    (fill yes (arc_segments 16) (thermal_gap 0.508) (thermal_bridge_width 0.508))
+    (polygon
+      (pts
+        (xy 74.25 70) (xy 74.5 69.75) (xy 75.75 69.75) (xy 76 70) (xy 76 70.75)
+        (xy 75.75 71) (xy 74.5 71) (xy 74.25 70.75)
+      )
+    )
+  )
+  (zone (net 0) (net_name "") (layer B.Mask) (hatch edge 0.508)
+    (priority 1)
+    (connect_pads yes (clearance 0.25))
+    (min_thickness 0.254)
+    (fill yes (arc_segments 16) (thermal_gap 0.508) (thermal_bridge_width 0.508))
+    (polygon
+      (pts
+        (xy 75.75 72.25) (xy 76 72.5) (xy 76 73.25) (xy 75.75 73.5) (xy 74.5 73.5)
+        (xy 74.25 73.25) (xy 74.25 72.5) (xy 74.5 72.25)
+      )
+    )
+  )
+  (zone (net 0) (net_name "") (layer B.Mask) (hatch edge 0.508)
+    (priority 1)
+    (connect_pads yes (clearance 0.25))
+    (min_thickness 0.254)
+    (fill yes (arc_segments 16) (thermal_gap 0.508) (thermal_bridge_width 0.508))
+    (polygon
+      (pts
+        (xy 75.75 69.75) (xy 76 70) (xy 76 70.75) (xy 75.75 71) (xy 74.5 71)
+        (xy 74.25 70.75) (xy 74.25 70) (xy 74.5 69.75)
+      )
+    )
+  )
+  (zone (net 0) (net_name "") (layer B.Mask) (hatch edge 0.508)
+    (priority 1)
+    (connect_pads yes (clearance 0.25))
+    (min_thickness 0.254)
+    (fill yes (arc_segments 16) (thermal_gap 0.508) (thermal_bridge_width 0.508))
+    (polygon
+      (pts
+        (xy 73 71) (xy 73.25 71.25) (xy 73.25 72) (xy 73 72.25) (xy 71.75 72.25)
+        (xy 71.5 72) (xy 71.5 71.25) (xy 71.75 71)
+      )
+    )
+  )
+  (zone (net 17) (net_name "Net-(C27-Pad1)") (layer B.Cu) (hatch edge 0.508)
+    (priority 1)
+    (connect_pads yes (clearance 0.25))
+    (min_thickness 0.254)
+    (fill yes (arc_segments 16) (thermal_gap 0.508) (thermal_bridge_width 0.508))
+    (polygon
+      (pts
+        (xy 69.5 72.5) (xy 69.75 72.25) (xy 71 72.25) (xy 71.25 72.5) (xy 71.25 73.25)
+        (xy 71 73.5) (xy 69.75 73.5) (xy 69.5 73.25)
+      )
+    )
+  )
+  (zone (net 0) (net_name "") (layer B.Mask) (hatch edge 0.508)
+    (priority 1)
+    (connect_pads yes (clearance 0.25))
+    (min_thickness 0.254)
+    (fill yes (arc_segments 16) (thermal_gap 0.508) (thermal_bridge_width 0.508))
+    (polygon
+      (pts
+        (xy 71 72.25) (xy 71.25 72.5) (xy 71.25 73.25) (xy 71 73.5) (xy 69.75 73.5)
+        (xy 69.5 73.25) (xy 69.5 72.5) (xy 69.75 72.25)
+      )
+    )
+  )
+  (zone (net 0) (net_name "") (layer B.Mask) (hatch edge 0.508)
+    (priority 1)
+    (connect_pads yes (clearance 0.25))
+    (min_thickness 0.254)
+    (fill yes (arc_segments 16) (thermal_gap 0.508) (thermal_bridge_width 0.508))
+    (polygon
+      (pts
+        (xy 71 67.75) (xy 71.25 68) (xy 71.25 68.75) (xy 71 69) (xy 69.75 69)
+        (xy 69.5 68.75) (xy 69.5 68) (xy 69.75 67.75)
+      )
+    )

Commit message: stmsp
Parts:
- removed T4, T5: testpoint, stmbl:Measurement_Point_Round-SMD-Pad_Small
- added REF**: STMSP_LOGO, stmbl:STMSP_LOGO, B.Cu at (78.5, 83.8)
- moved C9 0.25 mm to (73.2, 79.8)
Routing:
- net GND: track 177.3 -> 183.5 mm, vias 132 -> 135
- net Net-(P1-Pad3): track 6.16 -> 2.85 mm, vias 1 -> 0
- net Net-(P1-Pad2): track 4.89 -> 1.64 mm, vias 1 -> 0
- net +3V3: track 47.6 -> 46.5 mm, vias 19 -> 17
Other:
- board text added: "+ DC - 12-48V"
- board text added: "0 A B"
- board text added: "0V B/TX A/RX C VP"
- board text added: "1A 2A 1B 2B"
- board text added: "3/5V"
- board text added: "5V A1 B1 A0 B0 0V"
- board text added: "CL 0V IO RS"
- board text added: "DC O1 0V I1 5V DC O0 0V I0 5V"
- board text added: "STMSP V0.9"
- board text added: "STMSP V0.9 (GITHASH) github.com/rene-dev/stmbl"
