File: hw/kicad/stmsp/in.sch (KiCad schematic (older format))
At the start: 3 parts

Commit message: stmsp
Changed lines of the file:
@@
 $Descr A4 11693 8268
 encoding utf-8
-Sheet 9 10
+Sheet 7 10
 Title ""
 Date ""
@@
 AR Path="/594079D4/59409106" Ref="R31"  Part="1"
 AR Path="/5940FC3C/59409106" Ref="R36"  Part="1"
-F 0 "R36" V 4480 2200 50  0000 C CNN
+F 0 "R31" V 4480 2200 50  0000 C CNN
 F 1 "10k" V 4400 2200 50  0000 C CNN
 F 2 "stmbl:R_0603" V 4330 2200 50  0001 C CNN
@@
 AR Path="/594079D4/5940910D" Ref="R32"  Part="1"
 AR Path="/5940FC3C/5940910D" Ref="R37"  Part="1"
-F 0 "R37" V 4480 2700 50  0000 C CNN
+F 0 "R32" V 4480 2700 50  0000 C CNN
 F 1 "1k" V 4400 2700 50  0000 C CNN
 F 2 "stmbl:R_0603" V 4330 2700 50  0001 C CNN
@@
 AR Path="/594079D4/5940911B" Ref="C31"  Part="1"
 AR Path="/5940FC3C/5940911B" Ref="C32"  Part="1"
-F 0 "C32" H 4675 2800 50  0000 L CNN
+F 0 "C31" H 4675 2800 50  0000 L CNN
 F 1 "1n" H 4675 2600 50  0000 L CNN
 F 2 "stmbl:C_0603" H 4688 2550 50  0001 C CNN
@@
 	4650 2850 4650 3050
 $Comp
-L GND #PWR062
+L GND #PWR064
 U 1 1 59409131
 P 4650 3050
-AR Path="/594079D4/59409131" Ref="#PWR062"  Part="1"
-AR Path="/5940FC3C/59409131" Ref="#PWR065"  Part="1"
-F 0 "#PWR065" H 4650 2800 50  0001 C CNN
+AR Path="/594079D4/59409131" Ref="#PWR064"  Part="1"
+AR Path="/5940FC3C/59409131" Ref="#PWR067"  Part="1"
+F 0 "#PWR067" H 4650 2800 50  0001 C CNN
 F 1 "GND" H 4650 2900 50  0000 C CNN
 F 2 "" H 4650 3050 50  0000 C CNN

Commit message: stmsp
Changed lines of the file:
@@
 AR Path="/594079D4/59409106" Ref="R31"  Part="1"
 AR Path="/5940FC3C/59409106" Ref="R36"  Part="1"
-F 0 "R31" V 4480 2200 50  0000 C CNN
+F 0 "R36" V 4480 2200 50  0000 C CNN
 F 1 "10k" V 4400 2200 50  0000 C CNN
 F 2 "stmbl:R_0603" V 4330 2200 50  0001 C CNN
@@
 AR Path="/594079D4/5940910D" Ref="R32"  Part="1"
 AR Path="/5940FC3C/5940910D" Ref="R37"  Part="1"
-F 0 "R32" V 4480 2700 50  0000 C CNN
+F 0 "R37" V 4480 2700 50  0000 C CNN
 F 1 "1k" V 4400 2700 50  0000 C CNN
 F 2 "stmbl:R_0603" V 4330 2700 50  0001 C CNN
@@
 AR Path="/594079D4/5940911B" Ref="C31"  Part="1"
 AR Path="/5940FC3C/5940911B" Ref="C32"  Part="1"
-F 0 "C31" H 4675 2800 50  0000 L CNN
+F 0 "C32" H 4675 2800 50  0000 L CNN
 F 1 "1n" H 4675 2600 50  0000 L CNN
 F 2 "stmbl:C_0603" H 4688 2550 50  0001 C CNN

Commit message: stmsp
Parts:
- R32: value 1k -> 1.5k
Changed lines of the file:
@@
 $Descr A4 11693 8268
 encoding utf-8
-Sheet 7 10
+Sheet 9 10
 Title ""
 Date ""
@@
 AR Path="/5940FC3C/5940910D" Ref="R37"  Part="1"
 F 0 "R37" V 4480 2700 50  0000 C CNN
-F 1 "1k" V 4400 2700 50  0000 C CNN
+F 1 "1.5k" V 4400 2700 50  0000 C CNN
 F 2 "stmbl:R_0603" V 4330 2700 50  0001 C CNN
 F 3 "" H 4400 2700 50  0000 C CNN

Commit message: stmsp
Other:
- note added: "3.3 / 1.5V * (10k + 1.5k) = 25.3V"
Changed lines of the file:
@@
 $Descr A4 11693 8268
 encoding utf-8
-Sheet 9 10
+Sheet 7 10
 Title ""
 Date ""
@@
 AR Path="/594079D4/59409106" Ref="R31"  Part="1"
 AR Path="/5940FC3C/59409106" Ref="R36"  Part="1"
-F 0 "R36" V 4480 2200 50  0000 C CNN
+F 0 "R31" V 4480 2200 50  0000 C CNN
 F 1 "10k" V 4400 2200 50  0000 C CNN
 F 2 "stmbl:R_0603" V 4330 2200 50  0001 C CNN
@@
 AR Path="/594079D4/5940910D" Ref="R32"  Part="1"
 AR Path="/5940FC3C/5940910D" Ref="R37"  Part="1"
-F 0 "R37" V 4480 2700 50  0000 C CNN
+F 0 "R32" V 4480 2700 50  0000 C CNN
 F 1 "1.5k" V 4400 2700 50  0000 C CNN
 F 2 "stmbl:R_0603" V 4330 2700 50  0001 C CNN
@@
 AR Path="/594079D4/5940911B" Ref="C31"  Part="1"
 AR Path="/5940FC3C/5940911B" Ref="C32"  Part="1"
-F 0 "C32" H 4675 2800 50  0000 L CNN
+F 0 "C31" H 4675 2800 50  0000 L CNN
 F 1 "1n" H 4675 2600 50  0000 L CNN
 F 2 "stmbl:C_0603" H 4688 2550 50  0001 C CNN
@@
 AR Path="/594079D4/59409131" Ref="#PWR064"  Part="1"
 AR Path="/5940FC3C/59409131" Ref="#PWR067"  Part="1"
-F 0 "#PWR067" H 4650 2800 50  0001 C CNN
+F 0 "#PWR064" H 4650 2800 50  0001 C CNN
 F 1 "GND" H 4650 2900 50  0000 C CNN
 F 2 "" H 4650 3050 50  0000 C CNN
@@
 	4650 2550 4650 2450
 Connection ~ 4650 2450
+Text Notes 5000 2150 0    60   ~ 0
+3.3 / 1.5V * (10k + 1.5k) = 25.3V
 $EndSCHEMATC

Commit message: stmsp
Changed lines of the file:
@@
 $Descr A4 11693 8268
 encoding utf-8
-Sheet 7 10
+Sheet 9 10
 Title ""
 Date ""
@@
 AR Path="/594079D4/59409106" Ref="R31"  Part="1"
 AR Path="/5940FC3C/59409106" Ref="R36"  Part="1"
-F 0 "R31" V 4480 2200 50  0000 C CNN
+F 0 "R36" V 4480 2200 50  0000 C CNN
 F 1 "10k" V 4400 2200 50  0000 C CNN
 F 2 "stmbl:R_0603" V 4330 2200 50  0001 C CNN
@@
 AR Path="/594079D4/5940910D" Ref="R32"  Part="1"
 AR Path="/5940FC3C/5940910D" Ref="R37"  Part="1"
-F 0 "R32" V 4480 2700 50  0000 C CNN
+F 0 "R37" V 4480 2700 50  0000 C CNN
 F 1 "1.5k" V 4400 2700 50  0000 C CNN
 F 2 "stmbl:R_0603" V 4330 2700 50  0001 C CNN
@@
 AR Path="/594079D4/5940911B" Ref="C31"  Part="1"
 AR Path="/5940FC3C/5940911B" Ref="C32"  Part="1"
-F 0 "C31" H 4675 2800 50  0000 L CNN
+F 0 "C32" H 4675 2800 50  0000 L CNN
 F 1 "1n" H 4675 2600 50  0000 L CNN
 F 2 "stmbl:C_0603" H 4688 2550 50  0001 C CNN
@@
 AR Path="/594079D4/59409131" Ref="#PWR064"  Part="1"
 AR Path="/5940FC3C/59409131" Ref="#PWR067"  Part="1"
-F 0 "#PWR064" H 4650 2800 50  0001 C CNN
+F 0 "#PWR067" H 4650 2800 50  0001 C CNN
 F 1 "GND" H 4650 2900 50  0000 C CNN
 F 2 "" H 4650 3050 50  0000 C CNN
