File: hw/kicad/stmsp/drv.sch (KiCad schematic (older format))
At the start: 34 parts, among them P3 CONN_01X04, P4 CONN_01X02, U2 L6206Q

Commit message: stmsp
Parts:
- added C26: 10u, stmbl:c_elec_5x5.3, symbol CP
- added C30: 10n, stmbl:C_0603, symbol C
- added C33, C5: 100n, stmbl:C_0603, symbol C
- added D10, D11: D, stmbl:SOD-123, symbol D
- added R55: 1k, stmbl:R_0603, symbol R
- added R56: 100, stmbl:R_0603, symbol R
- added TH1: Thermistor_NTC, stmbl:R_0603, symbol Thermistor_NTC
- R12, R8: value 0.01 -> 0.015; footprint stmbl:R_0603 -> stmbl:R_0805
Connections:
- net +3V3: now also R55.2
- net GND: now also C26.2, TH1.2
- net VPP: now also C26.1
- net at P3.2 (P2), R18.1: now also U2.2 (OUT1A), U2.3 (OUT1A); no longer U2.38 (OUT2A), U2.39 (OUT2A)
- net at P3.1 (P1), R22.1: now also U2.38 (OUT2A), U2.39 (OUT2A); no longer U2.2 (OUT1A), U2.3 (OUT1A)
- net at U2.21 (VBOOT): now also C33.1, C5.1, D11.1 (K)
- net at U2.40 (VCP): now also C30.1
- new net: C30.2, R56.2
- new net: D10.1 (K), D11.2 (A), R56.1
- new net: C33.2, C5.2, D10.2 (A)
- new net TEMP: R55.1, TH1.1

Commit message: stmsp
Parts:
- added C38, C39: 1n, stmbl:C_0603, symbol C
- added P6: CONN_01X02, stmbl:akl182-2, symbol CONN_01X02
- C12, C14, C15, C20: value C -> 220n
- P3: footprint Pin_Headers:Pin_Header_Straight_1x04 -> stmbl:Pin_Header_Straight_1x04
- R13, R14: value 22 -> 10k
- R6, R7: value 10k -> 1k
Connections:
- net GND: now also C38.2, C39.2, P6.2 (P2)
- net VPP: now also P6.1 (P1)
- net at R14.1, U2.13 (OCDB), U2.20 (ENB): now also C39.1
- net at R13.1, U2.41 (ENA), U2.48 (OCDA): now also C38.1
Other:
- moved on the sheet: R13, R14
Changed lines of the file:
@@
 AR Path="/5918AB0C/5918AB0C/5918DE6E" Ref="C15"  Part="1"
 F 0 "C15" H 5225 6400 50  0000 L CNN
-F 1 "C" H 5225 6200 50  0000 L CNN
+F 1 "220n" H 5225 6200 50  0000 L CNN
 F 2 "stmbl:C_0805" H 5238 6150 50  0001 C CNN
 F 3 "" H 5200 6300 50  0000 C CNN
@@
 AR Path="/5918AB0C/5918AB0C/5918DE99" Ref="C14"  Part="1"
 F 0 "C14" H 4975 6400 50  0000 L CNN
-F 1 "C" H 4975 6200 50  0000 L CNN
+F 1 "220n" H 4975 6200 50  0000 L CNN
 F 2 "stmbl:C_0805" H 4988 6150 50  0001 C CNN
 F 3 "" H 4950 6300 50  0000 C CNN
@@
 AR Path="/5918AB0C/5918AB0C/5918DEB2" Ref="C12"  Part="1"
 F 0 "C12" H 4725 6400 50  0000 L CNN
-F 1 "C" H 4725 6200 50  0000 L CNN
+F 1 "220n" H 4725 6200 50  0000 L CNN
 F 2 "stmbl:C_0805" H 4738 6150 50  0001 C CNN
 F 3 "" H 4700 6300 50  0000 C CNN
@@
 L R R14
 U 1 1 5919412F
-P 4550 2900
+P 4150 2900
 AR Path="/5918AB0C/5919412F" Ref="R14"  Part="1"
 AR Path="/5918AB0C/5918AB0C/5919412F" Ref="R14"  Part="1"
-F 0 "R14" V 4630 2900 50  0000 C CNN
-F 1 "22" V 4550 2900 50  0000 C CNN
-F 2 "stmbl:R_0603" V 4480 2900 50  0001 C CNN
-F 3 "" H 4550 2900 50  0000 C CNN
-	1    4550 2900
+F 0 "R14" V 4230 2900 50  0000 C CNN
+F 1 "10k" V 4150 2900 50  0000 C CNN
+F 2 "stmbl:R_0603" V 4080 2900 50  0001 C CNN
+F 3 "" H 4150 2900 50  0000 C CNN
+	1    4150 2900
 	0    1    1    0
 $EndComp
@@
 L R R13
 U 1 1 5919419E
-P 4550 2500
+P 4150 2500
 AR Path="/5918AB0C/5919419E" Ref="R13"  Part="1"
 AR Path="/5918AB0C/5918AB0C/5919419E" Ref="R13"  Part="1"
-F 0 "R13" V 4630 2500 50  0000 C CNN
-F 1 "22" V 4550 2500 50  0000 C CNN
-F 2 "stmbl:R_0603" V 4480 2500 50  0001 C CNN
-F 3 "" H 4550 2500 50  0000 C CNN
-	1    4550 2500
-	0    1    1    0
-$EndComp
-Text HLabel 4300 2900 0    60   Input ~ 0
+F 0 "R13" V 4230 2500 50  0000 C CNN
+F 1 "10k" V 4150 2500 50  0000 C CNN
+F 2 "stmbl:R_0603" V 4080 2500 50  0001 C CNN
+F 3 "" H 4150 2500 50  0000 C CNN
+	1    4150 2500
+	0    1    1    0
+$EndComp
+Text HLabel 3900 2900 0    60   Input ~ 0
 ENB
-Text HLabel 4300 2500 0    60   Input ~ 0
+Text HLabel 3900 2500 0    60   Input ~ 0
 ENA
 $Comp
@@
 AR Path="/5918AB0C/5918AB0C/59194A21" Ref="R7"  Part="1"
 F 0 "R7" V 3430 2750 50  0000 C CNN
-F 1 "10k" V 3350 2750 50  0000 C CNN
+F 1 "1k" V 3350 2750 50  0000 C CNN
 F 2 "stmbl:R_0603" V 3280 2750 50  0001 C CNN
 F 3 "" H 3350 2750 50  0000 C CNN
@@
 AR Path="/5918AB0C/5918AB0C/59194A90" Ref="R6"  Part="1"
 F 0 "R6" V 3230 2750 50  0000 C CNN
-F 1 "10k" V 3150 2750 50  0000 C CNN
+F 1 "1k" V 3150 2750 50  0000 C CNN
 F 2 "stmbl:R_0603" V 3080 2750 50  0001 C CNN
 F 3 "" H 3150 2750 50  0000 C CNN
@@
 F 0 "P3" H 7050 2700 50  0000 C CNN
 F 1 "CONN_01X04" V 7150 2450 50  0000 C CNN
-F 2 "Pin_Headers:Pin_Header_Straight_1x04" H 7050 2450 50  0001 C CNN
+F 2 "stmbl:Pin_Header_Straight_1x04" H 7050 2450 50  0001 C CNN
 F 3 "" H 7050 2450 50  0000 C CNN
 	1    7050 2450
@@
 P 4450 6300
 F 0 "C20" H 4475 6400 50  0000 L CNN
-F 1 "C" H 4475 6200 50  0000 L CNN
+F 1 "220n" H 4475 6200 50  0000 L CNN
 F 2 "stmbl:C_0805" H 4488 6150 50  0001 C CNN
 F 3 "" H 4450 6300 50  0000 C CNN
@@
 	4800 2600 4800 2500
 Wire Wire Line
-	4700 2500 4900 2500
+	4300 2500 4900 2500
 Wire Wire Line
 	4900 3000 4800 3000
@@
 	4800 3000 4800 2900
 Wire Wire Line
-	4700 2900 4900 2900
+	4300 2900 4900 2900
 Connection ~ 4800 2500
 Connection ~ 4800 2900
 Wire Wire Line
-	4300 2500 4400 2500
-Wire Wire Line
-	4300 2900 4400 2900
+	3900 2500 4000 2500
+Wire Wire Line
+	3900 2900 4000 2900
 Wire Wire Line
 	4800 2800 4900 2800
@@
 Connection ~ 4450 6050
 Wire Wire Line
-	4050 6350 4150 6350
-Wire Wire Line
-	4150 6250 4050 6250
+	3600 6350 4150 6350
+Wire Wire Line
+	3600 6250 4150 6250
 Wire Wire Line
 	3600 4400 3700 4400
@@
 Wire Wire Line
 	5500 6550 5500 6450
+$Comp
+L CONN_01X02 P6
+U 1 1 593C4D39
+P 3400 6300
+F 0 "P6" H 3400 6450 50  0000 C CNN
+F 1 "CONN_01X02" V 3500 6300 50  0000 C CNN
+F 2 "stmbl:akl182-2" H 3400 6300 50  0001 C CNN
+F 3 "" H 3400 6300 50  0000 C CNN
+	1    3400 6300
+	-1   0    0    -1
+$EndComp
+Connection ~ 4050 6350
+Connection ~ 4050 6250
+$Comp
+L C C39
+U 1 1 593CC856
+P 4150 3100
+F 0 "C39" H 4175 3200 50  0000 L CNN
+F 1 "1n" H 4175 3000 50  0000 L CNN
+F 2 "stmbl:C_0603" H 4188 2950 50  0001 C CNN
+F 3 "" H 4150 3100 50  0000 C CNN
+	1    4150 3100
+	0    1    1    0
+$EndComp
+$Comp
+L C C38
+U 1 1 593CC99F
+P 4150 2700
+F 0 "C38" H 4175 2800 50  0000 L CNN
+F 1 "1n" H 4175 2600 50  0000 L CNN
+F 2 "stmbl:C_0603" H 4188 2550 50  0001 C CNN
+F 3 "" H 4150 2700 50  0000 C CNN
+	1    4150 2700
+	0    1    1    0
+$EndComp
+Wire Wire Line
+	4300 2700 4400 2700
+Wire Wire Line
+	4400 2700 4400 2500
+Connection ~ 4400 2500
+Wire Wire Line
+	4300 3100 4400 3100
+Wire Wire Line
+	4400 3100 4400 2900
+Connection ~ 4400 2900
+$Comp
+L GND #PWR024
+U 1 1 593CCC88
+P 3900 3100
+F 0 "#PWR024" H 3900 2850 50  0001 C CNN
+F 1 "GND" H 3900 2950 50  0000 C CNN
+F 2 "" H 3900 3100 50  0000 C CNN
+F 3 "" H 3900 3100 50  0000 C CNN
+	1    3900 3100
+	0    1    1    0
+$EndComp
+$Comp
+L GND #PWR025
+U 1 1 593CCD1D
+P 3900 2700
+F 0 "#PWR025" H 3900 2450 50  0001 C CNN
+F 1 "GND" H 3900 2550 50  0000 C CNN
+F 2 "" H 3900 2700 50  0000 C CNN
+F 3 "" H 3900 2700 50  0000 C CNN
+	1    3900 2700
+	0    1    1    0
+$EndComp
+Wire Wire Line
+	3900 2700 4000 2700
+Wire Wire Line
+	3900 3100 4000 3100
 $EndSCHEMATC

Commit message: stmsp
Parts:
- P3: footprint stmbl:Pin_Header_Straight_1x04 -> stmbl:Pin_Header_Straight_1x04_dual
- P6: footprint stmbl:akl182-2 -> stmbl:akl183-2
Connections:
- net VPP: now also C33.2, C5.2, D10.2 (A)
Changed lines of the file:
@@
 F 0 "P3" H 7050 2700 50  0000 C CNN
 F 1 "CONN_01X04" V 7150 2450 50  0000 C CNN
-F 2 "stmbl:Pin_Header_Straight_1x04" H 7050 2450 50  0001 C CNN
+F 2 "stmbl:Pin_Header_Straight_1x04_dual" H 7050 2450 50  0001 C CNN
 F 3 "" H 7050 2450 50  0000 C CNN
 	1    7050 2450
@@
 	2050 5450 2150 5450
 Wire Wire Line
-	3250 3500 3150 3500
+	3050 3500 3250 3500
 Wire Wire Line
 	3150 3500 3150 4150
@@
 F 0 "P6" H 3400 6450 50  0000 C CNN
 F 1 "CONN_01X02" V 3500 6300 50  0000 C CNN
-F 2 "stmbl:akl182-2" H 3400 6300 50  0001 C CNN
+F 2 "stmbl:akl183-2" H 3400 6300 50  0001 C CNN
 F 3 "" H 3400 6300 50  0000 C CNN
 	1    3400 6300
@@
 Wire Wire Line
 	3900 3100 4000 3100
+$Comp
+L VPP #PWR026
+U 1 1 593ED301
+P 3050 3400
+F 0 "#PWR026" H 3050 3250 50  0001 C CNN
+F 1 "VPP" H 3050 3550 50  0000 C CNN
+F 2 "" H 3050 3400 50  0000 C CNN
+F 3 "" H 3050 3400 50  0000 C CNN
+	1    3050 3400
+	1    0    0    -1
+$EndComp
+Wire Wire Line
+	3050 3400 3050 3500
+Connection ~ 3150 3500
 $EndSCHEMATC

Commit message: stmsp
Parts:
- C26: value 10u -> 22u
- C34, C35, C6: value C -> 18p
- R12, R8: value 0.015 -> 0.02
- R46, R47, R48: value R -> 3.9k
- R49, R50, R51: value R -> 120
Other:
- note added: "3.3V / 1k * (10k + 10k + 1k) = 69.3V"
- note added: "alt.: 470:15k"
Changed lines of the file:
@@
 AR Path="/5918AB0C/5918AB0C/5918E2CF" Ref="R12"  Part="1"
 F 0 "R12" V 4580 4850 50  0000 C CNN
-F 1 "0.015" V 4500 4850 50  0000 C CNN
+F 1 "0.02" V 4500 4850 50  0000 C CNN
 F 2 "stmbl:R_0805" V 4430 4850 50  0001 C CNN
 F 3 "" H 4500 4850 50  0000 C CNN
@@
 AR Path="/5918AB0C/5918AB0C/5918E363" Ref="R8"  Part="1"
 F 0 "R8" V 4180 4850 50  0000 C CNN
-F 1 "0.015" V 4100 4850 50  0000 C CNN
+F 1 "0.02" V 4100 4850 50  0000 C CNN
 F 2 "stmbl:R_0805" V 4030 4850 50  0001 C CNN
 F 3 "" H 4100 4850 50  0000 C CNN
@@
 P 3850 5100
 F 0 "R51" V 3930 5100 50  0000 C CNN
-F 1 "R" V 3850 5100 50  0000 C CNN
+F 1 "120" V 3850 5100 50  0000 C CNN
 F 2 "stmbl:R_0603" V 3780 5100 50  0001 C CNN
 F 3 "" H 3850 5100 50  0000 C CNN
@@
 P 3850 4600
 F 0 "R50" V 3930 4600 50  0000 C CNN
-F 1 "R" V 3850 4600 50  0000 C CNN
+F 1 "120" V 3850 4600 50  0000 C CNN
 F 2 "stmbl:R_0603" V 3780 4600 50  0001 C CNN
 F 3 "" H 3850 4600 50  0000 C CNN
@@
 P 3850 4400
 F 0 "R49" V 3930 4400 50  0000 C CNN
-F 1 "R" V 3850 4400 50  0000 C CNN
+F 1 "120" V 3850 4400 50  0000 C CNN
 F 2 "stmbl:R_0603" V 3780 4400 50  0001 C CNN
 F 3 "" H 3850 4400 50  0000 C CNN
@@
 P 2300 4650
 F 0 "R46" V 2380 4650 50  0000 C CNN
-F 1 "R" V 2300 4650 50  0000 C CNN
+F 1 "3.9k" V 2300 4650 50  0000 C CNN
 F 2 "stmbl:R_0603" V 2230 4650 50  0001 C CNN
 F 3 "" H 2300 4650 50  0000 C CNN
@@
 P 2300 4800
 F 0 "R47" V 2380 4800 50  0000 C CNN
-F 1 "R" V 2300 4800 50  0000 C CNN
+F 1 "3.9k" V 2300 4800 50  0000 C CNN
 F 2 "stmbl:R_0603" V 2230 4800 50  0001 C CNN
 F 3 "" H 2300 4800 50  0000 C CNN
@@
 P 2300 4950
 F 0 "R48" V 2380 4950 50  0000 C CNN
-F 1 "R" V 2300 4950 50  0000 C CNN
+F 1 "3.9k" V 2300 4950 50  0000 C CNN
 F 2 "stmbl:R_0603" V 2230 4950 50  0001 C CNN
 F 3 "" H 2300 4950 50  0000 C CNN
@@
 P 2300 5450
 F 0 "C6" H 2325 5550 50  0000 L CNN
-F 1 "C" H 2325 5350 50  0000 L CNN
+F 1 "18p" H 2325 5350 50  0000 L CNN
 F 2 "stmbl:C_0603" H 2338 5300 50  0001 C CNN
 F 3 "" H 2300 5450 50  0000 C CNN
@@
 P 2300 5650
 F 0 "C34" H 2325 5750 50  0000 L CNN
-F 1 "C" H 2325 5550 50  0000 L CNN
+F 1 "18p" H 2325 5550 50  0000 L CNN
 F 2 "stmbl:R_0603" H 2338 5500 50  0001 C CNN
 F 3 "" H 2300 5650 50  0000 C CNN
@@
 P 2300 5850
 F 0 "C35" H 2325 5950 50  0000 L CNN
-F 1 "C" H 2325 5750 50  0000 L CNN
+F 1 "18p" H 2325 5750 50  0000 L CNN
 F 2 "stmbl:R_0603" H 2338 5700 50  0001 C CNN
 F 3 "" H 2300 5850 50  0000 C CNN
@@
 P 5500 6300
 F 0 "C26" H 5525 6400 50  0000 L CNN
-F 1 "10u" H 5525 6200 50  0000 L CNN
+F 1 "22u" H 5525 6200 50  0000 L CNN
 F 2 "stmbl:c_elec_5x5.3" H 5538 6150 50  0001 C CNN
 F 3 "" H 5500 6300 50  0000 C CNN
@@
 	3050 3400 3050 3500
 Connection ~ 3150 3500
+Text Notes 8900 3850 0    60   ~ 0
+3.3V / 1k * (10k + 10k + 1k) = 69.3V
+Text Notes 2850 4850 0    60   ~ 0
+alt.: 470:15k
 $EndSCHEMATC

Commit message: stmsp
Parts:
- C34, C35: footprint stmbl:R_0603 -> stmbl:C_0603
- D10, D11: value D -> 1N4148
- TH1: value Thermistor_NTC -> 4.7k
Changed lines of the file:
@@
 F 0 "C34" H 2325 5750 50  0000 L CNN
 F 1 "18p" H 2325 5550 50  0000 L CNN
-F 2 "stmbl:R_0603" H 2338 5500 50  0001 C CNN
+F 2 "stmbl:C_0603" H 2338 5500 50  0001 C CNN
 F 3 "" H 2300 5650 50  0000 C CNN
 	1    2300 5650
@@
 F 0 "C35" H 2325 5950 50  0000 L CNN
 F 1 "18p" H 2325 5750 50  0000 L CNN
-F 2 "stmbl:R_0603" H 2338 5700 50  0001 C CNN
+F 2 "stmbl:C_0603" H 2338 5700 50  0001 C CNN
 F 3 "" H 2300 5850 50  0000 C CNN
 	1    2300 5850
@@
 P 2200 2800
 F 0 "TH1" V 2025 2800 50  0000 C CNN
-F 1 "Thermistor_NTC" V 2325 2800 50  0000 C CNN
+F 1 "4.7k" V 2325 2800 50  0000 C CNN
 F 2 "stmbl:R_0603" H 2200 2850 50  0001 C CNN
 F 3 "" H 2200 2850 50  0001 C CNN
@@
 P 3400 3500
 F 0 "D10" H 3400 3600 50  0000 C CNN
-F 1 "D" H 3400 3400 50  0000 C CNN
+F 1 "1N4148" H 3400 3400 50  0000 C CNN
 F 2 "stmbl:SOD-123" H 3400 3500 50  0001 C CNN
 F 3 "" H 3400 3500 50  0000 C CNN
@@
 P 3650 3750
 F 0 "D11" H 3650 3850 50  0000 C CNN
-F 1 "D" H 3650 3650 50  0000 C CNN
+F 1 "1N4148" H 3650 3650 50  0000 C CNN
 F 2 "stmbl:SOD-123" H 3650 3750 50  0001 C CNN
 F 3 "" H 3650 3750 50  0000 C CNN
