File: hw/kicad/stmsp/out.sch (KiCad schematic (older format))
At the start: 4 parts, among them Q1 Q_NJFET_GSD

Commit message: stmsp
Changed lines of the file:
@@
 $Descr A4 11693 8268
 encoding utf-8
-Sheet 10 10
+Sheet 8 10
 Title ""
 Date ""
@@
 AR Path="/5940CCE8/5940D06F" Ref="R34"  Part="1"
 AR Path="/59418122/5940D06F" Ref="R39"  Part="1"
-F 0 "R39" V 5280 2700 50  0000 C CNN
+F 0 "R34" V 5280 2700 50  0000 C CNN
 F 1 "1k" V 5200 2700 50  0000 C CNN
 F 2 "stmbl:R_0603" V 5130 2700 50  0001 C CNN
@@
 AR Path="/5940CCE8/5940D076" Ref="R35"  Part="1"
 AR Path="/59418122/5940D076" Ref="R40"  Part="1"
-F 0 "R40" V 5530 2450 50  0000 C CNN
+F 0 "R35" V 5530 2450 50  0000 C CNN
 F 1 "120" V 5450 2450 50  0000 C CNN
 F 2 "stmbl:R_0603" V 5380 2450 50  0001 C CNN
@@
 AR Path="/5940CCE8/5940D07D" Ref="Q1"  Part="1"
 AR Path="/59418122/5940D07D" Ref="Q2"  Part="1"
-F 0 "Q2" H 5200 2500 50  0000 R CNN
+F 0 "Q1" H 5200 2500 50  0000 R CNN
 F 1 "Q_NJFET_GSD" H 5550 2400 50  0000 R CNN
 F 2 "stmbl:SOT-23" H 5100 2550 50  0001 C CNN
@@
 AR Path="/5940CCE8/5940D084" Ref="D4"  Part="1"
 AR Path="/59418122/5940D084" Ref="D6"  Part="1"
-F 0 "D6" H 4800 2000 50  0000 C CNN
+F 0 "D4" H 4800 2000 50  0000 C CNN
 F 1 "ES1J" H 4800 1800 50  0000 C CNN
 F 2 "stmbl:SOD-123" H 4800 1900 50  0001 C CNN
@@
 	4800 2650 4800 3050
 $Comp
-L VPP #PWR063
+L VPP #PWR065
 U 1 1 5940D092
 P 4800 1650
-AR Path="/5940CCE8/5940D092" Ref="#PWR063"  Part="1"
-AR Path="/59418122/5940D092" Ref="#PWR066"  Part="1"
-F 0 "#PWR066" H 4800 1500 50  0001 C CNN
+AR Path="/5940CCE8/5940D092" Ref="#PWR065"  Part="1"
+AR Path="/59418122/5940D092" Ref="#PWR068"  Part="1"
+F 0 "#PWR068" H 4800 1500 50  0001 C CNN
 F 1 "VPP" H 4800 1800 50  0000 C CNN
 F 2 "" H 4800 1650 50  0000 C CNN
@@
 Connection ~ 4800 2950
 $Comp
-L GND #PWR064
+L GND #PWR066
 U 1 1 5940D09C
 P 4800 3050
-AR Path="/5940CCE8/5940D09C" Ref="#PWR064"  Part="1"
-AR Path="/59418122/5940D09C" Ref="#PWR067"  Part="1"
-F 0 "#PWR067" H 4800 2800 50  0001 C CNN
+AR Path="/5940CCE8/5940D09C" Ref="#PWR066"  Part="1"
+AR Path="/59418122/5940D09C" Ref="#PWR069"  Part="1"
+F 0 "#PWR069" H 4800 2800 50  0001 C CNN
 F 1 "GND" H 4800 2900 50  0000 C CNN
 F 2 "" H 4800 3050 50  0000 C CNN

Commit message: stmsp
Changed lines of the file:
@@
 AR Path="/5940CCE8/5940D06F" Ref="R34"  Part="1"
 AR Path="/59418122/5940D06F" Ref="R39"  Part="1"
-F 0 "R34" V 5280 2700 50  0000 C CNN
+F 0 "R39" V 5280 2700 50  0000 C CNN
 F 1 "1k" V 5200 2700 50  0000 C CNN
 F 2 "stmbl:R_0603" V 5130 2700 50  0001 C CNN
@@
 AR Path="/5940CCE8/5940D076" Ref="R35"  Part="1"
 AR Path="/59418122/5940D076" Ref="R40"  Part="1"
-F 0 "R35" V 5530 2450 50  0000 C CNN
+F 0 "R40" V 5530 2450 50  0000 C CNN
 F 1 "120" V 5450 2450 50  0000 C CNN
 F 2 "stmbl:R_0603" V 5380 2450 50  0001 C CNN
@@
 AR Path="/5940CCE8/5940D07D" Ref="Q1"  Part="1"
 AR Path="/59418122/5940D07D" Ref="Q2"  Part="1"
-F 0 "Q1" H 5200 2500 50  0000 R CNN
+F 0 "Q2" H 5200 2500 50  0000 R CNN
 F 1 "Q_NJFET_GSD" H 5550 2400 50  0000 R CNN
 F 2 "stmbl:SOT-23" H 5100 2550 50  0001 C CNN
@@
 AR Path="/5940CCE8/5940D084" Ref="D4"  Part="1"
 AR Path="/59418122/5940D084" Ref="D6"  Part="1"
-F 0 "D4" H 4800 2000 50  0000 C CNN
+F 0 "D6" H 4800 2000 50  0000 C CNN
 F 1 "ES1J" H 4800 1800 50  0000 C CNN
 F 2 "stmbl:SOD-123" H 4800 1900 50  0001 C CNN

Commit message: stmsp
Changed lines of the file:
@@
 AR Path="/5940CCE8/5940D06F" Ref="R34"  Part="1"
 AR Path="/59418122/5940D06F" Ref="R39"  Part="1"
-F 0 "R39" V 5280 2700 50  0000 C CNN
+F 0 "R34" V 5280 2700 50  0000 C CNN
 F 1 "1k" V 5200 2700 50  0000 C CNN
 F 2 "stmbl:R_0603" V 5130 2700 50  0001 C CNN
@@
 AR Path="/5940CCE8/5940D076" Ref="R35"  Part="1"
 AR Path="/59418122/5940D076" Ref="R40"  Part="1"
-F 0 "R40" V 5530 2450 50  0000 C CNN
+F 0 "R35" V 5530 2450 50  0000 C CNN
 F 1 "120" V 5450 2450 50  0000 C CNN
 F 2 "stmbl:R_0603" V 5380 2450 50  0001 C CNN
@@
 AR Path="/5940CCE8/5940D07D" Ref="Q1"  Part="1"
 AR Path="/59418122/5940D07D" Ref="Q2"  Part="1"
-F 0 "Q2" H 5200 2500 50  0000 R CNN
+F 0 "Q1" H 5200 2500 50  0000 R CNN
 F 1 "Q_NJFET_GSD" H 5550 2400 50  0000 R CNN
 F 2 "stmbl:SOT-23" H 5100 2550 50  0001 C CNN
@@
 AR Path="/5940CCE8/5940D084" Ref="D4"  Part="1"
 AR Path="/59418122/5940D084" Ref="D6"  Part="1"
-F 0 "D6" H 4800 2000 50  0000 C CNN
+F 0 "D4" H 4800 2000 50  0000 C CNN
 F 1 "ES1J" H 4800 1800 50  0000 C CNN
 F 2 "stmbl:SOD-123" H 4800 1900 50  0001 C CNN
@@
 AR Path="/5940CCE8/5940D092" Ref="#PWR065"  Part="1"
 AR Path="/59418122/5940D092" Ref="#PWR068"  Part="1"
-F 0 "#PWR068" H 4800 1500 50  0001 C CNN
+F 0 "#PWR065" H 4800 1500 50  0001 C CNN
 F 1 "VPP" H 4800 1800 50  0000 C CNN
 F 2 "" H 4800 1650 50  0000 C CNN
@@
 AR Path="/5940CCE8/5940D09C" Ref="#PWR066"  Part="1"
 AR Path="/59418122/5940D09C" Ref="#PWR069"  Part="1"
-F 0 "#PWR069" H 4800 2800 50  0001 C CNN
+F 0 "#PWR066" H 4800 2800 50  0001 C CNN
 F 1 "GND" H 4800 2900 50  0000 C CNN
 F 2 "" H 4800 3050 50  0000 C CNN

Commit message: stmsp
Changed lines of the file:
@@
 $Descr A4 11693 8268
 encoding utf-8
-Sheet 8 10
+Sheet 10 10
 Title ""
 Date ""
@@
 AR Path="/5940CCE8/5940D06F" Ref="R34"  Part="1"
 AR Path="/59418122/5940D06F" Ref="R39"  Part="1"
-F 0 "R34" V 5280 2700 50  0000 C CNN
+F 0 "R39" V 5280 2700 50  0000 C CNN
 F 1 "1k" V 5200 2700 50  0000 C CNN
 F 2 "stmbl:R_0603" V 5130 2700 50  0001 C CNN
@@
 AR Path="/5940CCE8/5940D076" Ref="R35"  Part="1"
 AR Path="/59418122/5940D076" Ref="R40"  Part="1"
-F 0 "R35" V 5530 2450 50  0000 C CNN
+F 0 "R40" V 5530 2450 50  0000 C CNN
 F 1 "120" V 5450 2450 50  0000 C CNN
 F 2 "stmbl:R_0603" V 5380 2450 50  0001 C CNN
@@
 AR Path="/5940CCE8/5940D07D" Ref="Q1"  Part="1"
 AR Path="/59418122/5940D07D" Ref="Q2"  Part="1"
-F 0 "Q1" H 5200 2500 50  0000 R CNN
+F 0 "Q2" H 5200 2500 50  0000 R CNN
 F 1 "Q_NJFET_GSD" H 5550 2400 50  0000 R CNN
 F 2 "stmbl:SOT-23" H 5100 2550 50  0001 C CNN
@@
 AR Path="/5940CCE8/5940D084" Ref="D4"  Part="1"
 AR Path="/59418122/5940D084" Ref="D6"  Part="1"
-F 0 "D4" H 4800 2000 50  0000 C CNN
+F 0 "D6" H 4800 2000 50  0000 C CNN
 F 1 "ES1J" H 4800 1800 50  0000 C CNN
 F 2 "stmbl:SOD-123" H 4800 1900 50  0001 C CNN
@@
 AR Path="/5940CCE8/5940D092" Ref="#PWR065"  Part="1"
 AR Path="/59418122/5940D092" Ref="#PWR068"  Part="1"
-F 0 "#PWR065" H 4800 1500 50  0001 C CNN
+F 0 "#PWR068" H 4800 1500 50  0001 C CNN
 F 1 "VPP" H 4800 1800 50  0000 C CNN
 F 2 "" H 4800 1650 50  0000 C CNN
@@
 AR Path="/5940CCE8/5940D09C" Ref="#PWR066"  Part="1"
 AR Path="/59418122/5940D09C" Ref="#PWR069"  Part="1"
-F 0 "#PWR066" H 4800 2800 50  0001 C CNN
+F 0 "#PWR069" H 4800 2800 50  0001 C CNN
 F 1 "GND" H 4800 2900 50  0000 C CNN
 F 2 "" H 4800 3050 50  0000 C CNN

Commit message: stmsp
Parts:
- D4: value ES1J -> 200V 1A
Changed lines of the file:
@@
 $Descr A4 11693 8268
 encoding utf-8
-Sheet 10 10
+Sheet 8 10
 Title ""
 Date ""
@@
 AR Path="/5940CCE8/5940D06F" Ref="R34"  Part="1"
 AR Path="/59418122/5940D06F" Ref="R39"  Part="1"
-F 0 "R39" V 5280 2700 50  0000 C CNN
+F 0 "R34" V 5280 2700 50  0000 C CNN
 F 1 "1k" V 5200 2700 50  0000 C CNN
 F 2 "stmbl:R_0603" V 5130 2700 50  0001 C CNN
@@
 AR Path="/5940CCE8/5940D076" Ref="R35"  Part="1"
 AR Path="/59418122/5940D076" Ref="R40"  Part="1"
-F 0 "R40" V 5530 2450 50  0000 C CNN
+F 0 "R35" V 5530 2450 50  0000 C CNN
 F 1 "120" V 5450 2450 50  0000 C CNN
 F 2 "stmbl:R_0603" V 5380 2450 50  0001 C CNN
@@
 AR Path="/5940CCE8/5940D07D" Ref="Q1"  Part="1"
 AR Path="/59418122/5940D07D" Ref="Q2"  Part="1"
-F 0 "Q2" H 5200 2500 50  0000 R CNN
+F 0 "Q1" H 5200 2500 50  0000 R CNN
 F 1 "Q_NJFET_GSD" H 5550 2400 50  0000 R CNN
 F 2 "stmbl:SOT-23" H 5100 2550 50  0001 C CNN
@@
 AR Path="/5940CCE8/5940D084" Ref="D4"  Part="1"
 AR Path="/59418122/5940D084" Ref="D6"  Part="1"
-F 0 "D6" H 4800 2000 50  0000 C CNN
-F 1 "ES1J" H 4800 1800 50  0000 C CNN
+F 0 "D4" H 4800 2000 50  0000 C CNN
+F 1 "200V 1A" H 4800 1800 50  0000 C CNN
 F 2 "stmbl:SOD-123" H 4800 1900 50  0001 C CNN
 F 3 "" H 4800 1900 50  0000 C CNN
