File: hw/kicad/stmsp/supply.sch (KiCad schematic (older format))
At the start: 14 parts, among them U5 MCP16331, U6 zldo1117

Commit message: stmsp
Parts:
- removed C26: 100n, stmbl:C_0603, symbol C
- removed U6: zldo1117, stmbl:SOT-223, symbol zldo1117
- added D12: Led_Small, stmbl:LED-0805-SIDE, symbol Led_Small
- added R1: 470, stmbl:R_0603, symbol R
- added U6: MIC55, stmbl:SOT-23-5, symbol MIC55
- C22, C24: value C -> 100n
- C23, C25: value C -> 2.2u
- D2: footprint stmbl:SMA_Standard -> stmbl:SOD-123
- L3: footprint (none) -> stmbl:SMD_INDUCTOR_32x25
- R25: value R -> 51k
- R26: value R -> 10k
Connections:
- net +3V3: now also U6.5 (VOUT)
- net +5V: now also D12.2 (A), U6.1 (VIN), U6.3 (EN)
- net GND: now also R1.2
- net at C23.2, C25.2: now also U6.2 (GND)
- new net: D12.1 (K), R1.1
Other:
- note added: "LQH2HPZ220MJRL"
- moved on the sheet: C21, C23, C25, C28
Changed lines of the file:
@@
 EESchema Schematic File Version 2
-LIBS:stmsp-rescue
+LIBS:stmbl
 LIBS:transistors
 LIBS:stm32
@@
 LIBS:video
 LIBS:Xicor
-LIBS:xilinx
-LIBS:Zilog
-LIBS:stmbl
 LIBS:stmsp-cache
 EELAYER 26 0
@@
 $Descr A4 11693 8268
 encoding utf-8
-Sheet 4 7
+Sheet 3 10
 Title ""
 Date ""
@@
 $EndComp
 $Comp
-L zldo1117 U6
-U 1 1 5918AC7A
-P 6100 5250
-F 0 "U6" H 6250 5054 50  0000 C CNN
-F 1 "zldo1117" H 6100 5450 50  0000 C CNN
-F 2 "stmbl:SOT-223" H 6100 5250 50  0001 C CNN
-F 3 "" H 6100 5250 50  0000 C CNN
-	1    6100 5250
-	1    0    0    -1
-$EndComp
-$Comp
 L INDUCTOR L3
 U 1 1 5918C529
@@
 F 0 "L3" V 7000 3400 50  0000 C CNN
 F 1 "INDUCTOR" V 7150 3400 50  0000 C CNN
-F 2 "" H 7050 3400 50  0001 C CNN
+F 2 "stmbl:SMD_INDUCTOR_32x25" H 7050 3400 50  0001 C CNN
 F 3 "" H 7050 3400 50  0000 C CNN
 	1    7050 3400
@@
 L C C23
 U 1 1 5918DD3D
-P 5600 5450
-F 0 "C23" H 5625 5550 50  0000 L CNN
-F 1 "C" H 5625 5350 50  0000 L CNN
-F 2 "stmbl:C_0603" H 5638 5300 50  0001 C CNN
-F 3 "" H 5600 5450 50  0000 C CNN
-	1    5600 5450
+P 5600 5550
+F 0 "C23" H 5625 5650 50  0000 L CNN
+F 1 "2.2u" H 5625 5450 50  0000 L CNN
+F 2 "stmbl:C_0603" H 5638 5400 50  0001 C CNN
+F 3 "" H 5600 5550 50  0000 C CNN
+	1    5600 5550
 	1    0    0    -1
 $EndComp
@@
 L C C25
 U 1 1 5918DD80
-P 6600 5450
-F 0 "C25" H 6625 5550 50  0000 L CNN
-F 1 "C" H 6625 5350 50  0000 L CNN
-F 2 "stmbl:C_0603" H 6638 5300 50  0001 C CNN
-F 3 "" H 6600 5450 50  0000 C CNN
-	1    6600 5450
-	1    0    0    -1
-$EndComp
-$Comp
-L C C26
-U 1 1 5918DDA3
-P 7750 3650
-F 0 "C26" H 7775 3750 50  0000 L CNN
-F 1 "100n" H 7775 3550 50  0000 L CNN
-F 2 "stmbl:C_0603" H 7788 3500 50  0001 C CNN
-F 3 "" H 7750 3650 50  0000 C CNN
-	1    7750 3650
+P 6600 5550
+F 0 "C25" H 6625 5650 50  0000 L CNN
+F 1 "2.2u" H 6625 5450 50  0000 L CNN
+F 2 "stmbl:C_0603" H 6638 5400 50  0001 C CNN
+F 3 "" H 6600 5550 50  0000 C CNN
+	1    6600 5550
 	1    0    0    -1
 $EndComp
@@
 P 6650 3150
 F 0 "C24" H 6675 3250 50  0000 L CNN
-F 1 "C" H 6675 3050 50  0000 L CNN
+F 1 "100n" H 6675 3050 50  0000 L CNN
 F 2 "stmbl:C_0603" H 6688 3000 50  0001 C CNN
 F 3 "" H 6650 3150 50  0000 C CNN
@@
 P 5450 3650
 F 0 "C22" H 5475 3750 50  0000 L CNN
-F 1 "C" H 5475 3550 50  0000 L CNN
+F 1 "100n" H 5475 3550 50  0000 L CNN
 F 2 "stmbl:C_0603" H 5488 3500 50  0001 C CNN
 F 3 "" H 5450 3650 50  0000 C CNN
@@
 P 7450 3650
 F 0 "R25" V 7530 3650 50  0000 C CNN
-F 1 "R" V 7450 3650 50  0000 C CNN
+F 1 "51k" V 7450 3650 50  0000 C CNN
 F 2 "stmbl:R_0603" V 7380 3650 50  0001 C CNN
 F 3 "" H 7450 3650 50  0000 C CNN
@@
 P 7450 4150
 F 0 "R26" V 7530 4150 50  0000 C CNN
-F 1 "R" V 7450 4150 50  0000 C CNN
+F 1 "10k" V 7450 4150 50  0000 C CNN
 F 2 "stmbl:R_0603" V 7380 4150 50  0001 C CNN
 F 3 "" H 7450 4150 50  0000 C CNN
@@
 F 0 "D2" H 6900 3000 50  0000 C CNN
 F 1 "D" H 6900 2800 50  0000 C CNN
-F 2 "stmbl:SMA_Standard" H 6900 2900 50  0001 C CNN
+F 2 "stmbl:SOD-123" H 6900 2900 50  0001 C CNN
 F 3 "" H 6900 2900 50  0000 C CNN
 	1    6900 2900
@@
 Connection ~ 6650 3400
 Wire Wire Line
-	7350 3400 8250 3400
+	7350 3400 8350 3400
 Wire Wire Line
 	7450 2900 7450 3500
@@
 	6650 4400 6650 3800
 Wire Wire Line
-	5450 4400 8250 4400
+	5450 4400 8350 4400
 Wire Wire Line
 	7450 4400 7450 4300
@@
 	6050 3950 6050 4400
 Connection ~ 6650 4400
-Wire Wire Line
-	7750 3400 7750 3500
 Connection ~ 7450 3400
-Wire Wire Line
-	7750 3800 7750 4400
 Connection ~ 7450 4400
 Wire Wire Line
@@
 Connection ~ 6050 4400
 $Comp
-L GND #PWR027
+L GND #PWR024
 U 1 1 59234F24
-P 8250 4500
-F 0 "#PWR027" H 8250 4250 50  0001 C CNN
-F 1 "GND" H 8250 4350 50  0000 C CNN
-F 2 "" H 8250 4500 50  0000 C CNN
-F 3 "" H 8250 4500 50  0000 C CNN
-	1    8250 4500
-	1    0    0    -1
-$EndComp
-$Comp
-L +5V #PWR028
+P 8050 4500
+F 0 "#PWR024" H 8050 4250 50  0001 C CNN
+F 1 "GND" H 8050 4350 50  0000 C CNN
+F 2 "" H 8050 4500 50  0000 C CNN
+F 3 "" H 8050 4500 50  0000 C CNN
+	1    8050 4500
+	1    0    0    -1
+$EndComp
+$Comp
+L +5V #PWR025
 U 1 1 59234FB8
-P 8250 3300
-F 0 "#PWR028" H 8250 3150 50  0001 C CNN
-F 1 "+5V" H 8250 3440 50  0000 C CNN
-F 2 "" H 8250 3300 50  0000 C CNN
-F 3 "" H 8250 3300 50  0000 C CNN
-	1    8250 3300
-	1    0    0    -1
-$EndComp
-$Comp
-L VPP #PWR029
+P 8050 3300
+F 0 "#PWR025" H 8050 3150 50  0001 C CNN
+F 1 "+5V" H 8050 3440 50  0000 C CNN
+F 2 "" H 8050 3300 50  0000 C CNN
+F 3 "" H 8050 3300 50  0000 C CNN
+	1    8050 3300
+	1    0    0    -1
+$EndComp
+$Comp
+L VPP #PWR026
 U 1 1 5923508D
 P 5450 3300
-F 0 "#PWR029" H 5450 3150 50  0001 C CNN
+F 0 "#PWR026" H 5450 3150 50  0001 C CNN
 F 1 "VPP" H 5450 3450 50  0000 C CNN
 F 2 "" H 5450 3300 50  0000 C CNN
@@
 $EndComp
 Connection ~ 5450 3400
-Connection ~ 7750 3400
-Connection ~ 7750 4400
 $Comp
 L C C21
 U 1 1 592353E2
-P 8000 3650
-F 0 "C21" H 8025 3750 50  0000 L CNN
-F 1 "10u" H 8025 3550 50  0000 L CNN
-F 2 "stmbl:C_0603" H 8038 3500 50  0001 C CNN
-F 3 "" H 8000 3650 50  0000 C CNN
-	1    8000 3650
+P 7750 3650
+F 0 "C21" H 7775 3750 50  0000 L CNN
+F 1 "10u" H 7775 3550 50  0000 L CNN
+F 2 "stmbl:C_0603" H 7788 3500 50  0001 C CNN
+F 3 "" H 7750 3650 50  0000 C CNN
+	1    7750 3650
 	1    0    0    -1
 $EndComp
@@
 L C C28
 U 1 1 5923540F
-P 8250 3650
-F 0 "C28" H 8275 3750 50  0000 L CNN
-F 1 "10u" H 8275 3550 50  0000 L CNN
-F 2 "stmbl:C_0603" H 8288 3500 50  0001 C CNN
-F 3 "" H 8250 3650 50  0000 C CNN
-	1    8250 3650
-	1    0    0    -1
-$EndComp
-Wire Wire Line
-	8000 4400 8000 3800
-Wire Wire Line
-	8250 3800 8250 4500
-Connection ~ 8000 4400
-Wire Wire Line
-	8250 3300 8250 3500
-Wire Wire Line
-	8000 3500 8000 3400
-Connection ~ 8000 3400
-Connection ~ 8250 4400
-Connection ~ 8250 3400
-Wire Wire Line
-	5700 5200 5600 5200
-Wire Wire Line
-	5600 5100 5600 5300
-Wire Wire Line
-	6500 5200 6600 5200
-Wire Wire Line
-	6600 5100 6600 5300
-Wire Wire Line
-	5600 5600 5600 5700
-Wire Wire Line
-	5600 5700 6600 5700
-Wire Wire Line
-	6600 5700 6600 5600
-Wire Wire Line
-	6100 5500 6100 5700
-Connection ~ 6100 5700
-$Comp
-L +3.3V #PWR030
+P 8050 3650
+F 0 "C28" H 8075 3750 50  0000 L CNN
+F 1 "10u" H 8075 3550 50  0000 L CNN
+F 2 "stmbl:C_0603" H 8088 3500 50  0001 C CNN
+F 3 "" H 8050 3650 50  0000 C CNN
+	1    8050 3650
+	1    0    0    -1
+$EndComp
+Wire Wire Line
+	7750 4400 7750 3800
+Wire Wire Line
+	8050 3800 8050 4500
+Connection ~ 7750 4400
+Wire Wire Line
+	8050 3300 8050 3500
+Wire Wire Line
+	7750 3500 7750 3400
+Connection ~ 7750 3400
+Connection ~ 8050 4400
+Connection ~ 8050 3400
+Wire Wire Line
+	5700 5100 5600 5100
+Wire Wire Line
+	5600 5000 5600 5400
+Wire Wire Line
+	6500 5100 6600 5100
+Wire Wire Line
+	6600 5000 6600 5400
+Wire Wire Line
+	5600 5700 5600 5800
+Wire Wire Line
+	5600 5800 6600 5800
+Wire Wire Line
+	6600 5800 6600 5700
+Wire Wire Line
+	6100 5500 6100 5800
+Connection ~ 6100 5800
+$Comp
+L +3.3V #PWR027
 U 1 1 59235CD1
-P 6600 5100
-F 0 "#PWR030" H 6600 4950 50  0001 C CNN
-F 1 "+3.3V" H 6600 5240 50  0000 C CNN
-F 2 "" H 6600 5100 50  0000 C CNN
-F 3 "" H 6600 5100 50  0000 C CNN
-	1    6600 5100
-	1    0    0    -1
-$EndComp
-Connection ~ 6600 5200
-$Comp
-L +5V #PWR031
+P 6600 5000
+F 0 "#PWR027" H 6600 4850 50  0001 C CNN
+F 1 "+3.3V" H 6600 5140 50  0000 C CNN
+F 2 "" H 6600 5000 50  0000 C CNN
+F 3 "" H 6600 5000 50  0000 C CNN
+	1    6600 5000
+	1    0    0    -1
+$EndComp
+Connection ~ 6600 5100
+$Comp
+L +5V #PWR028
 U 1 1 59235D71
-P 5600 5100
-F 0 "#PWR031" H 5600 4950 50  0001 C CNN
-F 1 "+5V" H 5600 5240 50  0000 C CNN
-F 2 "" H 5600 5100 50  0000 C CNN
-F 3 "" H 5600 5100 50  0000 C CNN
-	1    5600 5100
-	1    0    0    -1
-$EndComp
-Connection ~ 5600 5200
+P 5600 5000
+F 0 "#PWR028" H 5600 4850 50  0001 C CNN
+F 1 "+5V" H 5600 5140 50  0000 C CNN
+F 2 "" H 5600 5000 50  0000 C CNN
+F 3 "" H 5600 5000 50  0000 C CNN
+	1    5600 5000
+	1    0    0    -1
+$EndComp
+Connection ~ 5600 5100
+Text Notes 7550 2950 0    60   ~ 0
+LQH2HPZ220MJRL
+$Comp
+L MIC55 U6
+U 1 1 59444047
+P 6100 5200
+F 0 "U6" H 5850 5400 50  0000 L CNN
+F 1 "MIC55" H 6700 5400 50  0000 R CNN
+F 2 "stmbl:SOT-23-5" H 6750 4950 50  0001 C CIN
+F 3 "" H 6100 5200 50  0000 C CNN
+	1    6100 5200
+	1    0    0    -1
+$EndComp
+Wire Wire Line
+	5700 5300 5600 5300
+Connection ~ 5600 5300
+$Comp
+L Led_Small D12
+U 1 1 5944CEE5
+P 8350 3650
+F 0 "D12" H 8300 3775 50  0000 L CNN
+F 1 "Led_Small" H 8175 3550 50  0000 L CNN
+F 2 "stmbl:LED-0805-SIDE" V 8350 3650 50  0001 C CNN
+F 3 "" V 8350 3650 50  0000 C CNN
+	1    8350 3650
+	0    -1   -1   0
+$EndComp
+$Comp
+L R R1
+U 1 1 5944CF59
+P 8350 4150
+F 0 "R1" V 8430 4150 50  0000 C CNN
+F 1 "470" V 8350 4150 50  0000 C CNN
+F 2 "stmbl:R_0603" V 8280 4150 50  0001 C CNN
+F 3 "" H 8350 4150 50  0000 C CNN
+	1    8350 4150
+	1    0    0    -1
+$EndComp
+Wire Wire Line
+	8350 3400 8350 3550
+Wire Wire Line
+	8350 3750 8350 4000
+Wire Wire Line
+	8350 4400 8350 4300
 $EndSCHEMATC

Commit message: stmsp
Connections:
- net GND: now also C23.2, C25.2, U6.2 (GND)
Changed lines of the file:
@@
 Connection ~ 6050 4400
 $Comp
-L GND #PWR026
+L GND #PWR027
 U 1 1 59234F24
 P 8050 4500
-F 0 "#PWR026" H 8050 4250 50  0001 C CNN
+F 0 "#PWR027" H 8050 4250 50  0001 C CNN
 F 1 "GND" H 8050 4350 50  0000 C CNN
 F 2 "" H 8050 4500 50  0000 C CNN
@@
 $EndComp
 $Comp
-L +5V #PWR027
+L +5V #PWR028
 U 1 1 59234FB8
 P 8050 3300
-F 0 "#PWR027" H 8050 3150 50  0001 C CNN
+F 0 "#PWR028" H 8050 3150 50  0001 C CNN
 F 1 "+5V" H 8050 3440 50  0000 C CNN
 F 2 "" H 8050 3300 50  0000 C CNN
@@
 $EndComp
 $Comp
-L VPP #PWR028
+L VPP #PWR029
 U 1 1 5923508D
 P 5450 3300
-F 0 "#PWR028" H 5450 3150 50  0001 C CNN
+F 0 "#PWR029" H 5450 3150 50  0001 C CNN
 F 1 "VPP" H 5450 3450 50  0000 C CNN
 F 2 "" H 5450 3300 50  0000 C CNN
@@
 	6600 5800 6600 5700
 Wire Wire Line
-	6100 5500 6100 5800
+	6100 5500 6100 5900
 Connection ~ 6100 5800
-$Comp
-L +3.3V #PWR029
-U 1 1 59235CD1
-P 6600 5000
-F 0 "#PWR029" H 6600 4850 50  0001 C CNN
-F 1 "+3.3V" H 6600 5140 50  0000 C CNN
-F 2 "" H 6600 5000 50  0000 C CNN
-F 3 "" H 6600 5000 50  0000 C CNN
-	1    6600 5000
-	1    0    0    -1
-$EndComp
 Connection ~ 6600 5100
 $Comp
@@
 Wire Wire Line
 	8350 4400 8350 4300
+$Comp
+L GND #PWR031
+U 1 1 593D3F2D
+P 6100 5900
+F 0 "#PWR031" H 6100 5650 50  0001 C CNN
+F 1 "GND" H 6100 5750 50  0000 C CNN
+F 2 "" H 6100 5900 50  0000 C CNN
+F 3 "" H 6100 5900 50  0000 C CNN
+	1    6100 5900
+	1    0    0    -1
+$EndComp
+$Comp
+L +3.3V #PWR032
+U 1 1 594630A5
+P 6600 5000
+F 0 "#PWR032" H 6600 4850 50  0001 C CNN
+F 1 "+3.3V" H 6600 5140 50  0000 C CNN
+F 2 "" H 6600 5000 50  0000 C CNN
+F 3 "" H 6600 5000 50  0000 C CNN
+	1    6600 5000
+	1    0    0    -1
+$EndComp
 $EndSCHEMATC

Commit message: stmsp
Parts:
- U6: value MIC55 -> MIC5504-3.3YM5
Changed lines of the file:
@@
 P 6100 5200
 F 0 "U6" H 5850 5400 50  0000 L CNN
-F 1 "MIC55" H 6700 5400 50  0000 R CNN
+F 1 "MIC5504-3.3YM5" H 6700 5400 50  0000 R CNN
 F 2 "stmbl:SOT-23-5" H 6750 4950 50  0001 C CIN
 F 3 "" H 6100 5200 50  0000 C CNN

Commit message: stmsp
Other:
- note added: "0.816V * (51k + 10k) / 10k = 4.9776V"
Changed lines of the file:
@@
 	1    0    0    -1
 $EndComp
+Text Notes 8300 3200 0    60   ~ 0
+0.816V * (51k + 10k) / 10k = 4.9776V
 $EndSCHEMATC

Commit message: stmsp
Parts:
- C21, C28: footprint stmbl:C_0603 -> stmbl:C_0805
Connections:
- no-connect marks 0 -> 1
Changed lines of the file:
@@
 F 0 "C21" H 7775 3750 50  0000 L CNN
 F 1 "10u" H 7775 3550 50  0000 L CNN
-F 2 "stmbl:C_0603" H 7788 3500 50  0001 C CNN
+F 2 "stmbl:C_0805" H 7788 3500 50  0001 C CNN
 F 3 "" H 7750 3650 50  0000 C CNN
 	1    7750 3650
@@
 F 0 "C28" H 8075 3750 50  0000 L CNN
 F 1 "10u" H 8075 3550 50  0000 L CNN
-F 2 "stmbl:C_0603" H 8088 3500 50  0001 C CNN
+F 2 "stmbl:C_0805" H 8088 3500 50  0001 C CNN
 F 3 "" H 8050 3650 50  0000 C CNN
 	1    8050 3650
@@
 Text Notes 8300 3200 0    60   ~ 0
 0.816V * (51k + 10k) / 10k = 4.9776V
+NoConn ~ 5650 3600
 $EndSCHEMATC

Commit message: stmsp
Parts:
- D1: value D -> ss110
- D2: value D -> 1N4148
- L3: value INDUCTOR -> 22µ 650mA
Other:
- note added: "LQH32PN220MNCL"
- note removed: "LQH2HPZ220MJRL"
Changed lines of the file:
@@
 P 7050 3400
 F 0 "L3" V 7000 3400 50  0000 C CNN
-F 1 "INDUCTOR" V 7150 3400 50  0000 C CNN
+F 1 "22µ 650mA" V 7150 3400 50  0000 C CNN
 F 2 "stmbl:SMD_INDUCTOR_32x25" H 7050 3400 50  0001 C CNN
 F 3 "" H 7050 3400 50  0000 C CNN
@@
 P 6650 3650
 F 0 "D1" H 6650 3750 50  0000 C CNN
-F 1 "D" H 6650 3550 50  0000 C CNN
+F 1 "ss110" H 6650 3550 50  0000 C CNN
 F 2 "stmbl:SMA_Standard" H 6650 3650 50  0001 C CNN
 F 3 "" H 6650 3650 50  0000 C CNN
@@
 P 6900 2900
 F 0 "D2" H 6900 3000 50  0000 C CNN
-F 1 "D" H 6900 2800 50  0000 C CNN
+F 1 "1N4148" H 6900 2800 50  0000 C CNN
 F 2 "stmbl:SOD-123" H 6900 2900 50  0001 C CNN
 F 3 "" H 6900 2900 50  0000 C CNN
@@
 Connection ~ 5600 5100
 Text Notes 7550 2950 0    60   ~ 0
-LQH2HPZ220MJRL
+LQH32PN220MNCL
 $Comp
 L MIC55 U6
