File: hw/kicad/bob/ethernet_bob/flash.sch (KiCad schematic (older format))
At the start: 2 parts, among them U4 CAT250_EEPROM

Commit message: netbob lables
Parts:
- C22: footprint Capacitors_SMD:C_0603 -> stmbl:C_0603
Changed lines of the file:
@@
 EESchema Schematic File Version 2
-LIBS:ethernet_bob-rescue
 LIBS:power
 LIBS:device
@@
 LIBS:usblc
 LIBS:ethernet_bob-cache
-EELAYER 25 0
+EELAYER 26 0
 EELAYER END
 $Descr A4 11693 8268
@@
 F 0 "C22" H 7465 4046 50  0000 L CNN
 F 1 "C" H 7465 3955 50  0000 L CNN
-F 2 "Capacitors_SMD:C_0603" H 7388 3850 50  0001 C CNN
+F 2 "stmbl:C_0603" H 7388 3850 50  0001 C CNN
 F 3 "" H 7350 4000 50  0000 C CNN
 	1    7350 4000
@@
 $EndComp
 $Comp
-L +3.3V #PWR24
+L +3.3V #PWR022
 U 1 1 57FEB05E
 P 7350 3750
-F 0 "#PWR24" H 7350 3600 50  0001 C CNN
+F 0 "#PWR022" H 7350 3600 50  0001 C CNN
 F 1 "+3.3V" H 7365 3923 50  0000 C CNN
 F 2 "" H 7350 3750 50  0000 C CNN
@@
 $EndComp
 $Comp
-L GND #PWR25
+L GND #PWR023
 U 1 1 57FEB078
 P 7350 4250
-F 0 "#PWR25" H 7350 4000 50  0001 C CNN
+F 0 "#PWR023" H 7350 4000 50  0001 C CNN
 F 1 "GND" H 7355 4077 50  0000 C CNN
 F 2 "" H 7350 4250 50  0000 C CNN
@@
 $EndComp
 $Comp
-L GND #PWR23
+L GND #PWR024
 U 1 1 57FEB090
 P 5550 4300
-F 0 "#PWR23" H 5550 4050 50  0001 C CNN
+F 0 "#PWR024" H 5550 4050 50  0001 C CNN
 F 1 "GND" H 5555 4127 50  0000 C CNN
 F 2 "" H 5550 4300 50  0000 C CNN
@@
 	5550 4300 5550 4250
 $Comp
-L +3.3V #PWR22
+L +3.3V #PWR025
 U 1 1 57FEB0B4
 P 5550 3600
-F 0 "#PWR22" H 5550 3450 50  0001 C CNN
+F 0 "#PWR025" H 5550 3450 50  0001 C CNN
 F 1 "+3.3V" H 5565 3773 50  0000 C CNN
 F 2 "" H 5550 3600 50  0000 C CNN
