File: hw/kicad/11ua/11ua.sch (KiCad schematic (older format))
At the start: 17 parts, among them J1 RJ45, J2 RJ45, U1 LM393

Commit message: add index for 11ua, change to lm339
Parts:
- removed U1: LM393, stmbl:SOIC-8-N, symbol LM393
- added C10, C11, C12: C, stmbl:C_0603, symbol 11ua-rescue:C
- added C13, C14: CP, Capacitor_Tantalum_SMD:CP_EIA-2012-15_AVX-P, symbol Device:CP
- added C7, C8: 27p, stmbl:C_0603, symbol 11ua-rescue:C
- added C9: 100n, stmbl:C_0603, symbol 11ua-rescue:C
- added J3, J4: CONN_01X04, stmbl:RM3.81_1x4_UP, symbol stmbl:CONN_01X04
- added R10, R9: 100k, stmbl:R_0603, symbol 11ua-rescue:R
- added R11, R12: 120, stmbl:R_0603, symbol 11ua-rescue:R
- added U1: LM339, Package_SO:SOIC-14_3.9x8.7mm_P1.27mm, symbol Comparator:LM339
- C1, C2, C3, C4, C5, C6: symbol C -> 11ua-rescue:C
- J1, J2: symbol RJ45 -> 11ua-rescue:RJ45
- R1, R2, R3, R4, R5, R6, R7, R8: symbol R -> 11ua-rescue:R
Connections:
- wire segments 68 -> 161
Other:
- moved on the sheet: C1, C2, C3, C4, C5, C6, J1, J2, R1, R2, R3, R4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

Commit message: changed things
Parts:
- removed C9: 100n, stmbl:C_0603, symbol 11ua-rescue:C
- removed R11, R12, R5, R6: 120, stmbl:R_0603, symbol 11ua-rescue:R
Connections:
- net labels added: 2.5V
- wire segments 161 -> 157
Other:
- moved on the sheet: C6, R7, R8

Commit message: change rj45
Parts:
- removed J1, J2: RJ45, Connect:RJ45_8, symbol 11ua-rescue:RJ45
- added J1, J2: RJ45_LED, stmbl:RJ45_LED, symbol stmbl:RJ45_LED
Connections:
- net labels removed: GNDA
Other:
- moved on the sheet: J4
Changed lines of the file:
@@
 $EndDescr
-$Comp
-L 11ua-rescue:RJ45 J1
-U 1 1 592E009D
-P 3950 5350
-F 0 "J1" V 3375 5345 50  0000 C CNN
-F 1 "RJ45" V 3466 5345 50  0000 C CNN
-F 2 "Connect:RJ45_8" H 3950 5350 50  0001 C CNN
-F 3 "" H 3950 5350 50  0001 C CNN
-	1    3950 5350
-	0    -1   1    0
-$EndComp
-$Comp
-L 11ua-rescue:RJ45 J2
-U 1 1 592E00E5
-P 10650 5350
-F 0 "J2" V 10680 5830 50  0000 L CNN
-F 1 "RJ45" V 10771 5830 50  0000 L CNN
-F 2 "Connect:RJ45_8" H 10650 5350 50  0001 C CNN
-F 3 "" H 10650 5350 50  0001 C CNN
-	1    10650 5350
-	0    1    1    0
-$EndComp
-$Comp
-L power:GND #PWR05
-U 1 1 592E067C
-P 5550 5700
-F 0 "#PWR05" H 5550 5450 50  0001 C CNN
-F 1 "GND" V 5555 5572 50  0000 R CNN
-F 2 "" H 5550 5700 50  0001 C CNN
-F 3 "" H 5550 5700 50  0001 C CNN
-	1    5550 5700
-	0    -1   -1   0
-$EndComp
 $Comp
 L power:GND #PWR06
 U 1 1 592E06DB
+P 10100 5800
+F 0 "#PWR06" H 10100 5550 50  0001 C CNN
+F 1 "GND" V 10105 5672 50  0000 R CNN
+F 2 "" H 10100 5800 50  0001 C CNN
+F 3 "" H 10100 5800 50  0001 C CNN
+	1    10100 5800
+	0    1    1    0
+$EndComp
+$Comp
+L power:+5V #PWR08
+U 1 1 592E0780
 P 10100 5700
-F 0 "#PWR06" H 10100 5450 50  0001 C CNN
-F 1 "GND" V 10105 5572 50  0000 R CNN
+F 0 "#PWR08" H 10100 5550 50  0001 C CNN
+F 1 "+5V" V 10115 5828 50  0000 L CNN
 F 2 "" H 10100 5700 50  0001 C CNN
 F 3 "" H 10100 5700 50  0001 C CNN
 	1    10100 5700
-	0    1    1    0
-$EndComp
-$Comp
-L power:+5V #PWR07
-U 1 1 592E071C
-P 5550 5600
-F 0 "#PWR07" H 5550 5450 50  0001 C CNN
-F 1 "+5V" V 5565 5728 50  0000 L CNN
-F 2 "" H 5550 5600 50  0001 C CNN
-F 3 "" H 5550 5600 50  0001 C CNN
-	1    5550 5600
-	0    1    1    0
-$EndComp
-$Comp
-L power:+5V #PWR08
-U 1 1 592E0780
-P 10100 5600
-F 0 "#PWR08" H 10100 5450 50  0001 C CNN
-F 1 "+5V" V 10115 5728 50  0000 L CNN
-F 2 "" H 10100 5600 50  0001 C CNN
-F 3 "" H 10100 5600 50  0001 C CNN
-	1    10100 5600
 	0    -1   -1   0
 $EndComp
@@
 $EndComp
 Wire Wire Line
-	10100 5600 10200 5600
-Wire Wire Line
-	10200 5700 10100 5700
-Wire Wire Line
-	4400 5600 5250 5600
-Wire Wire Line
-	4400 5700 5150 5700
-Wire Wire Line
-	6150 7750 7300 7750
+	10100 5700 10200 5700
+Wire Wire Line
+	10200 5800 10100 5800
 Wire Wire Line
 	8000 8200 7300 8200
@@
 Wire Wire Line
 	4400 5200 5350 5200
-Wire Wire Line
-	6150 5200 6150 7750
 Connection ~ 7300 7750
 Wire Wire Line
@@
 Wire Wire Line
 	6250 2700 7250 2700
-Wire Wire Line
-	4400 5500 5350 5500
-Wire Wire Line
-	6250 5500 6250 7550
 Wire Wire Line
 	6250 7550 7300 7550
@@
 	10050 5100 10200 5100
 Wire Wire Line
-	10200 5500 9650 5500
-Wire Wire Line
-	9650 5500 9650 7500
-$Comp
-L power:GNDA #PWR013
-U 1 1 592E2042
-P 3600 6000
-F 0 "#PWR013" H 3600 5750 50  0001 C CNN
-F 1 "GNDA" H 3605 5827 50  0000 C CNN
-F 2 "" H 3600 6000 50  0001 C CNN
-F 3 "" H 3600 6000 50  0001 C CNN
-	1    3600 6000
-	1    0    0    -1
-$EndComp
-$Comp
-L power:GNDA #PWR014
-U 1 1 592E2078
-P 11000 6000
-F 0 "#PWR014" H 11000 5750 50  0001 C CNN
-F 1 "GNDA" H 11005 5827 50  0000 C CNN
-F 2 "" H 11000 6000 50  0001 C CNN
-F 3 "" H 11000 6000 50  0001 C CNN
-	1    11000 6000
-	1    0    0    -1
-$EndComp
-Wire Wire Line
-	11000 5900 11000 6000
-Wire Wire Line
-	3600 5900 3600 6000
+	10700 6050 10700 6150
 Wire Wire Line
 	7300 8200 7300 8550
@@
 	7350 5900 6650 5900
 Wire Wire Line
-	6650 5450 6650 5900
-Wire Wire Line
 	6650 6250 6750 6250
-Connection ~ 6650 5900
 Wire Wire Line
 	7400 5350 7750 5350
@@
 	7700 4800 7700 5200
 Wire Wire Line
-	4400 5400 5450 5400
-Wire Wire Line
-	6650 5400 6650 5450
-Connection ~ 6650 5450
-Wire Wire Line
 	4400 5300 5450 5300
 Wire Wire Line
@@
 	9100 5300 9100 5200
 Wire Wire Line
-	10200 5400 8950 5400
-Wire Wire Line
-	8950 5400 8950 5900
-Wire Wire Line
 	8950 5900 7750 5900
-$Comp
-L stmbl:CONN_01X04 J4
-U 1 1 5C702B75
-P 5350 5950
-F 0 "J4" V 5223 6130 50  0000 L CNN
-F 1 "CONN_01X04" V 5314 6130 50  0000 L CNN
-F 2 "stmbl:RM3.81_1x4_UP" H 5350 5950 50  0001 C CNN
-F 3 "" H 5350 5950 50  0001 C CNN
-	1    5350 5950
-	0    1    1    0
-$EndComp
 $Comp
 L stmbl:CONN_01X04 J3
@@
 Wire Wire Line
 	5350 4900 5350 5200
-Connection ~ 5350 5200
-Wire Wire Line
-	5350 5200 6150 5200
 Wire Wire Line
 	5450 4900 5450 5300
 Connection ~ 5450 5300
-Wire Wire Line
-	5450 5300 6650 5300
-Wire Wire Line
-	5450 5750 5450 5400
-Connection ~ 5450 5400
-Wire Wire Line
-	5450 5400 6650 5400
-Wire Wire Line
-	5350 5500 5350 5750
-Connection ~ 5350 5500
-Wire Wire Line
-	5350 5500 6250 5500
-Wire Wire Line
-	5250 5750 5250 5600
-Connection ~ 5250 5600
-Wire Wire Line
-	5250 5600 5550 5600
-Wire Wire Line
-	5150 5700 5150 5750
-Connection ~ 5150 5700
-Wire Wire Line
-	5150 5700 5550 5700
 $Comp
 L Comparator:LM339 U1
@@
 Wire Wire Line
 	13750 7050 13750 7150
+$Comp
+L stmbl:RJ45_LED J1
+U 1 1 5D7E41F6
+P 3900 5400
+F 0 "J1" V 3275 5400 50  0000 C CNN
+F 1 "RJ45_LED" V 3366 5400 50  0000 C CNN
+F 2 "stmbl:RJ45_LED" H 3900 5350 60  0001 C CNN
+F 3 "" H 3900 5350 60  0000 C CNN
+	1    3900 5400
+	0    -1   1    0
+$EndComp
+Wire Wire Line
+	6650 5500 6650 5450
+Connection ~ 6650 5900
+Connection ~ 5350 5200
+Wire Wire Line
+	5450 5300 6650 5300
+Wire Wire Line
+	6150 7750 7300 7750
+Wire Wire Line
+	5350 5200 6150 5200
+$Comp
+L power:GND #PWR05
+U 1 1 592E067C
+P 5550 5800
+F 0 "#PWR05" H 5550 5550 50  0001 C CNN
+F 1 "GND" V 5555 5672 50  0000 R CNN
+F 2 "" H 5550 5800 50  0001 C CNN
+F 3 "" H 5550 5800 50  0001 C CNN
+	1    5550 5800
+	0    -1   -1   0
+$EndComp
+$Comp
+L power:+5V #PWR07
+U 1 1 592E071C
+P 5550 5700
+F 0 "#PWR07" H 5550 5550 50  0001 C CNN
+F 1 "+5V" V 5565 5828 50  0000 L CNN
+F 2 "" H 5550 5700 50  0001 C CNN
+F 3 "" H 5550 5700 50  0001 C CNN
+	1    5550 5700
+	0    1    1    0
+$EndComp
+Wire Wire Line
+	4400 5700 5250 5700
+Wire Wire Line
+	4400 5800 5150 5800
+Wire Wire Line
+	6150 5200 6150 7750
+Wire Wire Line
+	4400 5600 5350 5600
+$Comp
+L stmbl:CONN_01X04 J4
+U 1 1 5C702B75
+P 5350 6050
+F 0 "J4" V 5223 6230 50  0000 L CNN
+F 1 "CONN_01X04" V 5314 6230 50  0000 L CNN
+F 2 "stmbl:RM3.81_1x4_UP" H 5350 6050 50  0001 C CNN
+F 3 "" H 5350 6050 50  0001 C CNN
+	1    5350 6050
+	0    1    1    0
+$EndComp
+Wire Wire Line
+	5450 5850 5450 5500
+Wire Wire Line
+	5350 5600 5350 5850
+Connection ~ 5350 5600
+Wire Wire Line
+	5350 5600 6250 5600
+Wire Wire Line
+	5250 5850 5250 5700
+Connection ~ 5250 5700
+Wire Wire Line
+	5250 5700 5550 5700
+Wire Wire Line
+	5150 5800 5150 5850
+Connection ~ 5150 5800
+Wire Wire Line
+	5150 5800 5550 5800
+Wire Wire Line
+	6250 5600 6250 7550
+Wire Wire Line
+	4400 5500 5450 5500
+Connection ~ 5450 5500
+Wire Wire Line
+	5450 5500 6650 5500
+Connection ~ 6650 5500
+Wire Wire Line
+	6650 5500 6650 5900
+Wire Wire Line
+	3900 6050 3900 6150
+$Comp
+L stmbl:RJ45_LED J2
+U 1 1 5D829B26
+P 10700 5400
+F 0 "J2" V 10075 5400 50  0000 C CNN
+F 1 "RJ45_LED" V 10166 5400 50  0000 C CNN
+F 2 "stmbl:RJ45_LED" H 10700 5350 60  0001 C CNN
+F 3 "" H 10700 5350 60  0000 C CNN
+	1    10700 5400
+	0    1    1    0
+$EndComp
+Wire Wire Line
+	10200 5600 9650 5600
+Wire Wire Line
+	9650 5600 9650 7500
+Wire Wire Line
+	10200 5500 8950 5500
+Wire Wire Line
+	8950 5500 8950 5900
+$Comp
+L power:GND #PWR?
+U 1 1 5D872060
+P 10700 6150
+F 0 "#PWR?" H 10700 5900 50  0001 C CNN
+F 1 "GND" H 10705 5977 50  0000 C CNN
+F 2 "" H 10700 6150 50  0001 C CNN
+F 3 "" H 10700 6150 50  0001 C CNN
+	1    10700 6150
+	-1   0    0    -1
+$EndComp
+$Comp
+L power:GND #PWR?
+U 1 1 5D872536
+P 3900 6150
+F 0 "#PWR?" H 3900 5900 50  0001 C CNN
+F 1 "GND" H 3905 5977 50  0000 C CNN
+F 2 "" H 3900 6150 50  0001 C CNN
+F 3 "" H 3900 6150 50  0001 C CNN
+	1    3900 6150
+	-1   0    0    -1
+$EndComp
 $EndSCHEMATC

Commit message: change to opamp....
Parts:
- removed U1: LM339, Package_SO:SOIC-14_3.9x8.7mm_P1.27mm, symbol Comparator:LM339
- added U1: OPA4376, Housings_SSOP:TSSOP-14_4.4x5mm_Pitch0.65mm, symbol Amplifier_Operational:OPA4376
- C1, C10, C11, C12, C2, C3, C4, C5, C6, C7, C8: footprint stmbl:C_0603 -> stmbl-kicad-lib:C_0603; symbol 11ua-rescue:C -> stmbl:C
- R1, R10, R2, R3, R4, R7, R8, R9: footprint stmbl:R_0603 -> stmbl-kicad-lib:R_0603; symbol 11ua-rescue:R -> stmbl:R
