File: hw/kicad/bob/ethernet_bob_base/psu.sch (KiCad schematic (older format))
At the start: 16 parts, among them U1 LM5017MR

Commit message: add outputs
Parts:
- added C10, C11: 20µ, Capacitors_SMD:CP_Elec_6.3x7.7, symbol stmbl:CP
Connections:
- net GND: now also C10.2, C11.2
- net VD: now also C10.1, C11.1
Changed lines of the file:
@@
 	5850 3150 6150 3150
 Connection ~ 5850 2550
+$Comp
+L stmbl:CP C10
+U 1 1 5C9805D5
+P 1900 4150
+F 0 "C10" H 2018 4241 50  0000 L CNN
+F 1 "20µ" H 2018 4150 50  0000 L CNN
+F 2 "Capacitors_SMD:CP_Elec_6.3x7.7" H 2800 3750 50  0001 L CNN
+F 3 "" H 1900 4150 50  0000 C CNN
+	1    1900 4150
+	1    0    0    -1
+$EndComp
+$Comp
+L stmbl:CP C11
+U 1 1 5C980A7A
+P 2350 4150
+F 0 "C11" H 2468 4241 50  0000 L CNN
+F 1 "20µ" H 2468 4150 50  0000 L CNN
+F 2 "Capacitors_SMD:CP_Elec_6.3x7.7" H 3250 3750 50  0001 L CNN
+F 3 "" H 2350 4150 50  0000 C CNN
+	1    2350 4150
+	1    0    0    -1
+$EndComp
+Wire Wire Line
+	1900 4000 2150 4000
+Wire Wire Line
+	1900 4300 2150 4300
+$Comp
+L stmbl:VD #PWR0136
+U 1 1 5C9839A3
+P 2150 4000
+F 0 "#PWR0136" H 2150 3850 50  0001 C CNN
+F 1 "VD" H 2167 4173 50  0000 C CNN
+F 2 "" H 2150 4000 50  0001 C CNN
+F 3 "" H 2150 4000 50  0001 C CNN
+	1    2150 4000
+	1    0    0    -1
+$EndComp
+Connection ~ 2150 4000
+Wire Wire Line
+	2150 4000 2350 4000
+$Comp
+L stmbl:GND #PWR0137
+U 1 1 5C983E19
+P 2150 4300
+F 0 "#PWR0137" H 2150 4050 50  0001 C CNN
+F 1 "GND" H 2155 4127 50  0000 C CNN
+F 2 "" H 2150 4300 50  0000 C CNN
+F 3 "" H 2150 4300 50  0000 C CNN
+	1    2150 4300
+	1    0    0    -1
+$EndComp
+Connection ~ 2150 4300
+Wire Wire Line
+	2150 4300 2350 4300
 $EndSCHEMATC

Commit message: routing
Parts:
- added C12, C13, C14, C15, C16, C17: 100n, stmbl:C_0805, symbol stmbl:C
Connections:
- net GND: now also C12.2, C13.2, C14.2, C15.2, C16.2, C17.2
- new net +3V3: C12.1, C13.1, C14.1, C15.1, C16.1, C17.1
Changed lines of the file:
@@
 Wire Wire Line
 	2150 4300 2350 4300
+$Comp
+L stmbl:C C12
+U 1 1 5CA7CA0A
+P 3600 4100
+F 0 "C12" H 3715 4146 50  0000 L CNN
+F 1 "100n" H 3715 4055 50  0000 L CNN
+F 2 "stmbl:C_0805" H 3638 3950 50  0001 C CNN
+F 3 "" H 3600 4100 50  0001 C CNN
+	1    3600 4100
+	1    0    0    -1
+$EndComp
+$Comp
+L stmbl:C C13
+U 1 1 5CA7CF46
+P 4050 4100
+F 0 "C13" H 4165 4146 50  0000 L CNN
+F 1 "100n" H 4165 4055 50  0000 L CNN
+F 2 "stmbl:C_0805" H 4088 3950 50  0001 C CNN
+F 3 "" H 4050 4100 50  0001 C CNN
+	1    4050 4100
+	1    0    0    -1
+$EndComp
+$Comp
+L stmbl:C C14
+U 1 1 5CA7D2B0
+P 4500 4100
+F 0 "C14" H 4615 4146 50  0000 L CNN
+F 1 "100n" H 4615 4055 50  0000 L CNN
+F 2 "stmbl:C_0805" H 4538 3950 50  0001 C CNN
+F 3 "" H 4500 4100 50  0001 C CNN
+	1    4500 4100
+	1    0    0    -1
+$EndComp
+$Comp
+L stmbl:C C15
+U 1 1 5CA7D4EB
+P 4950 4100
+F 0 "C15" H 5065 4146 50  0000 L CNN
+F 1 "100n" H 5065 4055 50  0000 L CNN
+F 2 "stmbl:C_0805" H 4988 3950 50  0001 C CNN
+F 3 "" H 4950 4100 50  0001 C CNN
+	1    4950 4100
+	1    0    0    -1
+$EndComp
+$Comp
+L stmbl:C C16
+U 1 1 5CA7D7C5
+P 5350 4100
+F 0 "C16" H 5465 4146 50  0000 L CNN
+F 1 "100n" H 5465 4055 50  0000 L CNN
+F 2 "stmbl:C_0805" H 5388 3950 50  0001 C CNN
+F 3 "" H 5350 4100 50  0001 C CNN
+	1    5350 4100
+	1    0    0    -1
+$EndComp
+$Comp
+L stmbl:C C17
+U 1 1 5CA7DB2B
+P 5750 4100
+F 0 "C17" H 5865 4146 50  0000 L CNN
+F 1 "100n" H 5865 4055 50  0000 L CNN
+F 2 "stmbl:C_0805" H 5788 3950 50  0001 C CNN
+F 3 "" H 5750 4100 50  0001 C CNN
+	1    5750 4100
+	1    0    0    -1
+$EndComp
+Wire Wire Line
+	3600 3950 4050 3950
+Connection ~ 4050 3950
+Wire Wire Line
+	4050 3950 4500 3950
+Connection ~ 4500 3950
+Wire Wire Line
+	4500 3950 4700 3950
+Connection ~ 4950 3950
+Wire Wire Line
+	4950 3950 5350 3950
+Connection ~ 5350 3950
+Wire Wire Line
+	5350 3950 5750 3950
+Wire Wire Line
+	3600 4250 4050 4250
+Connection ~ 4050 4250
+Wire Wire Line
+	4050 4250 4500 4250
+Connection ~ 4500 4250
+Wire Wire Line
+	4500 4250 4700 4250
+Connection ~ 4950 4250
+Wire Wire Line
+	4950 4250 5350 4250
+Connection ~ 5350 4250
+Wire Wire Line
+	5350 4250 5750 4250
+$Comp
+L stmbl:GND #PWR0142
+U 1 1 5CA8017C
+P 4700 4250
+F 0 "#PWR0142" H 4700 4000 50  0001 C CNN
+F 1 "GND" H 4705 4077 50  0000 C CNN
+F 2 "" H 4700 4250 50  0000 C CNN
+F 3 "" H 4700 4250 50  0000 C CNN
+	1    4700 4250
+	1    0    0    -1
+$EndComp
+Connection ~ 4700 4250
+Wire Wire Line
+	4700 4250 4950 4250
+$Comp
+L stmbl:+3.3V #PWR0143
+U 1 1 5CA80CBF
+P 4700 3950
+F 0 "#PWR0143" H 4700 3800 50  0001 C CNN
+F 1 "+3.3V" H 4715 4123 50  0000 C CNN
+F 2 "" H 4700 3950 50  0001 C CNN
+F 3 "" H 4700 3950 50  0001 C CNN
+	1    4700 3950
+	1    0    0    -1
+$EndComp
+Connection ~ 4700 3950
+Wire Wire Line
+	4700 3950 4950 3950
 $EndSCHEMATC
